File: bed-smart-plug/project.sch (KiCad schematic (older format))
At the start: 37 parts, among them J1 Prises, Q1 BT136-600, Q2 BT136-600, Q3 BT136-600, Q4 BT136-600, U1 MOC3021M, U2 MOC3021M, U3 MOC3021M, U4 MOC3021M, U5 ESP32-POE-ISO

Commit message: schematic
Parts:
- added AE1: Antenna, symbol Device:Antenna
- added D_OUT1, D_OUT2, D_OUT3, D_OUT4, D_STATUS1: LED, symbol Device:LED
- added HS1, HS2, HS3, HS4: Heatsink, symbol Mechanical:Heatsink
- added J_IR_LED1: Jack-DC, symbol Connector:Jack-DC
- added J_UART1: Conn_01x04_Female, symbol Connector:Conn_01x04_Female
- added Q5: 2N2222, Package_TO_SOT_THT:TO-92_Inline, symbol Transistor_BJT:2N3904
- added R17, R18, R19, R20, R21, R23: 100, symbol Device:R
- added R22: 4K7, symbol Device:R
- added R24: 1K, symbol Device:R
- added U6: DS18B20, Package_TO_SOT_THT:TO-92_Inline, symbol Sensor_Temperature:DS18B20
- added U7: RXB6, symbol mylife-symbols:RXB6
Connections:
- net GND: now also D_OUT1.1 (K), D_OUT2.1 (K), D_OUT3.1 (K), D_OUT4.1 (K), D_STATUS1.1 (K), J_UART1.4 (Pin_4), Q5.1 (E), U6.1 (GND), U7.2 (GND), U7.3 (GND), U7.8 (GND)
- net at R13.2, U5.14 (GPIO16): now also R17.1
- net at U5.10 (GPIO5): now also U7.7 (DATA)
- net at R16.2, U5.11 (GPIO13): now also R20.1
- net at R15.2, U5.12 (GPIO14): now also R19.1
- net at R14.2, U5.13 (GPIO15): now also R18.1
- net +3V3: now reaches U5.2 (+3.3V_(out))
- net +3V3: now also J_UART1.1 (Pin_1), R22.1, R23.1, U6.3 (VDD), U7.4 (VCC), U7.5 (VCC)
- net at U5.5 (GPIO0): now also R21.1
- net TX: now reaches U5.6 (GPIO1)
- net TX: now also J_UART1.2 (Pin_2)
- net at U5.7 (GPIO2): now also R22.2, U6.2 (DQ)
- net RX: now reaches U5.8 (GPIO3)
- net RX: now also J_UART1.3 (Pin_3)
- net at U5.9 (GPIO4): now also R24.1
- new net: D_OUT1.2 (A), R17.2
- new net: D_OUT2.2 (A), R18.2
- new net: D_OUT3.2 (A), R19.2
- new net: D_OUT4.2 (A), R20.2
- new net: D_STATUS1.2 (A), R21.2
- new net: AE1.1 (A), U7.1 (Antenna)
- new net: J_IR_LED1.1, R23.2
- new net: J_IR_LED1.2, Q5.3 (C)
- new net: Q5.2 (B), R24.2
Other:
- moved on the sheet: F2, PS1, U5

Commit message: wip footprints
Parts:
- removed J_UART1: Conn_01x04_Female, symbol Connector:Conn_01x04_Female
- removed U6: DS18B20, Package_TO_SOT_THT:TO-92_Inline, symbol Sensor_Temperature:DS18B20
- added D_POWER1: LED, LED_SMD:LED_1206_3216Metric_Pad1.42x1.75mm_HandSolder, symbol Device:LED
- added J_TEMP1: Conn_01x03_Male, Connector_PinHeader_2.54mm:PinHeader_1x03_P2.54mm_Vertical, symbol Connector:Conn_01x03_Male
- added J_UART1: Conn_01x04_Male, Connector_PinHeader_2.54mm:PinHeader_1x04_P2.54mm_Vertical, symbol Connector:Conn_01x04_Male
- added R25: 220, Resistor_SMD:R_1206_3216Metric_Pad1.42x1.75mm_HandSolder, symbol Device:R
- AE1: footprint (none) -> Connector_PinHeader_2.54mm:PinHeader_1x01_P2.54mm_Vertical
- C1, C3, C5, C7: footprint (none) -> Capacitor_THT:C_Rect_L9.0mm_W2.5mm_P7.50mm_MKT
- C2, C4, C6, C8: footprint (none) -> Capacitor_SMD:C_2220_5650Metric_Pad1.97x5.40mm_HandSolder
- D_OUT1, D_OUT2, D_OUT3, D_OUT4, D_STATUS1: footprint (none) -> LED_SMD:LED_1206_3216Metric_Pad1.42x1.75mm_HandSolder
- F1, F2: footprint (none) -> Fuse:Fuseholder_Cylinder-5x20mm_Schurter_0031_8201_Horizontal_Open
- HS1, HS2, HS3, HS4: footprint (none) -> Heatsink:Heatsink_Fischer_SK104-STC-STIC_35x13mm_2xDrill2.5mm
- J1: footprint (none) -> TerminalBlock:TerminalBlock_bornier-6_P5.08mm
- R1, R10, R4, R7: footprint (none) -> Resistor_THT:R_Axial_DIN0204_L3.6mm_D1.6mm_P7.62mm_Horizontal
- R11, R12, R13, R14, R15, R16, R17, R18, R19, R2, R20, R21, R22, R23, R24, R3, R5, R6, R8, R9: footprint (none) -> Resistor_SMD:R_1206_3216Metric_Pad1.42x1.75mm_HandSolder
- U1, U2, U3, U4: footprint (none) -> Package_DIP:DIP-6_W8.89mm_SMDSocket_LongPads
- renumbered U7 to U6
Connections:
- net +3V3: now also J_TEMP1.1 (Pin_1), J_UART1.1 (Pin_1)
- net +5V: now also R25.1
- net GND: now also D_POWER1.1 (K), J_TEMP1.3 (Pin_3), J_UART1.4 (Pin_4)
- net RX: now also J_UART1.3 (Pin_3)
- net TX: now also J_UART1.2 (Pin_2)
- net at R22.2, U5.7 (GPIO2): now also J_TEMP1.2 (Pin_2)
- new net: D_POWER1.2 (A), R25.2
