File: epanel-io/prototype-1/prototype.kicad_sch (KiCad schematic)
At the start: 20 parts, among them J1 Screw_Terminal_01x04, J2 Conn_01x02_Male, J3 Screw_Terminal_01x02, J4 Conn_01x03_Male, Q1 IRF830, U1 4N35, U2 H11AA1

Commit message: schematic wip
Parts:
- removed J1: Screw_Terminal_01x04, symbol Connector:Screw_Terminal_01x04
- removed J2: Conn_01x02_Male, symbol Connector:Conn_01x02_Male
- removed J4: Conn_01x03_Male, symbol Connector:Conn_01x03_Male
- added C3: 0.01uF, Capacitor_THT:C_Rect_L9.0mm_W2.5mm_P7.50mm_MKT, symbol Device:C
- added C4: 0.05uF, Capacitor_SMD:C_2220_5650Metric_Pad1.97x5.40mm_HandSolder, symbol Device:C
- added J1: Conn_01x05_Male, symbol Connector:Conn_01x05_Male
- added J2, J4: Screw_Terminal_01x02, symbol Connector:Screw_Terminal_01x02
- added Q2: BT136-600, Package_TO_SOT_THT:TO-220-3_Vertical, symbol Triac_Thyristor:BT136-600
- added R10: 470Ω, Resistor_SMD:R_1206_3216Metric_Pad1.42x1.75mm_HandSolder, symbol Device:R
- added R11: 360Ω, Resistor_SMD:R_1206_3216Metric_Pad1.42x1.75mm_HandSolder, symbol Device:R
- added R12: 220Ω, Resistor_SMD:R_1206_3216Metric_Pad1.42x1.75mm_HandSolder, symbol Device:R
- added R9: 39Ω, Resistor_THT:R_Axial_DIN0204_L3.6mm_D1.6mm_P7.62mm_Horizontal, symbol Device:R
- added U3: MOC3021M, Package_DIP:DIP-6_W8.89mm_SMDSocket_LongPads, symbol Relay_SolidState:MOC3021M
- R1, R2, R3, R4, R5, R8: footprint (none) -> Resistor_SMD:R_1206_3216Metric_Pad1.42x1.75mm_HandSolder
Connections:
- net +3V3: now reaches R8.2
- net +3V3: now also J1.1 (Pin_1)
- net at R8.1, U2.5: now also J1.5 (Pin_5)
- net GND: now reaches U2.4
- net GND: now also U1.2, J1.2 (Pin_2), U3.2
- net at D2.4: now also J2.1 (Pin_1)
- net at D2.3: now also J2.2 (Pin_2)
- net at R1.2: now also J1.3 (Pin_3)
- new net: C4.1, R10.2, R11.1
- new net: C3.2, C4.2, J4.2 (Pin_2), Q2.1 (A1)
- new net: R11.2, U3.6
- new net: J4.1 (Pin_1), Q2.2 (A2), R10.1, R9.1
- new net: C3.1, R9.2
- new net: R12.1, U3.1
- new net: Q2.3 (G), U3.4
- new net: J1.4 (Pin_4), R12.2
- no-connect marks 0 -> 2
Other:
- note added: "Mosfet-based dimmer"
- note added: "Triac-based dimmer"
- note added: "Zero crossing detector"
- note removed: "230V"
- note removed: "Lamp"
- moved on the sheet: C1, C2, D1, D2, D6, J3, Q1, R1, R2, R4, R5, R6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

Commit message: add JLPCB refs + footprints
Parts:
- J1: footprint (none) -> Connector_PinHeader_2.54mm:PinHeader_1x05_P2.54mm_Vertical
- J2, J3, J4: footprint (none) -> TerminalBlock:TerminalBlock_bornier-2_P5.08mm
- R1: footprint Resistor_SMD:R_1206_3216Metric_Pad1.42x1.75mm_HandSolder -> Resistor_SMD:R_0603_1608Metric; JLCPCB (none) -> C23138
- R10: footprint Resistor_SMD:R_1206_3216Metric_Pad1.42x1.75mm_HandSolder -> Resistor_SMD:R_0603_1608Metric; JLCPCB (none) -> C23179
- R11: footprint Resistor_SMD:R_1206_3216Metric_Pad1.42x1.75mm_HandSolder -> Resistor_SMD:R_0603_1608Metric; JLCPCB (none) -> C25194
- R12, R5: footprint Resistor_SMD:R_1206_3216Metric_Pad1.42x1.75mm_HandSolder -> Resistor_SMD:R_0603_1608Metric; JLCPCB (none) -> C22962
- R2: footprint Resistor_SMD:R_1206_3216Metric_Pad1.42x1.75mm_HandSolder -> Resistor_SMD:R_0603_1608Metric; JLCPCB (none) -> C31850
- R3, R4: footprint Resistor_SMD:R_1206_3216Metric_Pad1.42x1.75mm_HandSolder -> Resistor_SMD:R_0603_1608Metric; JLCPCB (none) -> C4216
- R6, R7: footprint (none) -> Resistor_SMD:R_0805_2012Metric; JLCPCB (none) -> C966118
- R8: footprint Resistor_SMD:R_1206_3216Metric_Pad1.42x1.75mm_HandSolder -> Resistor_SMD:R_0603_1608Metric; JLCPCB (none) -> C25804
- R9: footprint Resistor_THT:R_Axial_DIN0204_L3.6mm_D1.6mm_P7.62mm_Horizontal -> Resistor_SMD:R_0603_1608Metric; JLCPCB (none) -> C23154
- U1: footprint Package_DIP:DIP-6_W7.62mm -> (none); JLCPCB (none) -> C115444
- U2: footprint Package_DIP:DIP-6_W7.62mm -> (none); JLCPCB (none) -> C184383
- U3: footprint Package_DIP:DIP-6_W8.89mm_SMDSocket_LongPads -> (none); JLCPCB (none) -> C115465

Commit message: footprints + JLCPCB refs
Parts:
- C1: footprint (none) -> Capacitor_SMD:C_1206_3216Metric; JLCPCB (none) -> C50254
- C2: footprint (none) -> Capacitor_SMD:C_1210_3225Metric; JLCPCB (none) -> C340320
- C3: value 0.01uF -> 10nF; footprint Capacitor_THT:C_Rect_L9.0mm_W2.5mm_P7.50mm_MKT -> Capacitor_SMD:C_0805_2012Metric; JLCPCB (none) -> C106840
- C4: value 0.05uF -> 47nF; footprint Capacitor_SMD:C_2220_5650Metric_Pad1.97x5.40mm_HandSolder -> Capacitor_SMD:C_1206_3216Metric; JLCPCB (none) -> C309031
- D1: footprint Diode_SMD:D_MiniMELF -> Diode_SMD:D_SOD-123; JLCPCB (none) -> C173431
- D2: footprint (none) -> Diode_SMD:Diode_Bridge_Diotec_SO-DIL-Slim; JLCPCB (none) -> C169512
- D6: footprint Diode_THT:D_DO-41_SOD81_P10.16mm_Horizontal -> Diode_SMD:D_SMA; JLCPCB (none) -> C727081
- Q1: footprint Package_TO_SOT_THT:TO-220-3_Vertical -> Package_TO_SOT_SMD:TO-263-3_TabPin2; JLCPCB (none) -> C693297
- Q2: footprint Package_TO_SOT_THT:TO-220-3_Vertical -> Package_TO_SOT_SMD:TO-252-3_TabPin2; JLCPCB (none) -> C581425
- U1, U3: footprint (none) -> Package_DIP:SMDIP-6_W7.62mm
- U2: footprint (none) -> Package_DIP:SMDIP-6_W9.53mm

Commit message: place components
Connections:
- net at J2.1 (Pin_1): now also D2.3; no longer D2.4
- net at J2.2 (Pin_2): now also D2.4; no longer D2.3
- net at C3.2, C4.2, Q2.1 (A1): now also J4.1 (Pin_1); no longer J4.2 (Pin_2)
- net at Q2.2 (A2), R10.1, R9.1: now also J4.2 (Pin_2); no longer J4.1 (Pin_1)
Other:
- moved on the sheet: D2
Changed lines of the file:
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@@
     (pin "2")
   )
-  (symbol (lib_id "Connector:Screw_Terminal_01x02") (at 240.03 88.9 0) (unit 1)
-    (in_bom yes) (on_board yes)
-    (property "Reference" "J4" (id 0) (at 242.062 89.2615 0)
-      (effects (font (size 1.27 1.27)) (justify left))
-    )
-    (property "Value" "Screw_Terminal_01x02" (id 1) (at 242.062 92.0366 0)
-      (effects (font (size 1.27 1.27)) (justify left))
-    )
-    (property "Footprint" "TerminalBlock:TerminalBlock_bornier-2_P5.08mm" (id 2) (at 240.03 88.9 0)
-      (effects (font (size 1.27 1.27)) hide)
-    )
-    (property "Datasheet" "~" (id 3) (at 240.03 88.9 0)
+  (symbol (lib_id "Connector:Screw_Terminal_01x02") (at 240.03 91.44 0) (mirror x) (unit 1)
+    (in_bom yes) (on_board yes)
+    (property "Reference" "J4" (id 0) (at 242.062 91.0785 0)
+      (effects (font (size 1.27 1.27)) (justify left))
+    )
+    (property "Value" "Screw_Terminal_01x02" (id 1) (at 242.062 88.3034 0)
+      (effects (font (size 1.27 1.27)) (justify left))
+    )
+    (property "Footprint" "TerminalBlock:TerminalBlock_bornier-2_P5.08mm" (id 2) (at 240.03 91.44 0)
+      (effects (font (size 1.27 1.27)) hide)
+    )
+    (property "Datasheet" "~" (id 3) (at 240.03 91.44 0)
       (effects (font (size 1.27 1.27)) hide)
     )
@@
     (pin "2")
   )
-  (symbol (lib_id "Device:D_Bridge_+-AA") (at 212.09 43.18 90) (unit 1)
-    (in_bom yes) (on_board yes) (fields_autoplaced)
-    (property "Reference" "D2" (id 0) (at 223.3998 39.0865 90))
-    (property "Value" "4* 1N5408" (id 1) (at 223.3998 41.8616 90))
+  (symbol (lib_id "Device:D_Bridge_+-AA") (at 212.09 43.18 270) (mirror x) (unit 1)
+    (in_bom yes) (on_board yes) (fields_autoplaced)
+    (property "Reference" "D2" (id 0) (at 223.52 38.481 90))
+    (property "Value" "4* 1N5408" (id 1) (at 223.52 41.021 90))
     (property "Footprint" "Diode_SMD:Diode_Bridge_Diotec_SO-DIL-Slim" (id 2) (at 212.09 43.18 0)
       (effects (font (size 1.27 1.27)) hide)

Commit message: update tag name
Parts:
- C1: JLCPCB C50254 -> (none); LCSC (none) -> C50254
- C2: JLCPCB C340320 -> (none); LCSC (none) -> C340320
- C3: JLCPCB C106840 -> (none); LCSC (none) -> C106840
- C4: JLCPCB C309031 -> (none); LCSC (none) -> C309031
- D1: JLCPCB C173431 -> (none); LCSC (none) -> C173431
- D2: JLCPCB C169512 -> (none); LCSC (none) -> C169512
- D6: JLCPCB C727081 -> (none); LCSC (none) -> C727081
- Q1: JLCPCB C693297 -> (none); LCSC (none) -> C693297
- Q2: JLCPCB C581425 -> (none); LCSC (none) -> C581425
- R1: JLCPCB C23138 -> (none); LCSC (none) -> C23138
- R10: JLCPCB C23179 -> (none); LCSC (none) -> C23179
- R11: JLCPCB C25194 -> (none); LCSC (none) -> C25194
- R12, R5: JLCPCB C22962 -> (none); LCSC (none) -> C22962
- R2: JLCPCB C31850 -> (none); LCSC (none) -> C31850
- R3, R4: JLCPCB C4216 -> (none); LCSC (none) -> C4216
- R6, R7: JLCPCB C966118 -> (none); LCSC (none) -> C966118
- R8: JLCPCB C25804 -> (none); LCSC (none) -> C25804
- R9: JLCPCB C23154 -> (none); LCSC (none) -> C23154
- U1: JLCPCB C115444 -> (none); LCSC (none) -> C115444
- U2: JLCPCB C184383 -> (none); LCSC (none) -> C184383
- U3: JLCPCB C115465 -> (none); LCSC (none) -> C115465
Changed lines of the file:
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@@
       (effects (font (size 1.27 1.27)) hide)
     )
-    (property "JLCPCB" "C22962" (id 4) (at 173.99 30.48 90)
+    (property "LCSC" "C22962" (id 4) (at 173.99 30.48 90)
       (effects (font (size 1.27 1.27)) hide)
     )
@@
       (effects (font (size 1.27 1.27)) hide)
     )
-    (property "JLCPCB" "C23138" (id 4) (at 68.58 48.26 90)
+    (property "LCSC" "C23138" (id 4) (at 68.58 48.26 90)
       (effects (font (size 1.27 1.27)) hide)
     )
@@
       (effects (font (size 1.27 1.27)) (justify left) hide)
     )
-    (property "JLCPCB" "C693297" (id 4) (at 179.07 53.34 0)
+    (property "LCSC" "C693297" (id 4) (at 179.07 53.34 0)
       (effects (font (size 1.27 1.27)) hide)
     )
@@
       (effects (font (size 1.27 1.27)) hide)
     )
-    (property "JLCPCB" "C25804" (id 4) (at 166.37 144.78 0)
+    (property "LCSC" "C25804" (id 4) (at 166.37 144.78 0)
       (effects (font (size 1.27 1.27)) hide)
     )
@@
       (effects (font (size 1.27 1.27)) hide)
     )
-    (property "JLCPCB" "C309031" (id 4) (at 132.08 113.03 0)
+    (property "LCSC" "C309031" (id 4) (at 132.08 113.03 0)
       (effects (font (size 1.27 1.27)) hide)
     )
@@
       (effects (font (size 1.27 1.27)) hide)
     )
-    (property "JLCPCB" "C4216" (id 4) (at 104.14 36.83 0)
+    (property "LCSC" "C4216" (id 4) (at 104.14 36.83 0)
       (effects (font (size 1.27 1.27)) hide)
     )
@@
       (effects (font (size 1.27 1.27)) hide)
     )
-    (property "JLCPCB" "C25194" (id 4) (at 125.73 88.9 90)
+    (property "LCSC" "C25194" (id 4) (at 125.73 88.9 90)
       (effects (font (size 1.27 1.27)) hide)
     )
@@
       (effects (font (size 1.27 1.27)) (justify left) hide)
     )
-    (property "JLCPCB" "C115444" (id 4) (at 85.09 50.8 0)
+    (property "LCSC" "C115444" (id 4) (at 85.09 50.8 0)
       (effects (font (size 1.27 1.27)) hide)
     )
@@
       (effects (font (size 1.27 1.27)) hide)
     )
-    (property "JLCPCB" "C340320" (id 4) (at 163.83 46.99 0)
+    (property "LCSC" "C340320" (id 4) (at 163.83 46.99 0)
       (effects (font (size 1.27 1.27)) hide)
     )
@@
       (effects (font (size 1.27 1.27)) hide)
     )
-    (property "JLCPCB" "C966118" (id 4) (at 207.01 152.4 90)
+    (property "LCSC" "C966118" (id 4) (at 207.01 152.4 90)
       (effects (font (size 1.27 1.27)) hide)
     )
@@
       (effects (font (size 1.27 1.27)) hide)
     )
-    (property "JLCPCB" "C23154" (id 4) (at 158.75 97.79 0)
+    (property "LCSC" "C23154" (id 4) (at 158.75 97.79 0)
       (effects (font (size 1.27 1.27)) hide)
     )
@@
       (effects (font (size 1.27 1.27)) (justify left) hide)
     )
-    (property "JLCPCB" "C115465" (id 4) (at 111.76 91.44 0)
+    (property "LCSC" "C115465" (id 4) (at 111.76 91.44 0)
       (effects (font (size 1.27 1.27)) hide)
     )
@@
       (effects (font (size 1.27 1.27)) hide)
     )
-    (property "JLCPCB" "C106840" (id 4) (at 158.75 110.49 0)
+    (property "LCSC" "C106840" (id 4) (at 158.75 110.49 0)
       (effects (font (size 1.27 1.27)) hide)
     )
@@
       (effects (font (size 1.27 1.27)) hide)
     )
-    (property "JLCPCB" "C4216" (id 4) (at 128.27 30.48 90)
+    (property "LCSC" "C4216" (id 4) (at 128.27 30.48 90)
       (effects (font (size 1.27 1.27)) hide)
     )
@@
       (effects (font (size 1.27 1.27)) (justify left) hide)
     )
-    (property "JLCPCB" "C581425" (id 4) (at 143.51 101.6 0)
+    (property "LCSC" "C581425" (id 4) (at 143.51 101.6 0)
       (effects (font (size 1.27 1.27)) hide)
     )
@@
       (effects (font (size 1.27 1.27)) hide)
     )
-    (property "JLCPCB" "C23179" (id 4) (at 137.16 88.9 90)
+    (property "LCSC" "C23179" (id 4) (at 137.16 88.9 90)
       (effects (font (size 1.27 1.27)) hide)
     )
@@
       (effects (font (size 1.27 1.27)) hide)
     )
-    (property "JLCPCB" "C966118" (id 4) (at 207.01 142.24 90)
+    (property "LCSC" "C966118" (id 4) (at 207.01 142.24 90)
       (effects (font (size 1.27 1.27)) hide)
     )
@@
       (effects (font (size 1.27 1.27)) hide)
     )
-    (property "JLCPCB" "C727081" (id 4) (at 190.5 30.48 0)
+    (property "LCSC" "C727081" (id 4) (at 190.5 30.48 0)
       (effects (font (size 1.27 1.27)) hide)
     )
@@
       (effects (font (size 1.27 1.27)) hide)
     )
-    (property "JLCPCB" "C31850" (id 4) (at 104.14 58.42 0)
+    (property "LCSC" "C31850" (id 4) (at 104.14 58.42 0)
       (effects (font (size 1.27 1.27)) hide)
     )
@@
       (effects (font (size 1.27 1.27)) hide)
     )
-    (property "JLCPCB" "C22962" (id 4) (at 97.79 88.9 90)
+    (property "LCSC" "C22962" (id 4) (at 97.79 88.9 90)
       (effects (font (size 1.27 1.27)) hide)
     )
@@
       (effects (font (size 1.27 1.27)) (justify left) hide)
     )
-    (property "JLCPCB" "C184383" (id 4) (at 179.07 149.86 0)
+    (property "LCSC" "C184383" (id 4) (at 179.07 149.86 0)
       (effects (font (size 1.27 1.27)) hide)
     )
@@
       (effects (font (size 1.27 1.27)) hide)
     )
-    (property "JLCPCB" "C50254" (id 4) (at 144.78 46.99 0)
+    (property "LCSC" "C50254" (id 4) (at 144.78 46.99 0)
       (effects (font (size 1.27 1.27)) hide)
     )
@@
       (effects (font (size 1.27 1.27)) hide)
     )
-    (property "JLCPCB" "C173431" (id 4) (at 124.46 46.99 90)
+    (property "LCSC" "C173431" (id 4) (at 124.46 46.99 90)
       (effects (font (size 1.27 1.27)) hide)
     )
@@
       (effects (font (size 1.27 1.27)) hide)
     )
-    (property "JLCPCB" "C169512" (id 4) (at 212.09 43.18 90)
-      (effects (font (size 1.27 1.27)) hide)
-    )
+    (property "LCSC" "C169512" (id 4) (at 212.09 43.18 90)
+      (effects (font (size 1.27 1.27)) hide)
+    )
