File: epanel-io/prototype-2/prototype-2.kicad_pcb (KiCad board)
At the start: 2 copper layers, 87 x 68 mm, 30 parts, among them J1 Conn_01x05_Male, J2 Screw_Terminal_01x04, J3 Screw_Terminal_01x04, J4 Screw_Terminal_01x02, Q1 IRF830, Q2 IRF830, SW1 SW_Push, U1 Pico, U2 4N35, U3 4N35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

Commit message: wip pcb
Parts:
- moved U3 7.62 mm to (116.8, 94.0)
- moved U5 7.62 mm to (116.8, 83.8)
- moved R11 5.68 mm to (124.5, 81.3), turned to -90 degrees
- moved R7 5.14 mm to (124.5, 95.8), turned to -90 degrees
- moved R10 5.08 mm to (124.5, 86.4), turned to -90 degrees
Routing:
- net Net-(Q2-Pad1): track 62.4 -> 51.8 mm
- net Net-(PS2-Pad4): track 25.1 -> 35.6 mm
- net Net-(R9-Pad1): track 88.3 -> 80.7 mm
- net Net-(R11-Pad1): track 79.1 -> 73.5 mm
- net Net-(J3-Pad4): track 67.9 -> 64.1 mm
- net Net-(D2-Pad2): track 60.9 -> 63.3 mm
- net Net-(R10-Pad2): track 4.48 -> 3.37 mm
- net Net-(R11-Pad2): track 4.48 -> 3.53 mm

Commit message: wip pcb layout
Parts:
- moved J1 149.4 mm to (68.6, 167.6)
- moved U1 143.4 mm to (116.8, 182.9)
- moved SW1 142.9 mm to (147.3, 182.9)
- moved U6 64.4 mm to (170.2, 111.8)
- moved R12 63.5 mm to (179.4, 114.3)
- moved R13 63.4 mm to (179.4, 109.2)
- moved R2 22.7 mm to (111.8, 101.6)
- moved R5 18.0 mm to (113.5, 114.3), turned to 180 degrees
- moved R4 11.4 mm to (109.2, 88.9), turned to 180 degrees
- moved R1 11.4 mm to (111.8, 76.2)
- moved R3 5.68 mm to (109.2, 63.5), turned to 180 degrees
Routing:
- net GND: track 0.00 -> 112.9 mm
- net Net-(J4-Pad2): track 0.00 -> 6.78 mm
- net Net-(J4-Pad1): track 0.00 -> 6.78 mm
- net Net-(R13-Pad2): track 0.00 -> 4.62 mm
- net Net-(R12-Pad2): track 0.00 -> 3.57 mm
Changed lines of the file:
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@@
   )
   (footprint "MCU_RaspberryPi_and_Boards:RPi_Pico_SMD_TH" (layer "F.Cu")
-    (at 60.96 50.8)
+    (at 116.84 182.88)
     (descr "Through hole straight pin header, 2x20, 2.54mm pitch, double rows")
     (tags "Through hole pin header THT 2x20 2.54mm double row")
@@
   )
   (footprint "Button_Switch_SMD:SW_SPST_REED_CT05-XXXX-J1" (layer "F.Cu")
-    (at 81.82 55.88)
+    (at 147.32 182.88)
     (descr "Coto Technologies SPST Reed Switch CT05-XXXX-J1")
     (tags "Coto Reed SPST Switch")
@@
   )
   (footprint "Resistor_SMD:R_0603_1608Metric" (layer "F.Cu")
-    (at 95.685 111.76)
+    (at 113.475 114.3 180)
     (descr "Resistor SMD 0603 (1608 Metric), square (rectangular) end terminal, IPC_7351 nominal, (Body size source: IPC-SM-782 page 72, https://www.pcb-3d.com/wordpress/wp-content/uploads/ipc-sm-782a_amendment_1_and_2.pdf), generated with kicad-footprint-generator")
     (tags "resistor")
@@
     (fp_line (start -0.8 -0.4125) (end 0.8 -0.4125) (layer "F.Fab") (width 0.1))
     (fp_line (start 0.8 0.4125) (end -0.8 0.4125) (layer "F.Fab") (width 0.1))
-    (pad "1" smd roundrect locked (at -0.825 0) (size 0.8 0.95) (layers "F.Cu" "F.Paste" "F.Mask") (roundrect_rratio 0.25)
+    (pad "1" smd roundrect locked (at -0.825 0 180) (size 0.8 0.95) (layers "F.Cu" "F.Paste" "F.Mask") (roundrect_rratio 0.25)
       (net 28 "Net-(R5-Pad1)") (pintype "passive"))
-    (pad "2" smd roundrect locked (at 0.825 0) (size 0.8 0.95) (layers "F.Cu" "F.Paste" "F.Mask") (roundrect_rratio 0.25)
+    (pad "2" smd roundrect locked (at 0.825 0 180) (size 0.8 0.95) (layers "F.Cu" "F.Paste" "F.Mask") (roundrect_rratio 0.25)
       (net 26 "+3V3") (pintype "passive"))
     (model "${KICAD6_3DMODEL_DIR}/Resistor_SMD.3dshapes/R_0603_1608Metric.wrl"
@@
   )
   (footprint "Resistor_SMD:R_0805_2012Metric" (layer "F.Cu")
-    (at 116.005 111.76 180)
+    (at 179.4275 114.3 180)
     (descr "Resistor SMD 0805 (2012 Metric), square (rectangular) end terminal, IPC_7351 nominal, (Body size source: IPC-SM-782 page 72, https://www.pcb-3d.com/wordpress/wp-content/uploads/ipc-sm-782a_amendment_1_and_2.pdf), generated with kicad-footprint-generator")
     (tags "resistor")
@@
   )
   (footprint "Connector_PinHeader_2.54mm:PinHeader_1x05_P2.54mm_Vertical" (layer "F.Cu")
-    (at 22.86 25.405)
+    (at 68.58 167.64)
     (descr "Through hole straight pin header, 1x05, 2.54mm pitch, single row")
     (tags "Through hole pin header THT 1x05 2.54mm single row")
@@
   )
   (footprint "Resistor_SMD:R_0603_1608Metric" (layer "F.Cu")
-    (at 106.68 66.04 180)
+    (at 111.76 76.2 180)
     (descr "Resistor SMD 0603 (1608 Metric), square (rectangular) end terminal, IPC_7351 nominal, (Body size source: IPC-SM-782 page 72, https://www.pcb-3d.com/wordpress/wp-content/uploads/ipc-sm-782a_amendment_1_and_2.pdf), generated with kicad-footprint-generator")
     (tags "resistor")
@@
   )
   (footprint "Resistor_SMD:R_0603_1608Metric" (layer "F.Cu")
-    (at 99.06 83.82)
+    (at 109.22 88.9 180)
     (descr "Resistor SMD 0603 (1608 Metric), square (rectangular) end terminal, IPC_7351 nominal, (Body size source: IPC-SM-782 page 72, https://www.pcb-3d.com/wordpress/wp-content/uploads/ipc-sm-782a_amendment_1_and_2.pdf), generated with kicad-footprint-generator")
     (tags "resistor")
@@
     (fp_line (start -0.8 0.4125) (end -0.8 -0.4125) (layer "F.Fab") (width 0.1))
     (fp_line (start -0.8 -0.4125) (end 0.8 -0.4125) (layer "F.Fab") (width 0.1))
-    (pad "1" smd roundrect locked (at -0.825 0) (size 0.8 0.95) (layers "F.Cu" "F.Paste" "F.Mask") (roundrect_rratio 0.25)
+    (pad "1" smd roundrect locked (at -0.825 0 180) (size 0.8 0.95) (layers "F.Cu" "F.Paste" "F.Mask") (roundrect_rratio 0.25)
       (net 27 "Net-(R4-Pad1)") (pintype "passive"))
-    (pad "2" smd roundrect locked (at 0.825 0) (size 0.8 0.95) (layers "F.Cu" "F.Paste" "F.Mask") (roundrect_rratio 0.25)
+    (pad "2" smd roundrect locked (at 0.825 0 180) (size 0.8 0.95) (layers "F.Cu" "F.Paste" "F.Mask") (roundrect_rratio 0.25)
       (net 26 "+3V3") (pintype "passive"))
     (model "${KICAD6_3DMODEL_DIR}/Resistor_SMD.3dshapes/R_0603_1608Metric.wrl"
@@
   )
   (footprint "Resistor_SMD:R_0603_1608Metric" (layer "F.Cu")
-    (at 106.68 58.42)
+    (at 109.22 63.5 180)
     (descr "Resistor SMD 0603 (1608 Metric), square (rectangular) end terminal, IPC_7351 nominal, (Body size source: IPC-SM-782 page 72, https://www.pcb-3d.com/wordpress/wp-content/uploads/ipc-sm-782a_amendment_1_and_2.pdf), generated with kicad-footprint-generator")
     (tags "resistor")
@@
     (fp_line (start -0.8 -0.4125) (end 0.8 -0.4125) (layer "F.Fab") (width 0.1))
     (fp_line (start 0.8 -0.4125) (end 0.8 0.4125) (layer "F.Fab") (width 0.1))
-    (pad "1" smd roundrect locked (at -0.825 0) (size 0.8 0.95) (layers "F.Cu" "F.Paste" "F.Mask") (roundrect_rratio 0.25)
+    (pad "1" smd roundrect locked (at -0.825 0 180) (size 0.8 0.95) (layers "F.Cu" "F.Paste" "F.Mask") (roundrect_rratio 0.25)
       (net 25 "Net-(R3-Pad1)") (pintype "passive"))
-    (pad "2" smd roundrect locked (at 0.825 0) (size 0.8 0.95) (layers "F.Cu" "F.Paste" "F.Mask") (roundrect_rratio 0.25)
+    (pad "2" smd roundrect locked (at 0.825 0 180) (size 0.8 0.95) (layers "F.Cu" "F.Paste" "F.Mask") (roundrect_rratio 0.25)
       (net 26 "+3V3") (pintype "passive"))
     (model "${KICAD6_3DMODEL_DIR}/Resistor_SMD.3dshapes/R_0603_1608Metric.wrl"
@@
   )
   (footprint "Resistor_SMD:R_0805_2012Metric" (layer "F.Cu")
-    (at 116.005 109.22 180)
+    (at 179.4275 109.22 180)
     (descr "Resistor SMD 0805 (2012 Metric), square (rectangular) end terminal, IPC_7351 nominal, (Body size source: IPC-SM-782 page 72, https://www.pcb-3d.com/wordpress/wp-content/uploads/ipc-sm-782a_amendment_1_and_2.pdf), generated with kicad-footprint-generator")
     (tags "resistor")
@@
   )
   (footprint "Package_DIP:SMDIP-6_W9.53mm" (layer "F.Cu")
-    (at 105.845 109.22 180)
+    (at 170.18 111.76 180)
     (descr "6-lead surface-mounted (SMD) DIP package, row spacing 9.53 mm (375 mils)")
     (tags "SMD DIP DIL PDIP SMDIP 2.54mm 9.53mm 375mil")
@@
   )
   (footprint "Resistor_SMD:R_0603_1608Metric" (layer "F.Cu")
-    (at 91.44 91.44 180)
+    (at 111.76 101.6 180)
     (descr "Resistor SMD 0603 (1608 Metric), square (rectangular) end terminal, IPC_7351 nominal, (Body size source: IPC-SM-782 page 72, https://www.pcb-3d.com/wordpress/wp-content/uploads/ipc-sm-782a_amendment_1_and_2.pdf), generated with kicad-footprint-generator")
     (tags "resistor")
@@
   (segment (start 187.125 93.98) (end 178.635 93.98) (width 1) (layer "F.Cu") (net 8))
   (segment (start 178.635 93.98) (end 178.625 93.97) (width 1) (layer "F.Cu") (net 8))
+  (segment (start 160.02 101.6) (end 165.415 106.995) (width 0.25) (layer "F.Cu") (net 10))
+  (segment (start 116.84 68.58) (end 113.03 68.58) (width 0.25) (layer "F.Cu") (net 10))
+  (segment (start 112.075 55.88) (end 114.3 55.88) (width 0.25) (layer "F.Cu") (net 10))
+  (segment (start 116.84 58.42) (end 116.84 68.58) (width 0.25) (layer "F.Cu") (net 10))
+  (segment (start 119.38 101.6) (end 160.02 101.6) (width 0.25) (layer "F.Cu") (net 10))
+  (segment (start 116.84 93.98) (end 116.84 99.06) (width 0.25) (layer "F.Cu") (net 10))
+  (segment (start 116.84 81.28) (end 116.84 93.98) (width 0.25) (layer "F.Cu") (net 10))
+  (segment (start 165.415 106.995) (end 165.415 109.22) (width 0.25) (layer "F.Cu") (net 10))
+  (segment (start 116.84 93.98) (end 113.03 93.98) (width 0.25) (layer "F.Cu") (net 10))
+  (segment (start 116.84 68.58) (end 116.84 81.28) (width 0.25) (layer "F.Cu") (net 10))
+  (segment (start 116.84 81.28) (end 112.075 81.28) (width 0.25) (layer "F.Cu") (net 10))
+  (segment (start 116.84 99.06) (end 119.38 101.6) (width 0.25) (layer "F.Cu") (net 10))
+  (segment (start 114.3 55.88) (end 116.84 58.42) (width 0.25) (layer "F.Cu") (net 10))
   (segment (start 129.99625 86.36) (end 129.08375 85.4475) (width 0.25) (layer "F.Cu") (net 14))
   (segment (start 129.08375 85.4475) (end 124.46 85.4475) (width 0.25) (layer "F.Cu") (net 14))
@@
   (segment (start 159.3425 86.4) (end 134.66 86.4) (width 0.25) (layer "B.Cu") (net 14))
   (segment (start 161.9225 83.82) (end 187.125 83.82) (width 0.25) (layer "B.Cu") (net 14))
+  (segment (start 187.125 114.3) (end 180.34 114.3) (width 0.25) (layer "F.Cu") (net 15))
+  (segment (start 187.125 109.22) (end 180.34 109.22) (width 0.25) (layer "F.Cu") (net 16))
   (segment (start 139.7 58.42) (end 137.08 55.8) (width 0.25) (layer "F.Cu") (net 17))
   (segment (start 137.08 55.8) (end 129.9425 55.8) (width 0.25) (layer "F.Cu") (net 17))
@@
   (segment (start 122.8325 83.82) (end 121.605 83.82) (width 0.25) (layer "F.Cu") (net 32))
   (segment (start 124.46 82.1925) (end 122.8325 83.82) (width 0.25) (layer "F.Cu") (net 32))
+  (segment (start 178.515 114.3) (end 174.945 114.3) (width 0.25) (layer "F.Cu") (net 33))
+  (segment (start 178.515 109.22) (end 175.975 111.76) (width 0.25) (layer "F.Cu") (net 34))
+  (segment (start 175.975 111.76) (end 174.945 111.76) (width 0.25) (layer "F.Cu") (net 34))
   (segment (start 126.0875 53.34) (end 124.46 54.9675) (width 0.25) (layer "F.Cu") (net 77))
   (segment (start 134.62 53.34) (end 126.0875 53.34) (width 0.25) (layer "F.Cu") (net 77))

Commit message: wip pcb
Parts:
- moved R5 7.62 mm to (113.5, 106.7)
- moved R3 2.54 mm to (111.8, 63.5)
- moved R4 2.54 mm to (111.8, 88.9)
- turned R1 to 0 degrees
Routing:
- net Net-(R3-Pad1): track 0.00 -> 52.5 mm, vias 0 -> 1
- net +3V3: track 0.00 -> 50.7 mm
- net Net-(R1-Pad2): track 0.00 -> 33.1 mm, vias 0 -> 1
- net Net-(R4-Pad1): track 0.00 -> 22.1 mm, vias 0 -> 1
- net Net-(R1-Pad1): track 0.00 -> 11.4 mm
- net Net-(R2-Pad1): track 0.00 -> 7.85 mm, vias 0 -> 1
Changed lines of the file:
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@@
   )
   (footprint "Resistor_SMD:R_0603_1608Metric" (layer "F.Cu")
-    (at 113.475 114.3 180)
+    (at 113.475 106.68 180)
     (descr "Resistor SMD 0603 (1608 Metric), square (rectangular) end terminal, IPC_7351 nominal, (Body size source: IPC-SM-782 page 72, https://www.pcb-3d.com/wordpress/wp-content/uploads/ipc-sm-782a_amendment_1_and_2.pdf), generated with kicad-footprint-generator")
     (tags "resistor")
@@
   )
   (footprint "Resistor_SMD:R_0603_1608Metric" (layer "F.Cu")
-    (at 111.76 76.2 180)
+    (at 111.76 76.2)
     (descr "Resistor SMD 0603 (1608 Metric), square (rectangular) end terminal, IPC_7351 nominal, (Body size source: IPC-SM-782 page 72, https://www.pcb-3d.com/wordpress/wp-content/uploads/ipc-sm-782a_amendment_1_and_2.pdf), generated with kicad-footprint-generator")
     (tags "resistor")
@@
     (fp_line (start 0.8 0.4125) (end -0.8 0.4125) (layer "F.Fab") (width 0.1))
     (fp_line (start 0.8 -0.4125) (end 0.8 0.4125) (layer "F.Fab") (width 0.1))
-    (pad "1" smd roundrect locked (at -0.825 0 180) (size 0.8 0.95) (layers "F.Cu" "F.Paste" "F.Mask") (roundrect_rratio 0.25)
+    (pad "1" smd roundrect locked (at -0.825 0) (size 0.8 0.95) (layers "F.Cu" "F.Paste" "F.Mask") (roundrect_rratio 0.25)
       (net 21 "Net-(R1-Pad1)") (pintype "passive"))
-    (pad "2" smd roundrect locked (at 0.825 0 180) (size 0.8 0.95) (layers "F.Cu" "F.Paste" "F.Mask") (roundrect_rratio 0.25)
+    (pad "2" smd roundrect locked (at 0.825 0) (size 0.8 0.95) (layers "F.Cu" "F.Paste" "F.Mask") (roundrect_rratio 0.25)
       (net 22 "Net-(R1-Pad2)") (pintype "passive"))
     (model "${KICAD6_3DMODEL_DIR}/Resistor_SMD.3dshapes/R_0603_1608Metric.wrl"
@@
   )
   (footprint "Resistor_SMD:R_0603_1608Metric" (layer "F.Cu")
-    (at 109.22 88.9 180)
+    (at 111.76 88.9 180)
     (descr "Resistor SMD 0603 (1608 Metric), square (rectangular) end terminal, IPC_7351 nominal, (Body size source: IPC-SM-782 page 72, https://www.pcb-3d.com/wordpress/wp-content/uploads/ipc-sm-782a_amendment_1_and_2.pdf), generated with kicad-footprint-generator")
     (tags "resistor")
@@
   )
   (footprint "Resistor_SMD:R_0603_1608Metric" (layer "F.Cu")
-    (at 109.22 63.5 180)
+    (at 111.76 63.5 180)
     (descr "Resistor SMD 0603 (1608 Metric), square (rectangular) end terminal, IPC_7351 nominal, (Body size source: IPC-SM-782 page 72, https://www.pcb-3d.com/wordpress/wp-content/uploads/ipc-sm-782a_amendment_1_and_2.pdf), generated with kicad-footprint-generator")
     (tags "resistor")
@@
   (segment (start 157.48 81.28) (end 166.11 81.28) (width 0.25) (layer "F.Cu") (net 20))
   (segment (start 120.65 96.52) (end 121.92 96.52) (width 0.25) (layer "F.Cu") (net 20))
+  (segment (start 113.03 66.04) (end 112.395 66.04) (width 0.25) (layer "F.Cu") (net 21))
+  (segment (start 110.935 67.5) (end 110.935 76.2) (width 0.25) (layer "F.Cu") (net 21))
+  (segment (start 112.395 66.04) (end 110.935 67.5) (width 0.25) (layer "F.Cu") (net 21))
+  (segment (start 112.585 76.2) (end 114.3 76.2) (width 0.25) (layer "F.Cu") (net 22))
+  (via (at 114.3 76.2) (size 0.8) (drill 0.4) (layers "F.Cu" "B.Cu") (net 22))
+  (segment (start 114.3 76.2) (end 119.38 76.2) (width 0.25) (layer "B.Cu") (net 22))
+  (segment (start 119.38 76.2) (end 121.47048 78.29048) (width 0.25) (layer "B.Cu") (net 22))
+  (segment (start 121.47048 78.29048) (end 121.47048 101.6) (width 0.25) (layer "B.Cu") (net 22))
+  (segment (start 112.585 101.6) (end 114.3 101.6) (width 0.25) (layer "F.Cu") (net 23))
+  (via (at 114.3 101.6) (size 0.8) (drill 0.4) (layers "F.Cu" "B.Cu") (net 23))
+  (segment (start 114.3 101.6) (end 116.84 104.14) (width 0.25) (layer "B.Cu") (net 23))
+  (segment (start 116.84 104.14) (end 119.38 104.14) (width 0.25) (layer "B.Cu") (net 23))
+  (segment (start 114.3 61.785) (end 114.3 63.5) (width 0.25) (layer "F.Cu") (net 25))
+  (segment (start 114.3 63.5) (end 112.585 63.5) (width 0.25) (layer "F.Cu") (net 25))
+  (segment (start 114.3 59.745489) (end 114.3 61.785) (width 0.25) (layer "F.Cu") (net 25))
+  (segment (start 112.075 58.42) (end 112.974511 58.42) (width 0.25) (layer "F.Cu") (net 25))
+  (segment (start 112.974511 58.42) (end 114.3 59.745489) (width 0.25) (layer "F.Cu") (net 25))
+  (via (at 114.3 63.5) (size 0.8) (drill 0.4) (layers "F.Cu" "B.Cu") (net 25))
+  (segment (start 119.38 63.5) (end 121.92 66.04) (width 0.25) (layer "B.Cu") (net 25))
+  (segment (start 114.3 63.5) (end 119.38 63.5) (width 0.25) (layer "B.Cu") (net 25))
+  (segment (start 121.92 66.04) (end 121.92 78.74) (width 0.25) (layer "B.Cu") (net 25))
+  (segment (start 121.92 78.74) (end 121.92 101.6) (width 0.25) (layer "B.Cu") (net 25))
+  (segment (start 109.22 88.9) (end 110.935 88.9) (width 0.25) (layer "F.Cu") (net 26))
+  (segment (start 109.22 88.9) (end 109.22 111.76) (width 0.25) (layer "F.Cu") (net 26))
+  (segment (start 110.935 63.5) (end 109.22 65.215) (width 0.25) (layer "F.Cu") (net 26))
+  (segment (start 109.22 65.215) (end 109.22 88.9) (width 0.25) (layer "F.Cu") (net 26))
+  (segment (start 113.1875 83.82) (end 112.075 83.82) (width 0.25) (layer "F.Cu") (net 27))
+  (segment (start 114.3 84.9325) (end 114.3 88.9) (width 0.25) (layer "F.Cu") (net 27))
+  (segment (start 114.3 84.9325) (end 113.1875 83.82) (width 0.25) (layer "F.Cu") (net 27))
+  (segment (start 112.585 88.9) (end 114.3 88.9) (width 0.25) (layer "F.Cu") (net 27))
+  (via (at 114.3 88.9) (size 0.8) (drill 0.4) (layers "F.Cu" "B.Cu") (net 27))
+  (segment (start 114.3 88.9) (end 116.84 88.9) (width 0.25) (layer "B.Cu") (net 27))
+  (segment (start 116.84 88.9) (end 119.38 91.44) (width 0.25) (layer "B.Cu") (net 27))
+  (segment (start 119.38 93.98) (end 119.38 99.06) (width 0.25) (layer "B.Cu") (net 27))
+  (segment (start 119.38 91.44) (end 119.38 93.98) (width 0.25) (layer "B.Cu") (net 27))
   (segment (start 122.8325 61.8725) (end 121.92 60.96) (width 0.25) (layer "F.Cu") (net 29))
   (segment (start 124.46 61.8725) (end 122.8325 61.8725) (width 0.25) (layer "F.Cu") (net 29))

Commit message: remove pico from pcb
Parts:
- removed SW1: SW_Push, Button_Switch_SMD:SW_SPST_REED_CT05-XXXX-J1
- removed U1: Pico, MCU_RaspberryPi_and_Boards:RPi_Pico_SMD_TH
- J1: value Conn_01x05_Male -> Conn_01x07_Male; footprint Connector_PinHeader_2.54mm:PinHeader_1x05_P2.54mm_Vertical -> Connector_PinHeader_2.54mm:PinHeader_1x07_P2.54mm_Vertical
- moved J1 33.9 mm to (76.2, 134.6)
Connections:
- J1 pad 1: +5V -> +3V3
- J1 pad 3: Net-(J1-Pad3) -> Net-(R1-Pad2)
- J1 pad 4: Net-(J1-Pad4) -> Net-(R3-Pad1)
- J1 pad 5: Net-(J1-Pad5) -> Net-(R2-Pad2)

Commit message: wip prototype
Parts:
- moved J1 48.5 mm to (111.8, 101.6)
- moved R1 30.9 mm to (116.8, 106.7), turned to 180 degrees
- moved R2 11.4 mm to (116.8, 111.8)
- moved R5 10.7 mm to (116.8, 116.8), turned to 0 degrees
Routing:
- net Net-(R1-Pad1): track 11.4 -> 52.3 mm, vias 0 -> 2
- net Net-(R1-Pad2): track 33.1 -> 4.25 mm, vias 1 -> 0
- net Net-(R4-Pad1): track 22.1 -> 47.1 mm, vias 1 -> 2
- net Net-(R2-Pad1): track 7.85 -> 31.5 mm, vias 1 -> 2
- net Net-(R3-Pad1): track 52.5 -> 68.8 mm, vias 1 -> 2
- net +3V3: track 50.7 -> 41.6 mm
- net GND: track 112.9 -> 120.5 mm
- net Net-(R5-Pad1): track 0.00 -> 4.25 mm
- net Net-(R2-Pad2): track 0.00 -> 4.25 mm

Commit message: pcb ok
Routing:
- net Net-(R5-Pad1): track 4.25 -> 56.4 mm
- net +3V3: track 41.6 -> 64.3 mm
- net Net-(R2-Pad1): track 31.5 -> 30.1 mm
Changed lines of the file:
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@@
   (via (at 119.38 111.76) (size 0.8) (drill 0.4) (layers "F.Cu" "B.Cu") (net 19))
   (via (at 114.3 99.06) (size 0.8) (drill 0.4) (layers "F.Cu" "B.Cu") (net 19))
-  (segment (start 114.3 101.6) (end 114.3 109.22) (width 0.25) (layer "B.Cu") (net 19))
-  (segment (start 116.84 111.76) (end 119.38 111.76) (width 0.25) (layer "B.Cu") (net 19))
-  (segment (start 114.3 109.22) (end 116.84 111.76) (width 0.25) (layer "B.Cu") (net 19))
-  (segment (start 114.3 99.06) (end 114.3 101.6) (width 0.25) (layer "B.Cu") (net 19))
+  (segment (start 116.84 109.22) (end 119.38 111.76) (width 0.25) (layer "B.Cu") (net 19))
+  (segment (start 116.84 101.6) (end 116.84 109.22) (width 0.25) (layer "B.Cu") (net 19))
+  (segment (start 114.3 99.06) (end 116.84 101.6) (width 0.25) (layer "B.Cu") (net 19))
   (segment (start 111.76 111.76) (end 116.015 111.76) (width 0.25) (layer "F.Cu") (net 20))
   (segment (start 114.3 61.785) (end 114.3 63.5) (width 0.25) (layer "F.Cu") (net 21))
@@
   (segment (start 121.92 66.04) (end 121.92 78.74) (width 0.25) (layer "B.Cu") (net 21))
   (segment (start 121.92 78.74) (end 121.92 101.6) (width 0.25) (layer "B.Cu") (net 21))
+  (segment (start 111.273501 115.474511) (end 109.22 113.42101) (width 0.25) (layer "F.Cu") (net 22))
+  (segment (start 116.299511 115.474511) (end 111.273501 115.474511) (width 0.25) (layer "F.Cu") (net 22))
   (segment (start 109.22 99.06) (end 111.76 101.6) (width 0.25) (layer "F.Cu") (net 22))
+  (segment (start 109.22 104.14) (end 111.76 101.6) (width 0.25) (layer "F.Cu") (net 22))
   (segment (start 109.22 88.9) (end 110.935 88.9) (width 0.25) (layer "F.Cu") (net 22))
   (segment (start 110.935 63.5) (end 109.22 65.215) (width 0.25) (layer "F.Cu") (net 22))
+  (segment (start 109.22 113.42101) (end 109.22 104.14) (width 0.25) (layer "F.Cu") (net 22))
   (segment (start 109.22 88.9) (end 109.22 99.06) (width 0.25) (layer "F.Cu") (net 22))
   (segment (start 109.22 65.215) (end 109.22 88.9) (width 0.25) (layer "F.Cu") (net 22))
+  (segment (start 117.665 116.84) (end 116.299511 115.474511) (width 0.25) (layer "F.Cu") (net 22))
   (segment (start 113.1875 83.82) (end 112.075 83.82) (width 0.25) (layer "F.Cu") (net 23))
   (segment (start 114.3 84.9325) (end 114.3 88.9) (width 0.25) (layer "F.Cu") (net 23))
@@
   (segment (start 119.38 91.44) (end 119.38 93.98) (width 0.25) (layer "B.Cu") (net 23))
   (segment (start 111.76 116.84) (end 116.015 116.84) (width 0.25) (layer "F.Cu") (net 24))
+  (segment (start 159.53548 117.63952) (end 116.81452 117.63952) (width 0.25) (layer "F.Cu") (net 24))
+  (segment (start 165.415 111.76) (end 159.53548 117.63952) (width 0.25) (layer "F.Cu") (net 24))
+  (segment (start 116.81452 117.63952) (end 116.015 116.84) (width 0.25) (layer "F.Cu") (net 24))
   (segment (start 122.8325 61.8725) (end 121.92 60.96) (width 0.25) (layer "F.Cu") (net 25))
   (segment (start 124.46 61.8725) (end 122.8325 61.8725) (width 0.25) (layer "F.Cu") (net 25))
