File: epanel-io/prototype-2/prototype-2.kicad_pcb (KiCad board)
At the start: 2 copper layers, 87 x 68 mm, 28 parts, among them J1 Conn_01x07_Male, J2 Screw_Terminal_01x04, J3 Screw_Terminal_01x04, J4 Screw_Terminal_01x02, Q1 IRF830, Q2 IRF830, U2 4N35, U3 4N35, U4 H11AA1, U5 H11AA1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

Commit message: try to improve pcb
Routing:
- net +3V3: track 64.3 -> 65.3 mm
Changed lines of the file:
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@@
   (segment (start 121.92 66.04) (end 121.92 78.74) (width 0.25) (layer "B.Cu") (net 21))
   (segment (start 121.92 78.74) (end 121.92 101.6) (width 0.25) (layer "B.Cu") (net 21))
-  (segment (start 111.273501 115.474511) (end 109.22 113.42101) (width 0.25) (layer "F.Cu") (net 22))
-  (segment (start 116.299511 115.474511) (end 111.273501 115.474511) (width 0.25) (layer "F.Cu") (net 22))
-  (segment (start 109.22 99.06) (end 111.76 101.6) (width 0.25) (layer "F.Cu") (net 22))
-  (segment (start 109.22 104.14) (end 111.76 101.6) (width 0.25) (layer "F.Cu") (net 22))
+  (segment (start 116.299511 115.474511) (end 110.394511 115.474511) (width 0.25) (layer "F.Cu") (net 22))
+  (segment (start 117.665 116.84) (end 116.299511 115.474511) (width 0.25) (layer "F.Cu") (net 22))
+  (segment (start 111.76 101.6) (end 109.22 101.6) (width 0.25) (layer "F.Cu") (net 22))
+  (segment (start 110.394511 115.474511) (end 109.22 114.3) (width 0.25) (layer "F.Cu") (net 22))
   (segment (start 109.22 88.9) (end 110.935 88.9) (width 0.25) (layer "F.Cu") (net 22))
   (segment (start 110.935 63.5) (end 109.22 65.215) (width 0.25) (layer "F.Cu") (net 22))
-  (segment (start 109.22 113.42101) (end 109.22 104.14) (width 0.25) (layer "F.Cu") (net 22))
-  (segment (start 109.22 88.9) (end 109.22 99.06) (width 0.25) (layer "F.Cu") (net 22))
+  (segment (start 109.22 114.3) (end 109.22 101.6) (width 0.25) (layer "F.Cu") (net 22))
+  (segment (start 109.22 101.6) (end 109.22 88.9) (width 0.25) (layer "F.Cu") (net 22))
   (segment (start 109.22 65.215) (end 109.22 88.9) (width 0.25) (layer "F.Cu") (net 22))
-  (segment (start 117.665 116.84) (end 116.299511 115.474511) (width 0.25) (layer "F.Cu") (net 22))
   (segment (start 113.1875 83.82) (end 112.075 83.82) (width 0.25) (layer "F.Cu") (net 23))
   (segment (start 114.3 84.9325) (end 114.3 88.9) (width 0.25) (layer "F.Cu") (net 23))

Commit message: improve pcb
Routing:
- net Net-(R5-Pad1): track 56.4 -> 60.0 mm, vias 0 -> 1
- net GND: track 120.5 -> 119.2 mm
Changed lines of the file:
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@@
   (segment (start 178.635 93.98) (end 178.625 93.97) (width 1) (layer "F.Cu") (net 8))
   (segment (start 116.84 68.58) (end 113.03 68.58) (width 0.25) (layer "F.Cu") (net 9))
-  (segment (start 160.02 101.6) (end 165.415 106.995) (width 0.25) (layer "F.Cu") (net 9))
-  (segment (start 116.84 101.6) (end 160.02 101.6) (width 0.25) (layer "F.Cu") (net 9))
   (segment (start 112.075 55.88) (end 114.3 55.88) (width 0.25) (layer "F.Cu") (net 9))
   (segment (start 116.84 58.42) (end 116.84 68.58) (width 0.25) (layer "F.Cu") (net 9))
@@
   (segment (start 116.84 81.28) (end 116.84 93.98) (width 0.25) (layer "F.Cu") (net 9))
   (segment (start 116.84 93.98) (end 113.03 93.98) (width 0.25) (layer "F.Cu") (net 9))
-  (segment (start 165.415 106.995) (end 165.415 109.22) (width 0.25) (layer "F.Cu") (net 9))
   (segment (start 116.84 99.06) (end 116.84 101.6) (width 0.25) (layer "F.Cu") (net 9))
   (segment (start 116.84 68.58) (end 116.84 81.28) (width 0.25) (layer "F.Cu") (net 9))
   (segment (start 116.84 81.28) (end 112.075 81.28) (width 0.25) (layer "F.Cu") (net 9))
+  (segment (start 127 109.22) (end 119.38 101.6) (width 0.25) (layer "F.Cu") (net 9))
+  (segment (start 165.415 109.22) (end 127 109.22) (width 0.25) (layer "F.Cu") (net 9))
   (segment (start 114.3 55.88) (end 116.84 58.42) (width 0.25) (layer "F.Cu") (net 9))
+  (segment (start 116.84 101.6) (end 119.38 101.6) (width 0.25) (layer "F.Cu") (net 9))
   (segment (start 114.3 104.14) (end 111.76 104.14) (width 0.25) (layer "F.Cu") (net 9))
   (segment (start 129.99625 86.36) (end 129.08375 85.4475) (width 0.25) (layer "F.Cu") (net 10))
@@
   (segment (start 119.38 93.98) (end 119.38 99.06) (width 0.25) (layer "B.Cu") (net 23))
   (segment (start 119.38 91.44) (end 119.38 93.98) (width 0.25) (layer "B.Cu") (net 23))
+  (segment (start 165.415 111.76) (end 127 111.76) (width 0.25) (layer "F.Cu") (net 24))
   (segment (start 111.76 116.84) (end 116.015 116.84) (width 0.25) (layer "F.Cu") (net 24))
-  (segment (start 159.53548 117.63952) (end 116.81452 117.63952) (width 0.25) (layer "F.Cu") (net 24))
-  (segment (start 165.415 111.76) (end 159.53548 117.63952) (width 0.25) (layer "F.Cu") (net 24))
-  (segment (start 116.81452 117.63952) (end 116.015 116.84) (width 0.25) (layer "F.Cu") (net 24))
+  (via (at 127 111.76) (size 0.8) (drill 0.4) (layers "F.Cu" "B.Cu") (net 24))
+  (segment (start 121.92 116.84) (end 127 111.76) (width 0.25) (layer "B.Cu") (net 24))
+  (segment (start 111.76 116.84) (end 121.92 116.84) (width 0.25) (layer "B.Cu") (net 24))
   (segment (start 122.8325 61.8725) (end 121.92 60.96) (width 0.25) (layer "F.Cu") (net 25))
   (segment (start 124.46 61.8725) (end 122.8325 61.8725) (width 0.25) (layer "F.Cu") (net 25))
