File: epanel-io/prototype-2/prototype-2.kicad_sch (KiCad schematic)
At the start: 28 parts

Commit message: wip schematic
Parts:
- added SW1: SW_Push, symbol Switch:SW_Push
- added U1: Pico, RPi_Pico:RPi_Pico_SMD_TH, symbol MCU_RaspberryPi_and_Boards:Pico
- J1: renamed from J?; LCSC (none) -> C390682
- J2, J3: renamed from J?; footprint (none) -> TerminalBlock:TerminalBlock_bornier-4_P5.08mm
- PS1, PS2: renamed from PS?; LCSC (none) -> C209905
- gave numbers to parts that had none: 23
Connections:
- net +3V3: now also U1.36 (3V3); no longer J1.1 (Pin_1)
- net GND: now also SW1.2, U1.38 (GND)
- net at R4.1, U5.5: now also U1.16 (GPIO12)
- net at R1.2: now also U1.15 (GPIO11)
- net at R5.1, U6.5: now also U1.20 (GPIO15)
- net at R3.1, U4.5: now also U1.14 (GPIO10)
- net at J1.3 (Pin_3): now also U1.5 (GPIO3)
- net at J1.4 (Pin_4): now also U1.6 (GPIO4)
- net at J1.5 (Pin_5): now also U1.7 (GPIO5)
- net at R2.2: now also U1.17 (GPIO13)
- new net: SW1.1, U1.30 (RUN)
- new net +5V: J1.1 (Pin_1), U1.40 (VBUS)
Other:
- moved on the sheet: D1, D2, J1, J2, J3, J4, PS1, PS2, Q1, Q2, R1, R10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

Commit message: add footprints
Parts:
- SW1: footprint (none) -> Button_Switch_SMD:SW_SPST_REED_CT05-XXXX-J1; LCSC (none) -> C843669
Changed lines of the file:
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@@
     (property "Reference" "SW1" (id 0) (at 138.43 49.53 0))
     (property "Value" "SW_Push" (id 1) (at 138.43 52.07 0))
-    (property "Footprint" "" (id 2) (at 138.43 52.07 0)
+    (property "Footprint" "Button_Switch_SMD:SW_SPST_REED_CT05-XXXX-J1" (id 2) (at 138.43 52.07 0)
       (effects (font (size 1.27 1.27)) hide)
     )
     (property "Datasheet" "~" (id 3) (at 138.43 52.07 0)
+      (effects (font (size 1.27 1.27)) hide)
+    )
+    (property "LCSC" "C843669" (id 4) (at 138.43 57.15 0)
       (effects (font (size 1.27 1.27)) hide)
     )
@@
     )
     (path "/45442ab1-3603-477d-8386-dd6ae8b86d67"
-      (reference "SW1") (unit 1) (value "SW_Push") (footprint "")
+      (reference "SW1") (unit 1) (value "SW_Push") (footprint "Button_Switch_SMD:SW_SPST_REED_CT05-XXXX-J1")
     )
     (path "/15e614d5-b0e5-4340-a74c-5a64fbe16abe"

Commit message: wip pcb
Parts:
- U1: footprint RPi_Pico:RPi_Pico_SMD_TH -> MCU_RaspberryPi_and_Boards:RPi_Pico_SMD_TH
Connections:
- net at R8.1: now also J2.4 (Pin_4), PS1.2 (AC/N); no longer J2.3 (Pin_3)
- net at J3.4 (Pin_4), PS2.2 (AC/N): now also R10.1; no longer R11.1
- net at J3.3 (Pin_3): now also R11.1; no longer R10.1
- new net: J2.3 (Pin_3), R9.1
Changed lines of the file:
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@@
   (junction (at 224.79 177.8) (diameter 0) (color 0 0 0 0)
   )
+  (junction (at 355.6 64.77) (diameter 0) (color 0 0 0 0)
+  )
   (junction (at 355.6 57.15) (diameter 0) (color 0 0 0 0)
   )
@@
   (junction (at 236.22 154.94) (diameter 0) (color 0 0 0 0)
   )
-  (junction (at 359.41 64.77) (diameter 0) (color 0 0 0 0)
-  )
-  (junction (at 359.41 151.13) (diameter 0) (color 0 0 0 0)
-  )
   (junction (at 236.22 68.58) (diameter 0) (color 0 0 0 0)
   )
   (junction (at 355.6 143.51) (diameter 0) (color 0 0 0 0)
+  )
+  (junction (at 355.6 151.13) (diameter 0) (color 0 0 0 0)
   )
   (junction (at 250.19 68.58) (diameter 0) (color 0 0 0 0)
@@
     (stroke (width 0) (type default) (color 0 0 0 0))
   )
+  (wire (pts (xy 359.41 62.23) (xy 364.49 62.23))
+    (stroke (width 0) (type default) (color 0 0 0 0))
+  )
   (wire (pts (xy 234.95 224.79) (xy 240.03 224.79))
     (stroke (width 0) (type default) (color 0 0 0 0))
@@
     (stroke (width 0) (type default) (color 0 0 0 0))
   )
-  (wire (pts (xy 355.6 62.23) (xy 364.49 62.23))
-    (stroke (width 0) (type default) (color 0 0 0 0))
-  )
   (wire (pts (xy 52.07 34.29) (xy 52.07 46.99))
     (stroke (width 0) (type default) (color 0 0 0 0))
@@
     (stroke (width 0) (type default) (color 0 0 0 0))
   )
-  (wire (pts (xy 359.41 64.77) (xy 359.41 93.98))
-    (stroke (width 0) (type default) (color 0 0 0 0))
-  )
   (wire (pts (xy 134.62 30.48) (xy 134.62 31.75))
     (stroke (width 0) (type default) (color 0 0 0 0))
@@
     (stroke (width 0) (type default) (color 0 0 0 0))
   )
-  (wire (pts (xy 359.41 151.13) (xy 364.49 151.13))
+  (wire (pts (xy 355.6 151.13) (xy 364.49 151.13))
     (stroke (width 0) (type default) (color 0 0 0 0))
   )
@@
     (stroke (width 0) (type default) (color 0 0 0 0))
   )
-  (wire (pts (xy 359.41 151.13) (xy 359.41 180.34))
-    (stroke (width 0) (type default) (color 0 0 0 0))
-  )
   (wire (pts (xy 236.22 154.94) (xy 250.19 154.94))
     (stroke (width 0) (type default) (color 0 0 0 0))
@@
     (stroke (width 0) (type default) (color 0 0 0 0))
   )
-  (wire (pts (xy 355.6 148.59) (xy 355.6 170.18))
-    (stroke (width 0) (type default) (color 0 0 0 0))
-  )
   (wire (pts (xy 226.06 151.13) (xy 226.06 154.94))
     (stroke (width 0) (type default) (color 0 0 0 0))
   )
+  (wire (pts (xy 359.41 148.59) (xy 359.41 180.34))
+    (stroke (width 0) (type default) (color 0 0 0 0))
+  )
   (polyline (pts (xy 189.23 204.47) (xy 189.23 233.68))
     (stroke (width 0) (type default) (color 0 0 0 0))
@@
     (stroke (width 0) (type default) (color 0 0 0 0))
   )
-  (wire (pts (xy 350.52 64.77) (xy 359.41 64.77))
+  (wire (pts (xy 350.52 64.77) (xy 355.6 64.77))
     (stroke (width 0) (type default) (color 0 0 0 0))
   )
@@
     (stroke (width 0) (type default) (color 0 0 0 0))
   )
+  (wire (pts (xy 355.6 64.77) (xy 355.6 83.82))
+    (stroke (width 0) (type default) (color 0 0 0 0))
+  )
   (wire (pts (xy 250.19 147.32) (xy 250.19 154.94))
     (stroke (width 0) (type default) (color 0 0 0 0))
@@
     (stroke (width 0) (type default) (color 0 0 0 0))
   )
-  (wire (pts (xy 355.6 62.23) (xy 355.6 83.82))
-    (stroke (width 0) (type default) (color 0 0 0 0))
-  )
   (wire (pts (xy 234.95 180.34) (xy 240.03 180.34))
     (stroke (width 0) (type default) (color 0 0 0 0))
@@
     (stroke (width 0) (type default) (color 0 0 0 0))
   )
+  (wire (pts (xy 359.41 62.23) (xy 359.41 93.98))
+    (stroke (width 0) (type default) (color 0 0 0 0))
+  )
   (wire (pts (xy 200.66 142.24) (xy 200.66 147.32))
     (stroke (width 0) (type default) (color 0 0 0 0))
@@
     (stroke (width 0) (type default) (color 0 0 0 0))
   )
-  (wire (pts (xy 350.52 151.13) (xy 359.41 151.13))
+  (wire (pts (xy 350.52 151.13) (xy 355.6 151.13))
     (stroke (width 0) (type default) (color 0 0 0 0))
   )
@@
     (stroke (width 0) (type default) (color 0 0 0 0))
   )
-  (wire (pts (xy 355.6 148.59) (xy 364.49 148.59))
-    (stroke (width 0) (type default) (color 0 0 0 0))
-  )
   (wire (pts (xy 269.24 152.4) (xy 269.24 143.51))
     (stroke (width 0) (type default) (color 0 0 0 0))
@@
     (stroke (width 0) (type default) (color 0 0 0 0))
   )
+  (wire (pts (xy 359.41 148.59) (xy 364.49 148.59))
+    (stroke (width 0) (type default) (color 0 0 0 0))
+  )
   (wire (pts (xy 199.39 137.16) (xy 204.47 137.16))
     (stroke (width 0) (type default) (color 0 0 0 0))
@@
     (stroke (width 0) (type default) (color 0 0 0 0))
   )
+  (wire (pts (xy 355.6 151.13) (xy 355.6 170.18))
+    (stroke (width 0) (type default) (color 0 0 0 0))
+  )
   (wire (pts (xy 224.79 210.82) (xy 224.79 213.36))
     (stroke (width 0) (type default) (color 0 0 0 0))
@@
     (stroke (width 0) (type default) (color 0 0 0 0))
   )
-  (wire (pts (xy 359.41 64.77) (xy 364.49 64.77))
+  (wire (pts (xy 355.6 64.77) (xy 364.49 64.77))
     (stroke (width 0) (type default) (color 0 0 0 0))
   )
@@
     (property "Reference" "U1" (id 0) (at 105.41 24.13 0))
     (property "Value" "Pico" (id 1) (at 105.41 26.67 0))
-    (property "Footprint" "RPi_Pico:RPi_Pico_SMD_TH" (id 2) (at 105.41 55.88 90)
+    (property "Footprint" "MCU_RaspberryPi_and_Boards:RPi_Pico_SMD_TH" (id 2) (at 105.41 55.88 90)
       (effects (font (size 1.27 1.27)) hide)
     )
@@
     )
     (path "/15e614d5-b0e5-4340-a74c-5a64fbe16abe"
-      (reference "U1") (unit 1) (value "Pico") (footprint "RPi_Pico:RPi_Pico_SMD_TH")
+      (reference "U1") (unit 1) (value "Pico") (footprint "MCU_RaspberryPi_and_Boards:RPi_Pico_SMD_TH")
     )
     (path "/70396b64-ba42-4955-ac7d-aeff65748330"

Commit message: remove pico from pcb
Parts:
- removed J1: Conn_01x05_Male, Connector_PinHeader_2.54mm:PinHeader_1x05_P2.54mm_Vertical, symbol Connector:Conn_01x05_Male
- removed SW1: SW_Push, Button_Switch_SMD:SW_SPST_REED_CT05-XXXX-J1, symbol Switch:SW_Push
- removed U1: Pico, MCU_RaspberryPi_and_Boards:RPi_Pico_SMD_TH, symbol MCU_RaspberryPi_and_Boards:Pico
- added J1: Conn_01x07_Male, symbol Connector:Conn_01x07_Male
Connections:
- net +3V3: now also J1.1 (Pin_1)
- net GND: now also J1.2 (Pin_2)
- net at R4.1, U5.5: now also J1.6 (Pin_6)
- net at R1.2: now also J1.3 (Pin_3)
- net at R3.1, U4.5: now also J1.4 (Pin_4)
- net at R2.2: now also J1.5 (Pin_5)
- net at R5.1, U6.5: now also J1.7 (Pin_7)

Commit message: try other schematic
Parts:
- removed D2: 4* 1N5408, Diode_SMD:Diode_Bridge_Diotec_SO-DIL-Slim, symbol Device:D_Bridge_+-AA
- removed PS2: HLK-PM12, Converter_ACDC:Converter_ACDC_HiLink_HLK-PMxx, symbol Converter_ACDC:HLK-PM12
- added C1: 2.2uF/63V, Capacitor_SMD:C_1206_3216Metric, symbol Device:C_Polarized
- added D2: 10V/0.4W, Diode_SMD:D_SOD-123, symbol Diode:BZV55B10
- added D3: 1N4007, Diode_SMD:D_SMA, symbol Diode:1N4007
- added Q3: IRF830, Package_TO_SOT_SMD:TO-263-3_TabPin2, symbol Transistor_FET:IRF740
- added R14, R15: 33KΩ/0.5W, Resistor_SMD:R_0603_1608Metric, symbol Device:R
Connections:
- net at Q2.2 (D): now also J3.1 (Pin_1), D3.2 (A)
- net at Q2.3 (S), R7.2: now also C1.2, D2.2 (A), Q3.3 (S)
- net at J3.2 (Pin_2): now also Q3.2 (D)
- net at Q2.1 (G), R7.1, U3.4: now also Q3.1 (G)
- net at U3.5: now also C1.1, D2.1 (K), R14.2
- new net: D3.1 (K), R15.1
- new net: R14.1, R15.2

Commit message: update schematic
Parts:
- J1: footprint (none) -> Connector_PinHeader_2.54mm:PinHeader_1x07_P2.54mm_Vertical
Changed lines of the file:
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@@
     (property "Reference" "J1" (id 0) (at 42.545 68.58 0))
     (property "Value" "Conn_01x07_Male" (id 1) (at 42.545 71.12 0))
-    (property "Footprint" "" (id 2) (at 41.91 81.28 0)
+    (property "Footprint" "Connector_PinHeader_2.54mm:PinHeader_1x07_P2.54mm_Vertical" (id 2) (at 41.91 81.28 0)
       (effects (font (size 1.27 1.27)) hide)
     )
@@
     )
     (path "/e31efd23-be24-4c15-b84c-d88bbfadcb94"
-      (reference "J1") (unit 1) (value "Conn_01x07_Male") (footprint "")
+      (reference "J1") (unit 1) (value "Conn_01x07_Male") (footprint "Connector_PinHeader_2.54mm:PinHeader_1x07_P2.54mm_Vertical")
     )
     (path "/d32932d2-0f28-4db7-8df8-ecaa16aba6bd"

Commit message: update R refs
Parts:
- R14, R15: footprint Resistor_SMD:R_0603_1608Metric -> Resistor_SMD:R_0805_2012Metric
Changed lines of the file:
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@@
     (property "Reference" "R15" (id 0) (at 288.29 118.2075 90))
     (property "Value" "33KΩ/0.5W" (id 1) (at 288.29 120.9826 90))
-    (property "Footprint" "Resistor_SMD:R_0603_1608Metric" (id 2) (at 288.29 121.412 90)
-      (effects (font (size 1.27 1.27)) hide)
-    )
-    (property "Datasheet" "https://datasheet.lcsc.com/lcsc/1811091810_UNI-ROYAL-Uniroyal-Elec-0603WAF3302T5E_C4216.pdf" (id 3) (at 288.29 123.19 0)
+    (property "Footprint" "Resistor_SMD:R_0805_2012Metric" (id 2) (at 288.29 121.412 90)
+      (effects (font (size 1.27 1.27)) hide)
+    )
+    (property "Datasheet" "https://datasheet.lcsc.com/lcsc/2012181743_UNI-ROYAL-Uniroyal-Elec-AS05W2J0333T5E_C966118.pdf" (id 3) (at 288.29 123.19 0)
       (effects (font (size 1.27 1.27)) hide)
     )
@@
     (property "Reference" "R14" (id 0) (at 273.05 118.2075 90))
     (property "Value" "33KΩ/0.5W" (id 1) (at 273.05 120.9826 90))
-    (property "Footprint" "Resistor_SMD:R_0603_1608Metric" (id 2) (at 273.05 121.412 90)
-      (effects (font (size 1.27 1.27)) hide)
-    )
-    (property "Datasheet" "https://datasheet.lcsc.com/lcsc/1811091810_UNI-ROYAL-Uniroyal-Elec-0603WAF3302T5E_C4216.pdf" (id 3) (at 273.05 123.19 0)
+    (property "Footprint" "Resistor_SMD:R_0805_2012Metric" (id 2) (at 273.05 121.412 90)
+      (effects (font (size 1.27 1.27)) hide)
+    )
+    (property "Datasheet" "https://datasheet.lcsc.com/lcsc/2012181743_UNI-ROYAL-Uniroyal-Elec-AS05W2J0333T5E_C966118.pdf" (id 3) (at 273.05 123.19 0)
       (effects (font (size 1.27 1.27)) hide)
     )
@@
     )
     (path "/91131205-e84d-4112-aca5-975fc611e50f"
-      (reference "R14") (unit 1) (value "33KΩ/0.5W") (footprint "Resistor_SMD:R_0603_1608Metric")
+      (reference "R14") (unit 1) (value "33KΩ/0.5W") (footprint "Resistor_SMD:R_0805_2012Metric")
     )
     (path "/238a3140-61d8-47d2-a808-dbdb2b6fae29"
-      (reference "R15") (unit 1) (value "33KΩ/0.5W") (footprint "Resistor_SMD:R_0603_1608Metric")
+      (reference "R15") (unit 1) (value "33KΩ/0.5W") (footprint "Resistor_SMD:R_0805_2012Metric")
     )
     (path "/70396b64-ba42-4955-ac7d-aeff65748330"
