File: epanel-io/prototype-3/prototype-3.kicad_sch (KiCad schematic)
At the start: 35 parts, among them J1 Conn_01x07_Male, Q2 IRF830, Q3 IRF830, U3 4N35, U4 H11AA1, U5 H11AA1, U6 H11AA1

Commit message: wip proto 3
Parts:
- removed J1: Conn_01x07_Male, Connector_PinHeader_2.54mm:PinHeader_1x07_P2.54mm_Vertical, symbol Connector:Conn_01x07_Male
- added JP? (x2): Jumper_2_Bridged, symbol Jumper:Jumper_2_Bridged
- added PS?: HLK-PM01, Converter_ACDC:Converter_ACDC_HiLink_HLK-PMxx, symbol Converter_ACDC:HLK-PM01
- added U?: Pico, RPi_Pico:RPi_Pico_SMD_TH, symbol MCU_RaspberryPi_and_Boards:Pico
Connections:
- net +3V3: now also U?.36 (3V3)
- net GND: now also PS?.3 (-Vout), U?.38 (GND)
- net LINE: now also PS?.1 (AC/L)
- net NEUT: now also PS?.2 (AC/N)
- net at R4.1, U5.5: now also U?.21 (GPIO16)
- net at R5.1, U6.5: now also U?.17 (GPIO13)
- net at R3.1, U4.5: now also U?.19 (GPIO14)
- net at R?.2: now also U?.20 (GPIO15)
- net at R2.2: now also U?.22 (GPIO17)
- new net: JP?.1 (A), U?.39 (VSYS)
- new net +5V: JP?.2 (B), JP?.2 (B), PS?.4 (+Vout)

Commit message: wip proto 3
Parts:
- removed JP?: Jumper_2_Bridged, symbol Jumper:Jumper_2_Bridged
- added J1: Conn_01x05_Male, Connector_PinHeader_2.54mm:PinHeader_1x05_P2.54mm_Vertical, symbol Connector:Conn_01x05_Male
- J2, J3: renamed from J?; footprint (none) -> TerminalBlock:TerminalBlock_bornier-3_P5.08mm
- JP1: renamed from JP?; footprint (none) -> Connector_PinHeader_2.54mm:PinHeader_1x02_P2.54mm_Vertical
- U1: renamed from U?; footprint RPi_Pico:RPi_Pico_SMD_TH -> MCU_RaspberryPi_and_Boards:RPi_Pico_SMD_TH
- gave numbers to parts that had none: 11
- renumbered C1 to C2, D3 to D4, Q2 to Q3, Q3 to Q4, R8 to R10, R9 to R11, R10 to R12, R11 to R13, R12 to R14, R13 to R15, R15 to R17, R14 to R9
Connections:
- net +5V: now also J1.1 (Pin_1)
- net GND: now also J1.2 (Pin_2)
- net at U1.5 (GPIO3): now also J1.3 (Pin_3)
- net at U1.6 (GPIO4): now also J1.4 (Pin_4)
- net at U1.7 (GPIO5): now also J1.5 (Pin_5)
