File: epanel-energy-monitor/prototype-1/prototype-1.kicad_pcb (KiCad board)
At the start: 2 copper layers, 87 x 68 mm, 38 parts, among them J1 Conn_01x05_Male, J2 Screw_Terminal_01x03, J3 Screw_Terminal_01x03, Q1 IRF830, Q2 IRF830, Q3 IRF830, Q4 IRF830, U1 Pico, U2 4N35, U3 4N35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

Commit message: wip footprints
Parts:
- removed C1, C2: 2.2uF/63V, Capacitor_SMD:C_1206_3216Metric
- removed D1, D2: 10V/0.4W, Diode_SMD:D_SOD-123
- removed D3, D4: 1N4007, Diode_SMD:D_SMA
- removed J1: Conn_01x05_Male, Connector_PinHeader_2.54mm:PinHeader_1x05_P2.54mm_Vertical
- removed J2, J3: Screw_Terminal_01x03, TerminalBlock:TerminalBlock_bornier-3_P5.08mm
- removed JP1: Jumper_2_Bridged, Connector_PinHeader_2.54mm:PinHeader_1x02_P2.54mm_Vertical
- removed PS1: HLK-PM01, Converter_ACDC:Converter_ACDC_HiLink_HLK-PMxx
- removed Q1, Q2, Q3, Q4: IRF830, Package_TO_SOT_SMD:TO-263-3_TabPin2
- removed R1, R2: 330Ω, Resistor_SMD:R_0603_1608Metric
- removed R10, R11, R12, R13, R14, R15, R16, R17, R8, R9: 33KΩ/0.5W, Resistor_SMD:R_0805_2012Metric
- removed R3, R4, R5: 10KΩ, Resistor_SMD:R_0603_1608Metric
- removed R6, R7: 22KΩ, Resistor_SMD:R_0603_1608Metric
- removed U1: Pico, MCU_RaspberryPi_and_Boards:RPi_Pico_SMD_TH
- removed U2, U3: 4N35, Package_DIP:SMDIP-6_W7.62mm
- removed U4, U5, U6: H11AA1, Package_DIP:SMDIP-6_W9.53mm
Routing:
- net GND: track 166.4 -> 0.00 mm, vias 1 -> 0
- net NEUT: track 136.0 -> 0.00 mm, vias 5 -> 0
- net +5V: track 100.7 -> 0.00 mm, vias 2 -> 0
- net Net-(Q1-Pad1): track 87.5 -> 0.00 mm, vias 4 -> 0
- net Net-(R3-Pad1): track 77.3 -> 0.00 mm
- net Net-(R4-Pad1): track 74.4 -> 0.00 mm
- net LINE: track 68.3 -> 0.00 mm
- net Net-(Q3-Pad1): track 64.5 -> 0.00 mm, vias 4 -> 0
- net Net-(R5-Pad1): track 61.4 -> 0.00 mm
- net Net-(J1-Pad3): track 54.4 -> 0.00 mm
- net Net-(J1-Pad4): track 52.2 -> 0.00 mm
- net Net-(J1-Pad5): track 50.4 -> 0.00 mm
- net Net-(C1-Pad1): track 48.3 -> 0.00 mm, vias 2 -> 0
- net Net-(R15-Pad2): track 46.7 -> 0.00 mm
- net Net-(J2-Pad2): track 42.4 -> 0.00 mm
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Other:
- board text removed: "5V5"
- board text removed: "GND"
- board text removed: "I1"
- board text removed: "I2"
- board text removed: "INTR"
- board text removed: "O 1"
- board text removed: "O 2"
- board text removed: "SCL"
- board text removed: "SDA"

Commit message: wip pcb skeleton
Parts:
- added C1: 10uF/6V, Resistor_SMD:R_0603_1608Metric, F.Cu at (74.9, 80.0)
- added C2: 10uF/6V, Resistor_SMD:R_0603_1608Metric, F.Cu at (79.3, 77.1)
- added J1: Conn_01x06_Male, Connector_PinHeader_2.54mm:PinHeader_1x06_P2.54mm_Vertical, F.Cu at (83.7, 56.6)
- added J2: AudioJack4, Connector_Audio:Jack_3.5mm_PJ320D_Horizontal, F.Cu at (54.8, 81.3)
- added J3: AudioJack4, Connector_Audio:Jack_3.5mm_PJ320D_Horizontal, F.Cu at (90.6, 77.1)
- added J4: Screw_Terminal_01x02, TerminalBlock:TerminalBlock_bornier-2_P5.08mm, F.Cu at (64.6, 80.3)
- added J5: Screw_Terminal_01x02, TerminalBlock:TerminalBlock_bornier-2_P5.08mm, F.Cu at (89.2, 58.8)
- added J6: Conn_01x02_Male, Connector_PinHeader_2.54mm:PinHeader_1x02_P2.54mm_Vertical, F.Cu at (99.9, 56.6)
- added J7: Conn_01x02_Male, Connector_PinHeader_2.54mm:PinHeader_1x02_P2.54mm_Vertical, F.Cu at (88.3, 65.6)
- added PS1: HLK-PM01, Converter_ACDC:Converter_ACDC_HiLink_HLK-PMxx, F.Cu at (48.9, 62.5)
- added Q1: BS170, Package_TO_SOT_SMD:SOT-23, F.Cu at (48.0, 89.1)
- added R1: 1KΩ, Resistor_SMD:R_0603_1608Metric, F.Cu at (92.7, 64.6)
- added R10: 120Ω/0.5W, Resistor_SMD:R_0805_2012Metric, F.Cu at (52.6, 88.3)
- added R11: 4.7KΩ, Resistor_SMD:R_0603_1608Metric, F.Cu at (56.8, 88.1)
- added R2: 1KΩ, Resistor_SMD:R_0603_1608Metric, F.Cu at (64.8, 88.6)
- added R3: 10KΩ, Resistor_SMD:R_0603_1608Metric, F.Cu at (60.8, 88.6)
- added R4: 470KΩ, Resistor_SMD:R_0603_1608Metric, F.Cu at (67.4, 86.1)
- added R5: 470KΩ, Resistor_SMD:R_0603_1608Metric, F.Cu at (78.9, 80.0)
- added R6: 470KΩ, Resistor_SMD:R_0603_1608Metric, F.Cu at (92.7, 67.1)
- added R7: 470KΩ, Resistor_SMD:R_0603_1608Metric, F.Cu at (99.2, 64.6)
- added R8: 10KΩ, Resistor_SMD:R_0603_1608Metric, F.Cu at (63.4, 86.1)
- added R9: 22Ω/0.5W, Resistor_SMD:R_0805_2012Metric, F.Cu at (75.1, 77.3)
- added U1: LTV-814, Package_DIP:SMDIP-4_W7.62mm, F.Cu at (78.5, 86.0)

Commit message: wip pcb placement
Parts:
- moved J2 127.5 mm to (181.6, 94.0), turned to 180 degrees
- moved J4 124.3 mm to (186.7, 57.1), turned to -90 degrees
- moved PS1 122.6 mm to (171.4, 64.8), turned to 180 degrees
- moved R10 111.3 mm to (162.6, 105.4)
- moved R11 106.1 mm to (162.6, 78.7)
- moved Q1 101.4 mm to (148.9, 80.0)
- moved J5 101.0 mm to (188.0, 80.0), turned to -90 degrees
- moved J3 95.7 mm to (181.6, 106.7), turned to 180 degrees
- moved R2 93.9 mm to (157.5, 104.1)
- moved J7 89.3 mm to (168.9, 104.1)
- moved U1 87.8 mm to (166.4, 83.8)
- moved R8 86.5 mm to (149.9, 85.1)
- moved R9 85.9 mm to (159.1, 95.2)
- moved R3 82.0 mm to (142.2, 78.7)
- moved C2 81.3 mm to (152.8, 111.8)
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
Commit message: first draft
Parts:
- moved R5 41.0 mm to (170.2, 85.1)
- moved C1 39.6 mm to (170.2, 87.0), turned to 180 degrees
- moved R4 26.7 mm to (170.2, 83.2), turned to 180 degrees
- moved R3 24.3 mm to (166.4, 75.6)
- moved R7 23.9 mm to (170.2, 113.0)
- moved R8 22.9 mm to (166.4, 69.2)
- moved PS1 21.6 mm to (152.4, 54.6), turned to -90 degrees
- moved J7 20.7 mm to (189.2, 100.3)
- moved J6 20.4 mm to (189.2, 92.7)
- moved R1 19.1 mm to (170.2, 81.3)
- moved Q1 19.0 mm to (166.4, 72.4), turned to 180 degrees
- moved R9 18.8 mm to (174.0, 83.8), turned to -90 degrees
- moved R6 18.3 mm to (170.2, 111.1), turned to 180 degrees
- moved J1 17.7 mm to (111.8, 74.3)
- moved C2 17.6 mm to (170.2, 114.9), turned to 180 degrees
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Routing:
- net GND: track 0.00 -> 112.9 mm, vias 0 -> 3
- net +3V3: track 0.00 -> 102.2 mm, vias 0 -> 4
- net Net-(J1-Pad6): track 0.00 -> 74.4 mm
- net Net-(J1-Pad4): track 0.00 -> 65.2 mm
- net Net-(J1-Pad5): track 0.00 -> 60.5 mm
- net NEUT: track 0.00 -> 43.2 mm
- net LINE: track 0.00 -> 38.2 mm
- net +5V: track 0.00 -> 34.5 mm
- net Net-(J2-PadS): track 0.00 -> 30.1 mm
- net Net-(C2-Pad1): track 0.00 -> 30.1 mm
- net Net-(C1-Pad1): track 0.00 -> 26.5 mm
- net Net-(J3-PadS): track 0.00 -> 23.3 mm
- net Net-(J5-Pad1): track 0.00 -> 11.2 mm
- net Net-(J5-Pad2): track 0.00 -> 9.04 mm
- net Net-(R11-Pad2): track 0.00 -> 8.75 mm
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Other:
- board text added: "3V3"
- board text added: "5V"
- board text added: "CT0"
- board text added: "CT1"
- board text added: "GND"
- board text added: "Tele"
- board text added: "Teleinfo"
