File: epanel-io/v1/epanel-io.kicad_sch (KiCad schematic)
At the start: 10 parts, among them J1 Conn_01x05_Male, U1 Pico, U6 H11AA1

Commit message: wip schematic 10 io
Parts:
- added J? (x2): Screw_Terminal_01x03, symbol Connector:Screw_Terminal_01x03
Connections:
- net Input 9/RPI: now reaches U1.29 (GPIO22)
- net Input 10/RPI: now reaches U1.31 (GPIO26_ADC0)
- net Output 9/RPI: now reaches U1.32 (GPIO27_ADC1)
- net Output 10/RPI: now reaches U1.34 (GPIO28_ADC2)
- new net Input 10/INPUT: J?.3 (Pin_3)
- new net Input 10/NEUT: J?.1 (Pin_1)
- new net Input 9/INPUT: J?.2 (Pin_2)
- new net Output 10/LINE: J?.1 (Pin_1)
- new net Output 10/OUTPUT: J?.3 (Pin_3)
- new net Output 9/OUTPUT: J?.2 (Pin_2)
Other:
- added sheet Input 10 (input.kicad_sch)
- added sheet Input 9 (input.kicad_sch)
- added sheet Output 10 (output.kicad_sch)
- added sheet Output 9 (output.kicad_sch)
- moved on the sheet: R14, R15, R5, U6

Commit message: annotate
Parts:
- gave numbers to parts that had none: 6
- renumbered R5 to R1, R14 to R2, R15 to R3, U6 to U2

Commit message: ok let's go!
Parts:
- J2, J3, J4, J5: footprint (none) -> TerminalBlock:TerminalBlock_bornier-5_P5.08mm
- J6, J7: footprint (none) -> TerminalBlock:TerminalBlock_bornier-3_P5.08mm

Commit message: fix ZC line/neut
Connections:
- net Input 10/NEUT: now also R2.1
- net LINE: no longer R3.1
- net NEUT: no longer R2.1
- net Output 10/LINE: now also R3.1
Changed lines of the file:
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@@
   (junction (at 241.3 54.61) (diameter 0) (color 0 0 0 0)
   )
+  (junction (at 344.17 90.17) (diameter 0) (color 0 0 0 0)
+  )
   (junction (at 118.11 92.71) (diameter 0) (color 0 0 0 0)
   )
@@
   )
   (junction (at 238.76 93.98) (diameter 0) (color 0 0 0 0)
+  )
+  (junction (at 341.63 93.98) (diameter 0) (color 0 0 0 0)
   )
   (junction (at 118.11 158.75) (diameter 0) (color 0 0 0 0)
@@
     (stroke (width 0) (type default) (color 0 0 0 0))
   )
+  (wire (pts (xy 344.17 90.17) (xy 344.17 247.65))
+    (stroke (width 0) (type default) (color 0 0 0 0))
+  )
   (wire (pts (xy 220.98 259.08) (xy 220.98 260.35))
     (stroke (width 0) (type default) (color 0 0 0 0))
@@
     (stroke (width 0) (type default) (color 0 0 0 0))
   )
-  (wire (pts (xy 275.59 262.89) (xy 283.21 262.89))
+  (wire (pts (xy 275.59 262.89) (xy 294.64 262.89))
     (stroke (width 0) (type default) (color 0 0 0 0))
   )
@@
     (stroke (width 0) (type default) (color 0 0 0 0))
   )
+  (wire (pts (xy 341.63 93.98) (xy 341.63 245.11))
+    (stroke (width 0) (type default) (color 0 0 0 0))
+  )
   (wire (pts (xy 129.54 35.56) (xy 129.54 68.58))
     (stroke (width 0) (type default) (color 0 0 0 0))
@@
     (stroke (width 0) (type default) (color 0 0 0 0))
   )
+  (wire (pts (xy 341.63 245.11) (xy 292.1 245.11))
+    (stroke (width 0) (type default) (color 0 0 0 0))
+  )
   (wire (pts (xy 241.3 54.61) (xy 280.67 54.61))
     (stroke (width 0) (type default) (color 0 0 0 0))
@@
     (stroke (width 0) (type default) (color 0 0 0 0))
   )
+  (wire (pts (xy 292.1 245.11) (xy 292.1 252.73))
+    (stroke (width 0) (type default) (color 0 0 0 0))
+  )
   (wire (pts (xy 213.36 129.54) (xy 193.04 129.54))
     (stroke (width 0) (type default) (color 0 0 0 0))
@@
     (stroke (width 0) (type default) (color 0 0 0 0))
   )
+  (wire (pts (xy 344.17 247.65) (xy 294.64 247.65))
+    (stroke (width 0) (type default) (color 0 0 0 0))
+  )
   (wire (pts (xy 344.17 54.61) (xy 383.54 54.61))
     (stroke (width 0) (type default) (color 0 0 0 0))
@@
     (stroke (width 0) (type default) (color 0 0 0 0))
   )
+  (wire (pts (xy 275.59 252.73) (xy 292.1 252.73))
+    (stroke (width 0) (type default) (color 0 0 0 0))
+  )
   (wire (pts (xy 132.08 111.76) (xy 111.76 111.76))
     (stroke (width 0) (type default) (color 0 0 0 0))
@@
     (stroke (width 0) (type default) (color 0 0 0 0))
   )
+  (wire (pts (xy 294.64 247.65) (xy 294.64 262.89))
+    (stroke (width 0) (type default) (color 0 0 0 0))
+  )
   (wire (pts (xy 383.54 34.29) (xy 353.06 34.29))
     (stroke (width 0) (type default) (color 0 0 0 0))
@@
   )
   (wire (pts (xy 213.36 43.18) (xy 190.5 43.18))
-    (stroke (width 0) (type default) (color 0 0 0 0))
-  )
-  (wire (pts (xy 283.21 252.73) (xy 275.59 252.73))
     (stroke (width 0) (type default) (color 0 0 0 0))
   )
@@
     (pin "1")
   )
-  (symbol (lib_id "power:LINE") (at 283.21 262.89 0) (unit 1)
-    (in_bom yes) (on_board yes) (fields_autoplaced)
-    (property "Reference" "#PWR09" (id 0) (at 283.21 266.7 0)
-      (effects (font (size 1.27 1.27)) hide)
-    )
-    (property "Value" "LINE" (id 1) (at 283.21 257.81 0))
-    (property "Footprint" "" (id 2) (at 283.21 262.89 0)
-      (effects (font (size 1.27 1.27)) hide)
-    )
-    (property "Datasheet" "" (id 3) (at 283.21 262.89 0)
-      (effects (font (size 1.27 1.27)) hide)
-    )
-    (pin "1")
-  )
   (symbol (lib_id "Device:R") (at 271.78 262.89 270) (unit 1)
     (in_bom yes) (on_board yes) (fields_autoplaced)
@@
     (pin "5")
     (pin "6")
-  )
-  (symbol (lib_id "power:NEUT") (at 283.21 252.73 0) (unit 1)
-    (in_bom yes) (on_board yes) (fields_autoplaced)
-    (property "Reference" "#PWR08" (id 0) (at 283.21 256.54 0)
-      (effects (font (size 1.27 1.27)) hide)
-    )
-    (property "Value" "NEUT" (id 1) (at 283.21 247.65 0))
-    (property "Footprint" "" (id 2) (at 283.21 252.73 0)
-      (effects (font (size 1.27 1.27)) hide)
-    )
-    (property "Datasheet" "" (id 3) (at 283.21 252.73 0)
-      (effects (font (size 1.27 1.27)) hide)
-    )
-    (pin "1")
   )
   (symbol (lib_id "Connector:Screw_Terminal_01x05") (at 165.1 35.56 0) (unit 1)
@@
       (reference "#PWR07") (unit 1) (value "GND") (footprint "")
     )
-    (path "/cda037e7-389e-41d1-92e3-ae63dcb55333"
-      (reference "#PWR08") (unit 1) (value "NEUT") (footprint "")
-    )
-    (path "/8976ed33-631b-4eac-a707-8f367e5f14ae"
-      (reference "#PWR09") (unit 1) (value "LINE") (footprint "")
-    )
     (path "/80ac0b57-0388-409c-bf8b-2ee44690ae03/593bd94d-bb1f-4b56-85e8-ef6e8c44a556"
