File: epanel-io/v1/output.kicad_sch (KiCad schematic)
At the start: 10 parts

Commit message: ok let's go!
Parts:
- gave numbers to parts that had none: 10
Changed lines of the file:
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@@
   (symbol (lib_id "Isolator:4N35") (at 130.81 78.74 0)
     (in_bom yes) (on_board yes) (fields_autoplaced)
-    (property "Reference" "U?" (id 0) (at 130.81 70.9635 0))
+    (property "Reference" "U22" (id 0) (at 130.81 70.9635 0))
     (property "Value" "4N35" (id 1) (at 130.81 73.7386 0))
     (property "Footprint" "Package_DIP:SMDIP-6_W7.62mm" (id 2) (at 125.73 83.82 0)
@@
   (symbol (lib_id "Diode:1N4007") (at 220.98 62.23 0)
     (in_bom yes) (on_board yes) (fields_autoplaced)
-    (property "Reference" "D?" (id 0) (at 220.98 56.9935 0))
+    (property "Reference" "D20" (id 0) (at 220.98 56.9935 0))
     (property "Value" "1N4007" (id 1) (at 220.98 59.7686 0))
     (property "Footprint" "Diode_SMD:D_SMA" (id 2) (at 220.98 66.675 0)
@@
   (symbol (lib_id "Device:R") (at 207.01 62.23 270)
     (in_bom yes) (on_board yes) (fields_autoplaced)
-    (property "Reference" "R?" (id 0) (at 207.01 57.2475 90))
+    (property "Reference" "R73" (id 0) (at 207.01 57.2475 90))
     (property "Value" "33KΩ/0.5W" (id 1) (at 207.01 60.0226 90))
     (property "Footprint" "Resistor_SMD:R_0805_2012Metric" (id 2) (at 207.01 60.452 90)
@@
   (symbol (lib_id "Transistor_FET:IRF740") (at 236.22 72.39 0)
     (in_bom yes) (on_board yes) (fields_autoplaced)
-    (property "Reference" "Q?" (id 0) (at 241.427 71.4815 0)
+    (property "Reference" "Q19" (id 0) (at 241.427 71.4815 0)
       (effects (font (size 1.27 1.27)) (justify left))
     )
@@
   (symbol (lib_id "Transistor_FET:IRF740") (at 236.22 85.09 0) (mirror x)
     (in_bom yes) (on_board yes) (fields_autoplaced)
-    (property "Reference" "Q?" (id 0) (at 242.57 83.8199 0)
+    (property "Reference" "Q20" (id 0) (at 242.57 83.8199 0)
       (effects (font (size 1.27 1.27)) (justify left))
     )
@@
   (symbol (lib_id "Device:R") (at 191.77 62.23 270)
     (in_bom yes) (on_board yes) (fields_autoplaced)
-    (property "Reference" "R?" (id 0) (at 191.77 57.2475 90))
+    (property "Reference" "R72" (id 0) (at 191.77 57.2475 90))
     (property "Value" "33KΩ/0.5W" (id 1) (at 191.77 60.0226 90))
     (property "Footprint" "Resistor_SMD:R_0805_2012Metric" (id 2) (at 191.77 60.452 90)
@@
   (symbol (lib_id "Device:C_Polarized") (at 177.8 72.39 0)
     (in_bom yes) (on_board yes) (fields_autoplaced)
-    (property "Reference" "C?" (id 0) (at 180.721 70.5925 0)
+    (property "Reference" "C10" (id 0) (at 180.721 70.5925 0)
       (effects (font (size 1.27 1.27)) (justify left))
     )
@@
   (symbol (lib_id "power:GND") (at 119.38 86.36 0)
     (in_bom yes) (on_board yes)
-    (property "Reference" "#PWR?" (id 0) (at 119.38 92.71 0)
+    (property "Reference" "#PWR039" (id 0) (at 119.38 92.71 0)
       (effects (font (size 1.27 1.27)) hide)
     )
@@
   (symbol (lib_id "Device:R") (at 144.78 86.36 0)
     (in_bom yes) (on_board yes)
-    (property "Reference" "R?" (id 0) (at 140.97 85.09 0))
+    (property "Reference" "R71" (id 0) (at 140.97 85.09 0))
     (property "Value" "22KΩ" (id 1) (at 139.7 87.63 0))
     (property "Footprint" "Resistor_SMD:R_0603_1608Metric" (id 2) (at 143.002 86.36 90)
@@
   (symbol (lib_id "Device:R") (at 114.3 76.2 270)
     (in_bom yes) (on_board yes)
-    (property "Reference" "R?" (id 0) (at 113.03 71.12 90))
+    (property "Reference" "R70" (id 0) (at 113.03 71.12 90))
     (property "Value" "330Ω" (id 1) (at 114.3 73.66 90))
     (property "Footprint" "Resistor_SMD:R_0603_1608Metric" (id 2) (at 114.3 74.422 90)
@@
   (symbol (lib_id "Diode:BZV55B10") (at 160.02 72.39 270)
     (in_bom yes) (on_board yes) (fields_autoplaced)
-    (property "Reference" "D?" (id 0) (at 162.052 71.4815 90)
+    (property "Reference" "D19" (id 0) (at 162.052 71.4815 90)
       (effects (font (size 1.27 1.27)) (justify left))
     )

Commit message: fix ZC line/neut
Parts:
- renumbered C10 to C9, D19 to D17, D20 to D18, Q19 to Q17, Q20 to Q18, R70 to R63, R71 to R64, R72 to R65, R73 to R66, U22 to U20
Changed lines of the file:
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@@
   (symbol (lib_id "Isolator:4N35") (at 130.81 78.74 0)
     (in_bom yes) (on_board yes) (fields_autoplaced)
-    (property "Reference" "U22" (id 0) (at 130.81 70.9635 0))
+    (property "Reference" "U20" (id 0) (at 130.81 70.9635 0))
     (property "Value" "4N35" (id 1) (at 130.81 73.7386 0))
     (property "Footprint" "Package_DIP:SMDIP-6_W7.62mm" (id 2) (at 125.73 83.82 0)
@@
   (symbol (lib_id "Diode:1N4007") (at 220.98 62.23 0)
     (in_bom yes) (on_board yes) (fields_autoplaced)
-    (property "Reference" "D20" (id 0) (at 220.98 56.9935 0))
+    (property "Reference" "D18" (id 0) (at 220.98 56.9935 0))
     (property "Value" "1N4007" (id 1) (at 220.98 59.7686 0))
     (property "Footprint" "Diode_SMD:D_SMA" (id 2) (at 220.98 66.675 0)
@@
   (symbol (lib_id "Device:R") (at 207.01 62.23 270)
     (in_bom yes) (on_board yes) (fields_autoplaced)
-    (property "Reference" "R73" (id 0) (at 207.01 57.2475 90))
+    (property "Reference" "R66" (id 0) (at 207.01 57.2475 90))
     (property "Value" "33KΩ/0.5W" (id 1) (at 207.01 60.0226 90))
     (property "Footprint" "Resistor_SMD:R_0805_2012Metric" (id 2) (at 207.01 60.452 90)
@@
   (symbol (lib_id "Transistor_FET:IRF740") (at 236.22 72.39 0)
     (in_bom yes) (on_board yes) (fields_autoplaced)
-    (property "Reference" "Q19" (id 0) (at 241.427 71.4815 0)
+    (property "Reference" "Q17" (id 0) (at 241.427 71.4815 0)
       (effects (font (size 1.27 1.27)) (justify left))
     )
@@
   (symbol (lib_id "Transistor_FET:IRF740") (at 236.22 85.09 0) (mirror x)
     (in_bom yes) (on_board yes) (fields_autoplaced)
-    (property "Reference" "Q20" (id 0) (at 242.57 83.8199 0)
+    (property "Reference" "Q18" (id 0) (at 242.57 83.8199 0)
       (effects (font (size 1.27 1.27)) (justify left))
     )
@@
   (symbol (lib_id "Device:R") (at 191.77 62.23 270)
     (in_bom yes) (on_board yes) (fields_autoplaced)
-    (property "Reference" "R72" (id 0) (at 191.77 57.2475 90))
+    (property "Reference" "R65" (id 0) (at 191.77 57.2475 90))
     (property "Value" "33KΩ/0.5W" (id 1) (at 191.77 60.0226 90))
     (property "Footprint" "Resistor_SMD:R_0805_2012Metric" (id 2) (at 191.77 60.452 90)
@@
   (symbol (lib_id "Device:C_Polarized") (at 177.8 72.39 0)
     (in_bom yes) (on_board yes) (fields_autoplaced)
-    (property "Reference" "C10" (id 0) (at 180.721 70.5925 0)
+    (property "Reference" "C9" (id 0) (at 180.721 70.5925 0)
       (effects (font (size 1.27 1.27)) (justify left))
     )
@@
   (symbol (lib_id "power:GND") (at 119.38 86.36 0)
     (in_bom yes) (on_board yes)
-    (property "Reference" "#PWR039" (id 0) (at 119.38 92.71 0)
+    (property "Reference" "#PWR036" (id 0) (at 119.38 92.71 0)
       (effects (font (size 1.27 1.27)) hide)
     )
@@
   (symbol (lib_id "Device:R") (at 144.78 86.36 0)
     (in_bom yes) (on_board yes)
-    (property "Reference" "R71" (id 0) (at 140.97 85.09 0))
+    (property "Reference" "R64" (id 0) (at 140.97 85.09 0))
     (property "Value" "22KΩ" (id 1) (at 139.7 87.63 0))
     (property "Footprint" "Resistor_SMD:R_0603_1608Metric" (id 2) (at 143.002 86.36 90)
@@
   (symbol (lib_id "Device:R") (at 114.3 76.2 270)
     (in_bom yes) (on_board yes)
-    (property "Reference" "R70" (id 0) (at 113.03 71.12 90))
+    (property "Reference" "R63" (id 0) (at 113.03 71.12 90))
     (property "Value" "330Ω" (id 1) (at 114.3 73.66 90))
     (property "Footprint" "Resistor_SMD:R_0603_1608Metric" (id 2) (at 114.3 74.422 90)
@@
   (symbol (lib_id "Diode:BZV55B10") (at 160.02 72.39 270)
     (in_bom yes) (on_board yes) (fields_autoplaced)
-    (property "Reference" "D19" (id 0) (at 162.052 71.4815 90)
+    (property "Reference" "D17" (id 0) (at 162.052 71.4815 90)
       (effects (font (size 1.27 1.27)) (justify left))
     )
