File: epanel-io/v1/bottom/bottom.kicad_sch (KiCad schematic)
At the start: 12 parts, among them J1 Conn_01x05_Male, J2 Screw_Terminal_01x05, J3 Screw_Terminal_01x05, J4 Screw_Terminal_01x05, J5 Screw_Terminal_01x05, J6 Screw_Terminal_01x03, J7 Screw_Terminal_01x03, U1 Pico, U2 H11AA1

Commit message: bottom schematics
Parts:
- removed J2: Screw_Terminal_01x05, TerminalBlock:TerminalBlock_bornier-5_P5.08mm, symbol Connector:Screw_Terminal_01x05
- removed R1: 10KΩ, Resistor_SMD:R_0603_1608Metric, symbol Device:R
- removed R2, R3: 33KΩ/0.5W, Resistor_SMD:R_0805_2012Metric, symbol Device:R
- removed U1: Pico, MCU_RaspberryPi_and_Boards:RPi_Pico_SMD_TH, symbol MCU_RaspberryPi_and_Boards:Pico
- removed U2: H11AA1, Package_DIP:SMDIP-6_W9.53mm, symbol Isolator:H11AA1
- added J10, J9: Conn_01x04_Male, Connector_PinHeader_2.54mm:PinHeader_1x04_P2.54mm_Vertical, symbol Connector:Conn_01x04_Male
- added J2, J6: Conn_01x08_Male, Connector_PinHeader_2.54mm:PinHeader_1x08_P2.54mm_Vertical, symbol Connector:Conn_01x08_Male
- added J4: Screw_Terminal_01x05, TerminalBlock:TerminalBlock_bornier-5_P5.08mm, symbol Connector:Screw_Terminal_01x05
- added J5: Conn_01x05_Male, Connector_PinHeader_2.54mm:PinHeader_1x05_P2.54mm_Vertical, symbol Connector:Conn_01x05_Male
- added Q1, Q10, Q11, Q12, Q13, Q14, Q15, Q16, Q17, Q18, Q19, Q2, Q20, Q3, Q4, Q5, Q6, Q7, Q8, Q9: IRF830, Package_TO_SOT_SMD:TO-263-3_TabPin2, symbol Transistor_FET:IRF740
- renumbered J6 to J11, J7 to J12, J4 to J7, J5 to J8
Connections:
- net Output 1/LINE is gone; now on an unnamed net: J3.1 (Pin_1)
- net Output 1/OUTPUT is gone; now on an unnamed net: J3.2 (Pin_2)
- net Output 2/OUTPUT is gone; now on an unnamed net: J3.3 (Pin_3)
- net Output 3/OUTPUT is gone; now on an unnamed net: J3.4 (Pin_4)
- net Output 4/OUTPUT is gone; now on an unnamed net: J3.5 (Pin_5)
- net +5V: no longer names the net of J1.1 (Pin_1)
- net GND: no longer names the net of J1.2 (Pin_2)
- net Input 10/INPUT: no longer names the net of J11.3 (Pin_3)
- net Input 10/INPUT: now also J9.3 (Pin_3)
- net Input 10/NEUT: no longer names the net of J11.1 (Pin_1)
- net Input 10/NEUT: now also J9.1 (Pin_1)
- net Input 5/INPUT: no longer names the net of J7.2 (Pin_2)
- net Input 5/INPUT: now also J5.2 (Pin_2)
- net Input 5/NEUT: no longer names the net of J7.1 (Pin_1)
- net Input 5/NEUT: now also J5.1 (Pin_1)
- net Input 6/INPUT: no longer names the net of J7.3 (Pin_3)
- net Input 6/INPUT: now also J5.3 (Pin_3)
- net Input 7/INPUT: no longer names the net of J7.4 (Pin_4)
- net Input 7/INPUT: now also J5.4 (Pin_4)
- net Input 8/INPUT: no longer names the net of J7.5 (Pin_5)
- net Input 8/INPUT: now also J5.5 (Pin_5)
- net Input 9/INPUT: no longer names the net of J11.2 (Pin_2)
- net Input 9/INPUT: now also J9.2 (Pin_2)
- net Output 10/LINE: no longer names the net of J12.1 (Pin_1)
- net Output 10/LINE: now also J9.4 (Pin_4), Q17.2 (D), Q19.2 (D)
- net Output 10/OUTPUT: no longer names the net of J12.3 (Pin_3)
- net Output 10/OUTPUT: now also Q20.2 (D)
- net Output 5/LINE: no longer names the net of J8.1 (Pin_1)
- net Output 5/LINE: now also Q11.2 (D), Q13.2 (D), Q15.2 (D), Q9.2 (D)
- net Output 5/OUTPUT: no longer names the net of J8.2 (Pin_2)
- net Output 5/OUTPUT: now also Q10.2 (D)
- net Output 6/OUTPUT: no longer names the net of J8.4 (Pin_4)
- net Output 6/OUTPUT: now also Q14.2 (D)
- net Output 7/OUTPUT: no longer names the net of J8.3 (Pin_3)
- net Output 7/OUTPUT: now also Q12.2 (D)
- net Output 8/OUTPUT: no longer names the net of J8.5 (Pin_5)
- net Output 8/OUTPUT: now also Q16.2 (D)
- net Output 9/OUTPUT: no longer names the net of J12.2 (Pin_2)
- net Output 9/OUTPUT: now also Q18.2 (D)
- new net: J2.2 (Pin_2), Q1.1 (G), Q2.1 (G)
- new net: J4.1 (Pin_1), Q1.2 (D), Q3.2 (D), Q5.2 (D), Q7.2 (D)
- new net: J2.1 (Pin_1), Q1.3 (S), Q2.3 (S)
- new net: J4.2 (Pin_2), Q2.2 (D)
- new net: J4.3 (Pin_3), Q4.2 (D)
- new net: J4.4 (Pin_4), Q6.2 (D)
- new net: J4.5 (Pin_5), Q8.2 (D)
- new net: J10.4 (Pin_4), Q19.1 (G), Q20.1 (G)
- new net: J10.3 (Pin_3), Q19.3 (S), Q20.3 (S)
- new net: J2.6 (Pin_6), Q5.1 (G), Q6.1 (G)
- new net: J2.5 (Pin_5), Q5.3 (S), Q6.3 (S)
- new net: J10.1 (Pin_1), Q17.3 (S), Q18.3 (S)
- new net: J10.2 (Pin_2), Q17.1 (G), Q18.1 (G)
- new net: J6.8 (Pin_8), Q15.1 (G), Q16.1 (G)
- new net: J6.7 (Pin_7), Q15.3 (S), Q16.3 (S)
- new net: J6.1 (Pin_1), Q10.3 (S), Q9.3 (S)
- new net: J6.2 (Pin_2), Q10.1 (G), Q9.1 (G)
- new net: J6.3 (Pin_3), Q11.3 (S), Q12.3 (S)
- new net: J6.4 (Pin_4), Q11.1 (G), Q12.1 (G)
- new net: J6.5 (Pin_5), Q13.3 (S), Q14.3 (S)
- new net: J6.6 (Pin_6), Q13.1 (G), Q14.1 (G)
- new net: J2.4 (Pin_4), Q3.1 (G), Q4.1 (G)
- new net: J2.3 (Pin_3), Q3.3 (S), Q4.3 (S)
- new net: J2.8 (Pin_8), Q7.1 (G), Q8.1 (G)
- new net: J2.7 (Pin_7), Q7.3 (S), Q8.3 (S)
- no-connect marks 1 -> 0
Other:
- removed sheet Input 1
- removed sheet Input 10
- removed sheet Input 2
- removed sheet Input 3
- removed sheet Input 4
- removed sheet Input 5
- removed sheet Input 6
- removed sheet Input 7
- removed sheet Input 8
- removed sheet Input 9
- removed sheet Output 1
- removed sheet Output 10
- removed sheet Output 2
- removed sheet Output 3
- removed sheet Output 4
- removed sheet Output 5
- removed sheet Output 6
- removed sheet Output 7
- removed sheet Output 8
- removed sheet Output 9
- note removed: "Zero crossing detector"
- moved on the sheet: J11, J12, J7, J8

Commit message: bottom board first draft
Parts:
- added J? (x3): Conn_01x05_Male, Connector_PinHeader_2.54mm:PinHeader_1x05_P2.54mm_Vertical, symbol Connector:Conn_01x05_Male
Connections:
- new net: J?.1 (Pin_1), J?.1 (Pin_1), J?.1 (Pin_1)
- new net: J?.2 (Pin_2), J?.2 (Pin_2), J?.2 (Pin_2)
- new net: J?.3 (Pin_3), J?.3 (Pin_3), J?.3 (Pin_3)
- new net: J?.4 (Pin_4), J?.4 (Pin_4), J?.4 (Pin_4)
- new net: J?.5 (Pin_5), J?.5 (Pin_5), J?.5 (Pin_5)

Commit message: cleanup
Parts:
- gave numbers to parts that had none: 3
Changed lines of the file:
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@@
   (symbol (lib_id "Connector:Conn_01x05_Male") (at 278.13 189.23 0) (unit 1)
     (in_bom yes) (on_board yes)
-    (property "Reference" "J?" (id 0) (at 281.94 176.53 0))
+    (property "Reference" "J14" (id 0) (at 281.94 176.53 0))
     (property "Value" "Conn_01x05_Male" (id 1) (at 280.67 180.34 0))
     (property "Footprint" "Connector_PinHeader_2.54mm:PinHeader_1x05_P2.54mm_Vertical" (id 2) (at 278.13 189.23 0)
@@
   (symbol (lib_id "Connector:Conn_01x05_Male") (at 278.13 209.55 0) (unit 1)
     (in_bom yes) (on_board yes)
-    (property "Reference" "J?" (id 0) (at 281.94 196.85 0))
+    (property "Reference" "J15" (id 0) (at 281.94 196.85 0))
     (property "Value" "Conn_01x05_Male" (id 1) (at 280.67 200.66 0))
     (property "Footprint" "Connector_PinHeader_2.54mm:PinHeader_1x05_P2.54mm_Vertical" (id 2) (at 278.13 209.55 0)
@@
   (symbol (lib_id "Connector:Conn_01x05_Male") (at 278.13 168.91 0) (unit 1)
     (in_bom yes) (on_board yes)
-    (property "Reference" "J?" (id 0) (at 281.94 156.21 0))
+    (property "Reference" "J13" (id 0) (at 281.94 156.21 0))
     (property "Value" "Conn_01x05_Male" (id 1) (at 280.67 160.02 0))
     (property "Footprint" "Connector_PinHeader_2.54mm:PinHeader_1x05_P2.54mm_Vertical" (id 2) (at 278.13 168.91 0)
@@
       (reference "J12") (unit 1) (value "Screw_Terminal_01x03") (footprint "TerminalBlock:TerminalBlock_bornier-3_P5.08mm")
     )
+    (path "/fb7abf49-27cd-4c26-ba3a-f5fee1af179c"
+      (reference "J13") (unit 1) (value "Conn_01x05_Male") (footprint "Connector_PinHeader_2.54mm:PinHeader_1x05_P2.54mm_Vertical")
+    )
     (path "/1a40b32a-6c8c-448f-bf8b-56c1f528da37"
-      (reference "J?") (unit 1) (value "Conn_01x05_Male") (footprint "Connector_PinHeader_2.54mm:PinHeader_1x05_P2.54mm_Vertical")
+      (reference "J14") (unit 1) (value "Conn_01x05_Male") (footprint "Connector_PinHeader_2.54mm:PinHeader_1x05_P2.54mm_Vertical")
     )
     (path "/5564de75-9c7c-4b69-912b-824cbaa6df29"
-      (reference "J?") (unit 1) (value "Conn_01x05_Male") (footprint "Connector_PinHeader_2.54mm:PinHeader_1x05_P2.54mm_Vertical")
-    )
-    (path "/fb7abf49-27cd-4c26-ba3a-f5fee1af179c"
-      (reference "J?") (unit 1) (value "Conn_01x05_Male") (footprint "Connector_PinHeader_2.54mm:PinHeader_1x05_P2.54mm_Vertical")
+      (reference "J15") (unit 1) (value "Conn_01x05_Male") (footprint "Connector_PinHeader_2.54mm:PinHeader_1x05_P2.54mm_Vertical")
     )
     (path "/0a538e21-f9f7-41ac-9f9d-581175515cb0"
