File: epanel-io/v1/top/output.kicad_sch (KiCad schematic)
At the start: 10 parts, among them Q17 IRF830, Q18 IRF830, U20 4N35

Commit message: top schematic
Parts:
- removed Q17, Q18: IRF830, Package_TO_SOT_SMD:TO-263-3_TabPin2, symbol Transistor_FET:IRF740
- renumbered C9 to C?, D18 to D?, D17 to D?, R66 to R?, R65 to R?, R64 to R?, R63 to R?, U20 to U?
Connections:
- net GND: now also C?.2, D?.2 (A), R?.2
- net GATE: now reaches R?.1, U?.4
Changed lines of the file:
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@@
   (junction (at 177.8 62.23) (diameter 0) (color 0 0 0 0)
-  )
-  (junction (at 231.14 81.28) (diameter 0) (color 0 0 0 0)
-  )
-  (junction (at 238.76 78.74) (diameter 0) (color 0 0 0 0)
   )
   (junction (at 144.78 81.28) (diameter 0) (color 0 0 0 0)
@@
     (stroke (width 0) (type default) (color 0 0 0 0))
   )
-  (wire (pts (xy 224.79 62.23) (xy 257.81 62.23))
+  (wire (pts (xy 224.79 62.23) (xy 236.22 62.23))
     (stroke (width 0) (type default) (color 0 0 0 0))
   )
@@
     (stroke (width 0) (type default) (color 0 0 0 0))
   )
-  (wire (pts (xy 238.76 66.04) (xy 238.76 67.31))
-    (stroke (width 0) (type default) (color 0 0 0 0))
-  )
   (wire (pts (xy 177.8 62.23) (xy 177.8 68.58))
     (stroke (width 0) (type default) (color 0 0 0 0))
@@
     (stroke (width 0) (type default) (color 0 0 0 0))
   )
-  (wire (pts (xy 238.76 78.74) (xy 238.76 77.47))
-    (stroke (width 0) (type default) (color 0 0 0 0))
-  )
-  (wire (pts (xy 231.14 81.28) (xy 231.14 85.09))
-    (stroke (width 0) (type default) (color 0 0 0 0))
-  )
   (wire (pts (xy 118.11 76.2) (xy 123.19 76.2))
     (stroke (width 0) (type default) (color 0 0 0 0))
@@
     (stroke (width 0) (type default) (color 0 0 0 0))
   )
-  (wire (pts (xy 238.76 78.74) (xy 250.19 78.74))
-    (stroke (width 0) (type default) (color 0 0 0 0))
-  )
   (wire (pts (xy 96.52 76.2) (xy 110.49 76.2))
     (stroke (width 0) (type default) (color 0 0 0 0))
@@
     (stroke (width 0) (type default) (color 0 0 0 0))
   )
-  (wire (pts (xy 231.14 72.39) (xy 231.14 81.28))
-    (stroke (width 0) (type default) (color 0 0 0 0))
-  )
   (wire (pts (xy 187.96 62.23) (xy 177.8 62.23))
     (stroke (width 0) (type default) (color 0 0 0 0))
   )
-  (wire (pts (xy 238.76 78.74) (xy 238.76 80.01))
-    (stroke (width 0) (type default) (color 0 0 0 0))
-  )
   (wire (pts (xy 144.78 82.55) (xy 144.78 81.28))
     (stroke (width 0) (type default) (color 0 0 0 0))
   )
-  (wire (pts (xy 238.76 66.04) (xy 257.81 66.04))
-    (stroke (width 0) (type default) (color 0 0 0 0))
-  )
   (wire (pts (xy 119.38 81.28) (xy 119.38 86.36))
     (stroke (width 0) (type default) (color 0 0 0 0))
@@
     (stroke (width 0) (type default) (color 0 0 0 0))
   )
-  (wire (pts (xy 177.8 93.98) (xy 250.19 93.98))
-    (stroke (width 0) (type default) (color 0 0 0 0))
-  )
-  (wire (pts (xy 238.76 90.17) (xy 238.76 91.44))
+  (wire (pts (xy 177.8 93.98) (xy 236.22 93.98))
     (stroke (width 0) (type default) (color 0 0 0 0))
   )
@@
     (stroke (width 0) (type default) (color 0 0 0 0))
   )
-  (wire (pts (xy 250.19 93.98) (xy 250.19 78.74))
-    (stroke (width 0) (type default) (color 0 0 0 0))
-  )
-  (wire (pts (xy 238.76 91.44) (xy 260.35 91.44))
-    (stroke (width 0) (type default) (color 0 0 0 0))
-  )
-  (wire (pts (xy 144.78 81.28) (xy 231.14 81.28))
-    (stroke (width 0) (type default) (color 0 0 0 0))
-  )
-  (hierarchical_label "OUTPUT" (shape input) (at 260.35 91.44 0)
+  (wire (pts (xy 144.78 81.28) (xy 236.22 81.28))
+    (stroke (width 0) (type default) (color 0 0 0 0))
+  )
+  (hierarchical_label "GND" (shape input) (at 236.22 93.98 0)
     (effects (font (size 1.27 1.27)) (justify left))
   )
-  (hierarchical_label "LINE" (shape input) (at 257.81 66.04 0)
+  (hierarchical_label "GATE" (shape input) (at 236.22 81.28 0)
     (effects (font (size 1.27 1.27)) (justify left))
   )
-  (hierarchical_label "NEUT" (shape input) (at 257.81 62.23 0)
+  (hierarchical_label "NEUT" (shape input) (at 236.22 62.23 0)
     (effects (font (size 1.27 1.27)) (justify left))
   )
@@
   (symbol (lib_id "Isolator:4N35") (at 130.81 78.74 0)
     (in_bom yes) (on_board yes) (fields_autoplaced)
-    (property "Reference" "U20" (id 0) (at 130.81 70.9635 0))
+    (property "Reference" "U?" (id 0) (at 130.81 70.9635 0))
     (property "Value" "4N35" (id 1) (at 130.81 73.7386 0))
     (property "Footprint" "Package_DIP:SMDIP-6_W7.62mm" (id 2) (at 125.73 83.82 0)
@@
   (symbol (lib_id "Diode:1N4007") (at 220.98 62.23 0)
     (in_bom yes) (on_board yes) (fields_autoplaced)
-    (property "Reference" "D18" (id 0) (at 220.98 56.9935 0))
+    (property "Reference" "D?" (id 0) (at 220.98 56.9935 0))
     (property "Value" "1N4007" (id 1) (at 220.98 59.7686 0))
     (property "Footprint" "Diode_SMD:D_SMA" (id 2) (at 220.98 66.675 0)
@@
   (symbol (lib_id "Device:R") (at 207.01 62.23 270)
     (in_bom yes) (on_board yes) (fields_autoplaced)
-    (property "Reference" "R66" (id 0) (at 207.01 57.2475 90))
+    (property "Reference" "R?" (id 0) (at 207.01 57.2475 90))
     (property "Value" "33KΩ/0.5W" (id 1) (at 207.01 60.0226 90))
     (property "Footprint" "Resistor_SMD:R_0805_2012Metric" (id 2) (at 207.01 60.452 90)
@@
     (pin "2")
   )
-  (symbol (lib_id "Transistor_FET:IRF740") (at 236.22 72.39 0)
-    (in_bom yes) (on_board yes) (fields_autoplaced)
-    (property "Reference" "Q17" (id 0) (at 241.427 71.4815 0)
-      (effects (font (size 1.27 1.27)) (justify left))
-    )
-    (property "Value" "IRF830" (id 1) (at 241.427 74.2566 0)
-      (effects (font (size 1.27 1.27)) (justify left))
-    )
-    (property "Footprint" "Package_TO_SOT_SMD:TO-263-3_TabPin2" (id 2) (at 242.57 74.295 0)
-      (effects (font (size 1.27 1.27) italic) (justify left) hide)
-    )
-    (property "Datasheet" "https://datasheet.lcsc.com/lcsc/2006291614_VBsemi-Elec-IRF830ASTRL_C693297.pdf" (id 3) (at 236.22 72.39 0)
-      (effects (font (size 1.27 1.27)) (justify left) hide)
-    )
-    (property "LCSC" "C693297" (id 4) (at 236.22 72.39 0)
-      (effects (font (size 1.27 1.27)) hide)
-    )
-    (pin "1")
-    (pin "2")
-    (pin "3")
-  )
-  (symbol (lib_id "Transistor_FET:IRF740") (at 236.22 85.09 0) (mirror x)
-    (in_bom yes) (on_board yes) (fields_autoplaced)
-    (property "Reference" "Q18" (id 0) (at 242.57 83.8199 0)
-      (effects (font (size 1.27 1.27)) (justify left))
-    )
-    (property "Value" "IRF830" (id 1) (at 242.57 86.3599 0)
-      (effects (font (size 1.27 1.27)) (justify left))
-    )
-    (property "Footprint" "Package_TO_SOT_SMD:TO-263-3_TabPin2" (id 2) (at 242.57 83.185 0)
-      (effects (font (size 1.27 1.27) italic) (justify left) hide)
-    )
-    (property "Datasheet" "https://datasheet.lcsc.com/lcsc/2006291614_VBsemi-Elec-IRF830ASTRL_C693297.pdf" (id 3) (at 236.22 85.09 0)
-      (effects (font (size 1.27 1.27)) (justify left) hide)
-    )
-    (property "LCSC" "C693297" (id 4) (at 236.22 85.09 0)
-      (effects (font (size 1.27 1.27)) hide)
-    )
-    (pin "1")
-    (pin "2")
-    (pin "3")
-  )
   (symbol (lib_id "Device:R") (at 191.77 62.23 270)
     (in_bom yes) (on_board yes) (fields_autoplaced)
-    (property "Reference" "R65" (id 0) (at 191.77 57.2475 90))
+    (property "Reference" "R?" (id 0) (at 191.77 57.2475 90))
     (property "Value" "33KΩ/0.5W" (id 1) (at 191.77 60.0226 90))
     (property "Footprint" "Resistor_SMD:R_0805_2012Metric" (id 2) (at 191.77 60.452 90)
@@
   (symbol (lib_id "Device:C_Polarized") (at 177.8 72.39 0)
     (in_bom yes) (on_board yes) (fields_autoplaced)
-    (property "Reference" "C9" (id 0) (at 180.721 70.5925 0)
+    (property "Reference" "C?" (id 0) (at 180.721 70.5925 0)
       (effects (font (size 1.27 1.27)) (justify left))
     )
@@
   (symbol (lib_id "power:GND") (at 119.38 86.36 0)
     (in_bom yes) (on_board yes)
-    (property "Reference" "#PWR036" (id 0) (at 119.38 92.71 0)
+    (property "Reference" "#PWR?" (id 0) (at 119.38 92.71 0)
       (effects (font (size 1.27 1.27)) hide)
     )
@@
   (symbol (lib_id "Device:R") (at 144.78 86.36 0)
     (in_bom yes) (on_board yes)
-    (property "Reference" "R64" (id 0) (at 140.97 85.09 0))
+    (property "Reference" "R?" (id 0) (at 140.97 85.09 0))
     (property "Value" "22KΩ" (id 1) (at 139.7 87.63 0))
     (property "Footprint" "Resistor_SMD:R_0603_1608Metric" (id 2) (at 143.002 86.36 90)
@@
   (symbol (lib_id "Device:R") (at 114.3 76.2 270)
     (in_bom yes) (on_board yes)
-    (property "Reference" "R63" (id 0) (at 113.03 71.12 90))
+    (property "Reference" "R?" (id 0) (at 113.03 71.12 90))
     (property "Value" "330Ω" (id 1) (at 114.3 73.66 90))
     (property "Footprint" "Resistor_SMD:R_0603_1608Metric" (id 2) (at 114.3 74.422 90)
@@
   (symbol (lib_id "Diode:BZV55B10") (at 160.02 72.39 270)
     (in_bom yes) (on_board yes) (fields_autoplaced)
-    (property "Reference" "D17" (id 0) (at 162.052 71.4815 90)
+    (property "Reference" "D?" (id 0) (at 162.052 71.4815 90)
       (effects (font (size 1.27 1.27)) (justify left))
     )

Commit message: wip pcb
Parts:
- gave numbers to parts that had none: 8
Changed lines of the file:
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@@
   (symbol (lib_id "Isolator:4N35") (at 130.81 78.74 0)
     (in_bom yes) (on_board yes) (fields_autoplaced)
-    (property "Reference" "U?" (id 0) (at 130.81 70.9635 0))
+    (property "Reference" "U22" (id 0) (at 130.81 70.9635 0))
     (property "Value" "4N35" (id 1) (at 130.81 73.7386 0))
     (property "Footprint" "Package_DIP:SMDIP-6_W7.62mm" (id 2) (at 125.73 83.82 0)
@@
   (symbol (lib_id "Diode:1N4007") (at 220.98 62.23 0)
     (in_bom yes) (on_board yes) (fields_autoplaced)
-    (property "Reference" "D?" (id 0) (at 220.98 56.9935 0))
+    (property "Reference" "D20" (id 0) (at 220.98 56.9935 0))
     (property "Value" "1N4007" (id 1) (at 220.98 59.7686 0))
     (property "Footprint" "Diode_SMD:D_SMA" (id 2) (at 220.98 66.675 0)
@@
   (symbol (lib_id "Device:R") (at 207.01 62.23 270)
     (in_bom yes) (on_board yes) (fields_autoplaced)
-    (property "Reference" "R?" (id 0) (at 207.01 57.2475 90))
+    (property "Reference" "R73" (id 0) (at 207.01 57.2475 90))
     (property "Value" "33KΩ/0.5W" (id 1) (at 207.01 60.0226 90))
     (property "Footprint" "Resistor_SMD:R_0805_2012Metric" (id 2) (at 207.01 60.452 90)
@@
   (symbol (lib_id "Device:R") (at 191.77 62.23 270)
     (in_bom yes) (on_board yes) (fields_autoplaced)
-    (property "Reference" "R?" (id 0) (at 191.77 57.2475 90))
+    (property "Reference" "R72" (id 0) (at 191.77 57.2475 90))
     (property "Value" "33KΩ/0.5W" (id 1) (at 191.77 60.0226 90))
     (property "Footprint" "Resistor_SMD:R_0805_2012Metric" (id 2) (at 191.77 60.452 90)
@@
   (symbol (lib_id "Device:C_Polarized") (at 177.8 72.39 0)
     (in_bom yes) (on_board yes) (fields_autoplaced)
-    (property "Reference" "C?" (id 0) (at 180.721 70.5925 0)
+    (property "Reference" "C10" (id 0) (at 180.721 70.5925 0)
       (effects (font (size 1.27 1.27)) (justify left))
     )
@@
   (symbol (lib_id "power:GND") (at 119.38 86.36 0)
     (in_bom yes) (on_board yes)
-    (property "Reference" "#PWR?" (id 0) (at 119.38 92.71 0)
+    (property "Reference" "#PWR0117" (id 0) (at 119.38 92.71 0)
       (effects (font (size 1.27 1.27)) hide)
     )
@@
   (symbol (lib_id "Device:R") (at 144.78 86.36 0)
     (in_bom yes) (on_board yes)
-    (property "Reference" "R?" (id 0) (at 140.97 85.09 0))
+    (property "Reference" "R71" (id 0) (at 140.97 85.09 0))
     (property "Value" "22KΩ" (id 1) (at 139.7 87.63 0))
     (property "Footprint" "Resistor_SMD:R_0603_1608Metric" (id 2) (at 143.002 86.36 90)
@@
   (symbol (lib_id "Device:R") (at 114.3 76.2 270)
     (in_bom yes) (on_board yes)
-    (property "Reference" "R?" (id 0) (at 113.03 71.12 90))
+    (property "Reference" "R70" (id 0) (at 113.03 71.12 90))
     (property "Value" "330Ω" (id 1) (at 114.3 73.66 90))
     (property "Footprint" "Resistor_SMD:R_0603_1608Metric" (id 2) (at 114.3 74.422 90)
@@
   (symbol (lib_id "Diode:BZV55B10") (at 160.02 72.39 270)
     (in_bom yes) (on_board yes) (fields_autoplaced)
-    (property "Reference" "D?" (id 0) (at 162.052 71.4815 90)
+    (property "Reference" "D19" (id 0) (at 162.052 71.4815 90)
       (effects (font (size 1.27 1.27)) (justify left))
     )

Commit message: fix gnd
Parts:
- renumbered C10 to C9, D19 to D17, D20 to D18, R70 to R63, R71 to R64, R72 to R65, R73 to R66, U22 to U20
Connections:
- net GND: no longer C9.2, D17.2 (A), R64.2
- new net SOURCE: C9.2, D17.2 (A), R64.2
Changed lines of the file:
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@@
     (stroke (width 0) (type default) (color 0 0 0 0))
   )
-  (hierarchical_label "GND" (shape input) (at 236.22 93.98 0)
+  (hierarchical_label "SOURCE" (shape input) (at 236.22 93.98 0)
     (effects (font (size 1.27 1.27)) (justify left))
   )
@@
   (symbol (lib_id "Isolator:4N35") (at 130.81 78.74 0)
     (in_bom yes) (on_board yes) (fields_autoplaced)
-    (property "Reference" "U22" (id 0) (at 130.81 70.9635 0))
+    (property "Reference" "U20" (id 0) (at 130.81 70.9635 0))
     (property "Value" "4N35" (id 1) (at 130.81 73.7386 0))
     (property "Footprint" "Package_DIP:SMDIP-6_W7.62mm" (id 2) (at 125.73 83.82 0)
@@
   (symbol (lib_id "Diode:1N4007") (at 220.98 62.23 0)
     (in_bom yes) (on_board yes) (fields_autoplaced)
-    (property "Reference" "D20" (id 0) (at 220.98 56.9935 0))
+    (property "Reference" "D18" (id 0) (at 220.98 56.9935 0))
     (property "Value" "1N4007" (id 1) (at 220.98 59.7686 0))
     (property "Footprint" "Diode_SMD:D_SMA" (id 2) (at 220.98 66.675 0)
@@
   (symbol (lib_id "Device:R") (at 207.01 62.23 270)
     (in_bom yes) (on_board yes) (fields_autoplaced)
-    (property "Reference" "R73" (id 0) (at 207.01 57.2475 90))
+    (property "Reference" "R66" (id 0) (at 207.01 57.2475 90))
     (property "Value" "33KΩ/0.5W" (id 1) (at 207.01 60.0226 90))
     (property "Footprint" "Resistor_SMD:R_0805_2012Metric" (id 2) (at 207.01 60.452 90)
@@
   (symbol (lib_id "Device:R") (at 191.77 62.23 270)
     (in_bom yes) (on_board yes) (fields_autoplaced)
-    (property "Reference" "R72" (id 0) (at 191.77 57.2475 90))
+    (property "Reference" "R65" (id 0) (at 191.77 57.2475 90))
     (property "Value" "33KΩ/0.5W" (id 1) (at 191.77 60.0226 90))
     (property "Footprint" "Resistor_SMD:R_0805_2012Metric" (id 2) (at 191.77 60.452 90)
@@
   (symbol (lib_id "Device:C_Polarized") (at 177.8 72.39 0)
     (in_bom yes) (on_board yes) (fields_autoplaced)
-    (property "Reference" "C10" (id 0) (at 180.721 70.5925 0)
+    (property "Reference" "C9" (id 0) (at 180.721 70.5925 0)
       (effects (font (size 1.27 1.27)) (justify left))
     )
@@
   (symbol (lib_id "Device:R") (at 144.78 86.36 0)
     (in_bom yes) (on_board yes)
-    (property "Reference" "R71" (id 0) (at 140.97 85.09 0))
+    (property "Reference" "R64" (id 0) (at 140.97 85.09 0))
     (property "Value" "22KΩ" (id 1) (at 139.7 87.63 0))
     (property "Footprint" "Resistor_SMD:R_0603_1608Metric" (id 2) (at 143.002 86.36 90)
@@
   (symbol (lib_id "Device:R") (at 114.3 76.2 270)
     (in_bom yes) (on_board yes)
-    (property "Reference" "R70" (id 0) (at 113.03 71.12 90))
+    (property "Reference" "R63" (id 0) (at 113.03 71.12 90))
     (property "Value" "330Ω" (id 1) (at 114.3 73.66 90))
     (property "Footprint" "Resistor_SMD:R_0603_1608Metric" (id 2) (at 114.3 74.422 90)
@@
   (symbol (lib_id "Diode:BZV55B10") (at 160.02 72.39 270)
     (in_bom yes) (on_board yes) (fields_autoplaced)
-    (property "Reference" "D19" (id 0) (at 162.052 71.4815 90)
+    (property "Reference" "D17" (id 0) (at 162.052 71.4815 90)
       (effects (font (size 1.27 1.27)) (justify left))
     )
