File: epanel-io/v1/top/top.kicad_pcb (KiCad board)
At the start: 2 copper layers, 66.5 x 100.8 mm, 132 parts, among them J1 Conn_01x05_Male, J2 Conn_01x05_Female, J3 Conn_01x08_Female, J4 Conn_01x05_Female, J5 Conn_01x08_Female, J6 Conn_01x04_Female, J7 Conn_01x04_Female, U1 Pico, U10 4N35, U11 H11AA1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

Commit message: wip pcb
Routing:
- net +3V3: track 0.00 -> 102.7 mm, vias 0 -> 13
- net /Input 10/NEUT: track 67.3 -> 110.9 mm
Changed lines of the file:
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@@
   (segment (start 161.418 85.3195) (end 163.322 83.4155) (width 0.25) (layer "B.Cu") (net 8))
   (segment (start 164.592 82.1925) (end 164.592 83.4155) (width 0.25) (layer "B.Cu") (net 8))
+  (segment (start 127.762 141.415) (end 127.762 140.208) (width 0.25) (layer "F.Cu") (net 9))
+  (segment (start 127.701 64.199) (end 127.701 62.931) (width 0.25) (layer "F.Cu") (net 9))
+  (segment (start 127.701 82.235) (end 127.508 82.042) (width 0.25) (layer "F.Cu") (net 9))
+  (segment (start 127.762 111.252) (end 127.508 110.998) (width 0.25) (layer "F.Cu") (net 9))
+  (segment (start 127.508 77.216) (end 127.508 79.502) (width 0.25) (layer "F.Cu") (net 9))
+  (segment (start 127.701 83.503) (end 127.701 82.235) (width 0.25) (layer "F.Cu") (net 9))
+  (segment (start 127.762 130.556) (end 127.508 130.302) (width 0.25) (layer "F.Cu") (net 9))
+  (segment (start 127.508 110.998) (end 127.508 106.426) (width 0.25) (layer "F.Cu") (net 9))
+  (segment (start 127.762 140.208) (end 127.508 139.954) (width 0.25) (layer "F.Cu") (net 9))
+  (segment (start 127.762 112.459) (end 127.762 111.252) (width 0.25) (layer "F.Cu") (net 9))
+  (segment (start 127.762 101.6) (end 127.508 101.346) (width 0.25) (layer "F.Cu") (net 9))
+  (segment (start 127.6035 52.9275) (end 127.508 52.832) (width 0.25) (layer "F.Cu") (net 9))
+  (segment (start 127.762 91.948) (end 127.508 91.694) (width 0.25) (layer "F.Cu") (net 9))
+  (segment (start 127.701 73.851) (end 127.701 72.583) (width 0.25) (layer "F.Cu") (net 9))
+  (segment (start 127.762 93.155) (end 127.762 91.948) (width 0.25) (layer "F.Cu") (net 9))
+  (segment (start 127.762 122.111) (end 127.762 120.904) (width 0.25) (layer "F.Cu") (net 9))
+  (segment (start 127.762 102.807) (end 127.762 101.6) (width 0.25) (layer "F.Cu") (net 9))
+  (segment (start 127.762 131.763) (end 127.762 130.556) (width 0.25) (layer "F.Cu") (net 9))
+  (segment (start 127.701 62.931) (end 127.508 62.738) (width 0.25) (layer "F.Cu") (net 9))
+  (segment (start 127.6035 54.3885) (end 127.6035 52.9275) (width 0.25) (layer "F.Cu") (net 9))
+  (segment (start 127.762 120.904) (end 127.508 120.65) (width 0.25) (layer "F.Cu") (net 9))
+  (segment (start 127.701 72.583) (end 127.508 72.39) (width 0.25) (layer "F.Cu") (net 9))
+  (via (at 127.508 120.65) (size 0.8) (drill 0.4) (layers "F.Cu" "B.Cu") (net 9))
+  (via (at 127.508 101.346) (size 0.8) (drill 0.4) (layers "F.Cu" "B.Cu") (net 9))
+  (via (at 127.508 110.998) (size 0.8) (drill 0.4) (layers "F.Cu" "B.Cu") (net 9))
+  (via (at 127.508 91.694) (size 0.8) (drill 0.4) (layers "F.Cu" "B.Cu") (net 9))
+  (via (at 127.508 139.954) (size 0.8) (drill 0.4) (layers "F.Cu" "B.Cu") (net 9))
+  (via (at 127.508 62.738) (size 0.8) (drill 0.4) (layers "F.Cu" "B.Cu") (net 9))
+  (via (at 127.508 52.832) (size 0.8) (drill 0.4) (layers "F.Cu" "B.Cu") (net 9))
+  (via (at 127.508 72.39) (size 0.8) (drill 0.4) (layers "F.Cu" "B.Cu") (net 9))
+  (via (at 127.508 82.042) (size 0.8) (drill 0.4) (layers "F.Cu" "B.Cu") (net 9))
+  (via (at 127.508 77.216) (size 0.8) (drill 0.4) (layers "F.Cu" "B.Cu") (net 9))
+  (via (at 127.508 106.426) (size 0.8) (drill 0.4) (layers "F.Cu" "B.Cu") (net 9))
+  (via (at 127.508 130.302) (size 0.8) (drill 0.4) (layers "F.Cu" "B.Cu") (net 9))
+  (via (at 127.508 79.502) (size 0.8) (drill 0.4) (layers "F.Cu" "B.Cu") (net 9))
+  (segment (start 127.508 106.426) (end 127.508 101.346) (width 0.25) (layer "B.Cu") (net 9))
+  (segment (start 127.508 79.502) (end 127.508 82.042) (width 0.25) (layer "B.Cu") (net 9))
+  (segment (start 127.508 52.832) (end 127.508 62.738) (width 0.25) (layer "B.Cu") (net 9))
+  (segment (start 127.508 62.738) (end 127.508 72.39) (width 0.25) (layer "B.Cu") (net 9))
+  (segment (start 127.508 82.042) (end 127.508 91.694) (width 0.25) (layer "B.Cu") (net 9))
+  (segment (start 127.508 91.694) (end 127.508 101.346) (width 0.25) (layer "B.Cu") (net 9))
+  (segment (start 127.508 72.39) (end 127.508 77.216) (width 0.25) (layer "B.Cu") (net 9))
+  (segment (start 127.508 120.65) (end 127.508 130.302) (width 0.25) (layer "B.Cu") (net 9))
+  (segment (start 127.508 110.998) (end 127.508 120.65) (width 0.25) (layer "B.Cu") (net 9))
+  (segment (start 127.508 130.302) (end 127.508 139.954) (width 0.25) (layer "B.Cu") (net 9))
   (segment (start 165.608 143.764) (end 167.132 143.764) (width 0.25) (layer "F.Cu") (net 10))
   (segment (start 164.592 142.748) (end 165.608 143.764) (width 0.25) (layer "F.Cu") (net 10))
@@
   (via (at 130.81 76.2) (size 0.8) (drill 0.4) (layers "F.Cu" "B.Cu") (net 54))
   (via (at 117.856 90.678) (size 0.8) (drill 0.4) (layers "F.Cu" "B.Cu") (net 54))
-  (segment (start 157.416 105.854) (end 158.75 105.854) (width 0.25) (layer "B.Cu") (net 54))
-  (segment (start 157.036 95.948) (end 156.464 96.52) (width 0.25) (layer "B.Cu") (net 54))
+  (segment (start 157.416 105.854) (end 156.464 104.902) (width 0.25) (layer "B.Cu") (net 54))
+  (segment (start 124.714 86.36) (end 124.714 79.248) (width 0.25) (layer "B.Cu") (net 54))
+  (segment (start 124.714 79.248) (end 125.476 78.486) (width 0.25) (layer "B.Cu") (net 54))
+  (segment (start 156.464 86.106) (end 155.575 85.217) (width 0.25) (layer "B.Cu") (net 54))
   (segment (start 117.856 90.678) (end 119.38 90.678) (width 0.25) (layer "B.Cu") (net 54))
-  (segment (start 127.254 76.2) (end 130.81 76.2) (width 0.25) (layer "B.Cu") (net 54))
-  (segment (start 158.75 95.948) (end 157.036 95.948) (width 0.25) (layer "B.Cu") (net 54))
-  (segment (start 126.746 76.2) (end 127.254 76.2) (width 0.25) (layer "B.Cu") (net 54))
   (segment (start 120.2925 92.964) (end 121.8165 94.488) (width 0.25) (layer "B.Cu") (net 54))
   (segment (start 120.2925 92.964) (end 120.2925 90.7815) (width 0.25) (layer "B.Cu") (net 54))
+  (segment (start 158.75 105.854) (end 157.416 105.854) (width 0.25) (layer "B.Cu") (net 54))
   (segment (start 120.2925 90.7815) (end 120.396 90.678) (width 0.25) (layer "B.Cu") (net 54))
-  (segment (start 156.464 104.902) (end 157.416 105.854) (width 0.25) (layer "B.Cu") (net 54))
-  (segment (start 124.714 78.232) (end 126.746 76.2) (width 0.25) (layer "B.Cu") (net 54))
+  (segment (start 129.794 78.486) (end 130.81 77.47) (width 0.25) (layer "B.Cu") (net 54))
+  (segment (start 130.81 76.2) (end 152.4 76.2) (width 0.25) (layer "B.Cu") (net 54))
+  (segment (start 158.75 95.948) (end 156.528 95.948) (width 0.25) (layer "B.Cu") (net 54))
+  (segment (start 125.476 78.486) (end 129.794 78.486) (width 0.25) (layer "B.Cu") (net 54))
   (segment (start 121.8165 94.488) (end 121.8165 101.092) (width 0.25) (layer "B.Cu") (net 54))
-  (segment (start 124.714 86.36) (end 124.714 78.232) (width 0.25) (layer "B.Cu") (net 54))
+  (segment (start 130.81 77.47) (end 130.81 76.2) (width 0.25) (layer "B.Cu") (net 54))
+  (segment (start 156.528 95.948) (end 156.464 96.012) (width 0.25) (layer "B.Cu") (net 54))
   (segment (start 121.8165 101.092) (end 120.2925 102.616) (width 0.25) (layer "B.Cu") (net 54))
-  (segment (start 156.464 96.52) (end 156.464 104.902) (width 0.25) (layer "B.Cu") (net 54))
+  (segment (start 156.464 104.902) (end 156.464 96.012) (width 0.25) (layer "B.Cu") (net 54))
+  (segment (start 155.448 79.248) (end 155.448 85.09) (width 0.25) (layer "B.Cu") (net 54))
   (segment (start 120.396 90.678) (end 124.714 86.36) (width 0.25) (layer "B.Cu") (net 54))
   (segment (start 119.38 90.678) (end 120.396 90.678) (width 0.25) (layer "B.Cu") (net 54))
+  (segment (start 156.464 96.012) (end 156.464 86.106) (width 0.25) (layer "B.Cu") (net 54))
+  (segment (start 155.448 85.09) (end 155.575 85.217) (width 0.25) (layer "B.Cu") (net 54))
+  (segment (start 152.4 76.2) (end 155.448 79.248) (width 0.25) (layer "B.Cu") (net 54))
   (segment (start 158.75 91.948) (end 162.259 91.948) (width 0.25) (layer "B.Cu") (net 55))
   (segment (start 162.259 91.948) (end 162.306 91.995) (width 0.25) (layer "B.Cu") (net 55))

Commit message: wip pcb
Parts:
- moved R1 13.4 mm to (133.3, 73.9), turned to 180 degrees
Routing:
- net Net-(R1-Pad1): track 0.00 -> 15.8 mm
- net +3V3: track 102.7 -> 107.6 mm
Changed lines of the file:
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@@
     (property "Sheetname" "")
     (attr smd)
-    (fp_text reference "R2" (at 0 -1.65) (layer "F.SilkS")
+    (fp_text reference "R2" (at -2.6435 0) (layer "F.SilkS")
       (effects (font (size 1 1) (thickness 0.15)))
     )
@@
     (property "Sheetname" "")
     (attr smd)
-    (fp_text reference "R3" (at 0 1.778) (layer "F.SilkS")
+    (fp_text reference "R3" (at -2.6435 0) (layer "F.SilkS")
       (effects (font (size 1 1) (thickness 0.15)))
     )
@@
   )
   (footprint "Resistor_SMD:R_0603_1608Metric" (layer "F.Cu")
-    (at 146.558 71.628 90)
+    (at 133.35 73.914 180)
     (descr "Resistor SMD 0603 (1608 Metric), square (rectangular) end terminal, IPC_7351 nominal, (Body size source: IPC-SM-782 page 72, https://www.pcb-3d.com/wordpress/wp-content/uploads/ipc-sm-782a_amendment_1_and_2.pdf), generated with kicad-footprint-generator")
     (tags "resistor")
@@
     (property "Sheetname" "")
     (attr smd)
-    (fp_text reference "R1" (at 0 -1.43 90) (layer "F.SilkS")
+    (fp_text reference "R1" (at 0 1.524) (layer "F.SilkS")
       (effects (font (size 1 1) (thickness 0.15)))
     )
-    (fp_text value "10KΩ" (at 0 1.43 90) (layer "F.Fab")
+    (fp_text value "10KΩ" (at 0 1.43) (layer "F.Fab")
       (effects (font (size 1 1) (thickness 0.15)))
     )
-    (fp_text user "${REFERENCE}" (at 0 0 90) (layer "F.Fab")
+    (fp_text user "${REFERENCE}" (at 0 0) (layer "F.Fab")
       (effects (font (size 0.4 0.4) (thickness 0.06)))
     )
@@
     (fp_line (start -0.8 -0.4125) (end 0.8 -0.4125) (layer "F.Fab") (width 0.1))
     (fp_line (start 0.8 0.4125) (end -0.8 0.4125) (layer "F.Fab") (width 0.1))
-    (pad "1" smd roundrect locked (at -0.825 0 90) (size 0.8 0.95) (layers "F.Cu" "F.Paste" "F.Mask") (roundrect_rratio 0.25)
+    (pad "1" smd roundrect locked (at -0.825 0 180) (size 0.8 0.95) (layers "F.Cu" "F.Paste" "F.Mask") (roundrect_rratio 0.25)
       (net 6 "Net-(R1-Pad1)") (pintype "passive"))
-    (pad "2" smd roundrect locked (at 0.825 0 90) (size 0.8 0.95) (layers "F.Cu" "F.Paste" "F.Mask") (roundrect_rratio 0.25)
+    (pad "2" smd roundrect locked (at 0.825 0 180) (size 0.8 0.95) (layers "F.Cu" "F.Paste" "F.Mask") (roundrect_rratio 0.25)
       (net 9 "+3V3") (pintype "passive"))
     (model "${KICAD6_3DMODEL_DIR}/Resistor_SMD.3dshapes/R_0603_1608Metric.wrl"
@@
   (segment (start 164.592 72.2865) (end 164.592 73.5095) (width 0.25) (layer "B.Cu") (net 5))
   (segment (start 161.418 77.9065) (end 161.593 78.0815) (width 0.25) (layer "B.Cu") (net 5))
+  (segment (start 141.732 76.962) (end 141.732 74.422) (width 0.25) (layer "F.Cu") (net 6))
+  (segment (start 146.497 78.74) (end 143.51 78.74) (width 0.25) (layer "F.Cu") (net 6))
+  (segment (start 141.224 73.914) (end 134.175 73.914) (width 0.25) (layer "F.Cu") (net 6))
+  (segment (start 143.51 78.74) (end 141.732 76.962) (width 0.25) (layer "F.Cu") (net 6))
+  (segment (start 141.732 74.422) (end 141.224 73.914) (width 0.25) (layer "F.Cu") (net 6))
   (segment (start 164.4415 53.594) (end 165.4575 54.61) (width 0.25) (layer "F.Cu") (net 7))
   (segment (start 165.4575 54.61) (end 166.9815 54.61) (width 0.25) (layer "F.Cu") (net 7))
@@
   (segment (start 127.762 102.807) (end 127.762 101.6) (width 0.25) (layer "F.Cu") (net 9))
   (segment (start 127.762 131.763) (end 127.762 130.556) (width 0.25) (layer "F.Cu") (net 9))
+  (segment (start 132.525 73.914) (end 127.764 73.914) (width 0.25) (layer "F.Cu") (net 9))
+  (segment (start 127.764 73.914) (end 127.701 73.851) (width 0.25) (layer "F.Cu") (net 9))
   (segment (start 127.701 62.931) (end 127.508 62.738) (width 0.25) (layer "F.Cu") (net 9))
   (segment (start 127.6035 54.3885) (end 127.6035 52.9275) (width 0.25) (layer "F.Cu") (net 9))

Commit message: wip pcb
Routing:
- net GND: track 286.5 -> 310.8 mm
Changed lines of the file:
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@@
   (segment (start 125.161 98.044) (end 122.682 98.044) (width 0.25) (layer "F.Cu") (net 3))
   (segment (start 159.512 94.234) (end 161.798 94.234) (width 0.25) (layer "F.Cu") (net 3))
+  (segment (start 154.178 92.71) (end 151.284 92.71) (width 0.25) (layer "F.Cu") (net 3))
   (segment (start 161.798 104.14) (end 161.798 114.046) (width 0.25) (layer "F.Cu") (net 3))
   (segment (start 159.3615 54.61) (end 161.544 54.61) (width 0.25) (layer "F.Cu") (net 3))
@@
   (segment (start 161.798 64.516) (end 161.798 54.356) (width 0.25) (layer "F.Cu") (net 3))
   (segment (start 125.161 117.348) (end 122.682 117.348) (width 0.25) (layer "F.Cu") (net 3))
+  (segment (start 146.497 81.28) (end 146.497 91.379) (width 0.25) (layer "F.Cu") (net 3))
   (segment (start 125.0025 59.2775) (end 122.7775 59.2775) (width 0.25) (layer "F.Cu") (net 3))
   (segment (start 122.682 145.288) (end 123.698 146.304) (width 0.25) (layer "F.Cu") (net 3))
@@
   (segment (start 123.952 49.784) (end 122.682 51.054) (width 0.25) (layer "F.Cu") (net 3))
   (segment (start 161.798 142.748) (end 160.782 143.764) (width 0.25) (layer "F.Cu") (net 3))
+  (segment (start 155.702 94.234) (end 154.178 92.71) (width 0.25) (layer "F.Cu") (net 3))
   (segment (start 122.682 107.442) (end 122.682 110.236) (width 0.25) (layer "F.Cu") (net 3))
   (segment (start 125.1 69.088) (end 122.682 69.088) (width 0.25) (layer "F.Cu") (net 3))
@@
   (segment (start 161.798 64.516) (end 161.798 74.676) (width 0.25) (layer "F.Cu") (net 3))
   (segment (start 122.7775 59.2775) (end 122.682 59.182) (width 0.25) (layer "F.Cu") (net 3))
+  (segment (start 147.828 92.71) (end 151.284 92.71) (width 0.25) (layer "F.Cu") (net 3))
   (segment (start 159.512 114.1495) (end 161.6945 114.1495) (width 0.25) (layer "F.Cu") (net 3))
   (segment (start 122.682 88.392) (end 122.682 98.044) (width 0.25) (layer "F.Cu") (net 3))
@@
   (segment (start 161.6945 114.1495) (end 161.798 114.046) (width 0.25) (layer "F.Cu") (net 3))
   (segment (start 159.512 74.5255) (end 161.6475 74.5255) (width 0.25) (layer "F.Cu") (net 3))
+  (segment (start 146.497 91.379) (end 147.828 92.71) (width 0.25) (layer "F.Cu") (net 3))
   (segment (start 161.798 84.328) (end 161.798 94.234) (width 0.25) (layer "F.Cu") (net 3))
+  (segment (start 159.512 94.234) (end 155.702 94.234) (width 0.25) (layer "F.Cu") (net 3))
   (segment (start 159.512 84.4315) (end 161.6945 84.4315) (width 0.25) (layer "F.Cu") (net 3))
   (segment (start 122.682 59.182) (end 122.682 69.088) (width 0.25) (layer "F.Cu") (net 3))

Commit message: wip pcb
Routing:
- net /Output 1/RPI: track 0.00 -> 79.1 mm, vias 0 -> 1
- net /Output 2/RPI: track 0.00 -> 72.2 mm, vias 0 -> 1
- net /Output 3/RPI: track 0.00 -> 71.1 mm, vias 0 -> 1
- net /Output 4/RPI: track 0.00 -> 60.4 mm, vias 0 -> 1
- net Net-(R1-Pad1): track 15.8 -> 40.5 mm
- net /Input 10/NEUT: track 110.9 -> 121.8 mm, vias 2 -> 4
Changed lines of the file:
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@@
   (segment (start 161.418 77.9065) (end 161.593 78.0815) (width 0.25) (layer "B.Cu") (net 5))
   (segment (start 141.732 76.962) (end 141.732 74.422) (width 0.25) (layer "F.Cu") (net 6))
-  (segment (start 146.497 78.74) (end 143.51 78.74) (width 0.25) (layer "F.Cu") (net 6))
+  (segment (start 141.732 93.472) (end 139.954 95.25) (width 0.25) (layer "F.Cu") (net 6))
+  (segment (start 146.497 78.74) (end 141.732 78.74) (width 0.25) (layer "F.Cu") (net 6))
+  (segment (start 141.732 78.74) (end 141.732 93.472) (width 0.25) (layer "F.Cu") (net 6))
+  (segment (start 141.732 76.962) (end 141.732 78.74) (width 0.25) (layer "F.Cu") (net 6))
   (segment (start 141.224 73.914) (end 134.175 73.914) (width 0.25) (layer "F.Cu") (net 6))
-  (segment (start 143.51 78.74) (end 141.732 76.962) (width 0.25) (layer "F.Cu") (net 6))
+  (segment (start 139.954 95.25) (end 133.504 95.25) (width 0.25) (layer "F.Cu") (net 6))
   (segment (start 141.732 74.422) (end 141.224 73.914) (width 0.25) (layer "F.Cu") (net 6))
   (segment (start 164.4415 53.594) (end 165.4575 54.61) (width 0.25) (layer "F.Cu") (net 7))
@@
   (segment (start 111.188 81.188) (end 112.176 81.188) (width 0.25) (layer "F.Cu") (net 54))
   (segment (start 113.284 82.296) (end 113.284 89.916) (width 0.25) (layer "F.Cu") (net 54))
+  (segment (start 155.448 71.628) (end 130.81 71.628) (width 0.25) (layer "F.Cu") (net 54))
   (segment (start 112.176 81.188) (end 113.03 82.042) (width 0.25) (layer "F.Cu") (net 54))
   (segment (start 113.03 82.042) (end 113.284 82.296) (width 0.25) (layer "F.Cu") (net 54))
   (via (at 130.81 76.2) (size 0.8) (drill 0.4) (layers "F.Cu" "B.Cu") (net 54))
+  (via (at 155.448 71.628) (size 0.8) (drill 0.4) (layers "F.Cu" "B.Cu") (net 54))
   (via (at 117.856 90.678) (size 0.8) (drill 0.4) (layers "F.Cu" "B.Cu") (net 54))
+  (via (at 130.81 71.628) (size 0.8) (drill 0.4) (layers "F.Cu" "B.Cu") (net 54))
   (segment (start 157.416 105.854) (end 156.464 104.902) (width 0.25) (layer "B.Cu") (net 54))
   (segment (start 124.714 86.36) (end 124.714 79.248) (width 0.25) (layer "B.Cu") (net 54))
@@
   (segment (start 158.75 105.854) (end 157.416 105.854) (width 0.25) (layer "B.Cu") (net 54))
   (segment (start 120.2925 90.7815) (end 120.396 90.678) (width 0.25) (layer "B.Cu") (net 54))
+  (segment (start 130.81 71.628) (end 130.81 76.2) (width 0.25) (layer "B.Cu") (net 54))
   (segment (start 129.794 78.486) (end 130.81 77.47) (width 0.25) (layer "B.Cu") (net 54))
-  (segment (start 130.81 76.2) (end 152.4 76.2) (width 0.25) (layer "B.Cu") (net 54))
   (segment (start 158.75 95.948) (end 156.528 95.948) (width 0.25) (layer "B.Cu") (net 54))
   (segment (start 125.476 78.486) (end 129.794 78.486) (width 0.25) (layer "B.Cu") (net 54))
@@
   (segment (start 121.8165 101.092) (end 120.2925 102.616) (width 0.25) (layer "B.Cu") (net 54))
   (segment (start 156.464 104.902) (end 156.464 96.012) (width 0.25) (layer "B.Cu") (net 54))
+  (segment (start 155.448 79.248) (end 155.448 71.628) (width 0.25) (layer "B.Cu") (net 54))
   (segment (start 155.448 79.248) (end 155.448 85.09) (width 0.25) (layer "B.Cu") (net 54))
   (segment (start 120.396 90.678) (end 124.714 86.36) (width 0.25) (layer "B.Cu") (net 54))
@@
   (segment (start 156.464 96.012) (end 156.464 86.106) (width 0.25) (layer "B.Cu") (net 54))
   (segment (start 155.448 85.09) (end 155.575 85.217) (width 0.25) (layer "B.Cu") (net 54))
-  (segment (start 152.4 76.2) (end 155.448 79.248) (width 0.25) (layer "B.Cu") (net 54))
   (segment (start 158.75 91.948) (end 162.259 91.948) (width 0.25) (layer "B.Cu") (net 55))
   (segment (start 162.259 91.948) (end 162.306 91.995) (width 0.25) (layer "B.Cu") (net 55))
@@
   (segment (start 159.3615 52.07) (end 158.5995 52.07) (width 0.25) (layer "F.Cu") (net 72))
   (segment (start 157.7745 52.895) (end 156.8215 52.895) (width 0.25) (layer "F.Cu") (net 72))
+  (segment (start 146.05 62.0165) (end 146.05 69.85) (width 0.25) (layer "F.Cu") (net 73))
+  (segment (start 156.8215 51.245) (end 146.05 62.0165) (width 0.25) (layer "F.Cu") (net 73))
+  (via (at 146.05 69.85) (size 0.8) (drill 0.4) (layers "F.Cu" "B.Cu") (net 73))
+  (segment (start 146.05 108.104) (end 133.504 120.65) (width 0.25) (layer "B.Cu") (net 73))
+  (segment (start 146.05 69.85) (end 146.05 108.104) (width 0.25) (layer "B.Cu") (net 73))
   (segment (start 127.002 66.548) (end 127.701 65.849) (width 0.25) (layer "F.Cu") (net 74))
   (segment (start 125.1 66.548) (end 127.002 66.548) (width 0.25) (layer "F.Cu") (net 74))
@@
   (segment (start 158.5995 61.976) (end 157.7745 62.801) (width 0.25) (layer "F.Cu") (net 75))
   (segment (start 157.7745 62.801) (end 156.8215 62.801) (width 0.25) (layer "F.Cu") (net 75))
+  (segment (start 156.8215 61.151) (end 156.019 61.151) (width 0.25) (layer "F.Cu") (net 76))
+  (segment (start 156.019 61.151) (end 147.32 69.85) (width 0.25) (layer "F.Cu") (net 76))
+  (via (at 147.32 69.85) (size 0.8) (drill 0.4) (layers "F.Cu" "B.Cu") (net 76))
+  (segment (start 147.32 69.85) (end 146.49952 70.67048) (width 0.25) (layer "B.Cu") (net 76))
+  (segment (start 146.49952 110.19448) (end 133.504 123.19) (width 0.25) (layer "B.Cu") (net 76))
+  (segment (start 146.49952 70.67048) (end 146.49952 110.19448) (width 0.25) (layer "B.Cu") (net 76))
   (segment (start 162.1555 60.452) (end 164.4415 60.452) (width 0.25) (layer "B.Cu") (net 77))
   (segment (start 127.002 76.2) (end 127.701 75.501) (width 0.25) (layer "F.Cu") (net 78))
@@
   (segment (start 159.512 71.9855) (end 158.75 71.9855) (width 0.25) (layer "F.Cu") (net 81))
   (segment (start 158.75 71.9855) (end 157.925 72.8105) (width 0.25) (layer "F.Cu") (net 81))
+  (segment (start 155.6615 69.85) (end 148.59 69.85) (width 0.25) (layer "F.Cu") (net 82))
+  (segment (start 156.972 71.1605) (end 155.6615 69.85) (width 0.25) (layer "F.Cu") (net 82))
+  (via (at 148.59 69.85) (size 0.8) (drill 0.4) (layers "F.Cu" "B.Cu") (net 82))
+  (segment (start 148.59 69.85) (end 147.066 71.374) (width 0.25) (layer "B.Cu") (net 82))
+  (segment (start 147.066 71.374) (end 147.066 112.168) (width 0.25) (layer "B.Cu") (net 82))
+  (segment (start 147.066 112.168) (end 133.504 125.73) (width 0.25) (layer "B.Cu") (net 82))
   (segment (start 162.306 70.4615) (end 164.592 70.4615) (width 0.25) (layer "B.Cu") (net 83))
   (segment (start 127.002 85.852) (end 127.701 85.153) (width 0.25) (layer "F.Cu") (net 84))
@@
   (segment (start 157.925 82.7165) (end 156.972 82.7165) (width 0.25) (layer "F.Cu") (net 87))
   (segment (start 159.512 81.8915) (end 158.75 81.8915) (width 0.25) (layer "F.Cu") (net 87))
+  (segment (start 156.972 81.0665) (end 151.0895 81.0665) (width 0.25) (layer "F.Cu") (net 88))
+  (segment (start 151.0895 81.0665) (end 149.606 82.55) (width 0.25) (layer "F.Cu") (net 88))
+  (via (at 149.606 82.55) (size 0.8) (drill 0.4) (layers "F.Cu" "B.Cu") (net 88))
+  (segment (start 147.574 84.582) (end 147.574 114.2) (width 0.25) (layer "B.Cu") (net 88))
+  (segment (start 149.606 82.55) (end 147.574 84.582) (width 0.25) (layer "B.Cu") (net 88))
+  (segment (start 147.574 114.2) (end 133.504 128.27) (width 0.25) (layer "B.Cu") (net 88))
   (segment (start 162.306 80.3675) (end 164.592 80.3675) (width 0.25) (layer "B.Cu") (net 89))
   (segment (start 127.063 134.112) (end 127.762 133.413) (width 0.25) (layer "F.Cu") (net 90))
