File: epanel-io/v1/top/top.kicad_pcb (KiCad board)
At the start: 2 copper layers, 66.5 x 100.8 mm, 132 parts, among them J1 Conn_01x05_Male, J2 Conn_01x05_Female, J3 Conn_01x08_Female, J4 Conn_01x05_Female, J5 Conn_01x08_Female, J6 Conn_01x04_Female, J7 Conn_01x04_Female, U1 Pico, U10 4N35, U11 H11AA1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

Commit message: wip pcb
Routing:
- net /Input 3/RPI: track 2.89 -> 65.3 mm, vias 0 -> 3
- net +5V: track 0.00 -> 62.1 mm, vias 0 -> 2
- net /Input 1/RPI: track 2.89 -> 62.8 mm, vias 0 -> 1
- net /Input 2/RPI: track 2.89 -> 60.5 mm, vias 0 -> 1
- net /Input 4/RPI: track 2.89 -> 50.8 mm, vias 0 -> 1
- net /Input 5/RPI: track 2.89 -> 36.8 mm
- net /Input 6/RPI: track 2.89 -> 36.4 mm
- net +3V3: track 107.6 -> 140.2 mm
- net /Input 7/RPI: track 2.89 -> 26.5 mm
- net /Input 8/RPI: track 2.89 -> 18.8 mm
- net /Output 7/RPI: track 0.00 -> 15.1 mm
- net /Output 6/RPI: track 0.00 -> 14.2 mm
- net /Output 8/RPI: track 0.00 -> 8.67 mm
- net /Output 5/RPI: track 0.00 -> 6.72 mm
- net Net-(R1-Pad1): track 40.5 -> 39.8 mm, vias 0 -> 1
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
Commit message: wip pcb
Routing:
- net /Input 9/RPI: track 2.89 -> 90.4 mm, vias 0 -> 2
- net /Input 10/RPI: track 2.89 -> 88.5 mm, vias 0 -> 2
Changed lines of the file:
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@@
   (segment (start 130.048 85.09) (end 138.684 85.09) (width 0.25) (layer "F.Cu") (net 4))
   (segment (start 112.268 100.33) (end 126.238 100.33) (width 0.25) (layer "F.Cu") (net 4))
+  (segment (start 128.27 98.298) (end 126.238 100.33) (width 0.25) (layer "F.Cu") (net 4))
   (segment (start 138.684 85.09) (end 143.764 90.17) (width 0.25) (layer "F.Cu") (net 4))
   (segment (start 111.188 101.41) (end 112.268 100.33) (width 0.25) (layer "F.Cu") (net 4))
   (segment (start 143.764 90.17) (end 151.284 90.17) (width 0.25) (layer "F.Cu") (net 4))
-  (segment (start 126.238 100.33) (end 130.048 96.52) (width 0.25) (layer "F.Cu") (net 4))
   (segment (start 111.188 107.858) (end 111.188 101.41) (width 0.25) (layer "F.Cu") (net 4))
-  (via (at 130.048 96.52) (size 0.8) (drill 0.4) (layers "F.Cu" "B.Cu") (net 4))
+  (via (at 128.27 98.298) (size 0.8) (drill 0.4) (layers "F.Cu" "B.Cu") (net 4))
   (via (at 130.048 85.09) (size 0.8) (drill 0.4) (layers "F.Cu" "B.Cu") (net 4))
+  (segment (start 130.048 96.52) (end 128.27 98.298) (width 0.25) (layer "B.Cu") (net 4))
   (segment (start 130.048 96.52) (end 130.048 85.852) (width 0.25) (layer "B.Cu") (net 4))
   (segment (start 130.048 85.852) (end 130.048 85.09) (width 0.25) (layer "B.Cu") (net 4))
@@
   (segment (start 156.972 128.778) (end 153.924 125.73) (width 0.25) (layer "F.Cu") (net 112))
   (segment (start 162.306 110.0855) (end 164.592 110.0855) (width 0.25) (layer "B.Cu") (net 113))
-  (segment (start 125.161 95.504) (end 127.063 95.504) (width 0.25) (layer "F.Cu") (net 114))
-  (segment (start 127.063 95.504) (end 127.762 94.805) (width 0.25) (layer "F.Cu") (net 114))
+  (segment (start 127.762 94.805) (end 127.762 95.504) (width 0.25) (layer "F.Cu") (net 114))
+  (segment (start 127.762 95.504) (end 129.286 95.504) (width 0.25) (layer "F.Cu") (net 114))
+  (segment (start 149.098 115.57) (end 151.284 115.57) (width 0.25) (layer "F.Cu") (net 114))
+  (segment (start 130.556 108.712) (end 130.556 109.474) (width 0.25) (layer "F.Cu") (net 114))
+  (segment (start 125.161 95.504) (end 127.762 95.504) (width 0.25) (layer "F.Cu") (net 114))
+  (segment (start 129.286 95.504) (end 130.556 96.774) (width 0.25) (layer "F.Cu") (net 114))
+  (segment (start 146.05 139.192) (end 146.05 118.618) (width 0.25) (layer "F.Cu") (net 114))
+  (segment (start 146.05 118.618) (end 149.098 115.57) (width 0.25) (layer "F.Cu") (net 114))
+  (segment (start 130.556 96.774) (end 130.556 108.712) (width 0.25) (layer "F.Cu") (net 114))
+  (via (at 146.05 139.192) (size 0.8) (drill 0.4) (layers "F.Cu" "B.Cu") (net 114))
+  (via (at 130.556 109.474) (size 0.8) (drill 0.4) (layers "F.Cu" "B.Cu") (net 114))
+  (segment (start 130.556 109.474) (end 130.556 136.906) (width 0.25) (layer "B.Cu") (net 114))
+  (segment (start 132.588 139.192) (end 146.05 139.192) (width 0.25) (layer "B.Cu") (net 114))
+  (segment (start 130.556 137.16) (end 132.588 139.192) (width 0.25) (layer "B.Cu") (net 114))
+  (segment (start 130.556 136.906) (end 130.556 137.16) (width 0.25) (layer "B.Cu") (net 114))
   (segment (start 115.631 92.964) (end 118.11 92.964) (width 0.25) (layer "F.Cu") (net 115))
   (segment (start 118.11 92.964) (end 120.65 95.504) (width 0.25) (layer "F.Cu") (net 115))
@@
   (segment (start 162.306 100.076) (end 164.592 100.076) (width 0.25) (layer "B.Cu") (net 119))
   (segment (start 125.161 105.156) (end 127.063 105.156) (width 0.25) (layer "F.Cu") (net 120))
-  (segment (start 127.063 105.156) (end 127.762 104.457) (width 0.25) (layer "F.Cu") (net 120))
+  (segment (start 127.762 104.457) (end 127.762 105.156) (width 0.25) (layer "F.Cu") (net 120))
+  (segment (start 128.27 105.156) (end 129.54 106.426) (width 0.25) (layer "F.Cu") (net 120))
+  (segment (start 129.54 106.426) (end 129.54 108.712) (width 0.25) (layer "F.Cu") (net 120))
+  (segment (start 145.034 112.776) (end 147.32 110.49) (width 0.25) (layer "F.Cu") (net 120))
+  (segment (start 145.034 140.462) (end 145.034 112.776) (width 0.25) (layer "F.Cu") (net 120))
+  (segment (start 127.762 105.156) (end 128.27 105.156) (width 0.25) (layer "F.Cu") (net 120))
+  (segment (start 147.32 110.49) (end 151.284 110.49) (width 0.25) (layer "F.Cu") (net 120))
+  (segment (start 127.063 105.156) (end 127.762 105.156) (width 0.25) (layer "F.Cu") (net 120))
+  (via (at 129.54 108.712) (size 0.8) (drill 0.4) (layers "F.Cu" "B.Cu") (net 120))
+  (via (at 145.034 140.462) (size 0.8) (drill 0.4) (layers "F.Cu" "B.Cu") (net 120))
+  (segment (start 129.54 108.712) (end 129.54 137.668) (width 0.25) (layer "B.Cu") (net 120))
+  (segment (start 131.826 140.208) (end 132.08 140.462) (width 0.25) (layer "B.Cu") (net 120))
+  (segment (start 129.54 137.668) (end 129.54 137.922) (width 0.25) (layer "B.Cu") (net 120))
+  (segment (start 132.08 140.462) (end 145.034 140.462) (width 0.25) (layer "B.Cu") (net 120))
+  (segment (start 129.54 137.922) (end 131.826 140.208) (width 0.25) (layer "B.Cu") (net 120))
   (segment (start 118.11 102.616) (end 120.65 105.156) (width 0.25) (layer "F.Cu") (net 121))
   (segment (start 115.631 102.616) (end 118.11 102.616) (width 0.25) (layer "F.Cu") (net 121))

Commit message: pcb wired
Routing:
- net /Output 10/RPI: track 0.00 -> 15.6 mm
- net /Output 9/RPI: track 0.00 -> 11.6 mm
- net GND: track 311.1 -> 315.9 mm
Changed lines of the file:
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@@
   (segment (start 125.161 98.044) (end 122.682 98.044) (width 0.25) (layer "F.Cu") (net 3))
   (segment (start 159.512 94.234) (end 161.798 94.234) (width 0.25) (layer "F.Cu") (net 3))
-  (segment (start 154.178 92.71) (end 151.284 92.71) (width 0.25) (layer "F.Cu") (net 3))
   (segment (start 161.798 104.14) (end 161.798 114.046) (width 0.25) (layer "F.Cu") (net 3))
   (segment (start 159.3615 54.61) (end 161.544 54.61) (width 0.25) (layer "F.Cu") (net 3))
@@
   (segment (start 123.952 49.784) (end 122.682 51.054) (width 0.25) (layer "F.Cu") (net 3))
   (segment (start 161.798 142.748) (end 160.782 143.764) (width 0.25) (layer "F.Cu") (net 3))
-  (segment (start 155.702 94.234) (end 154.178 92.71) (width 0.25) (layer "F.Cu") (net 3))
+  (segment (start 153.67 91.44) (end 152.4 92.71) (width 0.25) (layer "F.Cu") (net 3))
   (segment (start 125.1 69.088) (end 122.682 69.088) (width 0.25) (layer "F.Cu") (net 3))
   (segment (start 125.161 107.696) (end 122.682 107.696) (width 0.25) (layer "F.Cu") (net 3))
@@
   (segment (start 159.512 74.5255) (end 161.6475 74.5255) (width 0.25) (layer "F.Cu") (net 3))
   (segment (start 161.798 84.328) (end 161.798 94.234) (width 0.25) (layer "F.Cu") (net 3))
-  (segment (start 159.512 94.234) (end 155.702 94.234) (width 0.25) (layer "F.Cu") (net 3))
+  (segment (start 153.67 88.091) (end 153.67 91.44) (width 0.25) (layer "F.Cu") (net 3))
   (segment (start 159.512 84.4315) (end 161.6945 84.4315) (width 0.25) (layer "F.Cu") (net 3))
   (segment (start 122.682 59.182) (end 122.682 69.088) (width 0.25) (layer "F.Cu") (net 3))
   (segment (start 122.52 110.398) (end 122.682 110.236) (width 0.25) (layer "F.Cu") (net 3))
+  (segment (start 159.512 84.4315) (end 157.3295 84.4315) (width 0.25) (layer "F.Cu") (net 3))
   (segment (start 161.798 94.234) (end 161.798 104.14) (width 0.25) (layer "F.Cu") (net 3))
   (segment (start 161.798 74.676) (end 161.798 84.328) (width 0.25) (layer "F.Cu") (net 3))
   (segment (start 161.544 54.61) (end 161.798 54.356) (width 0.25) (layer "F.Cu") (net 3))
   (segment (start 123.698 146.304) (end 125.161 146.304) (width 0.25) (layer "F.Cu") (net 3))
+  (segment (start 152.4 92.71) (end 151.284 92.71) (width 0.25) (layer "F.Cu") (net 3))
   (segment (start 122.682 107.696) (end 122.682 110.236) (width 0.25) (layer "F.Cu") (net 3))
   (segment (start 122.682 127) (end 122.682 136.652) (width 0.25) (layer "F.Cu") (net 3))
@@
   (segment (start 111.188 110.398) (end 122.52 110.398) (width 0.25) (layer "F.Cu") (net 3))
   (segment (start 125.161 127) (end 122.682 127) (width 0.25) (layer "F.Cu") (net 3))
+  (segment (start 157.3295 84.4315) (end 153.67 88.091) (width 0.25) (layer "F.Cu") (net 3))
   (segment (start 125.1 78.74) (end 122.682 78.74) (width 0.25) (layer "F.Cu") (net 3))
   (via (at 122.682 98.044) (size 0.8) (drill 0.4) (layers "F.Cu" "B.Cu") (net 3))
@@
   (segment (start 158.75 101.6) (end 157.925 102.425) (width 0.25) (layer "F.Cu") (net 117))
   (segment (start 159.512 101.6) (end 158.75 101.6) (width 0.25) (layer "F.Cu") (net 117))
+  (segment (start 156.972 100.775) (end 156.019 100.775) (width 0.25) (layer "F.Cu") (net 118))
+  (segment (start 153.924 107.95) (end 151.284 107.95) (width 0.25) (layer "F.Cu") (net 118))
+  (segment (start 154.94 106.934) (end 153.924 107.95) (width 0.25) (layer "F.Cu") (net 118))
+  (segment (start 156.019 100.775) (end 154.94 101.854) (width 0.25) (layer "F.Cu") (net 118))
+  (segment (start 154.94 101.854) (end 154.94 106.934) (width 0.25) (layer "F.Cu") (net 118))
   (segment (start 162.306 100.076) (end 164.592 100.076) (width 0.25) (layer "B.Cu") (net 119))
   (segment (start 125.161 105.156) (end 127.063 105.156) (width 0.25) (layer "F.Cu") (net 120))
@@
   (segment (start 158.75 91.694) (end 157.925 92.519) (width 0.25) (layer "F.Cu") (net 123))
   (segment (start 159.512 91.694) (end 158.75 91.694) (width 0.25) (layer "F.Cu") (net 123))
+  (segment (start 156.972 90.869) (end 156.147 90.869) (width 0.25) (layer "F.Cu") (net 124))
+  (segment (start 152.654 102.87) (end 151.284 102.87) (width 0.25) (layer "F.Cu") (net 124))
+  (segment (start 153.924 101.6) (end 152.654 102.87) (width 0.25) (layer "F.Cu") (net 124))
+  (segment (start 156.147 90.869) (end 153.924 93.092) (width 0.25) (layer "F.Cu") (net 124))
+  (segment (start 153.924 93.092) (end 153.924 101.6) (width 0.25) (layer "F.Cu") (net 124))
   (segment (start 162.306 90.17) (end 164.592 90.17) (width 0.25) (layer "B.Cu") (net 125))
   (segment (start 166.9815 57.15) (end 166.9815 59.3325) (width 0.25) (layer "F.Cu") (net 158))

Commit message: DRC
Routing:
- net /Output 3/GATE: track 11.8 -> 11.1 mm
- net /Output 1/GATE: track 20.8 -> 20.2 mm
- net /Input 1/NEUT: track 128.2 -> 127.7 mm
