File: epanel-io/v1/top/top.kicad_sch (KiCad schematic)
At the start: 12 parts, among them J1 Conn_01x05_Male, J2 Screw_Terminal_01x05, J3 Screw_Terminal_01x05, J4 Screw_Terminal_01x05, J5 Screw_Terminal_01x05, J6 Screw_Terminal_01x03, J7 Screw_Terminal_01x03, U1 Pico, U2 H11AA1

Commit message: top schematic
Parts:
- removed J2, J3, J4, J5: Screw_Terminal_01x05, TerminalBlock:TerminalBlock_bornier-5_P5.08mm, symbol Connector:Screw_Terminal_01x05
- removed J6, J7: Screw_Terminal_01x03, TerminalBlock:TerminalBlock_bornier-3_P5.08mm, symbol Connector:Screw_Terminal_01x03
- added J2, J4: Conn_01x05_Female, Connector_PinHeader_2.54mm:PinHeader_1x05_P2.54mm_Vertical, symbol Connector:Conn_01x05_Female
- added J3, J5: Conn_01x08_Female, Connector_PinHeader_2.54mm:PinHeader_1x08_P2.54mm_Vertical, symbol Connector:Conn_01x08_Female
- added J6, J7: Conn_01x04_Female, Connector_PinHeader_2.54mm:PinHeader_1x04_P2.54mm_Vertical, symbol Connector:Conn_01x04_Female
Connections:
- net Input 1/INPUT: now also J2.2 (Pin_2)
- net Input 1/NEUT: now also J2.1 (Pin_1)
- net Input 10/INPUT: now also J6.3 (Pin_3)
- net Input 10/NEUT: now also J6.1 (Pin_1)
- net Input 2/INPUT: now also J2.3 (Pin_3)
- net Input 3/INPUT: now also J2.4 (Pin_4)
- net Input 4/INPUT: now also J2.5 (Pin_5)
- net Input 5/INPUT: now also J4.4 (Pin_4)
- net Input 5/NEUT: now also J4.1 (Pin_1)
- net Input 5/RPI: now also U1.21 (GPIO16); no longer U1.19 (GPIO14)
- net Input 6/INPUT: now also J4.5 (Pin_5)
- net Input 6/RPI: now also U1.22 (GPIO17); no longer U1.20 (GPIO15)
- net Input 7/INPUT: now also J4.2 (Pin_2)
- net Input 7/RPI: now also U1.19 (GPIO14); no longer U1.21 (GPIO16)
- net Input 8/INPUT: now also J4.3 (Pin_3)
- net Input 8/RPI: now also U1.20 (GPIO15); no longer U1.22 (GPIO17)
- net Input 9/INPUT: now also J6.2 (Pin_2)
- net Output 5/RPI: now also U1.26 (GPIO20); no longer U1.24 (GPIO18)
- net Output 6/RPI: now also U1.27 (GPIO21); no longer U1.26 (GPIO20)
- net Output 7/RPI: now also U1.24 (GPIO18); no longer U1.25 (GPIO19)
- net Output 8/RPI: now also U1.25 (GPIO19); no longer U1.27 (GPIO21)
- net Output 10/LINE: no longer names the net of R3.1
- net Output 10/LINE: now also J6.4 (Pin_4)
- new net Output 1/GATE: J3.2 (Pin_2)
- new net Output 1/GND: J3.1 (Pin_1)
- new net Output 10/GATE: J7.4 (Pin_4)
- new net Output 10/GND: J7.3 (Pin_3)
- new net Output 2/GATE: J3.4 (Pin_4)
- new net Output 2/GND: J3.3 (Pin_3)
- new net Output 3/GATE: J3.6 (Pin_6)
- new net Output 3/GND: J3.5 (Pin_5)
- new net Output 4/GATE: J3.8 (Pin_8)
- new net Output 4/GND: J3.7 (Pin_7)
- new net Output 5/GATE: J5.6 (Pin_6)
- new net Output 5/GND: J5.5 (Pin_5)
- new net Output 6/GATE: J5.8 (Pin_8)
- new net Output 6/GND: J5.7 (Pin_7)
- new net Output 7/GATE: J5.2 (Pin_2)
- new net Output 7/GND: J5.1 (Pin_1)
- new net Output 8/GATE: J5.4 (Pin_4)
- new net Output 8/GND: J5.3 (Pin_3)
- new net Output 9/GATE: J7.2 (Pin_2)
- new net Output 9/GND: J7.1 (Pin_1)
Other:
- sheet Output 1 ports: added GATE, GND; removed LINE, OUTPUT
- sheet Output 10 ports: added GATE, GND; removed LINE, OUTPUT
- sheet Output 2 ports: added GATE, GND; removed LINE, OUTPUT
- sheet Output 3 ports: added GATE, GND; removed LINE, OUTPUT
- sheet Output 4 ports: added GATE, GND; removed LINE, OUTPUT
- sheet Output 5 ports: added GATE, GND; removed LINE, OUTPUT
- sheet Output 6 ports: added GATE, GND; removed LINE, OUTPUT
- sheet Output 7 ports: added GATE, GND; removed LINE, OUTPUT
- sheet Output 8 ports: added GATE, GND; removed LINE, OUTPUT
- sheet Output 9 ports: added GATE, GND; removed LINE, OUTPUT

Commit message: fix gnd
Connections:
- net Output 1/GND renamed Output 1/SOURCE
- net Output 10/GND renamed Output 10/SOURCE
- net Output 2/GND renamed Output 2/SOURCE
- net Output 3/GND renamed Output 3/SOURCE
- net Output 4/GND renamed Output 4/SOURCE
- net Output 5/GND renamed Output 5/SOURCE
- net Output 6/GND renamed Output 6/SOURCE
- net Output 7/GND renamed Output 7/SOURCE
- net Output 8/GND renamed Output 8/SOURCE
- net Output 9/GND renamed Output 9/SOURCE
Other:
- sheet Output 1 ports: added SOURCE; removed GND
- sheet Output 10 ports: added SOURCE; removed GND
- sheet Output 2 ports: added SOURCE; removed GND
- sheet Output 3 ports: added SOURCE; removed GND
- sheet Output 4 ports: added SOURCE; removed GND
- sheet Output 5 ports: added SOURCE; removed GND
- sheet Output 6 ports: added SOURCE; removed GND
- sheet Output 7 ports: added SOURCE; removed GND
- sheet Output 8 ports: added SOURCE; removed GND
- sheet Output 9 ports: added SOURCE; removed GND
Changed lines of the file:
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@@
       (effects (font (size 1.27 1.27)) (justify left))
     )
-    (pin "GND" input (at 232.41 86.36 0)
+    (pin "SOURCE" input (at 232.41 86.36 0)
       (effects (font (size 1.27 1.27)) (justify right))
     )
@@
       (effects (font (size 1.27 1.27)) (justify left))
     )
-    (pin "GND" input (at 111.76 171.45 0)
+    (pin "SOURCE" input (at 111.76 171.45 0)
       (effects (font (size 1.27 1.27)) (justify right))
     )
@@
       (effects (font (size 1.27 1.27)) (justify left))
     )
-    (pin "GND" input (at 232.41 172.72 0)
+    (pin "SOURCE" input (at 232.41 172.72 0)
       (effects (font (size 1.27 1.27)) (justify right))
     )
@@
       (effects (font (size 1.27 1.27)) (justify left))
     )
-    (pin "GND" input (at 232.41 129.54 0)
+    (pin "SOURCE" input (at 232.41 129.54 0)
       (effects (font (size 1.27 1.27)) (justify right))
     )
@@
       (effects (font (size 1.27 1.27)) (justify left))
     )
-    (pin "GND" input (at 335.28 86.36 0)
+    (pin "SOURCE" input (at 335.28 86.36 0)
       (effects (font (size 1.27 1.27)) (justify right))
     )
@@
       (effects (font (size 1.27 1.27)) (justify left))
     )
-    (pin "GND" input (at 111.76 85.09 0)
+    (pin "SOURCE" input (at 111.76 85.09 0)
       (effects (font (size 1.27 1.27)) (justify right))
     )
@@
       (effects (font (size 1.27 1.27)) (justify left))
     )
-    (pin "GND" input (at 111.76 128.27 0)
+    (pin "SOURCE" input (at 111.76 128.27 0)
       (effects (font (size 1.27 1.27)) (justify right))
     )
@@
       (effects (font (size 1.27 1.27)) (justify left))
     )
-    (pin "GND" input (at 335.28 43.18 0)
+    (pin "SOURCE" input (at 335.28 43.18 0)
       (effects (font (size 1.27 1.27)) (justify right))
     )
@@
       (effects (font (size 1.27 1.27)) (justify left))
     )
-    (pin "GND" input (at 111.76 41.91 0)
+    (pin "SOURCE" input (at 111.76 41.91 0)
       (effects (font (size 1.27 1.27)) (justify right))
     )
@@
       (effects (font (size 1.27 1.27)) (justify left))
     )
-    (pin "GND" input (at 232.41 43.18 0)
-      (effects (font (size 1.27 1.27)) (justify right))
-    )
+    (pin "SOURCE" input (at 232.41 43.18 0)
+      (effects (font (size 1.27 1.27)) (justify right))
+    )

Commit message: update rpi pinout
Parts:
- U1: footprint MCU_RaspberryPi_and_Boards:RPi_Pico_SMD_TH -> Custom:RPI_Pico_pinout
Changed lines of the file:
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@@
     (property "Reference" "U1" (id 0) (at 105.41 189.23 0))
     (property "Value" "Pico" (id 1) (at 105.41 191.77 0))
-    (property "Footprint" "MCU_RaspberryPi_and_Boards:RPi_Pico_SMD_TH" (id 2) (at 105.41 220.98 90)
+    (property "Footprint" "Custom:RPI_Pico_pinout" (id 2) (at 105.41 220.98 90)
       (effects (font (size 1.27 1.27)) hide)
     )
@@
     )
     (path "/547d4158-ddba-4752-97f0-70d1b9e258cb"
-      (reference "U1") (unit 1) (value "Pico") (footprint "MCU_RaspberryPi_and_Boards:RPi_Pico_SMD_TH")
+      (reference "U1") (unit 1) (value "Pico") (footprint "Custom:RPI_Pico_pinout")
     )
     (path "/c941acbf-ee78-4974-aae7-741801263b9b"

Commit message: update order + BOM
Parts:
- U2: LCSC C184383 -> C258253
Changed lines of the file:
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@@
       (effects (font (size 1.27 1.27)) (justify left) hide)
     )
-    (property "LCSC" "C184383" (id 4) (at 243.84 260.35 0)
+    (property "LCSC" "C258253" (id 4) (at 243.84 260.35 0)
       (effects (font (size 1.27 1.27)) hide)
     )
