File: garden-box/prototype-1/prototype.kicad_sch (KiCad schematic)
At the start: 16 parts, among them J1 Conn_01x05_Male, J2 Screw_Terminal_01x02, Q1 IRF830, U1 4N35

Commit message: wip garden box
Parts:
- added D?: LED, symbol Device:LED
- added D?: 1N4148, Diode_THT:D_DO-35_SOD27_P7.62mm_Horizontal, symbol Diode:1N4148
- added K?: G6E, Relay_THT:Relay_SPDT_Omron_G6E, symbol Relay:G6E
- added Q?: 2N3904, Package_TO_SOT_THT:TO-92_Inline, symbol Transistor_BJT:2N3904
- added R? (x2): 1KΩ, Resistor_SMD:R_0603_1608Metric, symbol Device:R
- added R?: 10KΩ, Resistor_SMD:R_0603_1608Metric, symbol Device:R
Connections:
- net GND: now also U?.2 (GND), Q?.1 (E), R?.2
- net +5V: now reaches U?.3 (VO)
- net +5V: now also D?.1 (K), K?.1, R?.1
- new net: D?.1 (K), D?.2 (A), K?.6, Q?.3 (C)
- new net: D?.2 (A), R?.2
- new net: Q?.2 (B), R?.1, R?.1
Other:
- moved on the sheet: T?, U?

Commit message: wip garden box proto
Parts:
- removed D?: LED, symbol Device:LED
- removed D?: 1N4148, Diode_THT:D_DO-35_SOD27_P7.62mm_Horizontal, symbol Diode:1N4148
- removed K?: G6E, Relay_THT:Relay_SPDT_Omron_G6E, symbol Relay:G6E
- removed Q?: 2N3904, Package_TO_SOT_THT:TO-92_Inline, symbol Transistor_BJT:2N3904
- removed R? (x2): 1KΩ, Resistor_SMD:R_0603_1608Metric, symbol Device:R
- removed R?: 10KΩ, Resistor_SMD:R_0603_1608Metric, symbol Device:R
- added J? (x8): Screw_Terminal_01x02, symbol Connector:Screw_Terminal_01x02
- added J?: Conn_01x04_Male, symbol Connector:Conn_01x04_Male
- added J?: Conn_01x02_Male, symbol Connector:Conn_01x02_Male
- added J?: Conn_01x03_Male, symbol Connector:Conn_01x03_Male
- added SW? (x6): SW_Push_DPDT, symbol Switch:SW_Push_DPDT
Connections:
- net GND: now also J?.2 (Pin_2)
- net at U?.1 (VI): now also J?.1 (Pin_1)
- net Relay Transfo/output2: now reaches T?.1 (AA)
- net at T?.2 (AB): now also J?.2 (Pin_2), SW?.4 (A), SW?.4 (A), SW?.4 (A), SW?.4 (A), SW?.4 (A), SW?.4 (A)
- net at T?.3 (SA): now also SW?.6 (C), SW?.6 (C), SW?.6 (C), SW?.6 (C), SW?.6 (C), SW?.6 (C)
- net at T?.4 (SB): now also T?.5 (SC)
- net at T?.6 (SD): now also SW?.3 (C), SW?.3 (C), SW?.3 (C), SW?.3 (C), SW?.3 (C), SW?.3 (C)
- new net: J?.1 (Pin_1), SW?.5 (B) (x6)
- new net Relay Transfo/output1: J?.1 (Pin_1), SW?.1 (A), SW?.1 (A), SW?.1 (A), SW?.1 (A), SW?.1 (A), SW?.1 (A)
- new net Relay1/output1: SW?.2 (B)
- new net Relay1/output2: J?.2 (Pin_2)
- new net Relay2/output1: SW?.2 (B)
- new net Relay2/output2: J?.2 (Pin_2)
- new net Relay3/output1: SW?.2 (B)
- new net Relay3/output2: J?.2 (Pin_2)
- new net Relay4/output1: SW?.2 (B)
- new net Relay4/output2: J?.2 (Pin_2)
- new net Relay5/output1: SW?.2 (B)
- new net Relay5/output2: J?.2 (Pin_2)
- new net Relay6/output1: SW?.2 (B)
- new net Relay6/output2: J?.2 (Pin_2)
Other:
- added sheet Relay Transfo (relay.kicad_sch)
- added sheet Relay1 (relay.kicad_sch)
- added sheet Relay2 (relay.kicad_sch)
- added sheet Relay3 (relay.kicad_sch)
- added sheet Relay4 (relay.kicad_sch)
- added sheet Relay5 (relay.kicad_sch)
- added sheet Relay6 (relay.kicad_sch)
- note added: "+"
- note added: "-"
- note added: "12v"
- note added: "220v"
- note added: "AO"
- note added: "DO"
- note added: "DS18B20"
- note added: "L"
- note added: "N"
- note added: "Switch"
- note added: "data"
- moved on the sheet: C1, C2, D1, D2, D6, J1, J2, Q1, R1, R2, R3, R4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

Commit message: wip garden-box schematic
Parts:
- removed C1: 2.2uF/63V, Capacitor_SMD:C_1206_3216Metric, symbol Device:C_Polarized
- removed C2: 220nF/275V, Capacitor_SMD:C_1210_3225Metric, symbol Device:C
- removed D1: 10V/0.4W, Diode_SMD:D_SOD-123, symbol Diode:BZV55B10
- removed D2: 4* 1N5408, Diode_SMD:Diode_Bridge_Diotec_SO-DIL-Slim, symbol Device:D_Bridge_+-AA
- removed D6: 1N4007, Diode_SMD:D_SMA, symbol Diode:1N4007
- removed J1: Conn_01x05_Male, Connector_PinHeader_2.54mm:PinHeader_1x05_P2.54mm_Vertical, symbol Connector:Conn_01x05_Male
- removed J2: Screw_Terminal_01x02, TerminalBlock:TerminalBlock_bornier-2_P5.08mm, symbol Connector:Screw_Terminal_01x02
- removed Q1: IRF830, Package_TO_SOT_SMD:TO-263-3_TabPin2, symbol Transistor_FET:IRF740
- removed R1: 330Ω, Resistor_SMD:R_0603_1608Metric, symbol Device:R
- removed R2: 22KΩ, Resistor_SMD:R_0603_1608Metric, symbol Device:R
- removed R3, R4: 33KΩ, Resistor_SMD:R_0603_1608Metric, symbol Device:R
- removed R5: 220Ω, Resistor_SMD:R_0603_1608Metric, symbol Device:R
- removed U1: 4N35, Package_DIP:SMDIP-6_W7.62mm, symbol Isolator:4N35
Connections:
- net +5V: now also J?.1 (Pin_1), J?.1 (Pin_1), J?.1 (Pin_1)
- net GND: now also J?.2 (Pin_2), J?.2 (Pin_2), J?.2 (Pin_2)
- no-connect marks 1 -> 0
Other:
- note added: "Moisture sensor"
- note removed: "Mosfet-based dimmer"
- moved on the sheet: J?
