File: garden-box/prototype-1/prototype-1.kicad_sch (KiCad schematic)
At the start: 15 parts, among them J1 Conn_01x02_Male, J2 Conn_01x03_Male, J3 Conn_01x04_Male, U2 ESP32-POE

Commit message: proto 1 schematic + footprint stuff
Parts:
- removed J1: Conn_01x02_Male, Connector_PinHeader_2.54mm:PinHeader_1x02_P2.54mm_Vertical, symbol Connector:Conn_01x02_Male
- added J?: USB_A, Connector_USB:USB_A_Molex_67643_Horizontal, symbol Connector:USB_A
- added PS1: RS PRO 5V 2A, Converter_ACDC:Converter_ACDC_Recom_RAC20-xxSK_THT, symbol Converter_ACDC:IRM-10-5
- added R1: 4.7KΩ, Resistor_SMD:R_0402_1005Metric, symbol Device:R
- K1: renamed from K?; value G6E -> G6DN-1A-L_DC5; footprint Relay_THT:Relay_SPDT_Omron_G6E -> rs-online:G6DN-1A-L; symbol Relay:G6E -> mylife-symbols:G6DN-1A-L_DC5
- T1: renamed from T?; footprint (none) -> rs-online:VCM36212
- gave numbers to parts that had none: 9
- renumbered U2 to U1
Connections:
- net +3V3: now also J2.2 (Pin_2), R1.1
- net +5V: now also J?.1 (VBUS), PS1.4 (+Vo); no longer J2.2 (Pin_2)
- net GND: now also J?.4 (GND), J?.5 (Shield), PS1.3 (-Vo)
- net at D1.1 (K), D2.2 (A), Q1.3 (C): now also K1.2; no longer K1.6
- net at J2.3 (Pin_3), U1.18 (GPIO35): now also R1.2
- net at T1.1 (AA): now also J5.1 (Pin_1), K1.8
- net at T1.2 (AB): now also J4.2 (Pin_2), J5.2 (Pin_2), PS1.1 (AC/N)
- net at J4.1 (Pin_1): now also K1.5, PS1.2 (AC/L); no longer K1.7
Other:
- moved on the sheet: J2, J3, J4, J5, J6, T1

Commit message: annotate
Parts:
- gave numbers to parts that had none: 1
Changed lines of the file:
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@@
   (symbol (lib_id "Connector:USB_A") (at 31.75 88.9 0) (unit 1)
     (in_bom yes) (on_board yes) (fields_autoplaced)
-    (property "Reference" "J?" (id 0) (at 31.75 76.2 0))
+    (property "Reference" "J1" (id 0) (at 31.75 76.2 0))
     (property "Value" "USB_A" (id 1) (at 31.75 78.74 0))
     (property "Footprint" "Connector_USB:USB_A_Molex_67643_Horizontal" (id 2) (at 35.56 90.17 0)
@@
   (symbol (lib_id "power:+5V") (at 44.45 81.28 0) (unit 1)
     (in_bom yes) (on_board yes) (fields_autoplaced)
-    (property "Reference" "#PWR0102" (id 0) (at 44.45 85.09 0)
+    (property "Reference" "#PWR02" (id 0) (at 44.45 85.09 0)
       (effects (font (size 1.27 1.27)) hide)
     )
@@
   (symbol (lib_id "power:GND") (at 46.99 156.21 0) (unit 1)
     (in_bom yes) (on_board yes)
-    (property "Reference" "#PWR03" (id 0) (at 46.99 162.56 0)
+    (property "Reference" "#PWR04" (id 0) (at 46.99 162.56 0)
       (effects (font (size 1.27 1.27)) hide)
     )
@@
   (symbol (lib_id "power:+3.3V") (at 63.5 67.31 0) (unit 1)
     (in_bom yes) (on_board yes) (fields_autoplaced)
-    (property "Reference" "#PWR09" (id 0) (at 63.5 71.12 0)
+    (property "Reference" "#PWR08" (id 0) (at 63.5 71.12 0)
       (effects (font (size 1.27 1.27)) hide)
     )
@@
   (symbol (lib_id "power:GND") (at 31.75 105.41 0) (unit 1)
     (in_bom yes) (on_board yes)
-    (property "Reference" "#PWR0101" (id 0) (at 31.75 111.76 0)
+    (property "Reference" "#PWR01" (id 0) (at 31.75 111.76 0)
       (effects (font (size 1.27 1.27)) hide)
     )
@@
   (symbol (lib_id "power:GND") (at 58.42 72.39 0) (unit 1)
     (in_bom yes) (on_board yes)
-    (property "Reference" "#PWR08" (id 0) (at 58.42 78.74 0)
+    (property "Reference" "#PWR07" (id 0) (at 58.42 78.74 0)
       (effects (font (size 1.27 1.27)) hide)
     )
@@
   (symbol (lib_id "power:GND") (at 46.99 130.81 0) (unit 1)
     (in_bom yes) (on_board yes)
-    (property "Reference" "#PWR02" (id 0) (at 46.99 137.16 0)
+    (property "Reference" "#PWR03" (id 0) (at 46.99 137.16 0)
       (effects (font (size 1.27 1.27)) hide)
     )
@@
   (symbol (lib_id "power:+3.3V") (at 64.77 111.76 0) (unit 1)
     (in_bom yes) (on_board yes) (fields_autoplaced)
-    (property "Reference" "#PWR07" (id 0) (at 64.77 115.57 0)
+    (property "Reference" "#PWR09" (id 0) (at 64.77 115.57 0)
       (effects (font (size 1.27 1.27)) hide)
     )
@@
   )
   (symbol_instances
+    (path "/705d7904-7783-4aa0-8d1a-24e75e472f89"
+      (reference "#PWR01") (unit 1) (value "GND") (footprint "")
+    )
+    (path "/3226b6bd-c8f2-4b15-a10a-d43df37b02fa"
+      (reference "#PWR02") (unit 1) (value "+5V") (footprint "")
+    )
     (path "/a9799945-6524-4792-9375-160ea9239fdb"
-      (reference "#PWR02") (unit 1) (value "GND") (footprint "")
+      (reference "#PWR03") (unit 1) (value "GND") (footprint "")
     )
     (path "/3d24ca64-8898-4a21-92dc-4bb372c9b113"
-      (reference "#PWR03") (unit 1) (value "GND") (footprint "")
+      (reference "#PWR04") (unit 1) (value "GND") (footprint "")
     )
     (path "/c0477393-31e8-40d5-b090-5fa2eaf7ba72"
@@
       (reference "#PWR06") (unit 1) (value "+5V") (footprint "")
     )
+    (path "/9c21d32b-1bd6-41c7-a0fb-1c1fb434cb30"
+      (reference "#PWR07") (unit 1) (value "GND") (footprint "")
+    )
+    (path "/47dd3c39-450c-4d60-835c-89b562cd20bd"
+      (reference "#PWR08") (unit 1) (value "+3.3V") (footprint "")
+    )
     (path "/c1c839fa-6054-424e-a156-b2a9bf37d803"
-      (reference "#PWR07") (unit 1) (value "+3.3V") (footprint "")
-    )
-    (path "/9c21d32b-1bd6-41c7-a0fb-1c1fb434cb30"
-      (reference "#PWR08") (unit 1) (value "GND") (footprint "")
-    )
-    (path "/47dd3c39-450c-4d60-835c-89b562cd20bd"
       (reference "#PWR09") (unit 1) (value "+3.3V") (footprint "")
     )
@@
       (reference "#PWR016") (unit 1) (value "+5V") (footprint "")
     )
-    (path "/705d7904-7783-4aa0-8d1a-24e75e472f89"
-      (reference "#PWR0101") (unit 1) (value "GND") (footprint "")
-    )
-    (path "/3226b6bd-c8f2-4b15-a10a-d43df37b02fa"
-      (reference "#PWR0102") (unit 1) (value "+5V") (footprint "")
-    )
     (path "/4f6aa278-908b-4606-ab16-3f89a1d8ebf8"
       (reference "D1") (unit 1) (value "LED") (footprint "Diode_SMD:D_0805_2012Metric")
@@
       (reference "D2") (unit 1) (value "1N4148") (footprint "Diode_SMD:D_SOD-123")
     )
+    (path "/046cc858-94d2-4a81-a286-14af2525c2b6"
+      (reference "J1") (unit 1) (value "USB_A") (footprint "Connector_USB:USB_A_Molex_67643_Horizontal")
+    )
     (path "/a92772ed-b0e6-4a03-a485-6f9febfd19d3"
       (reference "J2") (unit 1) (value "Conn_01x03_Male") (footprint "Connector_PinHeader_2.54mm:PinHeader_1x03_P2.54mm_Vertical")
@@
       (reference "J6") (unit 1) (value "Screw_Terminal_01x02") (footprint "TerminalBlock:TerminalBlock_bornier-2_P5.08mm")
     )
-    (path "/046cc858-94d2-4a81-a286-14af2525c2b6"
-      (reference "J?") (unit 1) (value "USB_A") (footprint "Connector_USB:USB_A_Molex_67643_Horizontal")
-    )
     (path "/c594017f-aa60-467a-ab4f-3544e1ac6b56"

Commit message: fix footprint
Parts:
- PS1: footprint Converter_ACDC:Converter_ACDC_Recom_RAC20-xxSK_THT -> mylife-footprints:RS PRO 5V 2A
Changed lines of the file:
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@@
     (property "Reference" "PS1" (id 0) (at 110.49 15.24 0))
     (property "Value" "RS PRO 5V 2A" (id 1) (at 110.49 17.78 0))
-    (property "Footprint" "Converter_ACDC:Converter_ACDC_Recom_RAC20-xxSK_THT" (id 2) (at 110.49 34.29 0)
+    (property "Footprint" "mylife-footprints:RS PRO 5V 2A" (id 2) (at 110.49 34.29 0)
       (effects (font (size 1.27 1.27)) hide)
     )
@@
     )
     (path "/2fb2622f-7997-48d2-bce0-8286d8a31d77"
-      (reference "PS1") (unit 1) (value "RS PRO 5V 2A") (footprint "Converter_ACDC:Converter_ACDC_Recom_RAC20-xxSK_THT")
+      (reference "PS1") (unit 1) (value "RS PRO 5V 2A") (footprint "mylife-footprints:RS PRO 5V 2A")
     )
     (path "/3b87441e-9545-4daa-bf5c-0e30f2dd4c01"
