File: garden-box/prototype-1/prototype-1.kicad_pcb (KiCad board)
At the start: 2 copper layers, 88.9 x 66 mm, 0 parts

Commit message: pcb size + screw
Parts:
- added D1: LED, Diode_SMD:D_0805_2012Metric, F.Cu at (444.1, 109.2)
- added D2: 1N4148, Diode_SMD:D_SOD-123, F.Cu at (531.7, 29.3)
- added J1: USB_A, Connector_USB:USB_A_Molex_67643_Horizontal, F.Cu at (469.2, 81.8)
- added J2: Conn_01x03_Male, Connector_PinHeader_2.54mm:PinHeader_1x03_P2.54mm_Vertical, F.Cu at (434.7, 110.0)
- added J3: Conn_01x04_Male, Connector_PinHeader_2.54mm:PinHeader_1x04_P2.54mm_Vertical, F.Cu at (531.1, 17.7)
- added J4: Screw_Terminal_01x02, TerminalBlock:TerminalBlock_bornier-2_P5.08mm, F.Cu at (424.0, 114.0)
- added J5: Screw_Terminal_01x02, TerminalBlock:TerminalBlock_bornier-2_P5.08mm, F.Cu at (536.7, 19.9)
- added J6: Screw_Terminal_01x02, TerminalBlock:TerminalBlock_bornier-2_P5.08mm, F.Cu at (412.5, 112.2)
- added K1: G6DN-1A-L_DC5, rs-online:G6DN-1A-L, F.Cu at (483.8, 105.1)
- added PS1: RS PRO 5V 2A, Converter_ACDC:Converter_ACDC_Recom_RAC20-xxSK_THT, F.Cu at (413.8, 82.9)
- added Q1: 2N3904, Package_TO_SOT_SMD:SOT-23, F.Cu at (439.4, 109.9)
- added R1: 4.7KΩ, Resistor_SMD:R_0402_1005Metric, F.Cu at (433.8, 118.4)
- added R2: 1KΩ, Resistor_SMD:R_0402_1005Metric, F.Cu at (413.6, 117.7)
- added R3: 10KΩ, Resistor_SMD:R_0402_1005Metric, F.Cu at (410.7, 117.7)
- added R4: 330Ω, Resistor_SMD:R_0402_1005Metric, F.Cu at (416.5, 117.7)
- added REF**: MountingHole_4.3mm_M4_Pad_Via, MountingHole:MountingHole_4.3mm_M4_Pad_Via, F.Cu at (245.9, 159.2)
- added REF**: MountingHole_4.3mm_M4_Pad_Via, MountingHole:MountingHole_4.3mm_M4_Pad_Via, F.Cu at (44.5, 159.2)
- added REF**: MountingHole_4.3mm_M4_Pad_Via, MountingHole:MountingHole_4.3mm_M4_Pad_Via, F.Cu at (44.5, 21.2)
- added REF**: MountingHole_4.3mm_M4_Pad_Via, MountingHole:MountingHole_4.3mm_M4_Pad_Via, F.Cu at (37.2, 90.2)
- added REF**: MountingHole_4.3mm_M4_Pad_Via, MountingHole:MountingHole_4.3mm_M4_Pad_Via, F.Cu at (253.2, 90.2)
- added REF**: MountingHole_4.3mm_M4_Pad_Via, MountingHole:MountingHole_4.3mm_M4_Pad_Via, F.Cu at (245.9, 21.2)
- added T1: Transformer_1P_2S, rs-online:VCM36212, F.Cu at (436.9, 29.4)
- added U1: ESP32-POE, mylife-footprints:ESP32-POE, F.Cu at (514.2, 60.0)
Other:
- board size 88.9 x 66 mm -> 230 x 150 mm

Commit message: proto1 PCB
Parts:
- added REF**: MountingHole_4.3mm_M4, MountingHole:MountingHole_4.3mm_M4, F.Cu at (88.5, 120.0)
- added REF**: MountingHole_4.3mm_M4, MountingHole:MountingHole_4.3mm_M4, F.Cu at (88.5, 26.1)
- PS1: footprint Converter_ACDC:Converter_ACDC_Recom_RAC20-xxSK_THT -> mylife-footprints:RS PRO 5V 2A
- moved J3 421.4 mm to (127.0, 137.2)
- moved U1 377.3 mm to (137.2, 73.7)
- moved PS1 351.3 mm to (66.3, 134.6)
- moved J5 340.4 mm to (212.7, 124.5)
- moved D2 330.4 mm to (209.6, 102.9), turned to 90 degrees
- moved J1 310.7 mm to (159.1, 101.3)
- moved R1 302.5 mm to (132.1, 141.0), turned to -90 degrees
- moved J2 298.7 mm to (137.2, 137.2)
- moved T1 254.1 mm to (183.2, 43.2)
- moved K1 248.6 mm to (235.2, 100.3)
- moved Q1 238.5 mm to (201.1, 102.3)
- moved D1 238.5 mm to (205.7, 102.2), turned to -90 degrees
- moved J4 231.2 mm to (193.0, 124.5)
- moved R2 211.1 mm to (202.8, 105.4)
- moved R4 211.1 mm to (205.7, 105.4)
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Routing:
- net Net-(J4-Pad2): track 0.00 -> 304.1 mm
- net +5V: track 0.00 -> 204.9 mm, vias 0 -> 2
- net Net-(J4-Pad1): track 0.00 -> 189.7 mm
- net GND: track 0.00 -> 171.4 mm
- net Net-(J5-Pad1): track 0.00 -> 127.8 mm
- net Net-(J6-Pad2): track 0.00 -> 105.3 mm
- net Net-(J3-Pad4): track 0.00 -> 92.7 mm
- net Net-(J2-Pad3): track 0.00 -> 92.3 mm
- net +3V3: track 0.00 -> 85.8 mm, vias 0 -> 1
- net Net-(R2-Pad2): track 0.00 -> 76.6 mm, vias 0 -> 1
- net Net-(J6-Pad1): track 0.00 -> 68.2 mm
- net Net-(D1-Pad1): track 0.00 -> 21.9 mm
- net Net-(T1-Pad4): track 0.00 -> 20.0 mm
- net Net-(Q1-Pad2): track 0.00 -> 4.12 mm
- net Net-(D1-Pad2): track 0.00 -> 2.45 mm
Other:
- board text added: "220V IN"
- board text added: "220V OUT"
- board text added: "24V~ OUT"
- board text added: "SWITCH"
