File: garden-box/v1/relay.kicad_sch (KiCad schematic)
At the start: 7 parts

Commit message: add relay footprints
Parts:
- D1: renamed from D?; footprint (none) -> Diode_SMD:D_0805_2012Metric; LCSC (none) -> C2297
- D2: renamed from D?; footprint Diode_THT:D_DO-35_SOD27_P7.62mm_Horizontal -> Diode_SMD:D_SOD-123; LCSC (none) -> C81598
- Q1: renamed from Q?; footprint Package_TO_SOT_THT:TO-92_Inline -> Package_TO_SOT_SMD:SOT-23; LCSC (none) -> C18536
- R1: renamed from R?; footprint Resistor_SMD:R_0603_1608Metric -> Resistor_SMD:R_0402_1005Metric; LCSC (none) -> C11702
- R2: renamed from R?; footprint Resistor_SMD:R_0603_1608Metric -> Resistor_SMD:R_0402_1005Metric; LCSC (none) -> C25744
- R3: renamed from R?; value 1KΩ -> 330Ω; footprint Resistor_SMD:R_0603_1608Metric -> Resistor_SMD:R_0402_1005Metric; LCSC (none) -> C25104
- gave numbers to parts that had none: 1
Changed lines of the file:
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@@
   (symbol (lib_id "power:+5V") (at 115.57 43.18 0)
     (in_bom yes) (on_board yes) (fields_autoplaced)
-    (property "Reference" "#PWR?" (id 0) (at 115.57 46.99 0)
+    (property "Reference" "#PWR0104" (id 0) (at 115.57 46.99 0)
       (effects (font (size 1.27 1.27)) hide)
     )
@@
   (symbol (lib_id "Transistor_BJT:2N3904") (at 110.49 72.39 0)
     (in_bom yes) (on_board yes) (fields_autoplaced)
-    (property "Reference" "Q?" (id 0) (at 115.3414 71.4815 0)
+    (property "Reference" "Q1" (id 0) (at 115.3414 71.4815 0)
       (effects (font (size 1.27 1.27)) (justify left))
     )
@@
       (effects (font (size 1.27 1.27)) (justify left))
     )
-    (property "Footprint" "Package_TO_SOT_THT:TO-92_Inline" (id 2) (at 115.57 74.295 0)
+    (property "Footprint" "Package_TO_SOT_SMD:SOT-23" (id 2) (at 115.57 74.295 0)
       (effects (font (size 1.27 1.27) italic) (justify left) hide)
     )
-    (property "Datasheet" "https://www.onsemi.com/pub/Collateral/2N3903-D.PDF" (id 3) (at 110.49 72.39 0)
+    (property "Datasheet" "https://datasheet.lcsc.com/lcsc/1806151220_KEC-Semicon-2N3904S-RTK-PS_C18536.pdf" (id 3) (at 110.49 72.39 0)
       (effects (font (size 1.27 1.27)) (justify left) hide)
+    )
+    (property "LCSC" "C18536" (id 4) (at 110.49 72.39 0)
+      (effects (font (size 1.27 1.27)) hide)
     )
     (pin "1")
@@
   (symbol (lib_id "Relay:G6E") (at 149.86 58.42 0)
     (in_bom yes) (on_board yes) (fields_autoplaced)
-    (property "Reference" "K?" (id 0) (at 160.782 57.5115 0)
+    (property "Reference" "K1" (id 0) (at 160.782 57.5115 0)
       (effects (font (size 1.27 1.27)) (justify left))
     )
@@
   (symbol (lib_id "power:GND") (at 105.41 93.98 0)
     (in_bom yes) (on_board yes)
-    (property "Reference" "#PWR?" (id 0) (at 105.41 100.33 0)
+    (property "Reference" "#PWR0102" (id 0) (at 105.41 100.33 0)
       (effects (font (size 1.27 1.27)) hide)
     )
@@
   (symbol (lib_id "Device:R") (at 105.41 83.82 0)
     (in_bom yes) (on_board yes)
-    (property "Reference" "R?" (id 0) (at 100.33 85.09 90))
+    (property "Reference" "R2" (id 0) (at 100.33 85.09 90))
     (property "Value" "10KΩ" (id 1) (at 102.87 83.82 90))
-    (property "Footprint" "Resistor_SMD:R_0603_1608Metric" (id 2) (at 103.632 83.82 90)
+    (property "Footprint" "Resistor_SMD:R_0402_1005Metric" (id 2) (at 103.632 83.82 90)
       (effects (font (size 1.27 1.27)) hide)
     )
-    (property "Datasheet" "" (id 3) (at 105.41 83.82 0)
+    (property "Datasheet" "https://datasheet.lcsc.com/lcsc/2206010100_UNI-ROYAL-Uniroyal-Elec-0402WGF1002TCE_C25744.pdf" (id 3) (at 105.41 83.82 0)
       (effects (font (size 1.27 1.27)) hide)
     )
-    (property "LCSC" "" (id 4) (at 105.41 83.82 90)
+    (property "LCSC" "C25744" (id 4) (at 105.41 83.82 90)
       (effects (font (size 1.27 1.27)) hide)
     )
@@
   (symbol (lib_id "Device:R") (at 97.79 72.39 270)
     (in_bom yes) (on_board yes)
-    (property "Reference" "R?" (id 0) (at 96.52 67.31 90))
+    (property "Reference" "R1" (id 0) (at 96.52 67.31 90))
     (property "Value" "1KΩ" (id 1) (at 97.79 69.85 90))
-    (property "Footprint" "Resistor_SMD:R_0603_1608Metric" (id 2) (at 97.79 70.612 90)
+    (property "Footprint" "Resistor_SMD:R_0402_1005Metric" (id 2) (at 97.79 70.612 90)
       (effects (font (size 1.27 1.27)) hide)
     )
-    (property "Datasheet" "" (id 3) (at 97.79 72.39 0)
+    (property "Datasheet" "https://datasheet.lcsc.com/lcsc/2206010216_UNI-ROYAL-Uniroyal-Elec-0402WGF1001TCE_C11702.pdf" (id 3) (at 97.79 72.39 0)
       (effects (font (size 1.27 1.27)) hide)
     )
-    (property "LCSC" "" (id 4) (at 97.79 72.39 90)
+    (property "LCSC" "C11702" (id 4) (at 97.79 72.39 90)
       (effects (font (size 1.27 1.27)) hide)
     )
@@
   (symbol (lib_id "Diode:1N4148") (at 128.27 57.15 270)
     (in_bom yes) (on_board yes) (fields_autoplaced)
-    (property "Reference" "D?" (id 0) (at 130.302 56.2415 90)
+    (property "Reference" "D2" (id 0) (at 130.302 56.2415 90)
       (effects (font (size 1.27 1.27)) (justify left))
     )
@@
       (effects (font (size 1.27 1.27)) (justify left))
     )
-    (property "Footprint" "Diode_THT:D_DO-35_SOD27_P7.62mm_Horizontal" (id 2) (at 123.825 57.15 0)
+    (property "Footprint" "Diode_SMD:D_SOD-123" (id 2) (at 123.825 57.15 0)
       (effects (font (size 1.27 1.27)) hide)
     )
-    (property "Datasheet" "https://assets.nexperia.com/documents/data-sheet/1N4148_1N4448.pdf" (id 3) (at 128.27 57.15 0)
+    (property "Datasheet" "https://datasheet.lcsc.com/lcsc/1811061725_ST-Semtech-1N4148W_C81598.pdf" (id 3) (at 128.27 57.15 0)
+      (effects (font (size 1.27 1.27)) hide)
+    )
+    (property "LCSC" "C81598" (id 4) (at 128.27 57.15 90)
       (effects (font (size 1.27 1.27)) hide)
     )
@@
   (symbol (lib_id "power:+5V") (at 144.78 43.18 0)
     (in_bom yes) (on_board yes) (fields_autoplaced)
-    (property "Reference" "#PWR?" (id 0) (at 144.78 46.99 0)
+    (property "Reference" "#PWR0101" (id 0) (at 144.78 46.99 0)
       (effects (font (size 1.27 1.27)) hide)
     )
@@
   (symbol (lib_id "Device:R") (at 115.57 49.53 0)
     (in_bom yes) (on_board yes)
-    (property "Reference" "R?" (id 0) (at 110.49 50.8 90))
-    (property "Value" "1KΩ" (id 1) (at 113.03 49.53 90))
-    (property "Footprint" "Resistor_SMD:R_0603_1608Metric" (id 2) (at 113.792 49.53 90)
+    (property "Reference" "R3" (id 0) (at 110.49 50.8 90))
+    (property "Value" "330Ω" (id 1) (at 113.03 49.53 90))
+    (property "Footprint" "Resistor_SMD:R_0402_1005Metric" (id 2) (at 113.792 49.53 90)
       (effects (font (size 1.27 1.27)) hide)
     )
-    (property "Datasheet" "" (id 3) (at 115.57 49.53 0)
+    (property "Datasheet" "https://datasheet.lcsc.com/lcsc/2205311900_UNI-ROYAL-Uniroyal-Elec-0402WGF3300TCE_C25104.pdf" (id 3) (at 115.57 49.53 0)
       (effects (font (size 1.27 1.27)) hide)
     )
-    (property "LCSC" "" (id 4) (at 115.57 49.53 90)
+    (property "LCSC" "C25104" (id 4) (at 115.57 49.53 90)
       (effects (font (size 1.27 1.27)) hide)
     )
@@
   (symbol (lib_id "Device:LED") (at 115.57 58.42 270) (mirror x)
     (in_bom yes) (on_board yes) (fields_autoplaced)
-    (property "Reference" "D?" (id 0) (at 117.602 59.099 90)
+    (property "Reference" "D1" (id 0) (at 117.602 59.099 90)
       (effects (font (size 1.27 1.27)) (justify left))
     )
@@
       (effects (font (size 1.27 1.27)) (justify left))
     )
-    (property "Footprint" "" (id 2) (at 115.57 58.42 0)
+    (property "Footprint" "Diode_SMD:D_0805_2012Metric" (id 2) (at 115.57 58.42 0)
       (effects (font (size 1.27 1.27)) hide)
     )
-    (property "Datasheet" "~" (id 3) (at 115.57 58.42 0)
+    (property "Datasheet" "https://datasheet.lcsc.com/lcsc/1806151820_Hubei-KENTO-Elec-C2297_C2297.pdf" (id 3) (at 115.57 58.42 0)
+      (effects (font (size 1.27 1.27)) hide)
+    )
+    (property "LCSC" "C2297" (id 4) (at 115.57 58.42 90)
       (effects (font (size 1.27 1.27)) hide)
     )
@@
   (symbol (lib_id "power:GND") (at 113.03 93.98 0)
     (in_bom yes) (on_board yes)
-    (property "Reference" "#PWR?" (id 0) (at 113.03 100.33 0)
+    (property "Reference" "#PWR0103" (id 0) (at 113.03 100.33 0)
       (effects (font (size 1.27 1.27)) hide)
     )

Commit message: add extension header + annotations
Parts:
- renumbered D1 to D13, D2 to D14, K1 to K7, Q1 to Q7, R1 to R19, R2 to R20, R3 to R21
Changed lines of the file:
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@@
   (symbol (lib_id "power:+5V") (at 115.57 43.18 0)
     (in_bom yes) (on_board yes) (fields_autoplaced)
-    (property "Reference" "#PWR0104" (id 0) (at 115.57 46.99 0)
+    (property "Reference" "#PWR0128" (id 0) (at 115.57 46.99 0)
       (effects (font (size 1.27 1.27)) hide)
     )
@@
   (symbol (lib_id "Transistor_BJT:2N3904") (at 110.49 72.39 0)
     (in_bom yes) (on_board yes) (fields_autoplaced)
-    (property "Reference" "Q1" (id 0) (at 115.3414 71.4815 0)
+    (property "Reference" "Q7" (id 0) (at 115.3414 71.4815 0)
       (effects (font (size 1.27 1.27)) (justify left))
     )
@@
   (symbol (lib_id "Relay:G6E") (at 149.86 58.42 0)
     (in_bom yes) (on_board yes) (fields_autoplaced)
-    (property "Reference" "K1" (id 0) (at 160.782 57.5115 0)
+    (property "Reference" "K7" (id 0) (at 160.782 57.5115 0)
       (effects (font (size 1.27 1.27)) (justify left))
     )
@@
   (symbol (lib_id "power:GND") (at 105.41 93.98 0)
     (in_bom yes) (on_board yes)
-    (property "Reference" "#PWR0102" (id 0) (at 105.41 100.33 0)
+    (property "Reference" "#PWR0126" (id 0) (at 105.41 100.33 0)
       (effects (font (size 1.27 1.27)) hide)
     )
@@
   (symbol (lib_id "Device:R") (at 105.41 83.82 0)
     (in_bom yes) (on_board yes)
-    (property "Reference" "R2" (id 0) (at 100.33 85.09 90))
+    (property "Reference" "R20" (id 0) (at 100.33 85.09 90))
     (property "Value" "10KΩ" (id 1) (at 102.87 83.82 90))
     (property "Footprint" "Resistor_SMD:R_0402_1005Metric" (id 2) (at 103.632 83.82 90)
@@
   (symbol (lib_id "Device:R") (at 97.79 72.39 270)
     (in_bom yes) (on_board yes)
-    (property "Reference" "R1" (id 0) (at 96.52 67.31 90))
+    (property "Reference" "R19" (id 0) (at 96.52 67.31 90))
     (property "Value" "1KΩ" (id 1) (at 97.79 69.85 90))
     (property "Footprint" "Resistor_SMD:R_0402_1005Metric" (id 2) (at 97.79 70.612 90)
@@
   (symbol (lib_id "Diode:1N4148") (at 128.27 57.15 270)
     (in_bom yes) (on_board yes) (fields_autoplaced)
-    (property "Reference" "D2" (id 0) (at 130.302 56.2415 90)
+    (property "Reference" "D14" (id 0) (at 130.302 56.2415 90)
       (effects (font (size 1.27 1.27)) (justify left))
     )
@@
   (symbol (lib_id "power:+5V") (at 144.78 43.18 0)
     (in_bom yes) (on_board yes) (fields_autoplaced)
-    (property "Reference" "#PWR0101" (id 0) (at 144.78 46.99 0)
+    (property "Reference" "#PWR0125" (id 0) (at 144.78 46.99 0)
       (effects (font (size 1.27 1.27)) hide)
     )
@@
   (symbol (lib_id "Device:R") (at 115.57 49.53 0)
     (in_bom yes) (on_board yes)
-    (property "Reference" "R3" (id 0) (at 110.49 50.8 90))
+    (property "Reference" "R21" (id 0) (at 110.49 50.8 90))
     (property "Value" "330Ω" (id 1) (at 113.03 49.53 90))
     (property "Footprint" "Resistor_SMD:R_0402_1005Metric" (id 2) (at 113.792 49.53 90)
@@
   (symbol (lib_id "Device:LED") (at 115.57 58.42 270) (mirror x)
     (in_bom yes) (on_board yes) (fields_autoplaced)
-    (property "Reference" "D1" (id 0) (at 117.602 59.099 90)
+    (property "Reference" "D13" (id 0) (at 117.602 59.099 90)
       (effects (font (size 1.27 1.27)) (justify left))
     )
@@
   (symbol (lib_id "power:GND") (at 113.03 93.98 0)
     (in_bom yes) (on_board yes)
-    (property "Reference" "#PWR0103" (id 0) (at 113.03 100.33 0)
+    (property "Reference" "#PWR0127" (id 0) (at 113.03 100.33 0)
       (effects (font (size 1.27 1.27)) hide)
     )

Commit message: cleanup + footprints
Parts:
- renumbered D13 to D1, D14 to D2, K7 to K1, Q7 to Q1, R19 to R1, R20 to R2, R21 to R3
Changed lines of the file:
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@@
   (symbol (lib_id "power:+5V") (at 115.57 43.18 0)
     (in_bom yes) (on_board yes) (fields_autoplaced)
-    (property "Reference" "#PWR0128" (id 0) (at 115.57 46.99 0)
+    (property "Reference" "#PWR0104" (id 0) (at 115.57 46.99 0)
       (effects (font (size 1.27 1.27)) hide)
     )
@@
   (symbol (lib_id "Transistor_BJT:2N3904") (at 110.49 72.39 0)
     (in_bom yes) (on_board yes) (fields_autoplaced)
-    (property "Reference" "Q7" (id 0) (at 115.3414 71.4815 0)
+    (property "Reference" "Q1" (id 0) (at 115.3414 71.4815 0)
       (effects (font (size 1.27 1.27)) (justify left))
     )
@@
   (symbol (lib_id "Relay:G6E") (at 149.86 58.42 0)
     (in_bom yes) (on_board yes) (fields_autoplaced)
-    (property "Reference" "K7" (id 0) (at 160.782 57.5115 0)
+    (property "Reference" "K1" (id 0) (at 160.782 57.5115 0)
       (effects (font (size 1.27 1.27)) (justify left))
     )
@@
   (symbol (lib_id "power:GND") (at 105.41 93.98 0)
     (in_bom yes) (on_board yes)
-    (property "Reference" "#PWR0126" (id 0) (at 105.41 100.33 0)
+    (property "Reference" "#PWR0102" (id 0) (at 105.41 100.33 0)
       (effects (font (size 1.27 1.27)) hide)
     )
@@
   (symbol (lib_id "Device:R") (at 105.41 83.82 0)
     (in_bom yes) (on_board yes)
-    (property "Reference" "R20" (id 0) (at 100.33 85.09 90))
+    (property "Reference" "R2" (id 0) (at 100.33 85.09 90))
     (property "Value" "10KΩ" (id 1) (at 102.87 83.82 90))
     (property "Footprint" "Resistor_SMD:R_0402_1005Metric" (id 2) (at 103.632 83.82 90)
@@
   (symbol (lib_id "Device:R") (at 97.79 72.39 270)
     (in_bom yes) (on_board yes)
-    (property "Reference" "R19" (id 0) (at 96.52 67.31 90))
+    (property "Reference" "R1" (id 0) (at 96.52 67.31 90))
     (property "Value" "1KΩ" (id 1) (at 97.79 69.85 90))
     (property "Footprint" "Resistor_SMD:R_0402_1005Metric" (id 2) (at 97.79 70.612 90)
@@
   (symbol (lib_id "Diode:1N4148") (at 128.27 57.15 270)
     (in_bom yes) (on_board yes) (fields_autoplaced)
-    (property "Reference" "D14" (id 0) (at 130.302 56.2415 90)
+    (property "Reference" "D2" (id 0) (at 130.302 56.2415 90)
       (effects (font (size 1.27 1.27)) (justify left))
     )
@@
   (symbol (lib_id "power:+5V") (at 144.78 43.18 0)
     (in_bom yes) (on_board yes) (fields_autoplaced)
-    (property "Reference" "#PWR0125" (id 0) (at 144.78 46.99 0)
+    (property "Reference" "#PWR0101" (id 0) (at 144.78 46.99 0)
       (effects (font (size 1.27 1.27)) hide)
     )
@@
   (symbol (lib_id "Device:R") (at 115.57 49.53 0)
     (in_bom yes) (on_board yes)
-    (property "Reference" "R21" (id 0) (at 110.49 50.8 90))
+    (property "Reference" "R3" (id 0) (at 110.49 50.8 90))
     (property "Value" "330Ω" (id 1) (at 113.03 49.53 90))
     (property "Footprint" "Resistor_SMD:R_0402_1005Metric" (id 2) (at 113.792 49.53 90)
@@
   (symbol (lib_id "Device:LED") (at 115.57 58.42 270) (mirror x)
     (in_bom yes) (on_board yes) (fields_autoplaced)
-    (property "Reference" "D13" (id 0) (at 117.602 59.099 90)
+    (property "Reference" "D1" (id 0) (at 117.602 59.099 90)
       (effects (font (size 1.27 1.27)) (justify left))
     )
@@
   (symbol (lib_id "power:GND") (at 113.03 93.98 0)
     (in_bom yes) (on_board yes)
-    (property "Reference" "#PWR0127" (id 0) (at 113.03 100.33 0)
+    (property "Reference" "#PWR0103" (id 0) (at 113.03 100.33 0)
       (effects (font (size 1.27 1.27)) hide)
     )
