File: garden-box/v1/garden-box.kicad_sch (KiCad schematic)
At the start: 19 parts

Commit message: v1 schematic
Parts:
- added U2: ESP32-POE-ISO, symbol mylife-symbols:ESP32-POE-ISO
- gave numbers to parts that had none: 19
Connections:
- net +5V: now also J1.2 (Pin_2), J2.2 (Pin_2), J3.3 (Pin_3), U2.1 (+5V); no longer J1.1 (Pin_1), J2.1 (Pin_1), J3.1 (Pin_1)
- net GND: now also J1.1 (Pin_1), J2.1 (Pin_1), J3.1 (Pin_1), U2.3 (GND); no longer J1.2 (Pin_2), J2.2 (Pin_2)
- net Relay1/input: now also U2.5 (GPIO0)
- net Relay2/input: now also U2.6 (GPIO1)
- net Relay3/input: now also U2.7 (GPIO2)
- net Relay4/input: now also U2.8 (GPIO3)
- net Relay5/input: now also U2.9 (GPIO4)
- net Relay6/input: now also U2.10 (GPIO5)
- net at J3.4 (Pin_4): now also U2.19 (GPIO36)
- net at J2.3 (Pin_3): now also U2.18 (GPIO35)
Other:
- note added: "GND"
- note added: "VCC"
- note removed: "DO"
- moved on the sheet: J8, T1

Commit message: add extension header + annotations
Parts:
- added J12, J13: Conn_01x06_Male, symbol Connector:Conn_01x06_Male
- J8: footprint (none) -> TerminalBlock:TerminalBlock_bornier-2_P5.08mm
Connections:
- net +5V: now also J12.3 (Pin_3), J12.4 (Pin_4)
- net GND: now also J12.1 (Pin_1), J12.2 (Pin_2)
- net at U2.11 (GPIO13): now also J13.1 (Pin_1)
- net at U2.12 (GPIO14): now also J13.2 (Pin_2)
- net at U2.13 (GPIO15): now also J13.3 (Pin_3)
- net at U2.14 (GPIO16): now also J13.4 (Pin_4)
- net at U2.15 (GPIO32): now also J13.5 (Pin_5)
- net at U2.16 (GPIO33): now also J13.6 (Pin_6)
- net +3V3: now reaches U2.2 (+3.3V_(out))
- net +3V3: now also J12.5 (Pin_5), J12.6 (Pin_6)

Commit message: cleanup + footprints
Parts:
- J1: footprint (none) -> Connector_PinHeader_2.54mm:PinHeader_1x02_P2.54mm_Vertical
- J10, J11, J4, J5, J6, J7, J9: footprint (none) -> TerminalBlock:TerminalBlock_bornier-2_P5.08mm
- J12, J13: footprint (none) -> Connector_PinHeader_2.54mm:PinHeader_1x06_P2.54mm_Vertical
- J2: footprint (none) -> Connector_PinHeader_2.54mm:PinHeader_1x03_P2.54mm_Vertical
- J3: footprint (none) -> Connector_PinHeader_2.54mm:PinHeader_1x04_P2.54mm_Vertical
Connections:
- net GND: now also J13.6 (Pin_6)
- net Relay Transfo/input: now also U2.16 (GPIO33)
Other:
- note removed: "+"
- note removed: "-"

Commit message: init new v1
Parts:
- removed J1: Conn_01x02_Male, Connector_PinHeader_2.54mm:PinHeader_1x02_P2.54mm_Vertical, symbol Connector:Conn_01x02_Male
- removed J10, J11, J7, J8, J9: Screw_Terminal_01x02, TerminalBlock:TerminalBlock_bornier-2_P5.08mm, symbol Connector:Screw_Terminal_01x02
- removed J12, J13: Conn_01x06_Male, Connector_PinHeader_2.54mm:PinHeader_1x06_P2.54mm_Vertical, symbol Connector:Conn_01x06_Male
- removed SW1, SW2, SW3, SW4, SW5, SW6: SW_Push_DPDT, symbol Switch:SW_Push_DPDT
- removed U1: LM7805_TO220, Package_TO_SOT_THT:TO-220-3_Vertical, symbol Regulator_Linear:LM7805_TO220
- added D1: LED, Diode_SMD:D_0805_2012Metric, symbol Device:LED
- added D2: 1N4148, Diode_SMD:D_SOD-123, symbol Diode:1N4148
- added J1: USB_A, rs-online:875200010BLF, symbol Connector:USB_A
- added K1: G6DN-1A-L_DC5, rs-online:G6DN-1A-L, symbol mylife-symbols:G6DN-1A-L_DC5
- added PS1: RS PRO 5V 2A, mylife-footprints:RS PRO 5V 2A, symbol Converter_ACDC:IRM-10-5
- added Q1: 2N3904, jlcpcb:SOT-23-3_L2.9-W1.3-P1.90-LS2.4-TR, symbol Transistor_BJT:2N3904
- added R1: 4.7KΩ, Resistor_SMD:R_0402_1005Metric, symbol Device:R
- added R2: 1KΩ, Resistor_SMD:R_0402_1005Metric, symbol Device:R
- added R3: 10KΩ, Resistor_SMD:R_0402_1005Metric, symbol Device:R
- added R4: 330Ω, Resistor_SMD:R_0402_1005Metric, symbol Device:R
- T1: footprint (none) -> rs-online:VCM36212
- U1: renamed from U2; value ESP32-POE-ISO -> ESP32-POE; footprint (none) -> mylife-footprints:ESP32-POE
Connections:
- net Relay Transfo/output2 is gone; now on an unnamed net: T1.1 (AA)
- net Relay1/output2 is gone; now on an unnamed net: J5.2 (Pin_2)
- net Relay2/output2 is gone; now on an unnamed net: J6.2 (Pin_2)
- net +3V3: now also J2.2 (Pin_2), R1.1
- net +5V: now also D2.1 (K), J1.1 (VBUS), K1.1, PS1.4 (+Vo), R4.1; no longer J2.2 (Pin_2)
- net GND: now also J1.4 (GND), J1.5 (Shield), PS1.3 (-Vo), Q1.1 (E), R3.2; no longer J4.2 (Pin_2)
- net at J6.1 (Pin_1): now also T1.3 (SA)
- net at T1.2 (AB): now also J4.2 (Pin_2), PS1.1 (AC/N)
- net at J5.1 (Pin_1): now also K1.8
- net at U1.11 (GPIO13): now also J2.3 (Pin_3), R1.2
- net at J4.1 (Pin_1): now also K1.5, PS1.2 (AC/L)
- net at U1.18 (GPIO35): no longer J2.3 (Pin_3)
- net Relay Transfo/input: no longer names the net of U1.16 (GPIO33)
- net Relay Transfo/input: now also R2.2
- net Relay1/input: no longer names the net of U1.5 (GPIO0)
- net Relay2/input: no longer names the net of U1.6 (GPIO1)
- net Relay3/input: no longer names the net of U1.7 (GPIO2)
- net Relay4/input: no longer names the net of U1.8 (GPIO3)
- net Relay5/input: no longer names the net of U1.9 (GPIO4)
- net Relay6/input: no longer names the net of U1.10 (GPIO5)
- new net: Q1.2 (B), R2.1, R3.1
- new net: D1.1 (K), D2.2 (A), K1.2, Q1.3 (C)
- new net: D1.2 (A), R4.2
Other:
- removed sheet Relay Transfo
- removed sheet Relay1
- removed sheet Relay2
- removed sheet Relay3
- removed sheet Relay4
- removed sheet Relay5
- removed sheet Relay6
- note added: "220v in"
- note added: "220v out"
- note added: "24V ~ out"
- note added: "SEN0308"
- note removed: "12v"
- note removed: "220v"
- note removed: "Moisture sensor"
- moved on the sheet: J2, J3

Commit message: update led resistor
Parts:
- R4: value 330Ω -> 1KΩ; LCSC C25104 -> C11702
Changed lines of the file:
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@@
     (in_bom yes) (on_board yes)
     (property "Reference" "R4" (id 0) (at 147.32 48.26 90))
-    (property "Value" "330Ω" (id 1) (at 149.86 46.99 90))
+    (property "Value" "1KΩ" (id 1) (at 149.86 46.99 90))
     (property "Footprint" "Resistor_SMD:R_0402_1005Metric" (id 2) (at 150.622 46.99 90)
       (effects (font (size 1.27 1.27)) hide)
     )
-    (property "Datasheet" "https://datasheet.lcsc.com/lcsc/2205311900_UNI-ROYAL-Uniroyal-Elec-0402WGF3300TCE_C25104.pdf" (id 3) (at 152.4 46.99 0)
-      (effects (font (size 1.27 1.27)) hide)
-    )
-    (property "LCSC" "C25104" (id 4) (at 152.4 46.99 90)
+    (property "Datasheet" "https://datasheet.lcsc.com/lcsc/2206010216_UNI-ROYAL-Uniroyal-Elec-0402WGF1001TCE_C11702.pdf" (id 3) (at 152.4 46.99 0)
+      (effects (font (size 1.27 1.27)) hide)
+    )
+    (property "LCSC" "C11702" (id 4) (at 152.4 46.99 90)
       (effects (font (size 1.27 1.27)) hide)
     )
@@
     )
     (path "/deba7d89-f9a2-4354-82a6-0d3192f950f8"
-      (reference "R4") (unit 1) (value "330Ω") (footprint "Resistor_SMD:R_0402_1005Metric")
+      (reference "R4") (unit 1) (value "1KΩ") (footprint "Resistor_SMD:R_0402_1005Metric")
     )
     (path "/be49853a-e63a-418f-add4-0398acbca9cd"

Commit message: update footprint on PCB
Parts:
- T1: footprint rs-online:VCM36212 -> mylife-footprints:VCM36212
Changed lines of the file:
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@@
     (property "Reference" "T1" (id 0) (at 246.38 85.0603 0))
     (property "Value" "Transformer_1P_2S" (id 1) (at 246.38 87.8354 0))
-    (property "Footprint" "rs-online:VCM36212" (id 2) (at 246.38 99.06 0)
+    (property "Footprint" "mylife-footprints:VCM36212" (id 2) (at 246.38 99.06 0)
       (effects (font (size 1.27 1.27)) hide)
     )
@@
     )
     (path "/be49853a-e63a-418f-add4-0398acbca9cd"
-      (reference "T1") (unit 1) (value "Transformer_1P_2S") (footprint "rs-online:VCM36212")
+      (reference "T1") (unit 1) (value "Transformer_1P_2S") (footprint "mylife-footprints:VCM36212")
     )
     (path "/a51d3ce6-8227-462c-b55f-ac7604ee63f5"

Commit message: wip v1 layout
Parts:
- removed D1: LED, Diode_SMD:D_0805_2012Metric, symbol Device:LED
- removed D2: 1N4148, Diode_SMD:D_SOD-123, symbol Diode:1N4148
- removed J5, J6: Screw_Terminal_01x02, TerminalBlock:TerminalBlock_bornier-2_P5.08mm, symbol Connector:Screw_Terminal_01x02
- removed K1: G6DN-1A-L_DC5, rs-online:G6DN-1A-L, symbol mylife-symbols:G6DN-1A-L_DC5
- removed Q1: 2N3904, jlcpcb:SOT-23-3_L2.9-W1.3-P1.90-LS2.4-TR, symbol Transistor_BJT:2N3904
- removed R2, R4: 1KΩ, Resistor_SMD:R_0402_1005Metric, symbol Device:R
- removed R3: 10KΩ, Resistor_SMD:R_0402_1005Metric, symbol Device:R
- added J? (x6): Conn_01x03_Male, Connector_PinHeader_2.54mm:PinHeader_1x03_P2.54mm_Vertical, symbol Connector:Conn_01x03_Male
- added J?: Screw_Terminal_01x06, TerminalBlock:TerminalBlock_bornier-2_P5.08mm, symbol Connector:Screw_Terminal_01x06
- added J? (x2): Screw_Terminal_01x04, TerminalBlock:TerminalBlock_bornier-2_P5.08mm, symbol Connector:Screw_Terminal_01x04
Connections:
- net at J4.2 (Pin_2), PS1.1 (AC/N), T1.2 (AB): now also J?.1 (Pin_1), J?.2 (Pin_2), J?.3 (Pin_3), J?.4 (Pin_4)
- net relay transfo/Output 1: now reaches J4.1 (Pin_1), PS1.2 (AC/L)
- net relay transfo/Output 1: now also J?.1 (Pin_1), J?.1 (Pin_1), J?.1 (Pin_1), J?.1 (Pin_1), J?.1 (Pin_1), J?.1 (Pin_1)
- net relay transfo/Logic input: now reaches U1.16 (GPIO33)
- net relay transfo/Output 2: now reaches T1.1 (AA)
- net at T1.3 (SA): now also J?.3 (Pin_3), J?.3 (Pin_3), J?.3 (Pin_3), J?.3 (Pin_3), J?.3 (Pin_3), J?.3 (Pin_3)
- net at T1.6 (SD): now also J?.1 (Pin_1), J?.2 (Pin_2), J?.3 (Pin_3), J?.4 (Pin_4)
- new net relay 1/Output 1: J?.2 (Pin_2)
- new net relay 1/Output 2: J?.1 (Pin_1)
- new net relay 2/Output 1: J?.2 (Pin_2)
- new net relay 2/Output 2: J?.2 (Pin_2)
- new net relay 3/Output 1: J?.2 (Pin_2)
- new net relay 3/Output 2: J?.3 (Pin_3)
- new net relay 4/Output 1: J?.2 (Pin_2)
- new net relay 4/Output 2: J?.4 (Pin_4)
- new net relay 5/Output 1: J?.2 (Pin_2)
- new net relay 5/Output 2: J?.5 (Pin_5)
- new net relay 6/Output 1: J?.2 (Pin_2)
- new net relay 6/Output 2: J?.6 (Pin_6)
Other:
- added sheet relay 1 (relay.kicad_sch)
- added sheet relay 2 (relay.kicad_sch)
- added sheet relay 3 (relay.kicad_sch)
- added sheet relay 4 (relay.kicad_sch)
- added sheet relay 5 (relay.kicad_sch)
- added sheet relay 6 (relay.kicad_sch)
- added sheet relay transfo (relay.kicad_sch)
- note added: "1-2 = 220v 2-3 = 24v"
- note added: "220v out (common)"
- note added: "24v out (common)"
- note added: "Relays out"
- note added: "~"
- note removed: "220v out"
- note removed: "24V ~ out"
- moved on the sheet: J1, J4, PS1, T1, U1
