File: garden-box/v1/garden-box.kicad_pcb (KiCad board)
At the start: 2 copper layers, 230 x 150 mm, 23 parts, among them J1 USB_A, J2 Conn_01x03_Male, J3 Conn_01x04_Male, J4 Screw_Terminal_01x02, J5 Screw_Terminal_01x02, J6 Screw_Terminal_01x02, K1 G6DN-1A-L_DC5, Q1 2N3904, T1 Transformer_1P_2S, U1 ESP32-POE

Commit message: fix term block footprint + init PCB design
Parts:
- added D10: 1N4148, Diode_SMD:D_SOD-123, F.Cu at (355.8, 151.5)
- added D11: LED, Diode_SMD:D_0805_2012Metric, F.Cu at (401.1, 151.4)
- added D12: 1N4148, Diode_SMD:D_SOD-123, F.Cu at (396.0, 151.5)
- added D13: LED, Diode_SMD:D_0805_2012Metric, F.Cu at (401.1, 137.9)
- added D14: 1N4148, Diode_SMD:D_SOD-123, F.Cu at (396.0, 138.1)
- added D3: LED, Diode_SMD:D_0805_2012Metric, F.Cu at (422.3, 115.6)
- added D4: 1N4148, Diode_SMD:D_SOD-123, F.Cu at (417.2, 115.7)
- added D5: LED, Diode_SMD:D_0805_2012Metric, F.Cu at (361.0, 137.9)
- added D6: 1N4148, Diode_SMD:D_SOD-123, F.Cu at (355.8, 138.1)
- added D7: LED, Diode_SMD:D_0805_2012Metric, F.Cu at (422.3, 102.1)
- added D8: 1N4148, Diode_SMD:D_SOD-123, F.Cu at (417.2, 102.3)
- added D9: LED, Diode_SMD:D_0805_2012Metric, F.Cu at (361.0, 151.4)
- added J10: Screw_Terminal_01x02, TerminalBlock:TerminalBlock_bornier-2_P5.08mm, F.Cu at (377.9, 107.9)
- added J11: Screw_Terminal_01x04, TerminalBlock:TerminalBlock_bornier-4_P5.08mm, F.Cu at (388.2, 98.9)
- added J12: Screw_Terminal_01x04, TerminalBlock:TerminalBlock_bornier-4_P5.08mm, F.Cu at (356.2, 107.9)
- added J13: Screw_Terminal_01x06, TerminalBlock:TerminalBlock_bornier-6_P5.08mm, F.Cu at (356.2, 98.9)
- added J7: Conn_01x03_Male, Connector_PinHeader_2.54mm:PinHeader_1x03_P2.54mm_Vertical, F.Cu at (355.3, 114.8)
- added J8: Conn_01x03_Male, Connector_PinHeader_2.54mm:PinHeader_1x03_P2.54mm_Vertical, F.Cu at (359.9, 114.8)
- added J9: Conn_01x03_Male, Connector_PinHeader_2.54mm:PinHeader_1x03_P2.54mm_Vertical, F.Cu at (364.6, 114.8)
- added K2: G6DN-1A-L_DC5, rs-online:G6DN-1A-L, F.Cu at (434.5, 109.7)
- added K3: G6DN-1A-L_DC5, rs-online:G6DN-1A-L, F.Cu at (373.2, 132.0)
- added K4: G6DN-1A-L_DC5, rs-online:G6DN-1A-L, F.Cu at (434.5, 96.2)
- added K5: G6DN-1A-L_DC5, rs-online:G6DN-1A-L, F.Cu at (373.2, 145.4)
- added K6: G6DN-1A-L_DC5, rs-online:G6DN-1A-L, F.Cu at (413.3, 145.4)
- added K7: G6DN-1A-L_DC5, rs-online:G6DN-1A-L, F.Cu at (413.3, 132.0)
- added Q2: 2N3904, jlcpcb:SOT-23-3_L2.9-W1.3-P1.90-LS2.4-TR, F.Cu at (438.8, 109.9)
- added Q3: 2N3904, jlcpcb:SOT-23-3_L2.9-W1.3-P1.90-LS2.4-TR, F.Cu at (377.5, 132.2)
- added Q4: 2N3904, jlcpcb:SOT-23-3_L2.9-W1.3-P1.90-LS2.4-TR, F.Cu at (438.8, 96.4)
- added Q5: 2N3904, jlcpcb:SOT-23-3_L2.9-W1.3-P1.90-LS2.4-TR, F.Cu at (377.5, 145.6)
- added Q6: 2N3904, jlcpcb:SOT-23-3_L2.9-W1.3-P1.90-LS2.4-TR, F.Cu at (417.6, 145.6)
- added Q7: 2N3904, jlcpcb:SOT-23-3_L2.9-W1.3-P1.90-LS2.4-TR, F.Cu at (417.6, 132.2)
- added R10: 1KΩ, Resistor_SMD:R_0402_1005Metric, F.Cu at (381.3, 131.1)
- added R11: 1KΩ, Resistor_SMD:R_0402_1005Metric, F.Cu at (437.9, 99.5)
- added R12: 10KΩ, Resistor_SMD:R_0402_1005Metric, F.Cu at (425.9, 101.6)
- added R13: 1KΩ, Resistor_SMD:R_0402_1005Metric, F.Cu at (442.6, 95.3)
- added R14: 1KΩ, Resistor_SMD:R_0402_1005Metric, F.Cu at (376.6, 148.7)
- added R15: 10KΩ, Resistor_SMD:R_0402_1005Metric, F.Cu at (364.6, 150.8)
- added R16: 1KΩ, Resistor_SMD:R_0402_1005Metric, F.Cu at (381.3, 144.6)
- added R17: 1KΩ, Resistor_SMD:R_0402_1005Metric, F.Cu at (416.7, 148.7)
- added R18: 10KΩ, Resistor_SMD:R_0402_1005Metric, F.Cu at (404.8, 150.8)
- added R19: 1KΩ, Resistor_SMD:R_0402_1005Metric, F.Cu at (421.4, 144.6)
- added R20: 1KΩ, Resistor_SMD:R_0402_1005Metric, F.Cu at (416.7, 135.3)
- added R21: 10KΩ, Resistor_SMD:R_0402_1005Metric, F.Cu at (404.8, 137.4)
- added R22: 1KΩ, Resistor_SMD:R_0402_1005Metric, F.Cu at (421.4, 131.1)
- added R5: 1KΩ, Resistor_SMD:R_0402_1005Metric, F.Cu at (437.9, 112.9)
- added R6: 10KΩ, Resistor_SMD:R_0402_1005Metric, F.Cu at (425.9, 115.0)
- added R7: 1KΩ, Resistor_SMD:R_0402_1005Metric, F.Cu at (442.6, 108.8)
- added R8: 1KΩ, Resistor_SMD:R_0402_1005Metric, F.Cu at (376.6, 135.3)
- added R9: 10KΩ, Resistor_SMD:R_0402_1005Metric, F.Cu at (364.6, 137.4)
- J4, J5, J6: value Screw_Terminal_01x02 -> Conn_01x03_Male; footprint TerminalBlock:TerminalBlock_bornier-2_P5.08mm -> Connector_PinHeader_2.54mm:PinHeader_1x03_P2.54mm_Vertical
- renumbered J2 to J1, J3 to J2, J1 to J3
Connections:
- net Net-(R2-Pad2) renamed /relay transfo/Logic input
- J4 pad 1: Net-(J4-Pad1) -> /relay transfo/Output 1
- J4 pad 2: Net-(J4-Pad2) -> /relay 1/Output 1
- J5 pad 1: Net-(J5-Pad1) -> /relay transfo/Output 1
- J5 pad 2: Net-(J4-Pad2) -> /relay 2/Output 1
- J6 pad 1: Net-(J6-Pad1) -> /relay transfo/Output 1
- J6 pad 2: Net-(J6-Pad2) -> /relay 3/Output 1
- K1 pad 5: Net-(J4-Pad1) -> /relay transfo/Output 2
- K1 pad 8: Net-(J5-Pad1) -> /relay transfo/Output 1
- PS1 pad 1: Net-(J4-Pad2) -> Net-(J10-Pad2)
- PS1 pad 2: Net-(J4-Pad1) -> /relay transfo/Output 1
- T1 pad 1: Net-(J5-Pad1) -> /relay transfo/Output 2
- T1 pad 2: Net-(J4-Pad2) -> Net-(J10-Pad2)
- T1 pad 3: Net-(J6-Pad1) -> Net-(J4-Pad3)
- T1 pad 6: Net-(J6-Pad2) -> Net-(J12-Pad1)
- U1 pad 10: unconnected-(U1-Pad10) -> /R6
- U1 pad 5: unconnected-(U1-Pad5) -> /R1
- U1 pad 6: unconnected-(U1-Pad6) -> /R2
- U1 pad 7: unconnected-(U1-Pad7) -> /R3
- U1 pad 8: unconnected-(U1-Pad8) -> /R4
- U1 pad 9: unconnected-(U1-Pad9) -> /R5
Routing:
- net /relay transfo/Output 1: track 0.00 -> 412.7 mm
- net Net-(J4-Pad3): track 0.00 -> 347.0 mm
- net Net-(J4-Pad2): track 347.0 -> 0.00 mm
- net Net-(J4-Pad1): track 196.1 -> 0.00 mm
- net Net-(J6-Pad1): track 116.8 -> 0.00 mm
- net Net-(J5-Pad1): track 99.8 -> 0.00 mm
- net Net-(J6-Pad2): track 84.3 -> 0.00 mm
- net Net-(J12-Pad1): track 0.00 -> 84.3 mm

Commit message: wip pcb
Parts:
- moved Q4 349.3 mm to (98.8, 176.5), turned to 90 degrees
- moved R13 349.2 mm to (103.2, 177.8)
- moved R11 345.5 mm to (100.3, 173.3)
- moved R12 336.2 mm to (97.5, 173.3), turned to 180 degrees
- moved R22 336.0 mm to (97.5, 220.3)
- moved Q7 336.0 mm to (93.1, 219.1), turned to 90 degrees
- moved R20 332.0 mm to (94.6, 215.9)
- moved Q6 330.6 mm to (93.1, 208.9), turned to 90 degrees
- moved R19 330.5 mm to (97.5, 210.2)
- moved D7 327.2 mm to (103.2, 174.6), turned to -90 degrees
- moved R17 327.1 mm to (94.6, 205.7)
- moved R21 322.6 mm to (91.8, 215.9), turned to 180 degrees
- moved D8 318.6 mm to (107.1, 175.2), turned to 90 degrees
- moved R18 317.7 mm to (91.8, 205.7), turned to 180 degrees
- moved K4 311.3 mm to (132.7, 172.7)
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Routing:
- net /relay transfo/Output 1: track 412.7 -> 20.6 mm
- net Net-(J4-Pad3): track 347.0 -> 68.6 mm
- net /relay transfo/Logic input: track 198.1 -> 0.00 mm
- net Net-(J10-Pad2): track 0.00 -> 89.4 mm
- net GND: track 282.4 -> 204.9 mm
- net Net-(J12-Pad1): track 84.3 -> 34.7 mm
- net /relay 6/Output 2: track 0.00 -> 37.9 mm, vias 0 -> 1
- net /relay 5/Output 2: track 0.00 -> 37.9 mm, vias 0 -> 1
- net /relay 2/Output 2: track 0.00 -> 37.9 mm, vias 0 -> 1
- net /relay 4/Output 2: track 0.00 -> 37.9 mm, vias 0 -> 1
- net /relay 3/Output 2: track 0.00 -> 37.9 mm, vias 0 -> 1
- net /relay 1/Output 2: track 0.00 -> 37.9 mm, vias 0 -> 1
- net Net-(D13-Pad1): track 0.00 -> 27.8 mm
- net Net-(D5-Pad1): track 0.00 -> 25.3 mm
- net Net-(D3-Pad1): track 0.00 -> 25.3 mm
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
Commit message: wip placement
Parts:
- moved D2 133.3 mm to (285.8, 92.7)
- moved Q1 133.3 mm to (277.5, 94.0)
- moved R3 133.3 mm to (276.2, 90.8)
- moved D1 133.3 mm to (281.9, 92.1)
- moved K1 133.3 mm to (311.4, 90.2)
- moved R2 133.3 mm to (279.0, 90.8)
- moved R4 133.3 mm to (281.9, 95.2)
- moved R10 48.5 mm to (103.2, 142.2)
- moved D5 48.5 mm to (103.2, 139.1)
- moved R9 48.5 mm to (97.5, 137.8)
- moved D6 48.5 mm to (107.1, 139.7)
- moved J5 48.5 mm to (139.1, 138.4)
- moved K3 48.5 mm to (132.7, 137.2)
- moved Q3 48.5 mm to (98.8, 141.0)
- moved R8 48.5 mm to (100.3, 137.8)
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
Commit message: restore switch pads
Parts:
- added REF**: MountingHole_4.3mm_M4, MountingHole:MountingHole_4.3mm_M4, F.Cu at (143.6, 84.7)
- added REF**: MountingHole_4.3mm_M4, MountingHole:MountingHole_4.3mm_M4, F.Cu at (49.6, 84.7)
- moved K1 142.7 mm to (168.9, 82.6)
- moved R3 125.8 mm to (151.9, 71.8)
- moved D1 125.8 mm to (157.6, 73.0)
- moved D2 125.8 mm to (161.4, 73.7)
- moved Q1 125.8 mm to (153.2, 74.9)
- moved R2 125.8 mm to (154.7, 71.8)
- moved R4 125.8 mm to (157.6, 76.2)
- moved D9 34.6 mm to (132.1, 135.3)
- moved R22 34.6 mm to (132.1, 153.7)
- moved R7 34.6 mm to (132.1, 115.6)
- moved D3 34.6 mm to (132.1, 112.4)
- moved D5 34.6 mm to (132.1, 120.0)
- moved D7 34.6 mm to (132.1, 127.6)
- moved D12 34.6 mm to (132.1, 142.9)
- moved D14 34.6 mm to (132.1, 150.5)
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Routing:
- net Net-(D1-Pad1): track 25.3 -> 18.1 mm
- net +5V: track 256.1 -> 259.8 mm
