File: epanel-energy-monitor/prototype-2/prototype-2.kicad_sch (KiCad schematic)
At the start: 31 parts, among them J1 Screw_Terminal_01x02, J10 Conn_01x02_Male, J2 Conn_01x03_Male, J3 Conn_01x01_Male, J4 Conn_01x01_Male, J5 Conn_01x01, J6 Conn_02x05, J7 Conn_02x05, J8 AudioJack4, J9 Screw_Terminal_01x02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

Commit message: wip PCB
Parts:
- J2: footprint (none) -> Connector_PinHeader_2.54mm:PinHeader_1x03_P2.54mm_Vertical
- J6, J7: symbol Connector_Generic:Conn_02x05_Counter_Clockwise -> Connector_Generic:Conn_02x05_Odd_Even
Connections:
- net at R12.2: now also J7.4 (Pin_4); no longer J7.9 (Pin_9)
- net at R7.2: now also J6.4 (Pin_4); no longer J6.9 (Pin_9)
- net at R9.2: now also J6.8 (Pin_8); no longer J6.7 (Pin_7)
- net at R15.2: now also J7.10 (Pin_10); no longer J7.6 (Pin_6)
- net at C1.1, J10.2 (Pin_2), J6.1 (Pin_1)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: now also J6.7 (Pin_7), J6.9 (Pin_9); no longer J6.2 (Pin_2), J6.4 (Pin_4)
- net at R14.2: now also J7.8 (Pin_8); no longer J7.7 (Pin_7)
- net at J6.10 (Pin_10): now also R10.2; no longer R6.2
- net at J6.6 (Pin_6): now also R8.2; no longer R10.2
- net at J7.1 (Pin_1), J7.3 (Pin_3), J7.5 (Pin_5)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: now also J7.7 (Pin_7), J7.9 (Pin_9); no longer J7.2 (Pin_2), J7.4 (Pin_4)
- net at R11.2: now also J7.2 (Pin_2); no longer J7.10 (Pin_10)
- net at R13.2: now also J7.6 (Pin_6); no longer J7.8 (Pin_8)
- new net: J6.2 (Pin_2), R6.2
Changed lines of the file:
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@@
     (pin "2")
   )
-  (symbol (lib_id "Connector_Generic:Conn_02x05_Counter_Clockwise") (at 220.98 154.94 0) (unit 1)
+  (symbol (lib_id "Connector_Generic:Conn_02x05_Odd_Even") (at 220.98 154.94 0) (unit 1)
     (in_bom yes) (on_board yes) (fields_autoplaced)
     (property "Reference" "J6" (id 0) (at 222.25 143.51 0))
@@
     (property "Reference" "J2" (id 0) (at 135.89 113.03 90))
     (property "Value" "Conn_01x03_Male" (id 1) (at 135.89 115.57 90))
-    (property "Footprint" "" (id 2) (at 135.89 118.11 0)
+    (property "Footprint" "Connector_PinHeader_2.54mm:PinHeader_1x03_P2.54mm_Vertical" (id 2) (at 135.89 118.11 0)
       (effects (font (size 1.27 1.27)) hide)
     )
@@
     (pin "1")
   )
-  (symbol (lib_id "Connector_Generic:Conn_02x05_Counter_Clockwise") (at 256.54 60.96 0) (unit 1)
+  (symbol (lib_id "Connector_Generic:Conn_02x05_Odd_Even") (at 256.54 60.96 0) (unit 1)
     (in_bom yes) (on_board yes) (fields_autoplaced)
     (property "Reference" "J7" (id 0) (at 257.81 49.53 0))
@@
     )
     (path "/66ddad46-33c9-4abd-9c24-c7e1b28436ab"
-      (reference "J2") (unit 1) (value "Conn_01x03_Male") (footprint "")
+      (reference "J2") (unit 1) (value "Conn_01x03_Male") (footprint "Connector_PinHeader_2.54mm:PinHeader_1x03_P2.54mm_Vertical")
     )
     (path "/c7adb180-cac4-4e08-bba9-6fc53c45552e"

Commit message: wip pcb
Parts:
- U1: value ESP32-POE-ISO -> ESP32-POE; footprint (none) -> mylife-footprints:ESP32-POE
Changed lines of the file:
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@@
     (in_bom yes) (on_board yes) (fields_autoplaced)
     (property "Reference" "U1" (id 0) (at 63.5 19.05 0))
-    (property "Value" "ESP32-POE-ISO" (id 1) (at 63.5 21.59 0))
-    (property "Footprint" "" (id 2) (at 63.5 20.32 0)
+    (property "Value" "ESP32-POE" (id 1) (at 63.5 21.59 0))
+    (property "Footprint" "mylife-footprints:ESP32-POE" (id 2) (at 63.5 20.32 0)
       (effects (font (size 1.27 1.27)) hide)
     )
@@
     )
     (path "/5d7b5a26-027a-4672-ad98-b9419fb008a1"
-      (reference "U1") (unit 1) (value "ESP32-POE-ISO") (footprint "")
+      (reference "U1") (unit 1) (value "ESP32-POE") (footprint "mylife-footprints:ESP32-POE")
     )
     (path "/245abd9d-3d35-4956-a9f0-7102dcf3248e"
