File: epanel-energy-monitor/prototype-2/prototype-2.kicad_pcb (KiCad board)
At the start: 2 copper layers, 87 x 68 mm, 23 parts, among them J1 Conn_01x06_Male, J2 AudioJack4, J3 AudioJack4, J4 Screw_Terminal_01x02, J5 Screw_Terminal_01x02, J6 Conn_01x02_Male, J7 Conn_01x02_Male, Q1 BS170, U1 LTV-814

Commit message: wip pcb
Parts:
- removed C2: 10uF/6V, Resistor_SMD:R_0603_1608Metric
- removed the J1 at (111.8, 74.3)
- removed J2: AudioJack4, Connector_Audio:Jack_3.5mm_PJ320D_Horizontal
- removed U1: LTV-814, Package_DIP:SMDIP-4_W7.62mm
- added J10: Conn_01x02_Male, Connector_PinHeader_2.54mm:PinHeader_1x02_P2.54mm_Vertical, F.Cu at (131.2, 92.1)
- added J4: Conn_01x01_Male, Connector_PinHeader_2.54mm:PinHeader_1x01_P2.54mm_Vertical, F.Cu at (135.8, 95.8)
- added J5: Conn_01x01, Connector_PinHeader_2.54mm:PinHeader_1x01_P2.54mm_Vertical, F.Cu at (103.0, 119.6)
- added J8: AudioJack4, Connector_Audio:Jack_3.5mm_PJ320D_Horizontal, F.Cu at (186.6, 85.1)
- added R12: 1.2KΩ, Resistor_SMD:R_0603_1608Metric, F.Cu at (116.4, 118.5)
- added R13: 2KΩ, Resistor_SMD:R_0603_1608Metric, F.Cu at (132.1, 104.4)
- added R14: 3.3KΩ, Resistor_SMD:R_0603_1608Metric, F.Cu at (135.2, 101.9)
- added R15: 4.7KΩ, Resistor_SMD:R_0603_1608Metric, F.Cu at (135.2, 99.4)
- added U2: MCP3208, Package_SO:SOIC-16_3.9x9.9mm_P1.27mm, F.Cu at (125.9, 110.3)
- added U3: LTV-814, Package_DIP:SMDIP-4_W7.62mm, F.Cu at (150.3, 82.0)
- J3: value AudioJack4 -> Conn_01x01_Male; footprint Connector_Audio:Jack_3.5mm_PJ320D_Horizontal -> Connector_PinHeader_2.54mm:PinHeader_1x01_P2.54mm_Vertical
- J6, J7: value Conn_01x02_Male -> Conn_02x05; footprint Connector_PinHeader_2.54mm:PinHeader_1x02_P2.54mm_Vertical -> Connector_PinHeader_2.54mm:PinHeader_2x05_P2.54mm_Vertical
- PS1: value HLK-PM01 -> Alim RS PRO 5V 1A; footprint Converter_ACDC:Converter_ACDC_HiLink_HLK-PMxx -> Converter_ACDC:Converter_ACDC_MeanWell_IRM-03-xx_THT
- Q1: value BS170 -> CJ2302
- R1, R2: value 1KΩ -> 470KΩ
- R10: value 120Ω/0.5W -> 33Ω/0.5W
- R11: value 4.7KΩ -> 1KΩ
- R4: value 470KΩ -> 1KΩ
- R5: value 470KΩ -> 10KΩ
- R6: value 470KΩ -> 220Ω/0.5W; footprint Resistor_SMD:R_0603_1608Metric -> Resistor_SMD:R_0805_2012Metric
- R7: value 470KΩ -> 150Ω/0.5W; footprint Resistor_SMD:R_0603_1608Metric -> Resistor_SMD:R_0805_2012Metric
- R8: value 10KΩ -> 120Ω/0.5W; footprint Resistor_SMD:R_0603_1608Metric -> Resistor_SMD:R_0805_2012Metric
- R9: value 22Ω/0.5W -> 75Ω/0.5W
- moved Q1 82.8 mm to (98.2, 119.5), turned to 0 degrees
- moved J3 75.6 mm to (107.7, 119.6), turned to 0 degrees
- moved R5 68.6 mm to (112.0, 121.4)
- moved R3 68.1 mm to (116.0, 121.4)
- moved J6 65.3 mm to (124.0, 92.1)
- moved R6 58.5 mm to (112.2, 118.7), turned to 0 degrees
- moved J7 53.1 mm to (139.8, 81.0)
- moved R10 50.5 mm to (123.8, 117.5), turned to 0 degrees
- moved R8 47.8 mm to (131.0, 101.4)
- moved R11 45.8 mm to (140.1, 97.2), turned to 0 degrees
- moved R7 41.8 mm to (131.0, 98.4)
- moved R4 32.2 mm to (140.1, 94.7), turned to 0 degrees
- moved PS1 30.5 mm to (121.9, 52.7)
- moved R2 29.6 mm to (151.1, 86.6)
- moved R9 27.3 mm to (146.9, 86.8), turned to 0 degrees
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- renumbered J4 to J1, J5 to J9
Connections:
- J6 pad 1: Net-(J2-PadS) -> Net-(C1-Pad1)
- J7 pad 1: Net-(J3-PadS) -> Net-(J7-Pad1)
- J7 pad 2: Net-(C2-Pad1) -> Net-(J7-Pad1)
- PS1 pad 3: GND -> NEUT
- Q1 pad 1: Net-(J1-Pad4) -> Net-(J3-Pad1)
- Q1 pad 2: Net-(Q1-Pad2) -> Net-(J5-Pad1)
- R1 pad 1: Net-(J1-Pad5) -> Net-(C1-Pad1)
- R1 pad 2: Net-(J2-PadS) -> +3V3
- R10 pad 1: Net-(J3-PadS) -> Net-(J10-Pad1)
- R10 pad 2: Net-(C2-Pad1) -> Net-(J6-Pad6)
- R11 pad 2: Net-(R11-Pad2) -> Net-(J7-Pad10)
- R2 pad 1: Net-(J1-Pad6) -> GND
- R2 pad 2: Net-(J3-PadS) -> Net-(C1-Pad1)
- R3 pad 1: Net-(J1-Pad4) -> Net-(J3-Pad1)
- R4 pad 1: Net-(C1-Pad1) -> Net-(J2-Pad2)
- R4 pad 2: +3V3 -> Net-(J10-Pad1)
- R5 pad 2: Net-(C1-Pad1) -> Net-(J5-Pad1)
- R6 pad 1: Net-(C2-Pad1) -> Net-(J10-Pad1)
- R6 pad 2: +3V3 -> Net-(J6-Pad10)
- R7 pad 1: GND -> Net-(J10-Pad1)
- R7 pad 2: Net-(C2-Pad1) -> Net-(J6-Pad9)
- R8 pad 1: GND -> Net-(J10-Pad1)
- R8 pad 2: Net-(Q1-Pad2) -> Net-(J6-Pad8)
- R9 pad 1: Net-(J2-PadS) -> Net-(J10-Pad1)
- R9 pad 2: Net-(C1-Pad1) -> Net-(J6-Pad7)
Routing:
- net GND: track 112.6 -> 0.00 mm, vias 3 -> 0
- net +3V3: track 102.2 -> 0.00 mm, vias 4 -> 0
- net Net-(J1-Pad6): track 74.4 -> 0.00 mm
- net Net-(J1-Pad4): track 65.2 -> 0.00 mm
- net Net-(J1-Pad5): track 60.5 -> 0.00 mm
- net NEUT: track 43.2 -> 0.00 mm
- net LINE: track 38.2 -> 0.00 mm
- net +5V: track 34.5 -> 0.00 mm
- net Net-(J2-PadS): track 30.1 -> 0.00 mm
- net Net-(C2-Pad1): track 30.1 -> 0.00 mm
- net Net-(C1-Pad1): track 26.5 -> 0.00 mm
- net Net-(J3-PadS): track 23.3 -> 0.00 mm
- net Net-(J9-Pad1): track 11.2 -> 0.00 mm
- net Net-(J9-Pad2): track 9.04 -> 0.00 mm
- net Net-(R11-Pad2): track 8.75 -> 0.00 mm
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Other:
- board text removed: "3V3"
- board text removed: "5V"
- board text removed: "CT0"
- board text removed: "CT1"
- board text removed: "GND"
- board text removed: "Tele"

Commit message: wip PCB
Parts:
- added J2: Conn_01x03_Male, Connector_PinHeader_2.54mm:PinHeader_1x03_P2.54mm_Vertical, F.Cu at (126.4, 83.8)
- moved R3 61.3 mm to (155.1, 74.3)
- moved R5 61.3 mm to (151.1, 74.3)
- moved J5 58.4 mm to (147.1, 81.3)
- moved J3 58.4 mm to (151.8, 81.3)
- moved Q1 58.4 mm to (142.3, 81.2)
- moved R12 56.9 mm to (138.4, 66.0)
- moved J6 52.8 mm to (175.9, 101.6)
- moved R13 36.4 mm to (138.4, 68.6)
- moved R11 33.8 mm to (138.4, 63.5)
- moved R14 31.0 mm to (138.6, 71.1)
- moved R6 29.2 mm to (141.0, 113.7)
- moved R15 25.9 mm to (138.4, 73.7)
- moved J10 24.5 mm to (155.6, 90.8)
- moved C1 22.9 mm to (143.3, 66.9)
- moved R9 22.9 mm to (143.5, 64.1)
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Connections:
- J6 pad 2: Net-(C1-Pad1) -> Net-(J6-Pad2)
- J6 pad 4: Net-(C1-Pad1) -> Net-(J6-Pad4)
- J6 pad 7: Net-(J6-Pad7) -> Net-(C1-Pad1)
- J6 pad 9: Net-(J6-Pad9) -> Net-(C1-Pad1)
- J7 pad 2: Net-(J7-Pad1) -> Net-(J7-Pad2)
- J7 pad 4: Net-(J7-Pad1) -> Net-(J7-Pad4)
- J7 pad 7: Net-(J7-Pad7) -> Net-(J7-Pad1)
- J7 pad 9: Net-(J7-Pad9) -> Net-(J7-Pad1)
- R10 pad 2: Net-(J6-Pad6) -> Net-(J6-Pad10)
- R11 pad 2: Net-(J7-Pad10) -> Net-(J7-Pad2)
- R12 pad 2: Net-(J7-Pad9) -> Net-(J7-Pad4)
- R13 pad 2: Net-(J7-Pad8) -> Net-(J7-Pad6)
- R14 pad 2: Net-(J7-Pad7) -> Net-(J7-Pad8)
- R15 pad 2: Net-(J7-Pad6) -> Net-(J7-Pad10)
- R6 pad 2: Net-(J6-Pad10) -> Net-(J6-Pad2)
- R7 pad 2: Net-(J6-Pad9) -> Net-(J6-Pad4)
- R8 pad 2: Net-(J6-Pad8) -> Net-(J6-Pad6)
- R9 pad 2: Net-(J6-Pad7) -> Net-(J6-Pad8)

Commit message: wip pcb
Parts:
- moved R9 54.8 mm to (182.2, 102.9), turned to 90 degrees
- moved R6 50.1 mm to (189.9, 102.9), turned to 90 degrees
- moved R7 45.8 mm to (187.3, 102.9), turned to 90 degrees
- moved R8 42.6 mm to (184.8, 102.9), turned to 90 degrees
- moved C1 42.3 mm to (174.6, 95.2), turned to 180 degrees
- moved J2 41.3 mm to (167.6, 83.8)
- moved R10 40.8 mm to (179.7, 102.9), turned to 90 degrees
- moved R2 39.9 mm to (174.6, 93.3)
- moved U2 39.0 mm to (158.1, 88.3), turned to 90 degrees
- moved R11 38.6 mm to (177.0, 66.0), turned to 180 degrees
- moved R12 38.6 mm to (177.0, 68.6), turned to 180 degrees
- moved R13 38.6 mm to (177.0, 71.1), turned to 180 degrees
- moved R15 38.6 mm to (177.0, 76.2), turned to 180 degrees
- moved R14 38.4 mm to (177.0, 73.7), turned to 180 degrees
- moved J4 35.8 mm to (153.7, 64.8)
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Routing:
- net GND: track 0.00 -> 98.3 mm
- net NEUT: track 0.00 -> 51.2 mm
- net +3V3: track 0.00 -> 50.8 mm, vias 0 -> 4
- net LINE: track 0.00 -> 44.7 mm
- net Net-(J10-Pad1): track 0.00 -> 44.3 mm, vias 0 -> 1
- net Net-(J9-Pad2): track 0.00 -> 37.1 mm, vias 0 -> 1
- net Net-(C1-Pad1): track 0.00 -> 32.5 mm
- net Net-(J9-Pad1): track 0.00 -> 20.3 mm
- net Net-(J2-Pad3): track 0.00 -> 19.1 mm, vias 0 -> 1
- net Net-(J7-Pad1): track 0.00 -> 15.8 mm
- net Net-(J5-Pad1): track 0.00 -> 13.9 mm
- net Net-(J3-Pad1): track 0.00 -> 8.46 mm
- net Net-(J7-Pad8): track 0.00 -> 7.88 mm
- net Net-(J7-Pad6): track 0.00 -> 7.88 mm
- net Net-(J7-Pad4): track 0.00 -> 7.88 mm
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Other:
- board text added: "1.2KΩ"
- board text added: "10A"
- board text added: "16A"
- board text added: "1KΩ"
- board text added: "20A"
- board text added: "2KΩ"
- board text added: "3.3KΩ"
- board text added: "32A"
- board text added: "4.7KΩ"
- board text added: "60A"

Commit message: wip pcb
Parts:
- added U1: ESP32-POE, mylife-footprints:ESP32-POE, F.Cu at (149.2, 102.2)
- moved J1 76.3 mm to (111.6, 55.9)
- moved PS1 31.8 mm to (120.0, 78.6), turned to 90 degrees
- moved J2 13.0 mm to (170.2, 71.1)
- moved C1 12.7 mm to (174.6, 82.5)
- moved J10 12.7 mm to (176.5, 71.1)
- moved J6 12.7 mm to (189.9, 82.5)
- moved J8 12.7 mm to (186.6, 72.4)
- moved R1 12.7 mm to (174.6, 78.7)
- moved R10 12.7 mm to (179.7, 90.2)
- moved R2 12.7 mm to (174.6, 80.6)
- moved R6 12.7 mm to (189.9, 90.2)
- moved R7 12.7 mm to (187.3, 90.2)
- moved R8 12.7 mm to (184.8, 90.2)
- moved R9 12.7 mm to (182.2, 90.2)
- moved J3 12.3 mm to (157.5, 68.6)
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Routing:
- net GND: track 98.3 -> 65.4 mm
- net NEUT: track 51.2 -> 24.8 mm
- net LINE: track 44.7 -> 26.2 mm
- net Net-(J9-Pad2): track 37.1 -> 22.5 mm
- net +3V3: track 50.8 -> 36.6 mm, vias 4 -> 3
- net Net-(J2-Pad3): track 19.1 -> 14.0 mm, vias 1 -> 0
- net Net-(J9-Pad1): track 20.3 -> 18.4 mm
- net Net-(J2-Pad2): track 4.79 -> 3.37 mm
- net Net-(J5-Pad1): track 13.9 -> 14.7 mm
- net Net-(J3-Pad1): track 8.46 -> 7.78 mm
- net Net-(J7-Pad1): track 15.8 -> 15.1 mm

Commit message: proto2 finish
Routing:
- net +5V: track 0.00 -> 62.1 mm
- net Net-(U1-Pad11): track 0.00 -> 59.1 mm
- net Net-(U1-Pad12): track 0.00 -> 58.5 mm
- net Net-(U1-Pad13): track 0.00 -> 58.0 mm
- net Net-(J2-Pad1): track 0.00 -> 54.7 mm
- net Net-(U1-Pad16): track 0.00 -> 42.8 mm, vias 0 -> 1
- net Net-(J3-Pad1): track 7.78 -> 37.9 mm
- net +3V3: track 36.6 -> 62.9 mm, vias 3 -> 4
- net Net-(J9-Pad2): track 22.5 -> 34.6 mm
- net GND: track 65.4 -> 75.9 mm
