File: epanel-energy-monitor/prototype-3/prototype-3.kicad_sch (KiCad schematic)
At the start: 31 parts, among them J1 Screw_Terminal_01x02, J10 Conn_01x02_Male, J2 Conn_01x03_Male, J3 Conn_01x01_Male, J4 Conn_01x01_Male, J5 Conn_01x01, J6 Conn_02x05, J7 Conn_02x05, J8 AudioJack4, J9 Screw_Terminal_01x02, Q1 CJ2302, U1 ESP32-POE, U2 MCP3208, U3 LTV-814

Commit message: update TIC
Parts:
- removed J7: Conn_02x05, Connector_PinHeader_2.54mm:PinHeader_2x05_P2.54mm_Vertical, symbol Connector_Generic:Conn_02x05_Odd_Even
- removed R12: 1.2KΩ, Resistor_SMD:R_0603_1608Metric, symbol Device:R
- removed R13: 2KΩ, Resistor_SMD:R_0603_1608Metric, symbol Device:R
- removed R14: 3.3KΩ, Resistor_SMD:R_0603_1608Metric, symbol Device:R
- removed R15: 4.7KΩ, Resistor_SMD:R_0603_1608Metric, symbol Device:R
- added D?: LED, Diode_SMD:D_0805_2012Metric, symbol Device:LED
- added R?: 1KΩ, Resistor_SMD:R_0603_1608Metric, symbol Device:R
- Q1: value CJ2302 -> BSS138; LCSC C2910175 -> C2938375
- R11: value 1KΩ -> 220Ω; LCSC C21190 -> C22962
- R5: value 10KΩ -> 3.3KΩ; LCSC C25804 -> C22978
Connections:
- net +3V3: now also D?.2 (A)
- net at J3.1 (Pin_1), Q1.1 (D), R3.1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: now also R?.1
- net at U3.1: now also R11.2
- new net: D?.1 (K), R?.2
Other:
- moved on the sheet: C1, J10, J3, J6, J8, R1, R10, R11, R2, R4, R6, R7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

Commit message: wip sensors
Parts:
- removed J10: Conn_01x02_Male, Connector_PinHeader_2.54mm:PinHeader_1x02_P2.54mm_Vertical, symbol Connector:Conn_01x02_Male
- removed J8: AudioJack4, Connector_Audio:Jack_3.5mm_PJ320D_Horizontal, symbol Connector:AudioJack4
- added C?: 1uF/6V, Resistor_SMD:R_0603_1608Metric, symbol Device:C
- added C? (x3): 10uF/6V, Resistor_SMD:R_0603_1608Metric, symbol Device:C
- added J? (x3): Conn_01x03_Male, Connector_PinHeader_2.54mm:PinHeader_1x03_P2.54mm_Vertical, symbol Connector:Conn_01x03_Male
- added J? (x4): Conn_02x03, Connector_PinHeader_2.54mm:PinHeader_2x03_P2.54mm_Vertical, symbol Connector_Generic:Conn_02x03_Odd_Even
- added J? (x2): Conn_02x05, Connector_PinHeader_2.54mm:PinHeader_2x05_P2.54mm_Vertical, symbol Connector_Generic:Conn_02x05_Odd_Even
- added J? (x3): Screw_Terminal_01x02, TerminalBlock:TerminalBlock_bornier-2_P5.08mm, symbol Connector:Screw_Terminal_01x02
- added R? (x2): 120Ω/0.5W, Resistor_SMD:R_0805_2012Metric, symbol Device:R
- added R? (x2): ??KΩ, Resistor_SMD:R_0603_1608Metric, symbol Device:R
- added R? (x6): 470KΩ, Resistor_SMD:R_0603_1608Metric, symbol Device:R
- added R? (x2): 33Ω/0.5W, Resistor_SMD:R_0805_2012Metric, symbol Device:R
- added R? (x2): 100Ω/0.5W, Resistor_SMD:R_0805_2012Metric, symbol Device:R
- added R? (x2): 62Ω/0.5W, Resistor_SMD:R_0805_2012Metric, symbol Device:R
- added R? (x2): 200Ω/0.5W, Resistor_SMD:R_0805_2012Metric, symbol Device:R
- added R? (x3): 1KΩ, Resistor_SMD:R_0603_1608Metric, symbol Device:R
- added R? (x2): 12KΩ, Resistor_SMD:R_0603_1608Metric, symbol Device:R
- added T?: Transformer_1P_1S, symbol Device:Transformer_1P_1S
- added U?: LMV321, Package_TO_SOT_SMD:SOT-23-5, symbol Amplifier_Operational:LMV321
- added U?: ADS1115, Package_SO:TSSOP-10_3x3mm_P0.5mm, symbol Analog_ADC:ADS1115IDGS
- R6: value 220Ω/0.5W -> 200Ω/0.5W; LCSC C966130 -> C560506
- R7: value 150Ω/0.5W -> 120Ω/0.5W; LCSC C560494 -> C543533
- R8: value 120Ω/0.5W -> 100Ω/0.5W; LCSC C966144 -> C417003
- R9: value 75Ω/0.5W -> 62Ω/0.5W; LCSC C441944 -> C560547
Connections:
- net +3V3: now also R?.2, R?.2, R?.2, R?.2, U?.5 (V+), U?.8 (VDD)
- net GND: now also C?.2, C?.2, C?.2, C?.2, R?.1, R?.1, R?.1, R?.1, U?.1 (ADDR), U?.2 (V-), U?.3 (GND)
- net LINE: now also T?.1 (AA)
- net NEUT: now also T?.2 (AB)
- net at J2.3 (Pin_3): now also J?.3 (Pin_3), J?.3 (Pin_3), J?.3 (Pin_3), U?.3 (-), U?.4; no longer U2.1 (CH0)
- net at U2.10 (~{CS}/SHDN): now also U1.14 (GPIO16); no longer U1.16 (GPIO33)
- net at U2.2 (CH1): now also J?.5 (Pin_5)
- net at U2.3 (CH2): now also J?.5 (Pin_5)
- net at U2.4 (CH3): now also J?.5 (Pin_5)
- net at R10.1, R4.2, R6.1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: now also J?.1 (Pin_1)
- net at J6.1 (Pin_1), J6.3 (Pin_3), J6.5 (Pin_5)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: now also J2.2 (Pin_2), J?.2 (Pin_2); no longer C1.1, R1.1, R2.2
- net at J2.1 (Pin_1): now also C1.1, R1.1, R2.2; no longer U1.15 (GPIO32)
- net at U1.18 (GPIO35): now also U?.9 (SDA)
- net at U1.19 (GPIO36): now also U?.10 (SCL)
- net at U1.7 (GPIO2): now also J3.1 (Pin_1), Q1.1 (D), R3.1, R?.1
- net at R4.1: now also J?.2 (Pin_2), J?.4 (Pin_4), J?.6 (Pin_6); no longer J2.2 (Pin_2)
- new net: J?.1 (Pin_1), R?.1, R?.1, R?.1, R?.1, R?.1, R?.2 (x2)
- new net: J?.4 (Pin_4), R?.2 (x2)
- new net: R?.1, R?.2, R?.2
- new net: R?.2, T?.4 (SB)
- new net: C?.1, J?.1 (Pin_1), R?.1, R?.2 (x3)
- new net: J?.2 (Pin_2), R?.1, T?.3 (SA)
- new net: J?.10 (Pin_10), R?.2 (x2)
- new net: J?.6 (Pin_6), R?.2 (x2)
- new net: J?.5 (Pin_5), U2.1 (CH0)
- new net: C?.1, R?.1, R?.2, U?.1 (+)
- new net: J?.8 (Pin_8), R?.2 (x2)
- new net: J?.2 (Pin_2), J?.4 (Pin_4), J?.6 (Pin_6), R?.1 (x3)
- new net: J?.3 (Pin_3), U?.7 (AIN3)
- new net: J?.2 (Pin_2), R?.2 (x2)
- new net: J?.1 (Pin_1), U1.15 (GPIO32)
- new net: J?.1 (Pin_1), U1.16 (GPIO33)
- new net: J?.3 (Pin_3), U?.4 (AIN0)
- new net: J?.1 (Pin_1), J?.2 (Pin_2), J?.2 (Pin_2), J?.3 (Pin_3), J?.5 (Pin_5), J?.7 (Pin_7), J?.9 (Pin_9) (x2)
- new net: J?.3 (Pin_3), U?.6 (AIN2)
- new net: J?.3 (Pin_3), U?.5 (AIN1)
- now unconnected: U1.8 (GPIO3)
Other:
- note added: "1-2 = ESP 3-4 = ADS 5-6 = MCP"
- note added: "1-2 = pont diviseur 2-3 = ampli op"
- note added: "CT0"
- note added: "CT1"
- note added: "CT2"
- note added: "Used by IO : - GPIO 3 (interrupt) - GPIO 4 (SDA) - GPIO 5 (SCL)"
- note added: "Voltage sensor"
- note removed: "CT - YHDC SCT-013-00"
- moved on the sheet: C1, D?, J1, J2, J3, J4, J5, J6, J9, PS1, Q1, R1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

Commit message: schematic
Parts:
- R?: value ??KΩ -> 100KΩ; LCSC C23178 -> C25803
- R?: value ??KΩ -> 12KΩ; LCSC C23178 -> C22790
- T?: value Transformer_1P_1S -> 230V - 6V; footprint (none) -> mylife-footprints:RS PRO 6V 0.35VA
Changed lines of the file:
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@@
       (effects (font (size 1.27 1.27)) (justify right))
     )
-    (property "Value" "??KΩ" (id 1) (at 316.738 37.4266 0)
+    (property "Value" "100KΩ" (id 1) (at 316.738 37.4266 0)
       (effects (font (size 1.27 1.27)) (justify right))
     )
@@
       (effects (font (size 1.27 1.27)) hide)
     )
-    (property "Datasheet" "https://datasheet.lcsc.com/lcsc/2206010116_UNI-ROYAL-Uniroyal-Elec-0603WAF4703T5E_C23178.pdf" (id 3) (at 314.96 35.56 0)
-      (effects (font (size 1.27 1.27)) hide)
-    )
-    (property "LCSC" "C23178" (id 4) (at 314.96 35.56 0)
+    (property "Datasheet" "https://datasheet.lcsc.com/lcsc/2206010045_UNI-ROYAL-Uniroyal-Elec-0603WAF1003T5E_C25803.pdf" (id 3) (at 314.96 35.56 0)
+      (effects (font (size 1.27 1.27)) hide)
+    )
+    (property "LCSC" "C25803" (id 4) (at 314.96 35.56 0)
       (effects (font (size 1.27 1.27)) hide)
     )
@@
     (in_bom yes) (on_board yes) (fields_autoplaced)
     (property "Reference" "T?" (id 0) (at 336.5373 33.02 0))
-    (property "Value" "Transformer_1P_1S" (id 1) (at 336.5373 35.56 0))
-    (property "Footprint" "" (id 2) (at 336.55 43.18 0)
-      (effects (font (size 1.27 1.27)) hide)
-    )
-    (property "Datasheet" "~" (id 3) (at 336.55 43.18 0)
+    (property "Value" "230V - 6V" (id 1) (at 336.5373 35.56 0))
+    (property "Footprint" "mylife-footprints:RS PRO 6V 0.35VA" (id 2) (at 336.55 43.18 0)
+      (effects (font (size 1.27 1.27)) hide)
+    )
+    (property "Datasheet" "https://docs.rs-online.com/5c0d/0900766b80f46e25.pdf" (id 3) (at 336.55 43.18 0)
       (effects (font (size 1.27 1.27)) hide)
     )
@@
       (effects (font (size 1.27 1.27)) (justify right))
     )
-    (property "Value" "??KΩ" (id 1) (at 316.738 52.6666 0)
+    (property "Value" "12KΩ" (id 1) (at 316.738 52.6666 0)
       (effects (font (size 1.27 1.27)) (justify right))
     )
@@
       (effects (font (size 1.27 1.27)) hide)
     )
-    (property "Datasheet" "https://datasheet.lcsc.com/lcsc/2206010116_UNI-ROYAL-Uniroyal-Elec-0603WAF4703T5E_C23178.pdf" (id 3) (at 314.96 50.8 0)
-      (effects (font (size 1.27 1.27)) hide)
-    )
-    (property "LCSC" "C23178" (id 4) (at 314.96 50.8 0)
+    (property "Datasheet" "https://datasheet.lcsc.com/lcsc/2206010130_UNI-ROYAL-Uniroyal-Elec-0603WAF1202T5E_C22790.pdf" (id 3) (at 314.96 50.8 0)
+      (effects (font (size 1.27 1.27)) hide)
+    )
+    (property "LCSC" "C22790" (id 4) (at 314.96 50.8 0)
       (effects (font (size 1.27 1.27)) hide)
     )
@@
     )
     (path "/080d6e4e-e338-42c4-a74a-4741aeddcb7e"
-      (reference "R?") (unit 1) (value "??KΩ") (footprint "Resistor_SMD:R_0603_1608Metric")
+      (reference "R?") (unit 1) (value "100KΩ") (footprint "Resistor_SMD:R_0603_1608Metric")
     )
     (path "/0c303439-92b4-41f4-a88c-f0d7c5a245fd"
@@
     )
     (path "/55df1ae4-d3b3-491d-9a0f-2b43e4fc59ed"
-      (reference "R?") (unit 1) (value "??KΩ") (footprint "Resistor_SMD:R_0603_1608Metric")
+      (reference "R?") (unit 1) (value "12KΩ") (footprint "Resistor_SMD:R_0603_1608Metric")
     )
     (path "/5e887bc3-0bbc-460d-9e7a-b6cd791564c9"
@@
     )
     (path "/35c8ca8a-5716-4892-b883-7f70694cf361"
-      (reference "T?") (unit 1) (value "Transformer_1P_1S") (footprint "")
+      (reference "T?") (unit 1) (value "230V - 6V") (footprint "mylife-footprints:RS PRO 6V 0.35VA")
     )
     (path "/5d7b5a26-027a-4672-ad98-b9419fb008a1"

Commit message: annotate
Parts:
- gave numbers to parts that had none: 44
- renumbered C1 to C3, J3 to J1, J2 to J11, J6 to J14, J4 to J2, J1 to J3, J5 to J4, J9 to J5, R2 to R10, R4 to R16, R3 to R2, R6 to R21, R7 to R22, R8 to R23, R9 to R24, R10 to R25, R5 to R3, R11 to R4, R1 to R9, U3 to U2, U2 to U3
