File: garden-box/prototype-2/prototype-2.kicad_sch (KiCad schematic)
At the start: 17 parts, among them J1 USB_A, J2 Conn_01x03_Male, J3 Conn_01x04_Male, J4 Screw_Terminal_01x02, J5 Screw_Terminal_01x02, J6 Screw_Terminal_01x02, K1 G6DN-1A-L_DC5, Q1 2N3904, T1 Transformer_1P_2S, U1 ESP32-POE

Commit message: fix Q1 pinout
Parts:
- Q1: footprint Package_TO_SOT_SMD:SOT-23 -> jlcpcb:SOT-23-3_L2.9-W1.3-P1.90-LS2.4-TR
Changed lines of the file:
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@@
       (effects (font (size 1.27 1.27)) (justify left))
     )
-    (property "Footprint" "Package_TO_SOT_SMD:SOT-23" (id 2) (at 152.4 71.755 0)
+    (property "Footprint" "jlcpcb:SOT-23-3_L2.9-W1.3-P1.90-LS2.4-TR" (id 2) (at 152.4 71.755 0)
       (effects (font (size 1.27 1.27) italic) (justify left) hide)
     )
@@
     )
     (path "/3b87441e-9545-4daa-bf5c-0e30f2dd4c01"
-      (reference "Q1") (unit 1) (value "2N3904") (footprint "Package_TO_SOT_SMD:SOT-23")
+      (reference "Q1") (unit 1) (value "2N3904") (footprint "jlcpcb:SOT-23-3_L2.9-W1.3-P1.90-LS2.4-TR")
     )
     (path "/edf8efa6-7dc9-40e5-9168-51551bfeb3ac"

Commit message: update usb connector
Parts:
- J1: footprint Connector_USB:USB_A_Molex_67643_Horizontal -> rs-online:875200010BLF
Changed lines of the file:
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@@
     (property "Reference" "J1" (id 0) (at 31.75 76.2 0))
     (property "Value" "USB_A" (id 1) (at 31.75 78.74 0))
-    (property "Footprint" "Connector_USB:USB_A_Molex_67643_Horizontal" (id 2) (at 35.56 90.17 0)
+    (property "Footprint" "rs-online:875200010BLF" (id 2) (at 35.56 90.17 0)
       (effects (font (size 1.27 1.27)) hide)
     )
@@
     )
     (path "/046cc858-94d2-4a81-a286-14af2525c2b6"
-      (reference "J1") (unit 1) (value "USB_A") (footprint "Connector_USB:USB_A_Molex_67643_Horizontal")
+      (reference "J1") (unit 1) (value "USB_A") (footprint "rs-online:875200010BLF")
     )
     (path "/a92772ed-b0e6-4a03-a485-6f9febfd19d3"

Commit message: improve silkscreen
Other:
- note added: "SEN0308"
- note removed: "Moisture sensor"
Changed lines of the file:
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@@
     (stroke (width 0) (type default) (color 0 0 0 0))
   )
-  (text "Moisture sensor" (at 12.7 148.59 0)
+  (text "SEN0308" (at 19.05 148.59 0)
     (effects (font (size 1.27 1.27)) (justify left bottom))
   )

Commit message: change sensor pin
Connections:
- net at U1.11 (GPIO13): now also J2.3 (Pin_3), R1.2
- now unconnected: U1.18 (GPIO35)
Changed lines of the file:
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@@
     (stroke (width 0) (type default) (color 0 0 0 0))
   )
-  (wire (pts (xy 101.6 73.66) (xy 113.03 73.66))
+  (wire (pts (xy 101.6 96.52) (xy 113.03 96.52))
     (stroke (width 0) (type default) (color 0 0 0 0))
   )
@@
     (stroke (width 0) (type default) (color 0 0 0 0))
   )
-  (wire (pts (xy 113.03 73.66) (xy 113.03 128.27))
+  (wire (pts (xy 113.03 96.52) (xy 113.03 128.27))
     (stroke (width 0) (type default) (color 0 0 0 0))
   )
