File: epanel-energy-monitor/v1/epanel-energy-monitor.kicad_sch (KiCad schematic)
At the start: 68 parts, among them J1 Conn_01x01_Male, J10 Conn_01x03_Male, J11 Conn_01x03_Male, J12 Conn_01x03_Male, J13 Conn_01x03_Male, J14 Conn_02x05, J15 Conn_02x05, J16 Conn_02x05, J17 Screw_Terminal_01x02, J18 Screw_Terminal_01x02, J19 Screw_Terminal_01x02, J2 Conn_01x01_Male, J3 Screw_Terminal_01x02, J4 Conn_01x01, J5 Screw_Terminal_01x02, J6 Conn_02x03, J7 Conn_02x03, J8 Conn_02x03, J9 Conn_02x03, Q1 BSS138, T1 230V - 6V, U1 ESP32-POE, U2 LTV-814, U3 MCP3208, U4 ADS1115, U5 LMV321

Commit message: skeleton
Parts:
- removed C2, C3, C4, C5: 10uF/6V, Resistor_SMD:R_0603_1608Metric, symbol Device:C
- removed J10, J11, J12, J13: Conn_01x03_Male, Connector_PinHeader_2.54mm:PinHeader_1x03_P2.54mm_Vertical, symbol Connector:Conn_01x03_Male
- removed J15, J16: Conn_02x05, Connector_PinHeader_2.54mm:PinHeader_2x05_P2.54mm_Vertical, symbol Connector_Generic:Conn_02x05_Odd_Even
- removed J18, J19: Screw_Terminal_01x02, TerminalBlock:TerminalBlock_bornier-2_P5.08mm, symbol Connector:Screw_Terminal_01x02
- removed J6, J7, J8, J9: Conn_02x03, Connector_PinHeader_2.54mm:PinHeader_2x03_P2.54mm_Vertical, symbol Connector_Generic:Conn_02x03_Odd_Even
- removed R10, R11, R12, R13, R14, R7, R8, R9: 470KΩ, Resistor_SMD:R_0603_1608Metric, symbol Device:R
- removed R17, R18: 1KΩ, Resistor_SMD:R_0603_1608Metric, symbol Device:R
- removed R26, R31: 200Ω/0.5W, Resistor_SMD:R_0805_2012Metric, symbol Device:R
- removed R27, R32: 120Ω/0.5W, Resistor_SMD:R_0805_2012Metric, symbol Device:R
- removed R28, R33: 100Ω/0.5W, Resistor_SMD:R_0805_2012Metric, symbol Device:R
- removed R29, R34: 62Ω/0.5W, Resistor_SMD:R_0805_2012Metric, symbol Device:R
- removed R30, R35: 33Ω/0.5W, Resistor_SMD:R_0805_2012Metric, symbol Device:R
- removed U4: ADS1115, Package_SO:TSSOP-10_3x3mm_P0.5mm, symbol Analog_ADC:ADS1115IDGS
Connections:
- net at R20.1, T1.3 (SA): now also J14.1 (Pin_1), J14.3 (Pin_3), J14.5 (Pin_5), J14.7 (Pin_7), J14.9 (Pin_9), J17.2 (Pin_2), U5.3 (-), U5.4
- net at U3.1 (CH0): now also R15.1
- net at U3.2 (CH1): now also R16.1
Other:
- note removed: "1-2 = ESP 3-4 = ADS 5-6 = MCP"
- note removed: "1-2 = pont diviseur 2-3 = ampli op"
- note removed: "CT0"
- note removed: "CT2"

Commit message: schematic wip
Parts:
- removed J1, J2: Conn_01x01_Male, Connector_PinHeader_2.54mm:PinHeader_1x01_P2.54mm_Vertical, symbol Connector:Conn_01x01_Male
- removed J14: Conn_02x05, Connector_PinHeader_2.54mm:PinHeader_2x05_P2.54mm_Vertical, symbol Connector_Generic:Conn_02x05_Odd_Even
- removed J17: Screw_Terminal_01x02, TerminalBlock:TerminalBlock_bornier-2_P5.08mm, symbol Connector:Screw_Terminal_01x02
- removed J4: Conn_01x01, Connector_PinHeader_2.54mm:PinHeader_1x01_P2.54mm_Vertical, symbol Connector:Conn_01x01_Male
- removed R16: 1KΩ, Resistor_SMD:R_0603_1608Metric, symbol Device:R
- removed R21: 200Ω/0.5W, Resistor_SMD:R_0805_2012Metric, symbol Device:R
- removed R22: 120Ω/0.5W, Resistor_SMD:R_0805_2012Metric, symbol Device:R
- removed R23: 100Ω/0.5W, Resistor_SMD:R_0805_2012Metric, symbol Device:R
- removed R24: 62Ω/0.5W, Resistor_SMD:R_0805_2012Metric, symbol Device:R
- removed R25: 33Ω/0.5W, Resistor_SMD:R_0805_2012Metric, symbol Device:R
- added J?: Conn_01x02_Male, symbol Connector:Conn_01x02_Male
- added J?: Conn_01x05_Male, Connector_PinHeader_2.54mm:PinHeader_1x05_P2.54mm_Vertical, symbol Connector:Conn_01x05_Male
- added SW?: SW_DPDT_x2, symbol Switch:SW_DPDT_x2
- added U?: MCP3208, Package_SO:SOIC-16_3.9x9.9mm_P1.27mm, symbol Analog_ADC:MCP3208
- Q1: footprint Package_TO_SOT_SMD:SOT-23 -> (none)
- T1: footprint mylife-footprints:RS PRO 6V 0.35VA -> mylife-footprints:RS PRO Transfo 6V 0.35VA
- U2: footprint Package_DIP:SMDIP-4_W7.62mm -> (none)
Connections:
- net +3V3: now also U?.15 (Vref), U?.16 (Vdd)
- net +5V: now also J?.1 (Pin_1)
- net GND: now also J?.2 (Pin_2), U?.14 (AGND), U?.9 (DGND)
- net LINE: now also SW?.1 (A); no longer PS1.1 (AC/L)
- net at R19.2, T1.4 (SB): now also J?.1 (Pin_1)
- net at R15.1: now also U?.1 (CH0); no longer U3.1 (CH0)
- net at U3.10 (~{CS}/SHDN): now also U1.16 (GPIO33); no longer U1.14 (GPIO16)
- net at U1.11 (GPIO13), U3.11 (Din): now also U?.11 (Din)
- net at U1.12 (GPIO14), U3.12 (Dout): now also U?.12 (Dout)
- net at U1.13 (GPIO15), U3.13 (CLK): now also U?.13 (CLK)
- net CT9: now reaches U3.2 (CH1)
- net CT10: now reaches U3.3 (CH2)
- net CT11: now reaches U3.4 (CH3)
- net CT12: now reaches U3.5 (CH4)
- net CT13: now reaches U3.6 (CH5)
- net CT14: now reaches U3.7 (CH6)
- net CT15: now reaches U3.8 (CH7)
- net CT Sensor 1/ZERO: now reaches R20.1, T1.3 (SA), U5.3 (-), U5.4
- net CT Sensor 1/ZERO: now also J?.2 (Pin_2)
- net at U1.10 (GPIO5): now also J?.5 (Pin_5)
- net at U1.15 (GPIO32): now also U?.10 (~{CS}/SHDN)
- net at U1.8 (GPIO3): now also J?.3 (Pin_3)
- net at U1.9 (GPIO4): now also J?.4 (Pin_4)
- new net: PS1.1 (AC/L), SW?.2 (B)
- new net CT1: U?.2 (CH1)
- new net CT2: U?.3 (CH2)
- new net CT3: U?.4 (CH3)
- new net CT4: U?.5 (CH4)
- new net CT5: U?.6 (CH5)
- new net CT6: U?.7 (CH6)
- new net CT7: U?.8 (CH7)
- new net CT8: U3.1 (CH0)
Other:
- added sheet CT Sensor 1 (ct_sensor.kicad_sch)
- added sheet CT Sensor 10 (ct_sensor.kicad_sch)
- added sheet CT Sensor 11 (ct_sensor.kicad_sch)
- added sheet CT Sensor 12 (ct_sensor.kicad_sch)
- added sheet CT Sensor 13 (ct_sensor.kicad_sch)
- added sheet CT Sensor 14 (ct_sensor.kicad_sch)
- added sheet CT Sensor 15 (ct_sensor.kicad_sch)
- added sheet CT Sensor 2 (ct_sensor.kicad_sch)
- added sheet CT Sensor 3 (ct_sensor.kicad_sch)
- added sheet CT Sensor 4 (ct_sensor.kicad_sch)
- added sheet CT Sensor 5 (ct_sensor.kicad_sch)
- added sheet CT Sensor 6 (ct_sensor.kicad_sch)
- added sheet CT Sensor 7 (ct_sensor.kicad_sch)
- added sheet CT Sensor 8 (ct_sensor.kicad_sch)
- added sheet CT Sensor 9 (ct_sensor.kicad_sch)
- note added: "IO"
- note added: "Transfo test"
- note removed: "CT1"
- note removed: "Used by IO : - GPIO 3 (interrupt) - GPIO 4 (SDA) - GPIO 5 (SCL)"
- moved on the sheet: C1, J3, PS1, R15, R19, R20, R5, R6, U5

Commit message: wip
Parts:
- J?: footprint (none) -> Connector_PinHeader_2.54mm:PinHeader_1x02_P2.54mm_Vertical

Commit message: annotate
Parts:
- gave numbers to parts that had none: 4
- renumbered J3 to J2, J5 to J3, R5 to R4, R6 to R5, R4 to R6, R15 to R7, R19 to R8, R20 to R9, U3 to U4

Commit message: fix mosfet pinout
Parts:
- Q1: footprint (none) -> Package_TO_SOT_SMD:SOT-23
Connections:
- net GND: now also Q1.2 (S); no longer Q1.3 (S)
- net at R3.2, U2.3: now also Q1.1 (G); no longer Q1.2 (G)
- net at R1.1, R2.1, U1.7 (GPIO2): now also Q1.3 (D); no longer Q1.1 (D)
Changed lines of the file:
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@@
   )
   (symbol (lib_id "Transistor_FET:BS170") (at 92.71 81.28 0) (mirror y) (unit 1)
-    (in_bom yes) (on_board yes) (fields_autoplaced)
-    (property "Reference" "Q1" (id 0) (at 87.5031 80.3715 0)
-      (effects (font (size 1.27 1.27)) (justify left))
-    )
-    (property "Value" "BSS138" (id 1) (at 87.5031 83.1466 0)
-      (effects (font (size 1.27 1.27)) (justify left))
-    )
-    (property "Footprint" "" (id 2) (at 87.63 83.185 0)
+    (in_bom yes) (on_board yes)
+    (property "Reference" "Q1" (id 0) (at 93.98 73.66 0)
+      (effects (font (size 1.27 1.27)) (justify left))
+    )
+    (property "Value" "BSS138" (id 1) (at 99.06 76.2 0)
+      (effects (font (size 1.27 1.27)) (justify left))
+    )
+    (property "Footprint" "Package_TO_SOT_SMD:SOT-23" (id 2) (at 97.79 83.185 0)
       (effects (font (size 1.27 1.27) italic) (justify left) hide)
     )
@@
       (effects (font (size 1.27 1.27)) hide)
     )
+    (pin "3")
     (pin "1")
     (pin "2")
-    (pin "3")
   )
   (symbol (lib_id "power:+3V3") (at 132.08 132.08 0) (unit 1)
@@
     )
     (path "/a6da1c49-f5f8-4bd8-8a1f-6e9f0765716a"
-      (reference "Q1") (unit 1) (value "BSS138") (footprint "")
+      (reference "Q1") (unit 1) (value "BSS138") (footprint "Package_TO_SOT_SMD:SOT-23")
     )
     (path "/63620899-db39-4076-b115-8a9f2685955e"

Commit message: wip schematic
Parts:
- U2: footprint (none) -> Package_DIP:SMDIP-4_W9.53mm

Commit message: cleanup
Other:
- note added: "Alim"
Changed lines of the file:
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@@
+    (effects (font (size 1.27 1.27)) (justify left bottom))
+  )
+  (text "Teleinfo" (at 177.8 80.01 0)
+    (effects (font (size 1.27 1.27)) (justify left bottom))
+  )
+  (text "Alim" (at 74.93 240.03 0)
     (effects (font (size 1.27 1.27)) (justify left bottom))
   )
@@
     (effects (font (size 1.27 1.27)) (justify left bottom))
   )
-  (label "Teleinfo" (at 177.8 80.01 0)
-    (effects (font (size 1.27 1.27)) (justify left bottom))
-  )

Commit message: add switch
Parts:
- SW1: footprint (none) -> mylife-footprints:RS PRO Switch MFP161D
Changed lines of the file:
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@@
     (property "Reference" "SW1" (id 0) (at 64.77 252.1925 0))
     (property "Value" "SW_DPDT_x2" (id 1) (at 64.77 254.9676 0))
-    (property "Footprint" "" (id 2) (at 64.77 259.08 0)
+    (property "Footprint" "mylife-footprints:RS PRO Switch MFP161D" (id 2) (at 64.77 259.08 0)
       (effects (font (size 1.27 1.27)) hide)
     )
@@
     )
     (path "/8455e93e-0497-4a1b-98ad-a5ed8aa30439"
-      (reference "SW1") (unit 1) (value "SW_DPDT_x2") (footprint "")
+      (reference "SW1") (unit 1) (value "SW_DPDT_x2") (footprint "mylife-footprints:RS PRO Switch MFP161D")
     )
     (path "/35c8ca8a-5716-4892-b883-7f70694cf361"
