File: epanel-controller/v1/epanel-controller.kicad_sch (KiCad schematic)
At the start: 6 parts, among them J1 Conn_01x05_Male

Commit message: wip controller
Connections:
- net +3V3: now also U?.2 (+3.3V_(out))
- net +5V: now also U?.1 (+5V)
- net CS1: now also U?.15 (GPIO32)
- net CS2: now also U?.16 (GPIO33)
- net GND: now also U?.3 (GND)
- net INTR: now also J1.3 (Pin_3), U?.8 (GPIO3)
- net MISO: now also U?.12 (GPIO14)
- net MOSI: now also U?.11 (GPIO13)
- net SCL: now also J1.5 (Pin_5), U?.10 (GPIO5)
- net SCLK: now also U?.13 (GPIO15)
- net SDA: now also J1.4 (Pin_4), U?.9 (GPIO4)
- net TIC: now also U?.7 (GPIO2)
Other:
- note added: "Energy Monitor"
- moved on the sheet: J1, J?, PS?, SW?A, U?

Commit message: controller schematic
Parts:
- J3: renamed from J?; value Conn_02x04_Counter_Clockwise -> Conn_02x04_Odd_Even; footprint (none) -> Connector_PinHeader_2.54mm:PinHeader_2x04_P2.54mm_Vertical
- SW1: renamed from SW?; footprint mylife-footprints:RS PRO Switch MFP161D -> mylife-footprints:RS PRO Switch 401-703
- gave numbers to parts that had none: 3

Commit message: controller pcb placement
Parts:
- U1: footprint (none) -> mylife-footprints:ESP32-POE
Changed lines of the file:
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@@
     (property "Reference" "U1" (id 0) (at 147.32 104.14 0))
     (property "Value" "ESP32-POE-ISO" (id 1) (at 147.32 106.68 0))
-    (property "Footprint" "" (id 2) (at 147.32 105.41 0)
+    (property "Footprint" "mylife-footprints:ESP32-POE" (id 2) (at 147.32 105.41 0)
       (effects (font (size 1.27 1.27)) hide)
     )
@@
     )
     (path "/d2f99d6e-0d4d-49fc-ad4d-c713356d660b"
-      (reference "U1") (unit 1) (value "ESP32-POE-ISO") (footprint "")
+      (reference "U1") (unit 1) (value "ESP32-POE-ISO") (footprint "mylife-footprints:ESP32-POE")
     )
   )
