File: epanel-controller/v1/epanel-controller.kicad_pcb (KiCad board)
At the start: 2 copper layers, 364 x 120.8 mm, 172 parts, among them J1 Conn_01x05_Male, J10 Screw_Terminal_01x02, J11 Screw_Terminal_01x02, J12 Screw_Terminal_01x02, J13 Screw_Terminal_01x02, J14 Screw_Terminal_01x02, J15 Screw_Terminal_01x02, J16 Screw_Terminal_01x02, J17 Screw_Terminal_01x02, J18 Screw_Terminal_01x02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

Commit message: controller pcb placement
Parts:
- removed C1: 1uF/6V, Resistor_SMD:R_0603_1608Metric
- removed D1: LED, Diode_SMD:D_0805_2012Metric
- removed J10, J11, J12, J13, J14, J15, J16, J17, J18, J19, J5, J6 (x15), J7, J8, J9: Screw_Terminal_01x02, mylife-footprints:RS PRO Terminal Small x2
- removed J4: Conn_01x02_Male, Connector_PinHeader_2.54mm:PinHeader_1x02_P2.54mm_Vertical
- removed Q1: BSS138, Package_TO_SOT_SMD:SOT-23
- removed R1, R10, R16, R22, R28, R34, R40, R46, R52, R58, R64, R7, R70, R76, R82, R88, R94: 1KΩ, Resistor_SMD:R_0603_1608Metric
- removed R11, R17, R23, R29, R35, R41, R47, R53, R59, R65, R71, R77, R83, R89, R95: 200Ω/0.5W, Resistor_SMD:R_0805_2012Metric
- removed R12, R18, R24, R30, R36, R42, R48, R54, R60, R66, R72, R78, R84, R90, R96: 120Ω/0.5W, Resistor_SMD:R_0805_2012Metric
- removed R13, R19, R25, R31, R37, R43, R49, R55, R61, R67, R73, R79, R85, R91, R97: 100Ω/0.5W, Resistor_SMD:R_0805_2012Metric
- removed R14, R20, R26, R32, R38, R44, R50, R56, R62, R68, R74, R80, R86, R92, R98: 62Ω/0.5W, Resistor_SMD:R_0805_2012Metric
- removed R15, R21, R27, R33, R39, R45, R51, R57, R63, R69, R75, R81, R87, R93, R99: 33Ω/0.5W, Resistor_SMD:R_0805_2012Metric
- removed R2: 10KΩ, Resistor_SMD:R_0603_1608Metric
- removed R3: 3.3KΩ, Resistor_SMD:R_0603_1608Metric
- removed R4, R5, R9: 12KΩ, Resistor_SMD:R_0603_1608Metric
- removed R6: 220Ω, Resistor_SMD:R_0603_1608Metric
- removed R8: 100KΩ, Resistor_SMD:R_0603_1608Metric
- removed S1, S10, S11, S12, S13, S14, S15, S2 (x15), S3, S4, S5, S6, S7, S8, S9: SS-10-15SPE, mylife-footprints:RS PRO SS-10-15SPE
- removed T1: 230V - 6V, mylife-footprints:RS PRO Transfo 6V 0.35VA
- removed U2: LTV-814, Package_DIP:SMDIP-4_W9.53mm
- removed U3, U4: MCP3208, Package_SO:SOIC-16_3.9x9.9mm_P1.27mm
- removed U5: LMV321, Package_TO_SOT_SMD:SOT-23-5
- J3: value Screw_Terminal_01x02 -> Conn_02x04_Odd_Even; footprint TerminalBlock:TerminalBlock_bornier-2_P5.08mm -> Connector_PinHeader_2.54mm:PinHeader_2x04_P2.54mm_Vertical
- SW1: footprint mylife-footprints:RS PRO Switch MFP161D -> mylife-footprints:RS PRO Switch 401-703
- U1: value ESP32-POE -> ESP32-POE-ISO
- moved J2 286.6 mm to (120.0, 55.1), turned to 180 degrees
- moved J1 232.4 mm to (103.5, 129.5), turned to 90 degrees
- moved J3 229.5 mm to (120.4, 131.4)
- moved SW1 161.5 mm to (121.9, 73.0), turned to 90 degrees
- moved PS1 33.5 mm to (108.7, 84.5), turned to 0 degrees
- moved U1 32.2 mm to (147.7, 94.3), turned to 0 degrees
Connections:
- net Net-(J1-Pad3) renamed /INTR
- net Net-(J1-Pad4) renamed /SDA
- net Net-(J1-Pad5) renamed /SCL
- J3 pad 1: Net-(J3-Pad1) -> +3V3
- J3 pad 2: Net-(J3-Pad2) -> GND
- U1 pad 11: Net-(U1-Pad11) -> /MOSI
- U1 pad 12: Net-(U1-Pad12) -> /MISO
- U1 pad 13: Net-(U1-Pad13) -> /SCLK
- U1 pad 15: Net-(U1-Pad15) -> /CS1
- U1 pad 16: Net-(U1-Pad16) -> /CS2
- U1 pad 7: Net-(Q1-Pad3) -> /TIC
Other:
- board size 364 x 120.8 mm -> 68 x 86.5 mm
- board text added: "3v3 TIC CS1 CS2"
- board text added: "5v GND INTR SDA SCL"
- board text added: "GND SCLK MISO MOSI"

Commit message: controller pcb
Routing:
- net GND: track 0.00 -> 75.5 mm
- net +3V3: track 0.00 -> 65.0 mm
- net +5V: track 0.00 -> 64.0 mm
- net /CS1: track 0.00 -> 60.8 mm, vias 0 -> 1
- net /TIC: track 0.00 -> 56.6 mm
- net /CS2: track 0.00 -> 56.5 mm, vias 0 -> 1
- net /SCLK: track 0.00 -> 48.5 mm
- net /MISO: track 0.00 -> 44.9 mm
- net /INTR: track 0.00 -> 44.5 mm
- net /SDA: track 0.00 -> 42.0 mm
- net NEUT: track 0.00 -> 41.5 mm
- net /MOSI: track 0.00 -> 41.3 mm
- net /SCL: track 0.00 -> 39.5 mm
- net LINE: track 0.00 -> 18.7 mm
- net Net-(PS1-Pad1): track 0.00 -> 16.4 mm
Changed lines of the file:
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@@
     (effects (font (size 0.8 0.8) (thickness 0.12)))
   )
+  (segment (start 126.5075 114.935) (end 117.475 114.935) (width 0.25) (layer "B.Cu") (net 1))
+  (segment (start 120.396 121.0465) (end 126.5075 114.935) (width 0.25) (layer "B.Cu") (net 1))
+  (segment (start 120.396 128.8542) (end 120.396 121.0465) (width 0.25) (layer "B.Cu") (net 1))
+  (segment (start 106.05 126.37) (end 106.05 129.54) (width 0.25) (layer "B.Cu") (net 1))
+  (segment (start 128.905 112.5375) (end 128.905 92.71) (width 0.25) (layer "B.Cu") (net 1))
+  (segment (start 117.475 114.935) (end 106.045 126.365) (width 0.25) (layer "B.Cu") (net 1))
+  (segment (start 132.305 89.31) (end 134.94 89.31) (width 0.25) (layer "B.Cu") (net 1))
+  (segment (start 106.045 126.365) (end 106.05 126.37) (width 0.25) (layer "B.Cu") (net 1))
+  (segment (start 128.905 92.71) (end 132.305 89.31) (width 0.25) (layer "B.Cu") (net 1))
+  (segment (start 126.5075 114.935) (end 128.905 112.5375) (width 0.25) (layer "B.Cu") (net 1))
+  (segment (start 103.51 129.54) (end 103.51 128.264282) (width 0.25) (layer "B.Cu") (net 2))
+  (segment (start 129.765 84.23) (end 134.94 84.23) (width 0.25) (layer "B.Cu") (net 2))
+  (segment (start 126.5075 109.855) (end 126.5075 87.4875) (width 0.25) (layer "B.Cu") (net 2))
+  (segment (start 103.51 128.264282) (end 121.919282 109.855) (width 0.25) (layer "B.Cu") (net 2))
+  (segment (start 126.5075 87.4875) (end 129.765 84.23) (width 0.25) (layer "B.Cu") (net 2))
+  (segment (start 121.919282 109.855) (end 126.5075 109.855) (width 0.25) (layer "B.Cu") (net 2))
+  (segment (start 120.396 131.3942) (end 122.9868 133.985) (width 0.25) (layer "B.Cu") (net 3))
+  (segment (start 136.935 86.77) (end 134.94 86.77) (width 0.25) (layer "B.Cu") (net 3))
+  (segment (start 139.065 88.9) (end 136.935 86.77) (width 0.25) (layer "B.Cu") (net 3))
+  (segment (start 122.9868 133.985) (end 130.81 133.985) (width 0.25) (layer "B.Cu") (net 3))
+  (segment (start 130.81 133.985) (end 139.065 125.73) (width 0.25) (layer "B.Cu") (net 3))
+  (segment (start 139.065 125.73) (end 139.065 88.9) (width 0.25) (layer "B.Cu") (net 3))
+  (segment (start 121.92 57.015) (end 120.015 55.11) (width 0.25) (layer "B.Cu") (net 4))
+  (segment (start 121.92 73.025) (end 121.92 57.015) (width 0.25) (layer "B.Cu") (net 4))
+  (segment (start 108.7275 89.535) (end 106.68 89.535) (width 0.25) (layer "B.Cu") (net 5))
+  (segment (start 104.775 87.63) (end 104.775 65.27) (width 0.25) (layer "B.Cu") (net 5))
+  (segment (start 106.68 89.535) (end 104.775 87.63) (width 0.25) (layer "B.Cu") (net 5))
+  (segment (start 104.775 65.27) (end 114.935 55.11) (width 0.25) (layer "B.Cu") (net 5))
+  (segment (start 108.59 118.103565) (end 124.683565 102.01) (width 0.25) (layer "F.Cu") (net 11))
+  (segment (start 108.59 129.54) (end 108.59 118.103565) (width 0.25) (layer "F.Cu") (net 11))
+  (segment (start 124.683565 102.01) (end 134.94 102.01) (width 0.25) (layer "F.Cu") (net 11))
+  (segment (start 122.779282 104.55) (end 134.94 104.55) (width 0.25) (layer "F.Cu") (net 15))
+  (segment (start 111.13 129.54) (end 111.13 116.199282) (width 0.25) (layer "F.Cu") (net 15))
+  (segment (start 111.13 116.199282) (end 122.779282 104.55) (width 0.25) (layer "F.Cu") (net 15))
+  (segment (start 113.67 120.607225) (end 113.665 120.602225) (width 0.25) (layer "F.Cu") (net 16))
+  (segment (start 120.875 107.09) (end 134.94 107.09) (width 0.25) (layer "F.Cu") (net 16))
+  (segment (start 113.665 114.3) (end 120.875 107.09) (width 0.25) (layer "F.Cu") (net 16))
+  (segment (start 113.67 129.54) (end 113.67 120.607225) (width 0.25) (layer "F.Cu") (net 16))
+  (segment (start 113.665 120.602225) (end 113.665 114.3) (width 0.25) (layer "F.Cu") (net 16))
+  (segment (start 122.936 131.3942) (end 122.936 132.969) (width 0.25) (layer "F.Cu") (net 17))
+  (segment (start 129.54 120.65) (end 139.065 111.125) (width 0.25) (layer "F.Cu") (net 17))
+  (segment (start 118.11 125.73) (end 123.19 120.65) (width 0.25) (layer "F.Cu") (net 17))
+  (segment (start 139.065 100.965) (end 137.57 99.47) (width 0.25) (layer "F.Cu") (net 17))
+  (segment (start 122.936 132.969) (end 121.92 133.985) (width 0.25) (layer "F.Cu") (net 17))
+  (segment (start 123.19 120.65) (end 129.54 120.65) (width 0.25) (layer "F.Cu") (net 17))
+  (segment (start 121.92 133.985) (end 118.745 133.985) (width 0.25) (layer "F.Cu") (net 17))
+  (segment (start 118.745 133.985) (end 118.11 133.35) (width 0.25) (layer "F.Cu") (net 17))
+  (segment (start 137.57 99.47) (end 134.94 99.47) (width 0.25) (layer "F.Cu") (net 17))
+  (segment (start 118.11 133.35) (end 118.11 125.73) (width 0.25) (layer "F.Cu") (net 17))
+  (segment (start 139.065 111.125) (end 139.065 100.965) (width 0.25) (layer "F.Cu") (net 17))
+  (segment (start 160.245 102.01) (end 160.34 102.01) (width 0.25) (layer "F.Cu") (net 18))
+  (segment (start 127.9652 123.825) (end 138.43 123.825) (width 0.25) (layer "F.Cu") (net 18))
+  (segment (start 122.936 128.8542) (end 127.9652 123.825) (width 0.25) (layer "F.Cu") (net 18))
+  (segment (start 138.43 123.825) (end 160.245 102.01) (width 0.25) (layer "F.Cu") (net 18))
+  (segment (start 128.27 133.985) (end 138.43 133.985) (width 0.25) (layer "F.Cu") (net 19))
+  (segment (start 127 133.985) (end 128.27 133.985) (width 0.25) (layer "F.Cu") (net 19))
+  (segment (start 125.73 132.715) (end 127 133.985) (width 0.25) (layer "F.Cu") (net 19))
+  (segment (start 138.43 133.985) (end 152.4 120.015) (width 0.25) (layer "F.Cu") (net 19))
+  (segment (start 157.48 114.935) (end 157.48 114.3) (width 0.25) (layer "F.Cu") (net 19))
+  (segment (start 125.476 132.461) (end 125.73 132.715) (width 0.25) (layer "F.Cu") (net 19))
+  (segment (start 125.476 131.3942) (end 125.476 132.461) (width 0.25) (layer "F.Cu") (net 19))
+  (segment (start 152.4 120.015) (end 157.48 114.935) (width 0.25) (layer "F.Cu") (net 19))
+  (via (at 157.48 114.3) (size 0.8) (drill 0.4) (layers "F.Cu" "B.Cu") (net 19))
+  (segment (start 157.48 114.3) (end 157.48 99.79) (width 0.25) (layer "B.Cu") (net 19))
+  (segment (start 157.48 99.79) (end 160.34 96.93) (width 0.25) (layer "B.Cu") (net 19))
+  (segment (start 160.34 104.55) (end 139.16 125.73) (width 0.25) (layer "F.Cu") (net 20))
+  (segment (start 125.476 128.8542) (end 128.6002 125.73) (width 0.25) (layer "F.Cu") (net 20))
+  (segment (start 128.6002 125.73) (end 133.35 125.73) (width 0.25) (layer "F.Cu") (net 20))
+  (segment (start 139.16 125.73) (end 138.43 125.73) (width 0.25) (layer "F.Cu") (net 20))
+  (segment (start 133.35 125.73) (end 138.43 125.73) (width 0.25) (layer "F.Cu") (net 20))
+  (segment (start 153.035 116.84) (end 155.575 114.3) (width 0.25) (layer "F.Cu") (net 21))
+  (segment (start 138.4808 131.3942) (end 153.035 116.84) (width 0.25) (layer "F.Cu") (net 21))
+  (segment (start 128.016 131.3942) (end 138.4808 131.3942) (width 0.25) (layer "F.Cu") (net 21))
+  (via (at 155.575 114.3) (size 0.8) (drill 0.4) (layers "F.Cu" "B.Cu") (net 21))
+  (segment (start 155.575 114.3) (end 155.575 99.155) (width 0.25) (layer "B.Cu") (net 21))
+  (segment (start 155.575 99.155) (end 160.34 94.39) (width 0.25) (layer "B.Cu") (net 21))
+  (segment (start 128.016 128.8542) (end 138.5758 128.8542) (width 0.25) (layer "F.Cu") (net 22))
+  (segment (start 138.5758 128.8542) (end 160.34 107.09) (width 0.25) (layer "F.Cu") (net 22))
+  (segment (start 111.125 84.455) (end 108.7275 84.455) (width 0.25) (layer "B.Cu") (net 24))
+  (segment (start 117.22 78.36) (end 111.125 84.455) (width 0.25) (layer "B.Cu") (net 24))
+  (segment (start 117.22 73.025) (end 117.22 78.36) (width 0.25) (layer "B.Cu") (net 24))
   (group "" (id 26dac7cb-1bb3-48fb-9339-9910ff5c9eb2)
     (members
