File: epanel-energy-monitor/v1.1/epanel-energy-monitor.kicad_pcb (KiCad board)
At the start: 2 copper layers, 103 x 86.5 mm, 143 parts, among them J1 Conn_02x04_Odd_Even, J10 Screw_Terminal_01x02, J11 Screw_Terminal_01x02, J12 Screw_Terminal_01x02, J13 Screw_Terminal_01x02, J14 Screw_Terminal_01x02, J15 Screw_Terminal_01x02, J16 Screw_Terminal_01x02, J17 Screw_Terminal_01x02, J18 Screw_Terminal_01x02, J19 Screw_Terminal_01x02, J2 Screw_Terminal_01x02, J3 Conn_01x02_Male, J4 Screw_Terminal_01x02, J5 Screw_Terminal_01x02, J6 Screw_Terminal_01x02, J7 Screw_Terminal_01x02, J8 Screw_Terminal_01x02, J9 Screw_Terminal_01x02, Q1 BSS138, T1 230V - 6V, U1 LTV-814, U2 MCP3208, U3 MCP3208, U4 LMV321

Commit message: wip fix pcb
Parts:
- moved R62 34.8 mm to (133.5, 136.1)
- moved R64 34.8 mm to (137.3, 136.1)
- moved R71 34.8 mm to (158.9, 128.5)
- moved R72 34.8 mm to (155.1, 128.5)
- moved R73 34.8 mm to (155.1, 132.3)
- moved R75 34.8 mm to (158.9, 132.3)
- moved R77 34.8 mm to (169.7, 128.5)
- moved R78 34.8 mm to (165.9, 128.5)
- moved R79 34.8 mm to (165.9, 132.4)
- moved R80 34.8 mm to (165.9, 136.2)
- moved R81 34.8 mm to (169.7, 132.4)
- moved R82 34.8 mm to (169.7, 136.2)
- moved R83 34.8 mm to (180.6, 128.5)
- moved R84 34.8 mm to (176.8, 128.5)
- moved R85 34.8 mm to (176.8, 132.4)
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Connections:
- S1 pad 1: Net-(R12-Pad2) -> Net-(R14-Pad2)
- S1 pad 2: /CT Sensor 1/ZERO -> Net-(R13-Pad2)
- S1 pad 3: Net-(R13-Pad2) -> /CT Sensor 1/ZERO
- S1 pad 4: Net-(R14-Pad2) -> Net-(R12-Pad2)
- S1 pad 5: Net-(R15-Pad2) -> unconnected-(S1-Pad5)
- S1 pad 6: Net-(R16-Pad2) -> /CT Sensor 1/ZERO
- S1 pad 7: /CT Sensor 1/ZERO -> Net-(R16-Pad2)
- S1 pad 8: unconnected-(S1-Pad8) -> Net-(R15-Pad2)
- S10 pad 1: Net-(R66-Pad2) -> Net-(R68-Pad2)
- S10 pad 2: /CT Sensor 1/ZERO -> Net-(R67-Pad2)
- S10 pad 3: Net-(R67-Pad2) -> /CT Sensor 1/ZERO
- S10 pad 4: Net-(R68-Pad2) -> Net-(R66-Pad2)
- S10 pad 5: Net-(R69-Pad2) -> unconnected-(S10-Pad5)
- S10 pad 6: Net-(R70-Pad2) -> /CT Sensor 1/ZERO
- S10 pad 7: /CT Sensor 1/ZERO -> Net-(R70-Pad2)
- S10 pad 8: unconnected-(S10-Pad8) -> Net-(R69-Pad2)
- S11 pad 1: Net-(R72-Pad2) -> Net-(R74-Pad2)
- S11 pad 2: /CT Sensor 1/ZERO -> Net-(R73-Pad2)
- S11 pad 3: Net-(R73-Pad2) -> /CT Sensor 1/ZERO
- S11 pad 4: Net-(R74-Pad2) -> Net-(R72-Pad2)
- S11 pad 5: Net-(R75-Pad2) -> unconnected-(S11-Pad5)
- S11 pad 6: Net-(R76-Pad2) -> /CT Sensor 1/ZERO
- S11 pad 7: /CT Sensor 1/ZERO -> Net-(R76-Pad2)
- S11 pad 8: unconnected-(S11-Pad8) -> Net-(R75-Pad2)
- S12 pad 1: Net-(R78-Pad2) -> Net-(R80-Pad2)
- S12 pad 2: /CT Sensor 1/ZERO -> Net-(R79-Pad2)
- S12 pad 3: Net-(R79-Pad2) -> /CT Sensor 1/ZERO
- S12 pad 4: Net-(R80-Pad2) -> Net-(R78-Pad2)
- S12 pad 5: Net-(R81-Pad2) -> unconnected-(S12-Pad5)
- S12 pad 6: Net-(R82-Pad2) -> /CT Sensor 1/ZERO
- S12 pad 7: /CT Sensor 1/ZERO -> Net-(R82-Pad2)
- S12 pad 8: unconnected-(S12-Pad8) -> Net-(R81-Pad2)
- S13 pad 1: Net-(R84-Pad2) -> Net-(R86-Pad2)
- S13 pad 2: /CT Sensor 1/ZERO -> Net-(R85-Pad2)
- S13 pad 3: Net-(R85-Pad2) -> /CT Sensor 1/ZERO
- S13 pad 4: Net-(R86-Pad2) -> Net-(R84-Pad2)
- S13 pad 5: Net-(R87-Pad2) -> unconnected-(S13-Pad5)
- S13 pad 6: Net-(R88-Pad2) -> /CT Sensor 1/ZERO
- S13 pad 7: /CT Sensor 1/ZERO -> Net-(R88-Pad2)
- S13 pad 8: unconnected-(S13-Pad8) -> Net-(R87-Pad2)
- S14 pad 1: Net-(R90-Pad2) -> Net-(R92-Pad2)
- S14 pad 2: /CT Sensor 1/ZERO -> Net-(R91-Pad2)
- S14 pad 3: Net-(R91-Pad2) -> /CT Sensor 1/ZERO
- S14 pad 4: Net-(R92-Pad2) -> Net-(R90-Pad2)
- S14 pad 5: Net-(R93-Pad2) -> unconnected-(S14-Pad5)
- S14 pad 6: Net-(R94-Pad2) -> /CT Sensor 1/ZERO
- S14 pad 7: /CT Sensor 1/ZERO -> Net-(R94-Pad2)
- S14 pad 8: unconnected-(S14-Pad8) -> Net-(R93-Pad2)
- S15 pad 1: Net-(R96-Pad2) -> Net-(R98-Pad2)
- S15 pad 2: /CT Sensor 1/ZERO -> Net-(R97-Pad2)
- S15 pad 3: Net-(R97-Pad2) -> /CT Sensor 1/ZERO
- S15 pad 4: Net-(R98-Pad2) -> Net-(R96-Pad2)
- S15 pad 5: Net-(R99-Pad2) -> unconnected-(S15-Pad5)
- S15 pad 6: Net-(R100-Pad2) -> /CT Sensor 1/ZERO
- S15 pad 7: /CT Sensor 1/ZERO -> Net-(R100-Pad2)
- S15 pad 8: unconnected-(S15-Pad8) -> Net-(R99-Pad2)
- S2 pad 1: Net-(R18-Pad2) -> Net-(R20-Pad2)
- S2 pad 2: /CT Sensor 1/ZERO -> Net-(R19-Pad2)
- S2 pad 3: Net-(R19-Pad2) -> /CT Sensor 1/ZERO
- S2 pad 4: Net-(R20-Pad2) -> Net-(R18-Pad2)
- S2 pad 5: Net-(R21-Pad2) -> unconnected-(S2-Pad5)
- S2 pad 6: Net-(R22-Pad2) -> /CT Sensor 1/ZERO
- S2 pad 7: /CT Sensor 1/ZERO -> Net-(R22-Pad2)
- S2 pad 8: unconnected-(S2-Pad8) -> Net-(R21-Pad2)
- S3 pad 1: Net-(R24-Pad2) -> Net-(R26-Pad2)
- S3 pad 2: /CT Sensor 1/ZERO -> Net-(R25-Pad2)
- S3 pad 3: Net-(R25-Pad2) -> /CT Sensor 1/ZERO
- S3 pad 4: Net-(R26-Pad2) -> Net-(R24-Pad2)
- S3 pad 5: Net-(R27-Pad2) -> unconnected-(S3-Pad5)
- S3 pad 6: Net-(R28-Pad2) -> /CT Sensor 1/ZERO
- S3 pad 7: /CT Sensor 1/ZERO -> Net-(R28-Pad2)
- S3 pad 8: unconnected-(S3-Pad8) -> Net-(R27-Pad2)
- S4 pad 1: Net-(R30-Pad2) -> Net-(R32-Pad2)
- S4 pad 2: /CT Sensor 1/ZERO -> Net-(R31-Pad2)
- S4 pad 3: Net-(R31-Pad2) -> /CT Sensor 1/ZERO
- S4 pad 4: Net-(R32-Pad2) -> Net-(R30-Pad2)
- S4 pad 5: Net-(R33-Pad2) -> unconnected-(S4-Pad5)
- S4 pad 6: Net-(R34-Pad2) -> /CT Sensor 1/ZERO
- S4 pad 7: /CT Sensor 1/ZERO -> Net-(R34-Pad2)
- S4 pad 8: unconnected-(S4-Pad8) -> Net-(R33-Pad2)
- S5 pad 1: Net-(R36-Pad2) -> Net-(R38-Pad2)
- S5 pad 2: /CT Sensor 1/ZERO -> Net-(R37-Pad2)
- S5 pad 3: Net-(R37-Pad2) -> /CT Sensor 1/ZERO
- S5 pad 4: Net-(R38-Pad2) -> Net-(R36-Pad2)
- S5 pad 5: Net-(R39-Pad2) -> unconnected-(S5-Pad5)
- S5 pad 6: Net-(R40-Pad2) -> /CT Sensor 1/ZERO
- S5 pad 7: /CT Sensor 1/ZERO -> Net-(R40-Pad2)
- S5 pad 8: unconnected-(S5-Pad8) -> Net-(R39-Pad2)
- S6 pad 1: Net-(R42-Pad2) -> Net-(R44-Pad2)
- S6 pad 2: /CT Sensor 1/ZERO -> Net-(R43-Pad2)
- S6 pad 3: Net-(R43-Pad2) -> /CT Sensor 1/ZERO
- S6 pad 4: Net-(R44-Pad2) -> Net-(R42-Pad2)
- S6 pad 5: Net-(R45-Pad2) -> unconnected-(S6-Pad5)
- S6 pad 6: Net-(R46-Pad2) -> /CT Sensor 1/ZERO
- S6 pad 7: /CT Sensor 1/ZERO -> Net-(R46-Pad2)
- S6 pad 8: unconnected-(S6-Pad8) -> Net-(R45-Pad2)
- S7 pad 1: Net-(R48-Pad2) -> Net-(R50-Pad2)
- S7 pad 2: /CT Sensor 1/ZERO -> Net-(R49-Pad2)
- S7 pad 3: Net-(R49-Pad2) -> /CT Sensor 1/ZERO
- S7 pad 4: Net-(R50-Pad2) -> Net-(R48-Pad2)
- S7 pad 5: Net-(R51-Pad2) -> unconnected-(S7-Pad5)
- S7 pad 6: Net-(R52-Pad2) -> /CT Sensor 1/ZERO
- S7 pad 7: /CT Sensor 1/ZERO -> Net-(R52-Pad2)
- S7 pad 8: unconnected-(S7-Pad8) -> Net-(R51-Pad2)
- S8 pad 1: Net-(R54-Pad2) -> Net-(R56-Pad2)
- S8 pad 2: /CT Sensor 1/ZERO -> Net-(R55-Pad2)
- S8 pad 3: Net-(R55-Pad2) -> /CT Sensor 1/ZERO
- S8 pad 4: Net-(R56-Pad2) -> Net-(R54-Pad2)
- S8 pad 5: Net-(R57-Pad2) -> unconnected-(S8-Pad5)
- S8 pad 6: Net-(R58-Pad2) -> /CT Sensor 1/ZERO
- S8 pad 7: /CT Sensor 1/ZERO -> Net-(R58-Pad2)
- S8 pad 8: unconnected-(S8-Pad8) -> Net-(R57-Pad2)
- S9 pad 1: Net-(R60-Pad2) -> Net-(R62-Pad2)
- S9 pad 2: /CT Sensor 1/ZERO -> Net-(R61-Pad2)
- S9 pad 3: Net-(R61-Pad2) -> /CT Sensor 1/ZERO
- S9 pad 4: Net-(R62-Pad2) -> Net-(R60-Pad2)
- S9 pad 5: Net-(R63-Pad2) -> unconnected-(S9-Pad5)
- S9 pad 6: Net-(R64-Pad2) -> /CT Sensor 1/ZERO
- S9 pad 7: /CT Sensor 1/ZERO -> Net-(R64-Pad2)
- S9 pad 8: unconnected-(S9-Pad8) -> Net-(R63-Pad2)
Routing:
- net /CT Sensor 1/ZERO: track 413.2 -> 377.8 mm
- net /CT15: track 33.8 -> 12.9 mm
- net Net-(J12-Pad1): track 31.1 -> 13.7 mm
- net /CT1: track 33.9 -> 18.1 mm
- net /CT13: track 18.2 -> 2.61 mm
- net /CT12: track 15.1 -> 0.00 mm
- net /CT11: track 19.1 -> 4.06 mm
- net /CT8: track 45.5 -> 31.1 mm
- net Net-(R55-Pad2): track 13.6 -> 0.00 mm
- net Net-(R67-Pad2): track 13.6 -> 0.00 mm
- net Net-(R61-Pad2): track 13.6 -> 0.00 mm
- net Net-(R85-Pad2): track 13.6 -> 0.00 mm
- net /CT7: track 31.7 -> 18.3 mm
- net /CT9: track 36.6 -> 24.0 mm
- net Net-(R98-Pad2): track 11.8 -> 24.1 mm
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
Commit message: pcb placement
Parts:
- added J13: Screw_Terminal_01x02, mylife-footprints:RS PRO Terminal Small x2, F.Cu at (129.6, 115.9)
- added J14: Screw_Terminal_01x02, mylife-footprints:RS PRO Terminal Small x2, F.Cu at (140.5, 115.9)
- added J15: Screw_Terminal_01x02, mylife-footprints:RS PRO Terminal Small x2, F.Cu at (151.4, 115.9)
- added J16: Screw_Terminal_01x02, mylife-footprints:RS PRO Terminal Small x2, F.Cu at (162.2, 115.9)
- added J17: Screw_Terminal_01x02, mylife-footprints:RS PRO Terminal Small x2, F.Cu at (173.1, 115.9)
- added J18: Screw_Terminal_01x02, mylife-footprints:RS PRO Terminal Small x2, F.Cu at (183.9, 115.9)
- added J19: Screw_Terminal_01x02, mylife-footprints:RS PRO Terminal Small x2, F.Cu at (194.8, 115.9)
- added R53: 1KΩ, Resistor_SMD:R_0603_1608Metric, F.Cu at (165.7, 92.4)
- added R53: 1KΩ, Resistor_SMD:R_0603_1608Metric, F.Cu at (133.1, 92.4)
- added R53: 1KΩ, Resistor_SMD:R_0603_1608Metric, F.Cu at (187.4, 92.4)
- added R53: 1KΩ, Resistor_SMD:R_0603_1608Metric, F.Cu at (176.6, 92.4)
- added R53: 1KΩ, Resistor_SMD:R_0603_1608Metric, F.Cu at (144.0, 92.4)
- added R53: 1KΩ, Resistor_SMD:R_0603_1608Metric, F.Cu at (198.3, 92.4)
- added R53: 1KΩ, Resistor_SMD:R_0603_1608Metric, F.Cu at (154.8, 92.4)
- added R54: 200Ω/0.5W, Resistor_SMD:R_0805_2012Metric, F.Cu at (194.5, 92.4)
- added R54: 200Ω/0.5W, Resistor_SMD:R_0805_2012Metric, F.Cu at (151.0, 92.4)
- added R54: 200Ω/0.5W, Resistor_SMD:R_0805_2012Metric, F.Cu at (129.3, 92.4)
- added R54: 200Ω/0.5W, Resistor_SMD:R_0805_2012Metric, F.Cu at (140.1, 92.4)
- added R54: 200Ω/0.5W, Resistor_SMD:R_0805_2012Metric, F.Cu at (161.9, 92.4)
- added R54: 200Ω/0.5W, Resistor_SMD:R_0805_2012Metric, F.Cu at (183.6, 92.4)
- added R54: 200Ω/0.5W, Resistor_SMD:R_0805_2012Metric, F.Cu at (172.8, 92.4)
- added R55: 120Ω/0.5W, Resistor_SMD:R_0805_2012Metric, F.Cu at (140.1, 96.2)
- added R55: 120Ω/0.5W, Resistor_SMD:R_0805_2012Metric, F.Cu at (129.3, 96.2)
- added R55: 120Ω/0.5W, Resistor_SMD:R_0805_2012Metric, F.Cu at (161.9, 96.2)
- added R55: 120Ω/0.5W, Resistor_SMD:R_0805_2012Metric, F.Cu at (194.5, 96.2)
- added R55: 120Ω/0.5W, Resistor_SMD:R_0805_2012Metric, F.Cu at (183.6, 96.2)
- added R55: 120Ω/0.5W, Resistor_SMD:R_0805_2012Metric, F.Cu at (172.8, 96.2)
- added R55: 120Ω/0.5W, Resistor_SMD:R_0805_2012Metric, F.Cu at (151.0, 96.2)
- added R56: 100Ω/0.5W, Resistor_SMD:R_0805_2012Metric, F.Cu at (151.0, 100.0)
- added R56: 100Ω/0.5W, Resistor_SMD:R_0805_2012Metric, F.Cu at (183.6, 100.0)
- added R56: 100Ω/0.5W, Resistor_SMD:R_0805_2012Metric, F.Cu at (140.1, 100.0)
- added R56: 100Ω/0.5W, Resistor_SMD:R_0805_2012Metric, F.Cu at (172.8, 100.0)
- added R56: 100Ω/0.5W, Resistor_SMD:R_0805_2012Metric, F.Cu at (161.9, 100.0)
- added R56: 100Ω/0.5W, Resistor_SMD:R_0805_2012Metric, F.Cu at (129.3, 100.0)
- added R56: 100Ω/0.5W, Resistor_SMD:R_0805_2012Metric, F.Cu at (194.5, 100.0)
- added R57: 62Ω/0.5W, Resistor_SMD:R_0805_2012Metric, F.Cu at (165.7, 96.2)
- added R57: 62Ω/0.5W, Resistor_SMD:R_0805_2012Metric, F.Cu at (144.0, 96.2)
- added R57: 62Ω/0.5W, Resistor_SMD:R_0805_2012Metric, F.Cu at (176.6, 96.2)
- added R57: 62Ω/0.5W, Resistor_SMD:R_0805_2012Metric, F.Cu at (187.4, 96.2)
- added R57: 62Ω/0.5W, Resistor_SMD:R_0805_2012Metric, F.Cu at (133.1, 96.2)
- added R57: 62Ω/0.5W, Resistor_SMD:R_0805_2012Metric, F.Cu at (198.3, 96.2)
- added R57: 62Ω/0.5W, Resistor_SMD:R_0805_2012Metric, F.Cu at (154.8, 96.2)
- added R58: 33Ω/0.5W, Resistor_SMD:R_0805_2012Metric, F.Cu at (176.6, 100.0)
- added R58: 33Ω/0.5W, Resistor_SMD:R_0805_2012Metric, F.Cu at (154.8, 100.0)
- added R58: 33Ω/0.5W, Resistor_SMD:R_0805_2012Metric, F.Cu at (144.0, 100.0)
- added R58: 33Ω/0.5W, Resistor_SMD:R_0805_2012Metric, F.Cu at (198.3, 100.0)
- added R58: 33Ω/0.5W, Resistor_SMD:R_0805_2012Metric, F.Cu at (187.4, 100.0)
- added R58: 33Ω/0.5W, Resistor_SMD:R_0805_2012Metric, F.Cu at (133.1, 100.0)
- added R58: 33Ω/0.5W, Resistor_SMD:R_0805_2012Metric, F.Cu at (165.7, 100.0)
- added S10: SS-10-15SPE, mylife-footprints:RS PRO SS-10-15SPE, F.Cu at (141.4, 107.4)
- added S11: SS-10-15SPE, mylife-footprints:RS PRO SS-10-15SPE, F.Cu at (152.3, 107.4)
- added S12: SS-10-15SPE, mylife-footprints:RS PRO SS-10-15SPE, F.Cu at (163.2, 107.4)
- added S13: SS-10-15SPE, mylife-footprints:RS PRO SS-10-15SPE, F.Cu at (174.0, 107.4)
- added S14: SS-10-15SPE, mylife-footprints:RS PRO SS-10-15SPE, F.Cu at (184.8, 107.4)
- added S15: SS-10-15SPE, mylife-footprints:RS PRO SS-10-15SPE, F.Cu at (195.7, 107.4)
- added S9: SS-10-15SPE, mylife-footprints:RS PRO SS-10-15SPE, F.Cu at (130.5, 107.4)
Routing:
- net Net-(J12-Pad1): track 13.7 -> 238.4 mm
- net Net-(R54-Pad2): track 0.00 -> 163.7 mm
- net Net-(R57-Pad2): track 0.00 -> 128.7 mm
- net /CT Sensor 1/ZERO: track 377.8 -> 488.7 mm
- net Net-(R55-Pad2): track 0.00 -> 89.6 mm
- net Net-(R58-Pad2): track 0.25 -> 74.1 mm
- net Net-(R56-Pad2): track 0.22 -> 34.4 mm

Commit message: wip pcb naming
Parts:
- removed the J13 at (136.3, 152.7)
- removed the J14 at (147.1, 152.6)
- removed the J15 at (157.9, 152.6)
- removed the J16 at (168.7, 152.6)
- removed the J17 at (179.5, 152.6)
- removed the J18 at (190.3, 152.6)
- removed the J19 at (201.2, 152.6)
- removed the R100 at (202.3, 136.2)
- removed the R59 at (137.3, 128.5)
- removed the R60 at (133.5, 128.5)
- removed the R61 at (133.5, 132.3)
- removed the R62 at (133.5, 136.1)
- removed the R63 at (137.3, 132.3)
- removed the R64 at (137.3, 136.1)
- removed the R65 at (148.0, 128.4)
- removed the R66 at (144.2, 128.4)
- removed the R67 at (144.2, 132.3)
- removed the R68 at (144.2, 136.1)
- removed the R69 at (148.0, 132.3)
- removed the R70 at (148.0, 136.1)
- removed the R71 at (158.9, 128.5)
- removed the R72 at (155.1, 128.5)
- removed the R73 at (155.1, 132.3)
- removed the R74 at (155.1, 136.1)
- removed the R75 at (158.9, 132.3)
- removed the R76 at (158.9, 136.1)
- removed the R77 at (169.7, 128.5)
- removed the R78 at (165.9, 128.5)
- removed the R79 at (165.9, 132.4)
- removed the R80 at (165.9, 136.2)
- removed the R81 at (169.7, 132.4)
- removed the R82 at (169.7, 136.2)
- removed the R83 at (180.6, 128.5)
- removed the R84 at (176.8, 128.5)
- removed the R85 at (176.8, 132.4)
- removed the R86 at (176.8, 136.2)
- removed the R87 at (180.6, 132.4)
- removed the R88 at (180.6, 136.2)
- removed the R89 at (191.4, 128.5)
- removed the R90 at (187.6, 128.5)
- removed the R91 at (187.6, 132.4)
- removed the R92 at (187.6, 136.2)
- removed the R93 at (191.4, 132.4)
- removed the R94 at (191.4, 136.2)
- removed the R95 at (202.3, 128.6)
- removed the R96 at (198.5, 128.6)
- removed the R97 at (198.5, 132.4)
- removed the R98 at (198.5, 136.2)
- removed the R99 at (202.3, 132.4)
- removed the S10 at (145.5, 143.5)
- removed the S11 at (156.3, 143.5)
- removed the S12 at (167.1, 143.5)
- removed the S13 at (178.0, 143.5)
- removed the S14 at (188.8, 143.6)
- removed the S15 at (199.7, 143.6)
- removed the S9 at (134.7, 143.5)
- renumbered R58 to R100, R53 to R59, R54 to R60, R55 to R61, R56 to R62, R57 to R63, R58 to R64, R53 to R65, R54 to R66, R55 to R67, R56 to R68, R57 to R69, R58 to R70, R53 to R71, R54 to R72, R55 to R73, R56 to R74, R57 to R75, R58 to R76, R53 to R77, R54 to R78, R55 to R79, R56 to R80, R57 to R81, R58 to R82, R53 to R83, R54 to R84, R55 to R85, R56 to R86, R57 to R87, R58 to R88, R53 to R89, R54 to R90, R55 to R91, R56 to R92, R57 to R93, R58 to R94, R53 to R95, R54 to R96, R55 to R97, R56 to R98, R57 to R99
Connections:
- J13 pad 1: Net-(J12-Pad1) -> Net-(J13-Pad1)
- J14 pad 1: Net-(J12-Pad1) -> Net-(J14-Pad1)
- J15 pad 1: Net-(J12-Pad1) -> Net-(J15-Pad1)
- J16 pad 1: Net-(J12-Pad1) -> Net-(J16-Pad1)
- J17 pad 1: Net-(J12-Pad1) -> Net-(J17-Pad1)
- J18 pad 1: Net-(J12-Pad1) -> Net-(J18-Pad1)
- J19 pad 1: Net-(J12-Pad1) -> Net-(J19-Pad1)
- R100 pad 1: Net-(J12-Pad1) -> Net-(J19-Pad1)
- R100 pad 2: Net-(R58-Pad2) -> Net-(R100-Pad2)
- R59 pad 1: /CT8 -> /CT9
- R59 pad 2: Net-(J12-Pad1) -> Net-(J13-Pad1)
- R60 pad 1: Net-(J12-Pad1) -> Net-(J13-Pad1)
- R60 pad 2: Net-(R54-Pad2) -> Net-(R60-Pad2)
- R61 pad 1: Net-(J12-Pad1) -> Net-(J13-Pad1)
- R61 pad 2: Net-(R55-Pad2) -> Net-(R61-Pad2)
- R62 pad 1: Net-(J12-Pad1) -> Net-(J13-Pad1)
- R62 pad 2: Net-(R56-Pad2) -> Net-(R62-Pad2)
- R63 pad 1: Net-(J12-Pad1) -> Net-(J13-Pad1)
- R63 pad 2: Net-(R57-Pad2) -> Net-(R63-Pad2)
- R64 pad 1: Net-(J12-Pad1) -> Net-(J13-Pad1)
- R64 pad 2: Net-(R58-Pad2) -> Net-(R64-Pad2)
- R65 pad 1: /CT8 -> /CT10
- R65 pad 2: Net-(J12-Pad1) -> Net-(J14-Pad1)
- R66 pad 1: Net-(J12-Pad1) -> Net-(J14-Pad1)
- R66 pad 2: Net-(R54-Pad2) -> Net-(R66-Pad2)
- R67 pad 1: Net-(J12-Pad1) -> Net-(J14-Pad1)
- R67 pad 2: Net-(R55-Pad2) -> Net-(R67-Pad2)
- R68 pad 1: Net-(J12-Pad1) -> Net-(J14-Pad1)
- R68 pad 2: Net-(R56-Pad2) -> Net-(R68-Pad2)
- R69 pad 1: Net-(J12-Pad1) -> Net-(J14-Pad1)
- R69 pad 2: Net-(R57-Pad2) -> Net-(R69-Pad2)
- R70 pad 1: Net-(J12-Pad1) -> Net-(J14-Pad1)
- R70 pad 2: Net-(R58-Pad2) -> Net-(R70-Pad2)
- R71 pad 1: /CT8 -> /CT11
- R71 pad 2: Net-(J12-Pad1) -> Net-(J15-Pad1)
- R72 pad 1: Net-(J12-Pad1) -> Net-(J15-Pad1)
- R72 pad 2: Net-(R54-Pad2) -> Net-(R72-Pad2)
- R73 pad 1: Net-(J12-Pad1) -> Net-(J15-Pad1)
- R73 pad 2: Net-(R55-Pad2) -> Net-(R73-Pad2)
- R74 pad 1: Net-(J12-Pad1) -> Net-(J15-Pad1)
- R74 pad 2: Net-(R56-Pad2) -> Net-(R74-Pad2)
- R75 pad 1: Net-(J12-Pad1) -> Net-(J15-Pad1)
- R75 pad 2: Net-(R57-Pad2) -> Net-(R75-Pad2)
- R76 pad 1: Net-(J12-Pad1) -> Net-(J15-Pad1)
- R76 pad 2: Net-(R58-Pad2) -> Net-(R76-Pad2)
- R77 pad 1: /CT8 -> /CT12
- R77 pad 2: Net-(J12-Pad1) -> Net-(J16-Pad1)
- R78 pad 1: Net-(J12-Pad1) -> Net-(J16-Pad1)
- R78 pad 2: Net-(R54-Pad2) -> Net-(R78-Pad2)
- R79 pad 1: Net-(J12-Pad1) -> Net-(J16-Pad1)
- R79 pad 2: Net-(R55-Pad2) -> Net-(R79-Pad2)
- R80 pad 1: Net-(J12-Pad1) -> Net-(J16-Pad1)
- R80 pad 2: Net-(R56-Pad2) -> Net-(R80-Pad2)
- R81 pad 1: Net-(J12-Pad1) -> Net-(J16-Pad1)
- R81 pad 2: Net-(R57-Pad2) -> Net-(R81-Pad2)
- R82 pad 1: Net-(J12-Pad1) -> Net-(J16-Pad1)
- R82 pad 2: Net-(R58-Pad2) -> Net-(R82-Pad2)
- R83 pad 1: /CT8 -> /CT13
- R83 pad 2: Net-(J12-Pad1) -> Net-(J17-Pad1)
- R84 pad 1: Net-(J12-Pad1) -> Net-(J17-Pad1)
- R84 pad 2: Net-(R54-Pad2) -> Net-(R84-Pad2)
- R85 pad 1: Net-(J12-Pad1) -> Net-(J17-Pad1)
- R85 pad 2: Net-(R55-Pad2) -> Net-(R85-Pad2)
- R86 pad 1: Net-(J12-Pad1) -> Net-(J17-Pad1)
- R86 pad 2: Net-(R56-Pad2) -> Net-(R86-Pad2)
- R87 pad 1: Net-(J12-Pad1) -> Net-(J17-Pad1)
- R87 pad 2: Net-(R57-Pad2) -> Net-(R87-Pad2)
- R88 pad 1: Net-(J12-Pad1) -> Net-(J17-Pad1)
- R88 pad 2: Net-(R58-Pad2) -> Net-(R88-Pad2)
- R89 pad 1: /CT8 -> /CT14
- R89 pad 2: Net-(J12-Pad1) -> Net-(J18-Pad1)
- R90 pad 1: Net-(J12-Pad1) -> Net-(J18-Pad1)
- R90 pad 2: Net-(R54-Pad2) -> Net-(R90-Pad2)
- R91 pad 1: Net-(J12-Pad1) -> Net-(J18-Pad1)
- R91 pad 2: Net-(R55-Pad2) -> Net-(R91-Pad2)
- R92 pad 1: Net-(J12-Pad1) -> Net-(J18-Pad1)
- R92 pad 2: Net-(R56-Pad2) -> Net-(R92-Pad2)
- R93 pad 1: Net-(J12-Pad1) -> Net-(J18-Pad1)
- R93 pad 2: Net-(R57-Pad2) -> Net-(R93-Pad2)
- R94 pad 1: Net-(J12-Pad1) -> Net-(J18-Pad1)
- R94 pad 2: Net-(R58-Pad2) -> Net-(R94-Pad2)
- R95 pad 1: /CT8 -> /CT15
- R95 pad 2: Net-(J12-Pad1) -> Net-(J19-Pad1)
- R96 pad 1: Net-(J12-Pad1) -> Net-(J19-Pad1)
- R96 pad 2: Net-(R54-Pad2) -> Net-(R96-Pad2)
- R97 pad 1: Net-(J12-Pad1) -> Net-(J19-Pad1)
- R97 pad 2: Net-(R55-Pad2) -> Net-(R97-Pad2)
- R98 pad 1: Net-(J12-Pad1) -> Net-(J19-Pad1)
- R98 pad 2: Net-(R56-Pad2) -> Net-(R98-Pad2)
- R99 pad 1: Net-(J12-Pad1) -> Net-(J19-Pad1)
- R99 pad 2: Net-(R57-Pad2) -> Net-(R99-Pad2)
- S10 pad 1: Net-(R56-Pad2) -> Net-(R68-Pad2)
- S10 pad 2: Net-(R55-Pad2) -> Net-(R67-Pad2)
- S10 pad 4: Net-(R54-Pad2) -> Net-(R66-Pad2)
- S10 pad 5: unconnected-(S8-Pad5) -> unconnected-(S10-Pad5)
- S10 pad 7: Net-(R58-Pad2) -> Net-(R70-Pad2)
- S10 pad 8: Net-(R57-Pad2) -> Net-(R69-Pad2)
- S11 pad 1: Net-(R56-Pad2) -> Net-(R74-Pad2)
- S11 pad 2: Net-(R55-Pad2) -> Net-(R73-Pad2)
- S11 pad 4: Net-(R54-Pad2) -> Net-(R72-Pad2)
- S11 pad 5: unconnected-(S8-Pad5) -> unconnected-(S11-Pad5)
- S11 pad 7: Net-(R58-Pad2) -> Net-(R76-Pad2)
- S11 pad 8: Net-(R57-Pad2) -> Net-(R75-Pad2)
- S12 pad 1: Net-(R56-Pad2) -> Net-(R80-Pad2)
- S12 pad 2: Net-(R55-Pad2) -> Net-(R79-Pad2)
- S12 pad 4: Net-(R54-Pad2) -> Net-(R78-Pad2)
- S12 pad 5: unconnected-(S8-Pad5) -> unconnected-(S12-Pad5)
- S12 pad 7: Net-(R58-Pad2) -> Net-(R82-Pad2)
- S12 pad 8: Net-(R57-Pad2) -> Net-(R81-Pad2)
- S13 pad 1: Net-(R56-Pad2) -> Net-(R86-Pad2)
- S13 pad 2: Net-(R55-Pad2) -> Net-(R85-Pad2)
- S13 pad 4: Net-(R54-Pad2) -> Net-(R84-Pad2)
- S13 pad 5: unconnected-(S8-Pad5) -> unconnected-(S13-Pad5)
- S13 pad 7: Net-(R58-Pad2) -> Net-(R88-Pad2)
- S13 pad 8: Net-(R57-Pad2) -> Net-(R87-Pad2)
- S14 pad 1: Net-(R56-Pad2) -> Net-(R92-Pad2)
- S14 pad 2: Net-(R55-Pad2) -> Net-(R91-Pad2)
- S14 pad 4: Net-(R54-Pad2) -> Net-(R90-Pad2)
- S14 pad 5: unconnected-(S8-Pad5) -> unconnected-(S14-Pad5)
- S14 pad 7: Net-(R58-Pad2) -> Net-(R94-Pad2)
- S14 pad 8: Net-(R57-Pad2) -> Net-(R93-Pad2)
- S15 pad 1: Net-(R56-Pad2) -> Net-(R98-Pad2)
- S15 pad 2: Net-(R55-Pad2) -> Net-(R97-Pad2)
- S15 pad 4: Net-(R54-Pad2) -> Net-(R96-Pad2)
- S15 pad 5: unconnected-(S8-Pad5) -> unconnected-(S15-Pad5)
- S15 pad 7: Net-(R58-Pad2) -> Net-(R100-Pad2)
- S15 pad 8: Net-(R57-Pad2) -> Net-(R99-Pad2)
- S9 pad 1: Net-(R56-Pad2) -> Net-(R62-Pad2)
- S9 pad 2: Net-(R55-Pad2) -> Net-(R61-Pad2)
- S9 pad 4: Net-(R54-Pad2) -> Net-(R60-Pad2)
- S9 pad 5: unconnected-(S8-Pad5) -> unconnected-(S9-Pad5)
- S9 pad 7: Net-(R58-Pad2) -> Net-(R64-Pad2)
- S9 pad 8: Net-(R57-Pad2) -> Net-(R63-Pad2)
Routing:
- net Net-(J12-Pad1): track 238.4 -> 29.8 mm
- net /CT Sensor 1/ZERO: track 488.7 -> 287.4 mm
- net Net-(R54-Pad2): track 163.7 -> 20.5 mm
- net Net-(R57-Pad2): track 128.7 -> 16.1 mm
- net Net-(R55-Pad2): track 89.6 -> 11.2 mm
- net Net-(R58-Pad2): track 74.1 -> 9.26 mm
- net Net-(R56-Pad2): track 34.4 -> 4.30 mm
- net Net-(R96-Pad2): track 0.00 -> 20.5 mm
- net Net-(R90-Pad2): track 0.00 -> 20.5 mm
- net Net-(R98-Pad2): track 24.1 -> 4.30 mm
- net Net-(R92-Pad2): track 24.1 -> 4.30 mm
- net Net-(R87-Pad2): track 0.00 -> 16.1 mm
- net Net-(R61-Pad2): track 0.00 -> 11.2 mm
- net Net-(R67-Pad2): track 0.00 -> 11.2 mm
- net Net-(R85-Pad2): track 0.00 -> 11.2 mm
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
Commit message: fix pcb
Routing:
- net /CT Sensor 1/ZERO: track 287.4 -> 408.2 mm, vias 0 -> 1
- net /CT15: track 12.9 -> 35.9 mm
- net /CT1: track 18.1 -> 34.6 mm
- net /CT7: track 18.3 -> 32.3 mm
- net /CT13: track 2.61 -> 16.6 mm
- net /CT8: track 31.1 -> 44.9 mm
- net /CT12: track 0.00 -> 13.5 mm
- net /CT11: track 4.06 -> 17.5 mm
- net /CT9: track 22.9 -> 36.1 mm
- net /CT6: track 11.4 -> 22.6 mm
- net /CT14: track 16.0 -> 26.5 mm
- net /CT10: track 16.8 -> 26.9 mm
- net /CT2: track 15.3 -> 24.9 mm
- net /CT3: track 6.83 -> 16.3 mm
- net /CT4: track 8.38 -> 16.6 mm
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