File: epanel-energy-monitor/v1.1/ct_sensor.kicad_sch (KiCad schematic)
At the start: 8 parts, among them J5 Screw_Terminal_01x02

Commit message: update PCB R200 to 220
Parts:
- R12: value 200Ω/0.5W -> 220Ω/0.5W; LCSC C560506 -> C966130
Changed lines of the file:
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@@
       (effects (font (size 1.27 1.27)))
     )
-    (property "Value" "200Ω/0.5W" (at 187.96 58.42 90)
+    (property "Value" "220Ω/0.5W" (at 187.96 58.42 90)
       (effects (font (size 1.27 1.27)))
     )
@@
       (effects (font (size 1.27 1.27)) hide)
     )
-    (property "Datasheet" "https://datasheet.lcsc.com/lcsc/2007231205_UNI-ROYAL-Uniroyal-Elec-AS05W2J0201T5E_C560506.pdf" (at 187.96 60.96 0)
+    (property "Datasheet" "https://datasheet.lcsc.com/lcsc/2012181744_UNI-ROYAL-Uniroyal-Elec-AS05W2J0221T5E_C966130.pdf" (at 187.96 60.96 0)
       (effects (font (size 1.27 1.27)) hide)
     )
-    (property "LCSC" "C560506" (at 187.96 60.96 0)
+    (property "LCSC" "C966130" (at 187.96 60.96 0)
       (effects (font (size 1.27 1.27)) hide)
     )
