File: rgb-spot-10w/v1/rgb-spot-10w.kicad_sch (KiCad schematic)
At the start: 5 parts, among them J1 Screw_Terminal_01x04

Commit message: pcb OK
Connections:
- net at R1.1: now also J1.1 (Pin_1); no longer J1.2 (Pin_2)
- net at D1.1 (A): now also J1.4 (Pin_4); no longer J1.1 (Pin_1)
- net at R2.1: now also J1.2 (Pin_2); no longer J1.3 (Pin_3)
- net at R3.1: now also J1.3 (Pin_3); no longer J1.4 (Pin_4)
Other:
- moved on the sheet: J1
