File: rgb-garden-box/v1/rgb-garden-box.kicad_pcb (KiCad board)
At the start: 2 copper layers, 230 x 150 mm, 74 parts, among them J1 Conn_01x03_Male, J10 Screw_Terminal_01x02, J11 Screw_Terminal_01x04, J12 Screw_Terminal_01x04, J13 Screw_Terminal_01x06, J2 Conn_01x04_Male, J3 USB_A, J4 Conn_01x03_Male, J5 Conn_01x03_Male, J6 Conn_01x03_Male, J7 Conn_01x03_Male, J8 Conn_01x03_Male, J9 Conn_01x03_Male, K1 G6DN-1A-L_DC5, K2 G6DN-1A-L_DC5, K3 G6DN-1A-L_DC5, K4 G6DN-1A-L_DC5, K5 G6DN-1A-L_DC5, K6 G6DN-1A-L_DC5, K7 G6DN-1A-L_DC5, Q1 2N3904, Q2 2N3904, Q3 2N3904, Q4 2N3904, Q5 2N3904, Q6 2N3904, Q7 2N3904, T1 Transformer_1P_2S, U1 ESP32-POE

Commit message: add footprints
Parts:
- removed D10, D12, D14, D6, D8: 1N4148, Diode_SMD:D_SOD-123
- removed D11, D13, D5, D7, D9: LED, Diode_SMD:D_0805_2012Metric
- removed J10: Screw_Terminal_01x02, TerminalBlock:TerminalBlock_bornier-2_P5.08mm
- removed J11, J12: Screw_Terminal_01x04, TerminalBlock:TerminalBlock_bornier-4_P5.08mm
- removed J13: Screw_Terminal_01x06, TerminalBlock:TerminalBlock_bornier-6_P5.08mm
- removed J6, J7, J8, J9: Conn_01x03_Male, Connector_PinHeader_2.54mm:PinHeader_1x03_P2.54mm_Vertical
- removed K3, K4, K5, K6, K7: G6DN-1A-L_DC5, rs-online:G6DN-1A-L
- removed R14, R16, R17, R19, R20, R22: 1KΩ, Resistor_SMD:R_0402_1005Metric
- removed R15, R18, R21: 10KΩ, Resistor_SMD:R_0402_1005Metric
- removed the REF** at (143.6, 84.7)
- removed the REF** at (49.6, 84.7)
- removed T1: Transformer_1P_2S, mylife-footprints:VCM36212
- added PS2: RS PRO 24V 833mA (20W), mylife-footprints:RS PRO Alim 5V 2A, F.Cu at (-110.7, 46.7)
- added PS4: Alim RS PRO 5V 1A, Converter_ACDC:Converter_ACDC_MeanWell_IRM-03-xx_THT, F.Cu at (-111.1, 75.6)
- added Q8: IRLZ44N, Package_TO_SOT_SMD:ATPAK-2, F.Cu at (-82.9, 115.8)
- J3: value USB_A -> Screw_Terminal_01x02; footprint rs-online:875200010BLF -> TerminalBlock:TerminalBlock_bornier-2_P5.08mm
- J4, J5: value Conn_01x03_Male -> Screw_Terminal_01x04; footprint Connector_PinHeader_2.54mm:PinHeader_1x03_P2.54mm_Vertical -> TerminalBlock:TerminalBlock_bornier-4_P5.08mm
- PS1: value RS PRO 5V 2A -> Mean Well 12V 2.5A (30W); footprint mylife-footprints:RS PRO 5V 2A -> mylife-footprints:IRM-30-12
- Q2, Q3, Q5, Q6, Q7: value 2N3904 -> IRLZ44N; footprint jlcpcb:SOT-23-3_L2.9-W1.3-P1.90-LS2.4-TR -> Package_TO_SOT_SMD:ATPAK-2
- R11, R13, R5, R8: value 1KΩ -> 10KΩ
- moved K1 269.1 mm to (-95.1, 112.0)
- moved K2 256.7 mm to (-95.1, 118.2)
- moved J4 244.9 mm to (-74.3, 76.0), turned to 0 degrees
- moved J5 244.7 mm to (-74.3, 85.1), turned to 0 degrees
- moved D1 240.1 mm to (-75.3, 113.3), turned to 0 degrees
- moved J1 239.0 mm to (-70.6, 101.9)
- moved R4 238.1 mm to (-76.1, 96.6)
- moved R1 236.6 mm to (-76.1, 90.6), turned to 0 degrees
- moved R2 235.2 mm to (-76.1, 92.6)
- moved J2 233.6 mm to (-75.3, 101.9)
- moved R3 232.7 mm to (-76.1, 94.6), turned to 0 degrees
- moved D2 227.3 mm to (-60.6, 101.2), turned to 0 degrees
- moved Q1 224.3 mm to (-65.9, 101.7), turned to 0 degrees
- moved U1 219.3 mm to (-129.9, 86.9), turned to 0 degrees
- moved Q5 215.4 mm to (-82.9, 91.6), turned to 0 degrees
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Connections:
- net /relay transfo/Logic input renamed Net-(U1-GPIO33)
- D3 pad 1: Net-(D3-Pad1) -> Net-(D3-K)
- D3 pad 2: Net-(D3-Pad2) -> Net-(D3-A)
- D4 pad 2: Net-(D3-Pad1) -> Net-(D3-K)
- J3 pad 1: +5V -> Net-(J3-Pin_1)
- J3 pad 2: unconnected-(J3-Pad2) -> Net-(J3-Pin_2)
- J4 pad 1: /relay transfo/Output 1 -> +12V
- J4 pad 2: /relay 1/Output 1 -> Net-(J4-Pin_2)
- J4 pad 3: Net-(J4-Pad3) -> Net-(J4-Pin_3)
- J5 pad 1: /relay transfo/Output 1 -> +24V
- J5 pad 2: /relay 2/Output 1 -> Net-(J5-Pin_2)
- J5 pad 3: Net-(J4-Pad3) -> Net-(J5-Pin_3)
- K1 pad 5: /relay transfo/Output 2 -> Net-(J3-Pin_1)
- K1 pad 8: /relay transfo/Output 1 -> Net-(PS1-AC/L)
- K2 pad 2: Net-(D3-Pad1) -> Net-(D3-K)
- K2 pad 5: /relay 1/Output 2 -> Net-(J3-Pin_1)
- K2 pad 8: /relay 1/Output 1 -> Net-(PS2-AC/L)
- PS1 pad 1: Net-(J10-Pad2) -> Net-(PS1-AC/L)
- PS1 pad 2: /relay transfo/Output 1 -> Net-(J3-Pin_2)
- PS1 pad 3: GND -> +12V
- PS1 pad 4: +5V -> GND
- Q2 pad 1: GND -> Net-(Q2-G)
- Q2 pad 2: Net-(Q2-Pad2) -> Net-(J5-Pin_2)
- Q2 pad 3: Net-(D3-Pad1) -> GND
- Q3 pad 1: GND -> Net-(Q3-G)
- Q3 pad 2: Net-(Q3-Pad2) -> Net-(J5-Pin_3)
- Q3 pad 3: Net-(D5-Pad1) -> GND
- Q4 pad 2: Net-(Q4-Pad2) -> Net-(Q4-B)
- Q4 pad 3: Net-(D7-Pad1) -> Net-(D3-K)
- Q5 pad 1: GND -> Net-(Q5-G)
- Q5 pad 2: Net-(Q5-Pad2) -> Net-(J5-Pin_4)
- Q5 pad 3: Net-(D10-Pad2) -> GND
- Q6 pad 1: GND -> Net-(Q6-G)
- Q6 pad 2: Net-(Q6-Pad2) -> Net-(J4-Pin_2)
- Q6 pad 3: Net-(D11-Pad1) -> GND
- Q7 pad 1: GND -> Net-(Q7-G)
- Q7 pad 2: Net-(Q7-Pad2) -> Net-(J4-Pin_3)
- Q7 pad 3: Net-(D13-Pad1) -> GND
- R10 pad 2: Net-(D5-Pad2) -> Net-(D3-A)
- R11 pad 1: Net-(Q4-Pad2) -> Net-(Q6-G)
- R11 pad 2: /R3 -> GND
- R12 pad 1: Net-(Q4-Pad2) -> Net-(Q7-G)
- R13 pad 1: +5V -> Net-(Q8-G)
- R13 pad 2: Net-(D7-Pad2) -> GND
- R5 pad 1: Net-(Q2-Pad2) -> Net-(Q2-G)
- R5 pad 2: /R1 -> GND
- R6 pad 1: Net-(Q2-Pad2) -> Net-(Q3-G)
- R7 pad 1: +5V -> Net-(Q4-B)
- R7 pad 2: Net-(D3-Pad2) -> Net-(U1-GPIO32)
- R8 pad 1: Net-(Q3-Pad2) -> Net-(Q4-B)
- R8 pad 2: /R2 -> GND
- R9 pad 1: Net-(Q3-Pad2) -> Net-(Q5-G)
- U1 pad 10: /R6 -> Net-(Q5-G)
- U1 pad 12: unconnected-(U1-Pad12) -> Net-(Q6-G)
- U1 pad 13: unconnected-(U1-Pad13) -> Net-(Q7-G)
- U1 pad 14: unconnected-(U1-Pad14) -> Net-(Q8-G)
- U1 pad 15: unconnected-(U1-Pad15) -> Net-(U1-GPIO32)
- U1 pad 5: /R1 -> unconnected-(U1-GPIO0-Pad5)
- U1 pad 6: /R2 -> unconnected-(U1-GPIO1-Pad6)
- U1 pad 7: /R3 -> unconnected-(U1-GPIO2-Pad7)
- U1 pad 8: /R4 -> Net-(Q2-G)
- U1 pad 9: /R5 -> Net-(Q3-G)
Routing:
- net Net-(J10-Pad2): track 392.0 -> 0.00 mm, vias 2 -> 0
- net +5V: track 361.6 -> 0.00 mm
- net GND: track 351.8 -> 0.00 mm, vias 1 -> 0
- net /relay transfo/Output 1: track 261.2 -> 0.00 mm
- net Net-(J4-Pad3): track 134.4 -> 0.00 mm
- net /R6: track 128.0 -> 0.00 mm, vias 2 -> 0
- net Net-(U1-GPIO33): track 127.7 -> 0.00 mm
- net /R5: track 122.9 -> 0.00 mm, vias 2 -> 0
- net /R4: track 117.9 -> 0.00 mm, vias 2 -> 0
- net /R3: track 112.8 -> 0.00 mm, vias 2 -> 0
- net /R2: track 107.7 -> 0.00 mm, vias 2 -> 0
- net +3V3: track 103.1 -> 0.00 mm
- net /R1: track 102.6 -> 0.00 mm, vias 2 -> 0
- net Net-(J2-Pin_4): track 92.8 -> 0.00 mm
- net Net-(J1-Pin_3): track 92.0 -> 0.00 mm
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Other:
- board text removed: "220V <- -> 24V"
- board text removed: "220V IN"
- board text removed: "220V OUT"
- board text removed: "24V~ OUT"
- board text removed: "3V3"
- board text removed: "5V"
- board text removed: "A0"
- board text removed: "DS18B20"
- board text removed: "GND"
- board text removed: "IN"
- board text removed: "L"
- board text removed: "N"
- board text removed: "OUT 1"
- board text removed: "OUT 2"
- board text removed: "OUT 3"
- board text removed: "OUT 4"
- board text removed: "OUT 5"
- board text removed: "OUT 6"
- board text removed: "SEN0308"
- board text removed: "SWITCH"

Commit message: enclosing box layout
Parts:
- moved REF** 53.1 mm to (91.6, 134.7)
- moved REF** 52.6 mm to (91.6, 44.7)
- moved REF** 46.8 mm to (84.0, 89.7)
- moved REF** 41.6 mm to (212.3, 134.7)
- moved REF** 41.0 mm to (212.3, 44.7)
- moved REF** 33.2 mm to (220.0, 89.7)
Other:
- board size 230 x 150 mm -> 149.3 x 102 mm
Changed lines of the file:
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@@
     )
     (fp_line (start -0.649987 -1.459995) (end -0.649987 -0.800102)
-      (stroke (width 0.254001) (type solid)) (layer "F.SilkS"))
+      (stroke (width 0.254) (type solid)) (layer "F.SilkS"))
     (fp_line (start -0.649987 -1.459995) (end 0.1651 -1.459995)
-      (stroke (width 0.254001) (type solid)) (layer "F.SilkS"))
+      (stroke (width 0.254) (type solid)) (layer "F.SilkS"))
     (fp_line (start -0.649987 -0.800102) (end -0.649987 -1.459995)
-      (stroke (width 0.254001) (type solid)) (layer "F.SilkS"))
+      (stroke (width 0.254) (type solid)) (layer "F.SilkS"))
     (fp_line (start -0.649987 -0.800102) (end -0.649987 -1.459995)
-      (stroke (width 0.254001) (type solid)) (layer "F.SilkS"))
+      (stroke (width 0.254) (type solid)) (layer "F.SilkS"))
     (fp_line (start -0.649987 1.459995) (end -0.649987 0.800102)
-      (stroke (width 0.254001) (type solid)) (layer "F.SilkS"))
+      (stroke (width 0.254) (type solid)) (layer "F.SilkS"))
     (fp_line (start 0.1651 1.459995) (end -0.649987 1.459995)
-      (stroke (width 0.254001) (type solid)) (layer "F.SilkS"))
+      (stroke (width 0.254) (type solid)) (layer "F.SilkS"))
     (fp_line (start 0.899924 0.299975) (end 0.899924 -0.299975)
       (stroke (width 0.2) (type solid)) (layer "F.SilkS"))
@@
       (stroke (width 0.059995) (type solid)) (fill none) (layer "F.SilkS"))
     (fp_circle (center 1.495809 -0.945136) (end 1.622809 -0.945136)
-      (stroke (width 0.254001) (type solid)) (fill none) (layer "F.Fab"))
+      (stroke (width 0.254) (type solid)) (fill none) (layer "F.Fab"))
     (pad "1" smd rect (at 1.249682 -0.949962 270) (size 0.7 1.250013) (layers "F.Cu" "F.Paste" "F.Mask")
       (net 4 "GND") (pinfunction "E") (pintype "passive"))
@@
   )
   (footprint "MountingHole:MountingHole_3.2mm_M3_Pad_Via" locked (layer "F.Cu")
-    (at 245.9 159.24)
+    (at 212.32 134.69)
     (descr "Mounting Hole 3.2mm, M3")
     (tags "mounting hole 3.2mm m3")
@@
   )
   (footprint "MountingHole:MountingHole_3.2mm_M3_Pad_Via" locked (layer "F.Cu")
-    (at 44.5 159.24)
+    (at 91.62 134.69)
     (descr "Mounting Hole 3.2mm, M3")
     (tags "mounting hole 3.2mm m3")
@@
   )
   (footprint "MountingHole:MountingHole_3.2mm_M3_Pad_Via" locked (layer "F.Cu")
-    (at 44.5 21.24)
+    (at 91.62 44.69)
     (descr "Mounting Hole 3.2mm, M3")
     (tags "mounting hole 3.2mm m3")
@@
   )
   (footprint "MountingHole:MountingHole_3.2mm_M3_Pad_Via" locked (layer "F.Cu")
-    (at 37.2 90.24)
+    (at 83.97 89.69)
     (descr "Mounting Hole 3.2mm, M3")
     (tags "mounting hole 3.2mm m3")
@@
   )
   (footprint "MountingHole:MountingHole_3.2mm_M3_Pad_Via" locked (layer "F.Cu")
-    (at 253.2 90.24)
+    (at 219.97 89.69)
     (descr "Mounting Hole 3.2mm, M3")
     (tags "mounting hole 3.2mm m3")
@@
     )
     (fp_line (start -0.649987 -1.459995) (end -0.649987 -0.800102)
-      (stroke (width 0.254001) (type solid)) (layer "F.SilkS"))
+      (stroke (width 0.254) (type solid)) (layer "F.SilkS"))
     (fp_line (start -0.649987 -1.459995) (end 0.1651 -1.459995)
-      (stroke (width 0.254001) (type solid)) (layer "F.SilkS"))
+      (stroke (width 0.254) (type solid)) (layer "F.SilkS"))
     (fp_line (start -0.649987 -0.800102) (end -0.649987 -1.459995)
-      (stroke (width 0.254001) (type solid)) (layer "F.SilkS"))
+      (stroke (width 0.254) (type solid)) (layer "F.SilkS"))
     (fp_line (start -0.649987 -0.800102) (end -0.649987 -1.459995)
-      (stroke (width 0.254001) (type solid)) (layer "F.SilkS"))
+      (stroke (width 0.254) (type solid)) (layer "F.SilkS"))
     (fp_line (start -0.649987 1.459995) (end -0.649987 0.800102)
-      (stroke (width 0.254001) (type solid)) (layer "F.SilkS"))
+      (stroke (width 0.254) (type solid)) (layer "F.SilkS"))
     (fp_line (start 0.1651 1.459995) (end -0.649987 1.459995)
-      (stroke (width 0.254001) (type solid)) (layer "F.SilkS"))
+      (stroke (width 0.254) (type solid)) (layer "F.SilkS"))
     (fp_line (start 0.899924 0.299975) (end 0.899924 -0.299975)
       (stroke (width 0.2) (type solid)) (layer "F.SilkS"))
@@
       (stroke (width 0.059995) (type solid)) (fill none) (layer "F.SilkS"))
     (fp_circle (center 1.495809 -0.945136) (end 1.622809 -0.945136)
-      (stroke (width 0.254001) (type solid)) (fill none) (layer "F.Fab"))
+      (stroke (width 0.254) (type solid)) (fill none) (layer "F.Fab"))
     (pad "1" smd rect (at 1.249682 -0.949962 270) (size 0.7 1.250013) (layers "F.Cu" "F.Paste" "F.Mask")
       (net 4 "GND") (pinfunction "E") (pintype "passive"))
@@
   )
   (footprint "MountingHole:MountingHole_3.2mm_M3_Pad_Via" locked (layer "F.Cu")
-    (at 245.9 21.24)
+    (at 212.32 44.69)
     (descr "Mounting Hole 3.2mm, M3")
     (tags "mounting hole 3.2mm m3")
@@
     )
   )
-  (gr_line locked (start 155.2 15.24) (end 251.2 15.24)
+  (gr_line locked (start 77.32 122.69) (end 86.32 122.69)
     (stroke (width 0.1) (type solid)) (layer "Edge.Cuts"))
-  (gr_line locked (start 30.2 147.24) (end 39.2 147.24)
+  (gr_line locked (start 217.62 140.69) (end 217.62 122.69)
     (stroke (width 0.1) (type solid)) (layer "Edge.Cuts"))
-  (gr_line locked (start 135.2 25.24) (end 155.2 25.24)
+  (gr_line locked (start 217.62 122.69) (end 226.62 122.69)
     (stroke (width 0.1) (type solid)) (layer "Edge.Cuts"))
-  (gr_line locked (start 251.2 165.24) (end 251.2 147.24)
+  (gr_line locked (start 226.62 56.69) (end 226.62 122.69)
     (stroke (width 0.1) (type solid)) (layer "Edge.Cuts"))
-  (gr_line locked (start 135.2 155.24) (end 155.2 155.24)
+  (gr_line locked (start 217.62 56.69) (end 217.62 38.69)
     (stroke (width 0.1) (type solid)) (layer "Edge.Cuts"))
-  (gr_line locked (start 251.2 147.24) (end 260.2 147.24)
+  (gr_line locked (start 86.32 140.69) (end 86.32 122.69)
     (stroke (width 0.1) (type solid)) (layer "Edge.Cuts"))
-  (gr_line locked (start 260.2 33.24) (end 260.2 147.24)
+  (gr_line locked (start 217.62 56.69) (end 226.62 56.69)
     (stroke (width 0.1) (type solid)) (layer "Edge.Cuts"))
-  (gr_line locked (start 155.2 15.24) (end 155.2 25.24)
+  (gr_line locked (start 217.62 140.69) (end 86.32 140.69)
     (stroke (width 0.1) (type solid)) (layer "Edge.Cuts"))
-  (gr_line locked (start 251.2 33.24) (end 251.2 15.24)
+  (gr_line locked (start 86.32 38.69) (end 217.62 38.69)
     (stroke (width 0.1) (type solid)) (layer "Edge.Cuts"))
-  (gr_line locked (start 155.2 155.24) (end 155.2 165.24)
+  (gr_line locked (start 77.32 122.69) (end 77.32 56.69)
     (stroke (width 0.1) (type solid)) (layer "Edge.Cuts"))
-  (gr_line locked (start 39.2 165.24) (end 39.2 147.24)
+  (gr_line locked (start 86.32 38.69) (end 86.32 56.69)
     (stroke (width 0.1) (type solid)) (layer "Edge.Cuts"))
-  (gr_line locked (start 251.2 33.24) (end 260.2 33.24)
-    (stroke (width 0.1) (type solid)) (layer "Edge.Cuts"))
-  (gr_line locked (start 135.2 165.24) (end 39.2 165.24)
-    (stroke (width 0.1) (type solid)) (layer "Edge.Cuts"))
-  (gr_line locked (start 39.2 15.24) (end 135.2 15.24)
-    (stroke (width 0.1) (type solid)) (layer "Edge.Cuts"))
-  (gr_line locked (start 251.2 165.24) (end 155.2 165.24)
-    (stroke (width 0.1) (type solid)) (layer "Edge.Cuts"))
-  (gr_line locked (start 135.2 15.24) (end 135.2 25.24)
-    (stroke (width 0.1) (type solid)) (layer "Edge.Cuts"))
-  (gr_line locked (start 30.2 147.24) (end 30.2 33.24)
-    (stroke (width 0.1) (type solid)) (layer "Edge.Cuts"))
-  (gr_line locked (start 135.2 155.24) (end 135.2 165.24)
-    (stroke (width 0.1) (type solid)) (layer "Edge.Cuts"))
-  (gr_line locked (start 39.2 15.24) (end 39.2 33.24)
-    (stroke (width 0.1) (type solid)) (layer "Edge.Cuts"))
-  (gr_line locked (start 30.2 33.24) (end 39.2 33.24)
+  (gr_line locked (start 77.32 56.69) (end 86.32 56.69)
     (stroke (width 0.1) (type solid)) (layer "Edge.Cuts"))
 )

Commit message: wip pcb placement
Parts:
- added J6: Screw_Terminal_01x04, TerminalBlock:TerminalBlock_bornier-4_P5.08mm, F.Cu at (214.0, 125.1)
- moved K1 321.1 mm to (221.6, 59.1), turned to 90 degrees
- moved K2 317.0 mm to (221.6, 102.9), turned to 90 degrees
- moved D3 292.5 mm to (217.1, 111.4)
- moved D1 291.7 mm to (211.5, 60.3)
- moved R8 284.9 mm to (211.4, 105.7)
- moved R7 284.9 mm to (211.4, 103.2)
- moved R10 284.8 mm to (211.6, 99.4)
- moved R2 284.0 mm to (206.0, 59.7)
- moved R4 283.8 mm to (205.9, 64.8)
- moved R3 283.8 mm to (205.8, 62.2)
- moved Q6 283.0 mm to (200.1, 97.4)
- moved Q7 283.0 mm to (200.1, 105.4)
- moved Q8 283.0 mm to (200.1, 113.5)
- moved Q4 281.8 mm to (215.9, 102.9)
- moved D2 280.2 mm to (216.5, 60.3)
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- renumbered PS4 to PS3
Connections:
- J5 pad 1: +24V -> +12V
- J5 pad 2: Net-(J5-Pin_2) -> Net-(J4-Pin_2)
- J5 pad 3: Net-(J5-Pin_3) -> Net-(J4-Pin_3)
- J5 pad 4: Net-(J5-Pin_4) -> Net-(J4-Pin_4)
- Q2 pad 2: Net-(J5-Pin_2) -> Net-(J6-Pin_2)
- Q3 pad 2: Net-(J5-Pin_3) -> Net-(J6-Pin_3)
- Q5 pad 2: Net-(J5-Pin_4) -> Net-(J6-Pin_4)

Commit message: wip pcb
Parts:
- moved D2 18.3 mm to (218.4, 78.5), turned to 90 degrees
- moved Q1 16.0 mm to (217.8, 63.2), turned to -90 degrees
- moved R2 14.5 mm to (218.4, 67.0), turned to 180 degrees
- moved D1 14.3 mm to (218.4, 72.8), turned to 90 degrees
- moved R3 14.1 mm to (218.4, 68.3)
- moved R4 13.5 mm to (218.4, 69.6)
- moved R10 9.58 mm to (218.4, 106.0)
- moved D4 7.42 mm to (218.4, 114.9), turned to 90 degrees
- moved R8 7.07 mm to (218.4, 104.8)
- moved R7 7.01 mm to (218.4, 103.5), turned to 180 degrees
- moved K2 4.45 mm to (221.6, 98.4)
- moved Q4 3.73 mm to (217.8, 99.7), turned to -90 degrees
- moved K1 2.91 mm to (221.6, 62.0)
- moved D3 2.57 mm to (218.4, 109.2), turned to 90 degrees
Routing:
- net +5V: track 0.00 -> 30.5 mm
- net Net-(D3-K): track 0.00 -> 19.7 mm
- net Net-(D1-K): track 0.00 -> 19.7 mm
- net GND: track 0.00 -> 8.83 mm
- net Net-(Q1-B): track 0.00 -> 5.13 mm
- net Net-(Q4-B): track 0.00 -> 5.13 mm
- net Net-(D1-A): track 0.00 -> 2.45 mm
- net Net-(D3-A): track 0.00 -> 2.45 mm

Commit message: wip pcb
Parts:
- moved PS2 49.6 mm to (145.2, 135.9), turned to 180 degrees
- moved R5 36.8 mm to (209.3, 106.3), turned to 180 degrees
- moved Q2 31.5 mm to (209.1, 113.5), turned to -90 degrees
- moved R6 28.9 mm to (201.1, 106.3), turned to 180 degrees
- moved R13 22.5 mm to (208.9, 100.5)
- moved Q8 22.0 mm to (208.9, 93.3), turned to 90 degrees
- moved R9 21.9 mm to (193.0, 106.3), turned to 180 degrees
- moved Q3 20.6 mm to (201.1, 113.5), turned to -90 degrees
- moved Q7 12.2 mm to (200.9, 93.3), turned to 90 degrees
- moved R12 11.6 mm to (200.8, 100.5)
- moved Q5 10.8 mm to (193.0, 113.5), turned to -90 degrees
- moved J2 9.61 mm to (156.2, 124.5), turned to 180 degrees
- moved Q6 8.35 mm to (192.8, 93.3), turned to 90 degrees
- moved J1 7.10 mm to (161.3, 121.9), turned to 180 degrees
- moved R11 4.06 mm to (192.7, 100.5)
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Routing:
- net GND: track 8.83 -> 404.5 mm
- net +5V: track 30.5 -> 299.4 mm, vias 0 -> 1
- net Net-(J3-Pin_1): track 0.00 -> 198.4 mm
- net Net-(J3-Pin_2): track 0.00 -> 160.2 mm
- net +24V: track 0.00 -> 121.1 mm
- net Net-(U1-GPIO33): track 0.00 -> 99.9 mm, vias 0 -> 1
- net Net-(PS1-AC/L): track 0.00 -> 99.4 mm
- net Net-(U1-GPIO32): track 0.00 -> 97.8 mm, vias 0 -> 2
- net Net-(Q8-G): track 0.00 -> 85.6 mm
- net Net-(PS2-AC/L): track 0.00 -> 83.6 mm
- net Net-(Q2-G): track 0.00 -> 79.9 mm
- net Net-(Q7-G): track 0.00 -> 74.7 mm
- net Net-(Q3-G): track 0.00 -> 68.9 mm
- net Net-(Q6-G): track 0.00 -> 61.6 mm
- net Net-(Q5-G): track 0.00 -> 57.9 mm
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
Commit message: DRC OK
Routing:
- net +3V3: track 50.3 -> 54.0 mm
- net Net-(J1-Pin_3): track 48.4 -> 51.6 mm
Changed lines of the file:
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@@
     (property "ki_description" "0.2A Ic, 40V Vce, Small Signal NPN Transistor, TO-92")
     (property "ki_keywords" "NPN Transistor")
-    (attr through_hole)
-    (fp_text reference "Q1" (at 0.655318 2.560318 -180) (layer "F.SilkS")
+    (attr smd)
+    (fp_text reference "Q1" (at -0.351602 2.570318) (layer "F.SilkS")
         (effects (font (size 1 1) (thickness 0.15)))
     )
@@
     (tags "mounting hole 3.2mm m3")
     (attr exclude_from_pos_files exclude_from_bom)
-    (fp_text reference "REF**" (at 0 -4.2) (layer "F.SilkS")
+    (fp_text reference "REF**" (at -2.055 -4.2) (layer "F.SilkS")
         (effects (font (size 1 1) (thickness 0.15)))
     )
@@
     (property "ki_description" "0.2A Ic, 40V Vce, Small Signal NPN Transistor, TO-92")
     (property "ki_keywords" "NPN Transistor")
-    (attr through_hole)
-    (fp_text reference "Q4" (at 0.655318 2.560318 180) (layer "F.SilkS")
+    (attr smd)
+    (fp_text reference "Q4" (at 0.655318 2.560318) (layer "F.SilkS")
         (effects (font (size 1 1) (thickness 0.15)))
     )
@@
   (segment (start 156.21 121.92) (end 156.21 124.46) (width 0.25) (layer "F.Cu") (net 4))
   (segment (start 213.36 100.37) (end 211.215 98.225) (width 1) (layer "F.Cu") (net 4))
+  (segment (start 162.685 117.985) (end 161.29 119.38) (width 0.25) (layer "F.Cu") (net 5))
+  (segment (start 164.465 117.985) (end 162.685 117.985) (width 0.25) (layer "F.Cu") (net 5))
   (segment (start 128.905 118.11) (end 120.015 109.22) (width 0.25) (layer "B.Cu") (net 5))
   (segment (start 155.575 113.665) (end 151.13 118.11) (width 0.25) (layer "B.Cu") (net 5))
@@
   (segment (start 150.495 83.82) (end 140.335 83.82) (width 0.25) (layer "F.Cu") (net 8))
   (segment (start 151.765 107.315) (end 150.495 107.315) (width 0.25) (layer "F.Cu") (net 8))
+  (segment (start 164.34 116.84) (end 164.465 116.965) (width 0.25) (layer "F.Cu") (net 8))
   (segment (start 161.29 116.84) (end 151.765 107.315) (width 0.25) (layer "F.Cu") (net 8))
+  (segment (start 161.29 116.84) (end 164.34 116.84) (width 0.25) (layer "F.Cu") (net 8))
   (via (at 150.495 83.82) (size 0.8) (drill 0.4) (layers "F.Cu" "B.Cu") (net 8))
   (via (at 150.495 107.315) (size 0.8) (drill 0.4) (layers "F.Cu" "B.Cu") (net 8))
