File: rgb-garden-box/v1/rgb-garden-box.kicad_pcb (KiCad board)
At the start: 2 copper layers, 149.3 x 102 mm, 43 parts, among them J1 Conn_01x03_Male, J2 Conn_01x04_Male, J3 Screw_Terminal_01x02, J4 Screw_Terminal_01x04, J5 Screw_Terminal_01x04, J6 Screw_Terminal_01x04, K1 G6DN-1A-L_DC5, K2 G6DN-1A-L_DC5, Q1 2N3904, Q2 IRLZ44N, Q3 IRLZ44N, Q4 2N3904, Q5 IRLZ44N, Q6 IRLZ44N, Q7 IRLZ44N, Q8 IRLZ44N, U1 ESP32-POE

Commit message: PCB OK
Other:
- board text added: "+ R G B"
- board text added: "12V"
- board text added: "220V"
- board text added: "24V"
- board text added: "3V3"
- board text added: "5V"
- board text added: "A0"
- board text added: "B G R +"
- board text added: "DS18B20"
- board text added: "GND"
- board text added: "IN"
- board text added: "L"
- board text added: "N"
- board text added: "SEN0308"
- board text added: "TODO: texts sur connectors"
Changed lines of the file:
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@@
     (tags "mounting hole 3.2mm m3")
     (attr exclude_from_pos_files exclude_from_bom)
-    (fp_text reference "REF**" (at 0 -4.2) (layer "F.SilkS")
+    (fp_text reference "REF**" (at 0 5.01) (layer "F.SilkS")
         (effects (font (size 1 1) (thickness 0.15)))
     )
@@
     (property "ki_keywords" "screw terminal")
     (attr through_hole)
-    (fp_text reference "J5" (at 7.6 -4.8) (layer "F.SilkS")
+    (fp_text reference "J5" (at -3.81 1.27) (layer "F.SilkS")
         (effects (font (size 1 1) (thickness 0.15)))
     )
@@
     (property "ki_keywords" "screw terminal")
     (attr through_hole)
-    (fp_text reference "J6" (at 7.6 -4.8) (layer "F.SilkS")
+    (fp_text reference "J6" (at -1.27 4.445) (layer "F.SilkS")
         (effects (font (size 1 1) (thickness 0.15)))
     )
@@
     (property "ki_keywords" "R res resistor")
     (attr smd)
-    (fp_text reference "R1" (at 1.905 -0.125 180) (layer "F.SilkS")
+    (fp_text reference "R1" (at 0 1.905 180) (layer "F.SilkS")
         (effects (font (size 1 1) (thickness 0.15)))
     )
@@
   (gr_line locked (start 77.32 56.69) (end 86.32 56.69)
     (stroke (width 0.1) (type solid)) (layer "Edge.Cuts"))
+  (gr_text "B    G    R    +" (at 198.12 131.445) (layer "F.SilkS")
+    (effects (font (size 1.5 1.5) (thickness 0.3) bold) (justify left bottom))
+  )
+  (gr_text "SEN0308" (at 154.305 127.635) (layer "F.SilkS")
+    (effects (font (size 1 1) (thickness 0.15)))
+  )
+  (gr_text "GND" (at 164.465 121.92) (layer "F.SilkS")
+    (effects (font (size 0.6 0.6) (thickness 0.125)))
+  )
+  (gr_text "DS18B20" (at 162.56 125.095) (layer "F.SilkS")
+    (effects (font (size 1 1) (thickness 0.15)))
+  )
+  (gr_text "L" (at 184.785 130.175) (layer "F.SilkS")
+    (effects (font (size 1.5 1.5) (thickness 0.3) bold) (justify left bottom))
+  )
+  (gr_text "3V3" (at 164.465 120.015) (layer "F.SilkS")
+    (effects (font (size 0.6 0.6) (thickness 0.125)))
+  )
+  (gr_text "TODO: texts sur connectors" (at 194.945 25.4) (layer "F.SilkS")
+    (effects (font (size 1.5 1.5) (thickness 0.3) bold) (justify left bottom))
+  )
+  (gr_text "12V" (at 203.835 62.865) (layer "F.SilkS")
+    (effects (font (size 1.5 1.5) (thickness 0.3) bold) (justify left bottom))
+  )
+  (gr_text "GND" (at 153.035 121.92) (layer "F.SilkS")
+    (effects (font (size 0.6 0.6) (thickness 0.125)))
+  )
+  (gr_text "5V" (at 153.035 119.38) (layer "F.SilkS")
+    (effects (font (size 0.6 0.6) (thickness 0.125)))
+  )
+  (gr_text "IN" (at 164.465 115.57) (layer "F.SilkS")
+    (effects (font (size 0.6 0.6) (thickness 0.125)))
+  )
+  (gr_text "24V" (at 204.47 133.985) (layer "F.SilkS")
+    (effects (font (size 1.5 1.5) (thickness 0.3) bold) (justify left bottom))
+  )
+  (gr_text "+    R    G    B" (at 197.485 77.47) (layer "F.SilkS")
+    (effects (font (size 1.5 1.5) (thickness 0.3) bold) (justify left bottom))
+  )
+  (gr_text "N" (at 184.785 135.255) (layer "F.SilkS")
+    (effects (font (size 1.5 1.5) (thickness 0.3) bold) (justify left bottom))
+  )
+  (gr_text "220V" (at 178.435 132.715) (layer "F.SilkS")
+    (effects (font (size 1.5 1.5) (thickness 0.3) bold) (justify left bottom))
+  )
+  (gr_text "12V" (at 204.47 75.565) (layer "F.SilkS")
+    (effects (font (size 1.5 1.5) (thickness 0.3) bold) (justify left bottom))
+  )
+  (gr_text "GND" (at 153.035 124.46) (layer "F.SilkS")
+    (effects (font (size 0.6 0.6) (thickness 0.125)))
+  )
+  (gr_text "A0" (at 153.035 116.84) (layer "F.SilkS")
+    (effects (font (size 0.6 0.6) (thickness 0.125)))
+  )
+  (gr_text "+    R    G    B" (at 198.12 59.69) (layer "F.SilkS")
+    (effects (font (size 1.5 1.5) (thickness 0.3) bold) (justify left bottom))
+  )
   (segment (start 220.005 72.14442) (end 218.45 73.69942) (width 0.25) (layer "F.Cu") (net 1))
   (segment (start 218.45 76.82692) (end 218.83 77.20692) (width 0.25) (layer "F.Cu") (net 1))

Commit message: cleanup
Other:
- board text removed: "TODO: texts sur connectors"
Changed lines of the file:
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@@
     (effects (font (size 0.6 0.6) (thickness 0.125)))
-  )
-  (gr_text "TODO: texts sur connectors" (at 194.945 25.4) (layer "F.SilkS")
-    (effects (font (size 1.5 1.5) (thickness 0.3) bold) (justify left bottom))
   )
   (gr_text "12V" (at 203.835 62.865) (layer "F.SilkS")
