File: rgb-garden-box/v1/rgb-garden-box.kicad_sch (KiCad schematic)
At the start: 36 parts, among them J1 Conn_01x03_Male, J2 Conn_01x04_Male, J3 Screw_Terminal_01x02, J4 Screw_Terminal_01x04, J5 Screw_Terminal_01x04, K1 G6DN-1A-L_DC5, K2 G6DN-1A-L_DC5, Q1 2N3904, Q2 IRLZ44N, Q3 IRLZ44N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

Commit message: add footprints
Parts:
- PS1: footprint (none) -> mylife-footprints:IRM-30-12; symbol Converter_ACDC:IRM-10-5 -> Converter_ACDC:IRM-60-12
- PS2: footprint (none) -> mylife-footprints:RS PRO Alim 5V 2A
Connections:
- net +12V: now also PS1.3 (+Vout); no longer PS1.4 (+Vo)
- net GND: now also PS1.4 (-Vout); no longer PS1.3 (-Vo)
- net at J3.2 (Pin_2), PS1.3 (AC/N), PS2.1 (AC/N): now also PS1.2 (AC/N); no longer PS1.1 (AC/N)
- net at K1.8: now also PS1.1 (AC/L); no longer PS1.2 (AC/L)
Changed lines of the file:
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@@
       (effects (font (size 1.27 1.27)))
     )
-    (property "Footprint" "" (at 204.47 69.85 0)
+    (property "Footprint" "mylife-footprints:RS PRO Alim 5V 2A" (at 204.47 69.85 0)
       (effects (font (size 1.27 1.27)) hide)
     )
@@
     )
   )
-  (symbol (lib_id "Converter_ACDC:IRM-10-5") (at 160.02 31.75 0) (mirror y) (unit 1)
-    (in_bom yes) (on_board yes) (dnp no) (fields_autoplaced)
+  (symbol (lib_id "Converter_ACDC:IRM-60-12") (at 160.02 31.75 0) (mirror y) (unit 1)
+    (in_bom yes) (on_board yes) (dnp no)
     (property "Reference" "PS1" (at 160.02 21.59 0)
       (effects (font (size 1.27 1.27)))
@@
       (effects (font (size 1.27 1.27)))
     )
-    (property "Footprint" "" (at 160.02 40.64 0)
-      (effects (font (size 1.27 1.27)) hide)
-    )
-    (property "Datasheet" "https://docs.rs-online.com/3f08/0900766b815c75c9.pdf" (at 160.02 41.91 0)
-      (effects (font (size 1.27 1.27)) hide)
-    )
+    (property "Footprint" "mylife-footprints:IRM-30-12" (at 160.02 41.91 0)
+      (effects (font (size 1.27 1.27)) hide)
+    )
+    (property "Datasheet" "http://www.meanwellusa.com/productPdf.aspx?i=687" (at 160.02 31.75 0)
+      (effects (font (size 1.27 1.27)) hide)
+    )

Commit message: wip pcb placement
Parts:
- added J4: Screw_Terminal_01x04, TerminalBlock:TerminalBlock_bornier-4_P5.08mm, symbol Connector:Screw_Terminal_01x04
- renumbered J4 to J5, J5 to J6
Connections:
- net +12V: now also J4.1 (Pin_1)
- net at J5.2 (Pin_2), Q6.2 (D): now also J4.2 (Pin_2)
- net at J5.4 (Pin_4), Q8.2 (D): now also J4.4 (Pin_4)
- net at J5.3 (Pin_3), Q7.2 (D): now also J4.3 (Pin_3)

Commit message: switch IRLZ44N to TO220
Parts:
- Q2, Q3, Q5, Q6, Q7, Q8: footprint Package_TO_SOT_SMD:ATPAK-2 -> Package_TO_SOT_THT:TO-220-3_Vertical; LCSC C538199 -> (none)
Changed lines of the file:
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@@
       (effects (font (size 1.27 1.27)) (justify left))
     )
-    (property "Footprint" "Package_TO_SOT_SMD:ATPAK-2" (at 190.5 127.635 0)
+    (property "Footprint" "Package_TO_SOT_THT:TO-220-3_Vertical" (at 190.5 127.635 0)
       (effects (font (size 1.27 1.27) italic) (justify left) hide)
     )
-    (property "Datasheet" "https://datasheet.lcsc.com/lcsc/2005300013_Infineon-Technologies-IRLZ44NSTRLPBF_C538199.pdf" (at 184.15 125.73 0)
+    (property "Datasheet" "" (at 184.15 125.73 0)
       (effects (font (size 1.27 1.27)) (justify left) hide)
     )
-    (property "LCSC" "C538199" (at 184.15 125.73 0)
+    (property "LCSC" "" (at 184.15 125.73 0)
       (effects (font (size 1.27 1.27)) hide)
     )
@@
       (effects (font (size 1.27 1.27)) (justify left))
     )
-    (property "Footprint" "Package_TO_SOT_SMD:ATPAK-2" (at 157.48 167.005 0)
+    (property "Footprint" "Package_TO_SOT_THT:TO-220-3_Vertical" (at 157.48 167.005 0)
       (effects (font (size 1.27 1.27) italic) (justify left) hide)
     )
-    (property "Datasheet" "https://datasheet.lcsc.com/lcsc/2005300013_Infineon-Technologies-IRLZ44NSTRLPBF_C538199.pdf" (at 151.13 165.1 0)
+    (property "Datasheet" "" (at 151.13 165.1 0)
       (effects (font (size 1.27 1.27)) (justify left) hide)
     )
-    (property "LCSC" "C538199" (at 151.13 165.1 0)
+    (property "LCSC" "" (at 151.13 165.1 0)
       (effects (font (size 1.27 1.27)) hide)
     )
@@
       (effects (font (size 1.27 1.27)) (justify left))
     )
-    (property "Footprint" "Package_TO_SOT_SMD:ATPAK-2" (at 227.33 127.635 0)
+    (property "Footprint" "Package_TO_SOT_THT:TO-220-3_Vertical" (at 227.33 127.635 0)
       (effects (font (size 1.27 1.27) italic) (justify left) hide)
     )
-    (property "Datasheet" "https://datasheet.lcsc.com/lcsc/2005300013_Infineon-Technologies-IRLZ44NSTRLPBF_C538199.pdf" (at 220.98 125.73 0)
+    (property "Datasheet" "" (at 220.98 125.73 0)
       (effects (font (size 1.27 1.27)) (justify left) hide)
     )
-    (property "LCSC" "C538199" (at 220.98 125.73 0)
+    (property "LCSC" "" (at 220.98 125.73 0)
       (effects (font (size 1.27 1.27)) hide)
     )
@@
       (effects (font (size 1.27 1.27)) (justify left))
     )
-    (property "Footprint" "Package_TO_SOT_SMD:ATPAK-2" (at 138.43 167.005 0)
+    (property "Footprint" "Package_TO_SOT_THT:TO-220-3_Vertical" (at 138.43 167.005 0)
       (effects (font (size 1.27 1.27) italic) (justify left) hide)
     )
-    (property "Datasheet" "https://datasheet.lcsc.com/lcsc/2005300013_Infineon-Technologies-IRLZ44NSTRLPBF_C538199.pdf" (at 132.08 165.1 0)
+    (property "Datasheet" "" (at 132.08 165.1 0)
       (effects (font (size 1.27 1.27)) (justify left) hide)
     )
-    (property "LCSC" "C538199" (at 132.08 165.1 0)
+    (property "LCSC" "" (at 132.08 165.1 0)
       (effects (font (size 1.27 1.27)) hide)
     )
@@
       (effects (font (size 1.27 1.27)) (justify left))
     )
-    (property "Footprint" "Package_TO_SOT_SMD:ATPAK-2" (at 208.28 127.635 0)
+    (property "Footprint" "Package_TO_SOT_THT:TO-220-3_Vertical" (at 208.28 127.635 0)
       (effects (font (size 1.27 1.27) italic) (justify left) hide)
     )
-    (property "Datasheet" "https://datasheet.lcsc.com/lcsc/2005300013_Infineon-Technologies-IRLZ44NSTRLPBF_C538199.pdf" (at 201.93 125.73 0)
+    (property "Datasheet" "" (at 201.93 125.73 0)
       (effects (font (size 1.27 1.27)) (justify left) hide)
     )
-    (property "LCSC" "C538199" (at 201.93 125.73 0)
+    (property "LCSC" "" (at 201.93 125.73 0)
       (effects (font (size 1.27 1.27)) hide)
     )
@@
       (effects (font (size 1.27 1.27)) (justify left))
     )
-    (property "Footprint" "Package_TO_SOT_SMD:ATPAK-2" (at 120.65 167.005 0)
+    (property "Footprint" "Package_TO_SOT_THT:TO-220-3_Vertical" (at 120.65 167.005 0)
       (effects (font (size 1.27 1.27) italic) (justify left) hide)
     )
-    (property "Datasheet" "https://datasheet.lcsc.com/lcsc/2005300013_Infineon-Technologies-IRLZ44NSTRLPBF_C538199.pdf" (at 114.3 165.1 0)
+    (property "Datasheet" "" (at 114.3 165.1 0)
       (effects (font (size 1.27 1.27)) (justify left) hide)
     )
-    (property "LCSC" "C538199" (at 114.3 165.1 0)
-      (effects (font (size 1.27 1.27)) hide)
-    )
+    (property "LCSC" "" (at 114.3 165.1 0)
+      (effects (font (size 1.27 1.27)) hide)
+    )
