File: garage-door-driver/v1/garage-door-driver.kicad_pcb (KiCad board)
At the start: 2 copper layers, 45 x 45 mm, 5 parts, among them J1 Screw_Terminal_01x04

Commit message: clean PCB + add edge cuts
Parts:
- removed D1: LED_ARGB, mylife-footprints:LED RGB 10W
- removed J1: Screw_Terminal_01x04, mylife-footprints:RS PRO Terminal Small x4
- removed R1, R2: 5.1Ω/1W, Resistor_SMD:R_2512_6332Metric
- removed R3: 10Ω/1W, Resistor_SMD:R_2512_6332Metric
Routing:
- net Net-(J1-Pin_2): track 56.6 -> 0.00 mm
- net Net-(J1-Pin_3): track 26.2 -> 0.00 mm
- net Net-(D1-RK): track 25.3 -> 0.00 mm, vias 1 -> 0
- net Net-(D1-BK): track 25.2 -> 0.00 mm, vias 1 -> 0
- net Net-(J1-Pin_1): track 21.3 -> 0.00 mm
- net Net-(D1-GK): track 11.6 -> 0.00 mm, vias 1 -> 0
- net Net-(D1-A): track 7.84 -> 0.00 mm
Other:
- board size 45 x 45 mm -> 95 x 50 mm
- board text removed: "+ R G B"

Commit message: pcb
Parts:
- added C1: 10μF/50V, Capacitor_SMD:C_1206_3216Metric, F.Cu at (96.4, 76.0)
- added C2: 22μF/10V, Capacitor_SMD:C_0805_2012Metric, F.Cu at (95.8, 79.1)
- added D1: LED, Diode_SMD:D_0805_2012Metric, F.Cu at (168.9, 96.2)
- added D2: LED, Diode_SMD:D_0805_2012Metric, F.Cu at (161.3, 93.3)
- added D3: LED, Diode_SMD:D_0805_2012Metric, F.Cu at (171.4, 96.2)
- added D4: LED, Diode_SMD:D_0805_2012Metric, F.Cu at (161.3, 90.8)
- added D5: LED, Diode_SMD:D_0805_2012Metric, F.Cu at (178.8, 96.5)
- added J1: Conn_01x03_Male, Connector_PinHeader_2.54mm:PinHeader_1x03_P2.54mm_Vertical, F.Cu at (160.7, 103.4)
- added J2: Screw_Terminal_01x02, mylife-footprints:RS PRO Terminal Small x2, F.Cu at (180.3, 104.9)
- added J3: Screw_Terminal_01x02, mylife-footprints:RS PRO Terminal Small x2, F.Cu at (171.4, 104.9)
- added J4: Conn_01x07_Pin, Connector_PinHeader_2.54mm:PinHeader_1x07_P2.54mm_Vertical, F.Cu at (190.2, 61.0)
- added R1: 4.7KΩ, Resistor_SMD:R_0402_1005Metric, F.Cu at (95.0, 81.6)
- added R10: 2.2KΩ, Resistor_SMD:R_0603_1608Metric, F.Cu at (84.7, 103.6)
- added R11: 220Ω, Resistor_SMD:R_0603_1608Metric, F.Cu at (84.7, 106.1)
- added R12: 1KΩ, Resistor_SMD:R_0603_1608Metric, F.Cu at (88.7, 96.1)
- added R13: 10KΩ, Resistor_SMD:R_0603_1608Metric, F.Cu at (88.7, 98.6)
- added R14: 2.2KΩ, Resistor_SMD:R_0603_1608Metric, F.Cu at (88.7, 101.1)
- added R2: 1KΩ, Resistor_SMD:R_0603_1608Metric, F.Cu at (80.7, 96.1)
- added R3: 10KΩ, Resistor_SMD:R_0603_1608Metric, F.Cu at (80.7, 98.6)
- added R4: 1KΩ, Resistor_SMD:R_0603_1608Metric, F.Cu at (80.7, 101.1)
- added R5: 2.2KΩ, Resistor_SMD:R_0603_1608Metric, F.Cu at (80.7, 103.6)
- added R6: 1KΩ, Resistor_SMD:R_0603_1608Metric, F.Cu at (80.7, 106.1)
- added R7: 220Ω, Resistor_SMD:R_0603_1608Metric, F.Cu at (84.7, 96.1)
- added R8: 10KΩ, Resistor_SMD:R_0603_1608Metric, F.Cu at (84.7, 98.6)
- added R9: 1KΩ, Resistor_SMD:R_0603_1608Metric, F.Cu at (84.7, 101.1)
- added U1: R-785.0-1.0, Converter_DCDC:Converter_DCDC_RECOM_R-78E-0.5_THT, F.Cu at (188.7, 105.1)
- added U2: WeMos_D1_mini, Module:WEMOS_D1_mini_light, F.Cu at (122.6, 102.2)
- added U3: 4N35, Package_DIP:DIP-6_W8.89mm_SMDSocket_LongPads, F.Cu at (58.7, 63.8)
- added U4: 4N35, Package_DIP:DIP-6_W8.89mm_SMDSocket_LongPads, F.Cu at (58.7, 73.1)
- added U5: 4N35, Package_DIP:DIP-6_W8.89mm_SMDSocket_LongPads, F.Cu at (58.7, 82.5)
- added U6: 4N35, Package_DIP:DIP-6_W8.89mm_SMDSocket_LongPads, F.Cu at (58.7, 91.8)
- added U7: 4N35, Package_DIP:DIP-6_W8.89mm_SMDSocket_LongPads, F.Cu at (58.7, 101.2)
Other:
- board text added: "24v"
- board text added: "3V3"
- board text added: "Bornier noir"
- board text added: "DS18B20"
- board text added: "GND"
- board text added: "IN"
- board text added: "Moteur"
- board text added: "Partiel"
- board text added: "Total"

Commit message: pcb
Parts:
- moved U4 137.0 mm to (195.6, 68.6), turned to 180 degrees
- moved U6 122.0 mm to (180.3, 82.5), turned to 90 degrees
- moved R7 117.0 mm to (200.0, 76.2), turned to 90 degrees
- moved U5 112.8 mm to (171.4, 82.5), turned to 90 degrees
- moved U3 105.6 mm to (162.6, 82.5), turned to 90 degrees
- moved C2 104.2 mm to (198.8, 95.2), turned to 90 degrees
- moved C1 103.3 mm to (198.8, 90.2), turned to -90 degrees
- moved U7 96.8 mm to (153.7, 82.5), turned to 90 degrees
- moved R11 95.7 mm to (179.1, 90.2)
- moved R12 94.2 mm to (182.9, 96.5)
- moved R6 93.8 mm to (174.0, 96.5), turned to -90 degrees
- moved R8 88.7 mm to (170.2, 74.9), turned to 180 degrees
- moved R10 86.6 mm to (170.3, 90.2), turned to 180 degrees
- moved R2 85.7 mm to (166.4, 96.5), turned to -90 degrees
- moved R3 84.0 mm to (161.3, 74.9), turned to 180 degrees
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Routing:
- net +5V: track 0.00 -> 73.8 mm, vias 0 -> 1
- net GND: track 0.00 -> 69.8 mm, vias 0 -> 1
- net +24V: track 0.00 -> 51.6 mm, vias 0 -> 1
- net Net-(J4-Pin_7): track 0.00 -> 20.8 mm
- net Net-(J4-Pin_3): track 0.00 -> 13.4 mm, vias 0 -> 1
- net Net-(R7-Pad2): track 0.00 -> 4.25 mm

Commit message: pcb
Parts:
- moved R14 18.0 mm to (170.2, 90.2)
- moved R13 17.8 mm to (170.2, 74.9)
- moved U7 17.8 mm to (171.4, 82.5)
- moved R10 8.89 mm to (161.4, 90.2)
- moved R8 8.89 mm to (161.3, 74.9)
- moved U3 8.89 mm to (153.7, 82.5)
- moved R3 8.89 mm to (152.4, 74.9)
- moved R5 8.89 mm to (152.4, 90.2)
- moved U5 8.89 mm to (162.6, 82.5)
- turned D2 to 180 degrees
- turned D4 to 180 degrees
- turned R1 to 180 degrees
- turned R11 to 180 degrees
- turned R12 to 180 degrees
- turned R2 to 90 degrees
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Routing:
- net GND: track 69.8 -> 206.0 mm, vias 1 -> 9
- net +3V3: track 0.00 -> 111.2 mm, vias 0 -> 4
- net Net-(D2-A): track 0.00 -> 106.8 mm
- net Net-(U2-MOSI/D7): track 0.00 -> 82.9 mm, vias 0 -> 1
- net Net-(D4-A): track 0.00 -> 74.7 mm, vias 0 -> 2
- net Net-(U2-MISO/D6): track 0.00 -> 72.6 mm, vias 0 -> 1
- net Net-(U2-SCK/D5): track 0.00 -> 69.1 mm, vias 0 -> 1
- net Net-(J1-Pin_3): track 0.00 -> 44.7 mm, vias 0 -> 1
- net Net-(J3-Pin_1): track 0.00 -> 37.2 mm, vias 0 -> 2
- net Net-(J3-Pin_2): track 0.00 -> 36.0 mm, vias 0 -> 1
- net Net-(J2-Pin_2): track 0.00 -> 25.6 mm, vias 0 -> 1
- net Net-(J2-Pin_1): track 0.00 -> 23.8 mm, vias 0 -> 1
- net Net-(J4-Pin_7): track 20.8 -> 37.3 mm
- net +5V: track 73.8 -> 88.3 mm, vias 1 -> 2
- net Net-(J4-Pin_3): track 13.4 -> 9.80 mm, vias 1 -> 0
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