File: bed-smart-plug/prototype-1/bed-smart-plug.kicad_sch (KiCad schematic)
At the start: 24 parts, among them J1 Main, J2 Prises, J3 Triac gate protection, J4 Triac snubber, J5 Opto snubber, J6 Opto snubber 2, J7 Conn_01x03_Male, Q1 BT136-600E, U1 MOC3021M, U2 ESP32-POE, U6 AM-RX12A-433P

Commit message: jack
Parts:
- added J10: Conn_01x02_Male, Connector_PinHeader_2.54mm:PinHeader_1x02_P2.54mm_Vertical, symbol Connector:Conn_01x04_Pin
- added J9: 3.5mm headphone jack, Connector_Audio:Jack_3.5mm_PJ320D_Horizontal, symbol Connector:AudioJack4
- J3, J4, J6: symbol Connector_Generic:Conn_01x02 -> Connector:Conn_01x02_Pin
- J5: symbol Connector_Generic:Conn_01x03 -> Connector:Conn_01x03_Pin
Connections:
- new net: J10.3 (Pin_3), J9.R1
- new net: J10.2 (Pin_2), J9.R2
- new net: J10.1 (Pin_1), J9.S
- new net: J10.4 (Pin_4), J9.T
Changed lines of the file:
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@@
+    (stroke (width 0) (type default))
+  )
+  (wire (pts (xy 143.51 140.97) (xy 153.67 140.97))
     (stroke (width 0) (type default))
   )
@@
     (stroke (width 0) (type default))
   )
+  (wire (pts (xy 143.51 143.51) (xy 153.67 143.51))
+    (stroke (width 0) (type default))
+  )
   (wire (pts (xy 195.58 68.58) (xy 199.39 68.58))
     (stroke (width 0) (type default))
@@
   )
   (wire (pts (xy 224.79 93.98) (xy 224.79 97.79))
+    (stroke (width 0) (type default))
+  )
+  (wire (pts (xy 143.51 146.05) (xy 153.67 146.05))
+    (stroke (width 0) (type default))
+  )
+  (wire (pts (xy 143.51 148.59) (xy 153.67 148.59))
     (stroke (width 0) (type default))
   )
@@
   )
   (text "GND" (at 29.21 109.22 0)
-    (effects (font (size 1.27 1.27)) (justify left bottom))
-  )
-  (label "TODO: jack pinout" (at 25.4 21.59 0) (fields_autoplaced)
     (effects (font (size 1.27 1.27)) (justify left bottom))
   )
@@
         (path "/099096e4-8c2a-4d84-a16f-06b4b6330e7a"
           (reference "AE1") (unit 1)
+        )
+      )
+    )
+  )
+  (symbol (lib_id "Connector:AudioJack4") (at 158.75 143.51 0) (mirror y) (unit 1)
+    (in_bom yes) (on_board yes) (dnp no)
+    (property "Reference" "J9" (at 160.02 138.43 0)
+      (effects (font (size 1.27 1.27)) (justify right))
+    )
+    (property "Value" "3.5mm headphone jack" (at 154.94 152.4 0)
+      (effects (font (size 1.27 1.27)) (justify right))
+    )
+    (property "Footprint" "Connector_Audio:Jack_3.5mm_PJ320D_Horizontal" (at 158.75 143.51 0)
+      (effects (font (size 1.27 1.27)) hide)
+    )
+    (property "Datasheet" "https://datasheet.lcsc.com/lcsc/2005041005_USAKRO-PJ-320D_C521460.pdf" (at 158.75 143.51 0)
+      (effects (font (size 1.27 1.27)) hide)
+    )
+    (property "LCSC" "C521460" (at 158.75 143.51 0)
+      (effects (font (size 1.27 1.27)) hide)
+    )
+    (pin "R1")
+    (pin "R2")
+    (pin "S")
+    (pin "T")
+    (instances
+      (project "bed-smart-plug"
+        (path "/099096e4-8c2a-4d84-a16f-06b4b6330e7a"
+          (reference "J9") (unit 1)
+        )
+      )
+      (project "prototype-2"
+        (path "/9e00edb4-f0f4-46bc-a82d-075ebfd0d3ed"
+          (reference "J8") (unit 1)
         )
       )
@@
     )
   )
-  (symbol (lib_id "Connector_Generic:Conn_01x02") (at 264.16 109.22 0) (unit 1)
-    (in_bom yes) (on_board yes) (dnp no)
-    (property "Reference" "J4" (at 266.7 109.855 0)
-      (effects (font (size 1.27 1.27)) (justify left))
-    )
-    (property "Value" "Triac snubber" (at 266.7 112.395 0)
+  (symbol (lib_id "Connector:Conn_01x02_Pin") (at 264.16 109.22 0) (mirror y) (unit 1)
+    (in_bom yes) (on_board yes) (dnp no)
+    (property "Reference" "J4" (at 267.97 109.22 0)
+      (effects (font (size 1.27 1.27)) (justify left))
+    )
+    (property "Value" "Triac snubber" (at 278.13 111.76 0)
       (effects (font (size 1.27 1.27)) (justify left))
     )
@@
     )
   )
+  (symbol (lib_id "Connector:Conn_01x04_Pin") (at 138.43 143.51 0) (unit 1)
+    (in_bom yes) (on_board yes) (dnp no)
+    (property "Reference" "J10" (at 137.7188 143.8715 0)
+      (effects (font (size 1.27 1.27)) (justify right))
+    )
+    (property "Value" "Conn_01x02_Male" (at 147.32 139.7 0)
+      (effects (font (size 1.27 1.27)) (justify right))
+    )
+    (property "Footprint" "Connector_PinHeader_2.54mm:PinHeader_1x02_P2.54mm_Vertical" (at 138.43 143.51 0)
+      (effects (font (size 1.27 1.27)) hide)
+    )
+    (property "Datasheet" "~" (at 138.43 143.51 0)
+      (effects (font (size 1.27 1.27)) hide)
+    )
+    (pin "1")
+    (pin "2")
+    (pin "3")
+    (pin "4")
+    (instances
+      (project "bed-smart-plug"
+        (path "/099096e4-8c2a-4d84-a16f-06b4b6330e7a"
+          (reference "J10") (unit 1)
+        )
+      )
+      (project "prototype-2"
+        (path "/9e00edb4-f0f4-46bc-a82d-075ebfd0d3ed"
+          (reference "J10") (unit 1)
+        )
+      )
+    )
+  )
   (symbol (lib_id "Device:LED") (at 157.48 110.49 270) (mirror x) (unit 1)
     (in_bom yes) (on_board yes) (dnp no) (fields_autoplaced)
@@
     )
   )
-  (symbol (lib_id "Connector_Generic:Conn_01x02") (at 229.87 81.28 0) (mirror x) (unit 1)
-    (in_bom yes) (on_board yes) (dnp no)
-    (property "Reference" "J6" (at 228.6 85.09 0)
-      (effects (font (size 1.27 1.27)) (justify left))
-    )
-    (property "Value" "Opto snubber 2" (at 222.25 86.36 0)
+  (symbol (lib_id "Connector:Conn_01x02_Pin") (at 229.87 81.28 180) (unit 1)
+    (in_bom yes) (on_board yes) (dnp no)
+    (property "Reference" "J6" (at 233.68 77.47 0)
+      (effects (font (size 1.27 1.27)) (justify left))
+    )
+    (property "Value" "Opto snubber 2" (at 242.57 80.01 0)
       (effects (font (size 1.27 1.27)) (justify left))
     )
@@
   (symbol (lib_id "Device:R") (at 157.48 99.06 0) (unit 1)
     (in_bom yes) (on_board yes) (dnp no)
-    (property "Reference" "R3" (at 152.2222 99.06 90)
-      (effects (font (size 1.27 1.27)))
-    )
-    (property "Value" "220Ω" (at 154.5336 99.06 90)
+    (property "Reference" "R3" (at 153.67 97.79 0)
+      (effects (font (size 1.27 1.27)))
+    )
+    (property "Value" "220Ω" (at 153.67 100.33 0)
       (effects (font (size 1.27 1.27)))
     )
@@
     )
   )
-  (symbol (lib_id "Connector_Generic:Conn_01x03") (at 222.25 78.74 0) (mirror x) (unit 1)
-    (in_bom yes) (on_board yes) (dnp no)
-    (property "Reference" "J5" (at 220.98 72.39 0)
-      (effects (font (size 1.27 1.27)) (justify left))
-    )
-    (property "Value" "Opto snubber" (at 215.9 69.85 0)
+  (symbol (lib_id "Connector:Conn_01x03_Pin") (at 222.25 78.74 180) (unit 1)
+    (in_bom yes) (on_board yes) (dnp no)
+    (property "Reference" "J5" (at 223.52 72.39 0)
+      (effects (font (size 1.27 1.27)) (justify left))
+    )
+    (property "Value" "Opto snubber" (at 228.6 69.85 0)
       (effects (font (size 1.27 1.27)) (justify left))
     )
@@
     )
   )
-  (symbol (lib_id "Connector_Generic:Conn_01x02") (at 193.04 63.5 90) (unit 1)
-    (in_bom yes) (on_board yes) (dnp no)
-    (property "Reference" "J3" (at 193.675 60.96 0)
-      (effects (font (size 1.27 1.27)) (justify left))
-    )
-    (property "Value" "Triac gate protection" (at 196.215 60.96 0)
-      (effects (font (size 1.27 1.27)) (justify left))
-    )
+  (symbol (lib_id "Connector:Conn_01x02_Pin") (at 193.04 63.5 90) (mirror x) (unit 1)
+    (in_bom yes) (on_board yes) (dnp no)
+    (property "Reference" "J3" (at 194.31 58.42 90)
+      (effects (font (size 1.27 1.27)) (justify left))
+    )
+    (property "Value" "Triac gate protection" (at 203.2 60.96 90)
+      (effects (font (size 1.27 1.27)) (justify left))
+    )

Commit message: annotate
Parts:
- renumbered J7 to J1, J10 to J2, J9 to J3, J3 to J4, J1 to J7, J4 to J8, J2 to J9, PS2 to PS1, R4 to R1, R3 to R2, R9 to R3, R10 to R4, R2 to R5, R1 to R6, U2 to U1, U6 to U2, U1 to U3

Commit message: wip pcb
Parts:
- J7, J9: footprint TerminalBlock:TerminalBlock_bornier-6_P5.08mm -> TerminalBlock:TerminalBlock_bornier-2_P5.08mm
Changed lines of the file:
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@@
       (effects (font (size 1.27 1.27)) (justify left))
     )
-    (property "Footprint" "TerminalBlock:TerminalBlock_bornier-6_P5.08mm" (at 264.16 26.67 0)
+    (property "Footprint" "TerminalBlock:TerminalBlock_bornier-2_P5.08mm" (at 264.16 26.67 0)
       (effects (font (size 1.27 1.27)) hide)
     )
@@
       (effects (font (size 1.27 1.27)) (justify left))
     )
-    (property "Footprint" "TerminalBlock:TerminalBlock_bornier-6_P5.08mm" (at 275.59 120.65 0)
-      (effects (font (size 1.27 1.27)) hide)
-    )
+    (property "Footprint" "TerminalBlock:TerminalBlock_bornier-2_P5.08mm" (at 275.59 120.65 0)
+      (effects (font (size 1.27 1.27)) hide)
+    )

Commit message: placement
Parts:
- J1: value Conn_01x03_Male -> DS18b20
- J2: footprint Connector_PinHeader_2.54mm:PinHeader_1x02_P2.54mm_Vertical -> Connector_PinHeader_2.54mm:PinHeader_1x04_P2.54mm_Vertical
Other:
- note removed: "DS18B20"
Changed lines of the file:
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@@
     (stroke (width 0) (type default))
-  )
-  (text "DS18B20" (at 19.05 111.76 0)
-    (effects (font (size 1.27 1.27)) (justify left bottom))
   )
   (text "VCC" (at 29.21 111.76 0)
@@
       (effects (font (size 1.27 1.27)))
     )
-    (property "Value" "Conn_01x03_Male" (at 34.29 101.8351 0)
+    (property "Value" "DS18b20" (at 34.29 101.8351 0)
       (effects (font (size 1.27 1.27)))
     )
@@
       (effects (font (size 1.27 1.27)) (justify right))
     )
-    (property "Footprint" "Connector_PinHeader_2.54mm:PinHeader_1x02_P2.54mm_Vertical" (at 138.43 143.51 0)
-      (effects (font (size 1.27 1.27)) hide)
-    )
+    (property "Footprint" "Connector_PinHeader_2.54mm:PinHeader_1x04_P2.54mm_Vertical" (at 138.43 143.51 0)
+      (effects (font (size 1.27 1.27)) hide)
+    )
