File: bed-smart-plug/prototype-1/bed-smart-plug.kicad_pcb (KiCad board)
At the start: 2 copper layers, 0 parts

Commit message: wip pcb
Parts:
- added AE1: Antenna, Connector_PinHeader_2.54mm:PinHeader_1x01_P2.54mm_Vertical, F.Cu at (77.5, 114.3)
- added C1: 47nF/400V, Capacitor_SMD:C_1206_3216Metric, F.Cu at (191.0, 77.1)
- added C2: 10nF/400V, Capacitor_SMD:C_0805_2012Metric, F.Cu at (194.4, 84.9)
- added D1: LED, Diode_SMD:D_0805_2012Metric, F.Cu at (208.6, 97.3)
- added F1: 3A, Fuse:Fuseholder_Cylinder-5x20mm_Schurter_0031_8201_Horizontal_Open, F.Cu at (176.0, 95.4)
- added HS1: Heatsink, Heatsink:Heatsink_Fischer_SK104-STC-STIC_35x13mm_2xDrill2.5mm, F.Cu at (238.4, 56.7)
- added J1: Conn_01x03_Male, Connector_PinHeader_2.54mm:PinHeader_1x03_P2.54mm_Vertical, F.Cu at (181.2, 77.7)
- added J2: Conn_01x02_Male, Connector_PinHeader_2.54mm:PinHeader_1x02_P2.54mm_Vertical, F.Cu at (201.2, 73.8)
- added J3: 3.5mm headphone jack, Connector_Audio:Jack_3.5mm_PJ320D_Horizontal, F.Cu at (113.0, 49.2)
- added J4: Triac gate protection, Connector_PinHeader_2.54mm:PinHeader_1x02_P2.54mm_Vertical, F.Cu at (205.8, 73.8)
- added J5: Opto snubber, Connector_PinHeader_2.54mm:PinHeader_1x03_P2.54mm_Vertical, F.Cu at (185.9, 77.7)
- added J6: Opto snubber 2, Connector_PinHeader_2.54mm:PinHeader_1x02_P2.54mm_Vertical, F.Cu at (210.5, 73.8)
- added J7: Main, TerminalBlock:TerminalBlock_bornier-2_P5.08mm, F.Cu at (223.5, 100.3)
- added J8: Triac snubber, Connector_PinHeader_2.54mm:PinHeader_1x02_P2.54mm_Vertical, F.Cu at (215.1, 73.8)
- added J9: Prises, TerminalBlock:TerminalBlock_bornier-2_P5.08mm, F.Cu at (223.5, 119.4)
- added PS1: Alim RS PRO 5V 1A, Converter_ACDC:Converter_ACDC_MeanWell_IRM-03-xx_THT, F.Cu at (78.9, 40.6)
- added Q1: BT136-600E, Package_TO_SOT_THT:TO-220-3_Vertical, F.Cu at (235.9, 61.0)
- added R1: 4.7KΩ, Resistor_SMD:R_0402_1005Metric, F.Cu at (207.8, 99.9)
- added R2: 220Ω, Resistor_SMD:R_0603_1608Metric, F.Cu at (190.2, 80.0)
- added R3: 220Ω, Resistor_SMD:R_0603_1608Metric, F.Cu at (190.2, 82.5)
- added R4: 360Ω/0.5W, Resistor_SMD:R_1210_3225Metric, F.Cu at (203.6, 92.0)
- added R5: 470Ω/0.5W, Resistor_SMD:R_1210_3225Metric, F.Cu at (203.6, 96.2)
- added R6: 39Ω/0.5W, Resistor_SMD:R_1210_3225Metric, F.Cu at (203.6, 100.4)
- added U1: ESP32-POE, mylife-footprints:ESP32-POE, F.Cu at (135.8, 82.7)
- added U2: AM-RX12A-433P, mylife-footprints:AMRX12A433P, F.Cu at (91.4, 124.6)
- added U3: MOC3021M, Package_DIP:SMDIP-6_W9.53mm, F.Cu at (185.5, 70.8)

Commit message: placement
Parts:
- J1: value Conn_01x03_Male -> DS18b20
- J2: footprint Connector_PinHeader_2.54mm:PinHeader_1x02_P2.54mm_Vertical -> Connector_PinHeader_2.54mm:PinHeader_1x04_P2.54mm_Vertical
- moved Q1 187.6 mm to (48.3, 61.4)
- moved HS1 187.6 mm to (50.8, 57.1)
- moved J8 169.6 mm to (45.5, 75.6), turned to 180 degrees
- moved J6 167.5 mm to (43.8, 90.8), turned to 180 degrees
- moved R5 162.3 mm to (41.3, 99.0)
- moved J9 160.2 mm to (80.0, 48.3), turned to 180 degrees
- moved R6 153.5 mm to (52.5, 73.0)
- moved C1 151.7 mm to (39.4, 79.4), turned to 90 degrees
- moved J5 147.1 mm to (39.4, 90.8), turned to 180 degrees
- moved D1 145.0 mm to (63.8, 104.1)
- moved R4 144.2 mm to (59.7, 83.2), turned to 90 degrees
- moved C2 142.5 mm to (52.2, 76.8), turned to 180 degrees
- moved J4 141.3 mm to (64.8, 81.9)
- moved J7 138.4 mm to (95.2, 48.3), turned to 180 degrees
- moved U3 135.7 mm to (53.3, 101.6)
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Other:
- board outline added: 122.6 x 80.6 mm
- board text added: "3V3"
- board text added: "Close x2=ON"
- board text added: "Close=OFF"
- board text added: "Close=ON"
- board text added: "DATA"
- board text added: "GND"
- board text added: "Open=ON"

Commit message: routing
Parts:
- turned R2 to 180 degrees
Routing:
- net GND: track 0.00 -> 189.9 mm
- net +3V3: track 0.00 -> 134.3 mm, vias 0 -> 1
- net NEUT: track 0.00 -> 97.6 mm
- net Net-(U1-GPIO2): track 0.00 -> 93.8 mm
- net +5V: track 0.00 -> 81.2 mm
- net Net-(J5-Pin_3): track 0.00 -> 78.1 mm
- net LINE: track 0.00 -> 63.4 mm
- net Net-(J8-Pin_2): track 0.00 -> 62.5 mm
- net Net-(Q1-G): track 0.00 -> 47.7 mm
- net Net-(U1-GPIO36): track 0.00 -> 34.1 mm, vias 0 -> 1
- net Net-(J4-Pin_2): track 0.00 -> 32.1 mm
- net Net-(J4-Pin_1): track 0.00 -> 28.5 mm
- net Net-(J1-Pin_3): track 0.00 -> 26.6 mm
- net Net-(J5-Pin_1): track 0.00 -> 21.9 mm
- net Net-(R3-Pad1): track 0.00 -> 20.2 mm, vias 0 -> 2
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