File: bed-smart-plug/prototype-3/bed-smart-plug.kicad_pcb (KiCad board)
At the start: 2 copper layers, 154 x 84 mm, 10 parts, among them J3 3.5mm headphone jack, Q1 BT136-600E, U1 ESP32-POE

Commit message: update PCB
Parts:
- moved J3 13.3 mm to (215.5, 77.7)
- moved ? 9.27 mm to (168.7, 54.9)
- moved ? 9.27 mm to (168.7, 82.8)
- moved U1 9.27 mm to (185.0, 68.8)
- moved ? 9.27 mm to (92.4, 56.3)
- moved ? 9.27 mm to (92.4, 110.5)
- moved HS1 9.27 mm to (104.5, 65.0)
- moved Q1 9.27 mm to (108.0, 67.6)
- moved ? 9.27 mm to (207.1, 56.3)
- moved ? 9.27 mm to (207.1, 110.5)
Changed lines of the file:
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@@
   (net 27 "unconnected-(U1-GPIO36-Pad19)")
   (footprint "" (layer "F.Cu")
-    (at 159.385 54.61)
+    (at 168.656 54.864)
     (fp_text reference "" (at 0 0) (layer "F.SilkS")
         (effects (font (size 1.27 1.27) (thickness 0.15)))
@@
   )
   (footprint "" (layer "F.Cu")
-    (at 197.875 56.025)
+    (at 207.146 56.279)
     (fp_text reference "" (at 0 0) (layer "F.SilkS")
         (effects (font (size 1.27 1.27) (thickness 0.15)))
@@
   )
   (footprint "Heatsink:Heatsink_Fischer_SK104-STC-STIC_35x13mm_2xDrill2.5mm" (layer "F.Cu")
-    (at 95.25 64.77 90)
+    (at 104.521 65.024 90)
     (descr "Heatsink, 35mm x 13mm, 2x Fixation 2,5mm Drill, Soldering, Fischer SK104-STC-STIC,")
     (tags "Heatsink fischer TO-220")
@@
   )
   (footprint "" (layer "F.Cu")
-    (at 83.125 56.025)
+    (at 92.396 56.279)
     (fp_text reference "" (at 0 0) (layer "F.SilkS")
         (effects (font (size 1.27 1.27) (thickness 0.15)))
@@
   )
   (footprint "" (layer "F.Cu")
-    (at 197.875 110.275)
+    (at 207.146 110.529)
     (fp_text reference "" (at 0 0) (layer "F.SilkS")
         (effects (font (size 1.27 1.27) (thickness 0.15)))
@@
   )
   (footprint "mylife-footprints:ESP32-POE" (layer "F.Cu")
-    (at 175.765 68.54 90)
+    (at 185.036 68.794 90)
     (property "Sheetfile" "bed-smart-plug.kicad_sch")
     (property "Sheetname" "")
@@
   )
   (footprint "Connector_Audio:Jack_3.5mm_PJ320D_Horizontal" (layer "F.Cu")
-    (at 206.553 87.63 180)
+    (at 215.459 77.724 180)
     (descr "Headphones with microphone connector, 3.5mm, 4 pins (http://www.qingpu-electronics.com/en/products/WQP-PJ320D-72.html)")
     (tags "3.5mm jack mic microphone phones headphones 4pins audio plug")
@@
   )
   (footprint "Package_TO_SOT_THT:TO-220-3_Vertical" (layer "F.Cu")
-    (at 98.735 67.31 90)
+    (at 108.006 67.564 90)
     (descr "TO-220-3, Vertical, RM 2.54mm, see https://www.vishay.com/docs/66542/to-220-1.pdf")
     (tags "TO-220-3 Vertical RM 2.54mm")
@@
   )
   (footprint "" (layer "F.Cu")
-    (at 83.125 110.275)
+    (at 92.396 110.529)
     (fp_text reference "" (at 0 0) (layer "F.SilkS")
         (effects (font (size 1.27 1.27) (thickness 0.15)))
@@
   )
   (footprint "" (layer "F.Cu")
-    (at 159.385 82.55)
+    (at 168.656 82.804)
     (fp_text reference "" (at 0 0) (layer "F.SilkS")
         (effects (font (size 1.27 1.27) (thickness 0.15)))
@@
     (pad "1" thru_hole circle (at 0 0) (size 8 8) (drill 5) (layers "*.Cu" "*.Mask"))
   )
-  (gr_circle (center 213 120.65) (end 217.5 120.65)
+  (gr_rect (start 77.271 90.904) (end 187.271 120.904)
+    (stroke (width 0.15) (type default)) (fill none) (layer "F.SilkS"))
+  (gr_circle (center 222.271 120.904) (end 226.771 120.904)
     (stroke (width 0.1) (type default)) (fill none) (layer "Edge.Cuts"))
-  (gr_circle (center 68 120.65) (end 72.5 120.65)
+  (gr_circle (center 77.271 120.904) (end 81.771 120.904)
     (stroke (width 0.1) (type default)) (fill none) (layer "Edge.Cuts"))
-  (gr_rect (start 68 45.65) (end 213 120.65)
+  (gr_rect (start 77.271 45.904) (end 222.271 120.904)
     (stroke (width 0.1) (type default)) (fill none) (layer "Edge.Cuts"))
-  (gr_circle (center 213 45.65) (end 217.5 45.65)
+  (gr_circle (center 222.271 45.904) (end 226.771 45.904)
     (stroke (width 0.1) (type default)) (fill none) (layer "Edge.Cuts"))
-  (gr_circle (center 68 45.65) (end 72.5 45.65)
+  (gr_circle (center 77.271 45.904) (end 81.771 45.904)
     (stroke (width 0.1) (type default)) (fill none) (layer "Edge.Cuts"))
   (group "" (id aa676b0e-43df-40bd-a189-b9438bbf0dca)
@@
     )
   )
+  (group "" (id d873e063-1830-4c9e-87b8-e724d0f76482)
+    (members
+      c124f288-ad60-40d1-9fa3-8e8b6013e3b3
+    )
+  )
+  (group "" (id 8dfabb76-7ca3-4096-acee-d093274d5469)
+    (members
+      4bf9e2b3-2087-4ee8-8d71-0b3b39ee3929
+      5e42b57e-66bc-4378-a3c3-0148e6af08fe
+    )
+  )
