File: bed-smart-plug/v1/bed-smart-plug.kicad_sch (KiCad schematic)
At the start: 38 parts, among them J2 3.5mm headphone jack, J5 Sorties, J7 Main, Q1 BT136-600E, Q2 BT136-600E, Q3 BT136-600E, Q4 BT136-600E, U1 ESP32-POE, U2 QAM-RX10-433, U3 MOC3021M, U4 MOC3021M, U5 MOC3021M, U6 MOC3021M

Commit message: note
Parts:
- HS1, HS3: value Heatsink -> Heatsink (shared by 2 triacs)
Changed lines of the file:
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@@
       (effects (font (size 1.27 1.27)) (justify left))
     )
-    (property "Value" "Heatsink" (at 195.3768 62.738 0)
+    (property "Value" "Heatsink (shared by 2 triacs)" (at 195.3768 62.738 0)
       (effects (font (size 1.27 1.27)) (justify left))
     )
@@
       (effects (font (size 1.27 1.27)) (justify left))
     )
-    (property "Value" "Heatsink" (at 195.3768 123.698 0)
-      (effects (font (size 1.27 1.27)) (justify left))
-    )
+    (property "Value" "Heatsink (shared by 2 triacs)" (at 195.3768 123.698 0)
+      (effects (font (size 1.27 1.27)) (justify left))
+    )

Commit message: wip pcb v1
Parts:
- removed J5: Sorties, symbol Connector:Screw_Terminal_01x04
- removed J7: Main, TerminalBlock:TerminalBlock_bornier-2_P5.08mm, symbol Connector:Screw_Terminal_01x02
- added J2: Main + Sorties, TerminalBlock:TerminalBlock_bornier-6_P5.08mm, symbol Connector:Screw_Terminal_01x06
- renumbered HS3 to HS2, J2 to J1, R9 to R10, R12 to R11, R15 to R12, R4 to R13, R10 to R14, R13 to R15, R5 to R2, R6 to R3, R7 to R4, R2 to R5, R8 to R6, R11 to R7, R14 to R8, R3 to R9
Connections:
- net LINE: now also J2.1 (Pin_1)
- net NEUT: now also J2.2 (Pin_2)
- net at Q1.1 (A1): now also J2.3 (Pin_3)
- net at Q4.1 (A1): now also J2.6 (Pin_6)
- net at Q3.1 (A1): now also J2.5 (Pin_5)
- net at Q2.1 (A1): now also J2.4 (Pin_4)
