File: bed-smart-plug/v1.1/bed-smart-plug.kicad_pcb (KiCad board)
At the start: 2 copper layers, 145 x 75 mm, 42 parts, among them J1 3.5mm headphone jack, J2 Main + Sorties, Q1 BT136-600E, Q2 BT136-600E, Q3 BT136-600E, Q4 BT136-600E, U1 ESP32-POE, U2 QAM-RX10-433, U3 MOC3021M, U4 MOC3021M, U5 MOC3021M, U6 MOC3021M

Commit message: pcb size
Parts:
- removed the ? at (202.0, 57.2)
- removed the ? at (163.5, 83.7)
- removed the ? at (87.2, 57.2)
- removed the ? at (163.5, 55.8)
- removed the ? at (202.0, 111.4)
- added ?: , , F.Cu at (209.3, 115.7)
- added ?: , , F.Cu at (94.5, 61.5)
- added ?: , , F.Cu at (170.8, 60.1)
- added ?: , , F.Cu at (209.3, 61.5)
- added ?: , , F.Cu at (170.8, 88.0)
- moved D4 8.47 mm to (161.0, 91.9)
- moved R8 8.47 mm to (161.0, 88.1)
- moved AE1 8.47 mm to (171.4, 52.8)
- moved J2 8.47 mm to (139.8, 55.5)
- moved Q2 8.47 mm to (89.7, 76.2)
- moved R1 8.47 mm to (208.4, 83.5)
- moved R11 8.47 mm to (176.2, 79.9)
- moved R14 8.47 mm to (158.4, 69.7)
- moved R16 8.47 mm to (183.8, 69.7)
- moved R9 8.47 mm to (150.8, 79.9)
- moved U2 8.47 mm to (194.9, 55.5)
- moved U3 8.47 mm to (152.1, 72.9)
- moved U4 8.47 mm to (164.8, 72.9)
- moved U6 8.47 mm to (190.2, 72.9)
- moved Q1 8.47 mm to (82.8, 71.1)
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Connections:
- AE1 pad 1: Net-(AE1-A) -> (no net)
- D1 pad 1: GND -> (no net)
- D1 pad 2: Net-(D1-A) -> (no net)
- D2 pad 1: GND -> (no net)
- D2 pad 2: Net-(D2-A) -> (no net)
- D3 pad 1: GND -> (no net)
- D3 pad 2: Net-(D3-A) -> (no net)
- D4 pad 1: GND -> (no net)
- D4 pad 2: Net-(D4-A) -> (no net)
- F1 pad 1: LINE -> (no net)
- F1 pad 2: Net-(Q1-A2) -> (no net)
- J1 pad R1: Net-(U1-GPIO13) -> (no net)
- J1 pad R2: Net-(U1-GPIO13) -> (no net)
- J1 pad S: GND -> (no net)
- J1 pad T: +3V3 -> (no net)
- J2 pad 1: LINE -> (no net)
- J2 pad 2: NEUT -> (no net)
- J2 pad 3: Net-(J2-Pin_3) -> (no net)
- J2 pad 4: Net-(J2-Pin_4) -> (no net)
- J2 pad 5: Net-(J2-Pin_5) -> (no net)
- J2 pad 6: Net-(J2-Pin_6) -> (no net)
- PS1 pad 1: LINE -> (no net)
- PS1 pad 14: GND -> (no net)
- PS1 pad 16: +5V -> (no net)
- PS1 pad 3: NEUT -> (no net)
- PS1 pad 5: unconnected-(PS1-NC-Pad5) -> (no net)
- Q1 pad 1: Net-(J2-Pin_3) -> (no net)
- Q1 pad 2: Net-(Q1-A2) -> (no net)
- Q1 pad 3: Net-(Q1-G) -> (no net)
- Q2 pad 1: Net-(J2-Pin_4) -> (no net)
- Q2 pad 2: Net-(Q1-A2) -> (no net)
- Q2 pad 3: Net-(Q2-G) -> (no net)
- Q3 pad 1: Net-(J2-Pin_5) -> (no net)
- Q3 pad 2: Net-(Q1-A2) -> (no net)
- Q3 pad 3: Net-(Q3-G) -> (no net)
- Q4 pad 1: Net-(J2-Pin_6) -> (no net)
- Q4 pad 2: Net-(Q1-A2) -> (no net)
- Q4 pad 3: Net-(Q4-G) -> (no net)
- R1 pad 1: +3V3 -> (no net)
- R1 pad 2: Net-(U1-GPIO13) -> (no net)
- R10 pad 1: Net-(R10-Pad1) -> (no net)
- R10 pad 2: Net-(U1-GPIO3) -> (no net)
- R11 pad 1: Net-(R11-Pad1) -> (no net)
- R11 pad 2: Net-(U1-GPIO4) -> (no net)
- R12 pad 1: Net-(R12-Pad1) -> (no net)
- R12 pad 2: Net-(U1-GPIO5) -> (no net)
- R13 pad 1: Net-(Q1-A2) -> (no net)
- R13 pad 2: Net-(R13-Pad2) -> (no net)
- R14 pad 1: Net-(Q1-A2) -> (no net)
- R14 pad 2: Net-(R14-Pad2) -> (no net)
- R15 pad 1: Net-(Q1-A2) -> (no net)
- R15 pad 2: Net-(R15-Pad2) -> (no net)
- R16 pad 1: Net-(Q1-A2) -> (no net)
- R16 pad 2: Net-(R16-Pad2) -> (no net)
- R2 pad 1: Net-(U1-GPIO36) -> (no net)
- R2 pad 2: Net-(R2-Pad2) -> (no net)
- R3 pad 1: Net-(U1-GPIO36) -> (no net)
- R3 pad 2: Net-(R3-Pad2) -> (no net)
- R4 pad 1: Net-(R3-Pad2) -> (no net)
- R4 pad 2: GND -> (no net)
- R5 pad 1: Net-(U1-GPIO2) -> (no net)
- R5 pad 2: Net-(D1-A) -> (no net)
- R6 pad 1: Net-(U1-GPIO3) -> (no net)
- R6 pad 2: Net-(D2-A) -> (no net)
- R7 pad 1: Net-(U1-GPIO4) -> (no net)
- R7 pad 2: Net-(D3-A) -> (no net)
- R8 pad 1: Net-(U1-GPIO5) -> (no net)
- R8 pad 2: Net-(D4-A) -> (no net)
- R9 pad 1: Net-(R9-Pad1) -> (no net)
- R9 pad 2: Net-(U1-GPIO2) -> (no net)
- U1 pad 1: +5V -> (no net)
- U1 pad 10: Net-(U1-GPIO5) -> (no net)
- U1 pad 11: Net-(U1-GPIO13) -> (no net)
- U1 pad 12: unconnected-(U1-GPIO14-Pad12) -> (no net)
- U1 pad 13: unconnected-(U1-GPIO15-Pad13) -> (no net)
- U1 pad 14: unconnected-(U1-GPIO16-Pad14) -> (no net)
- U1 pad 15: unconnected-(U1-GPIO32-Pad15) -> (no net)
- U1 pad 16: unconnected-(U1-GPIO33-Pad16) -> (no net)
- U1 pad 17: unconnected-(U1-GPIO34-Pad17) -> (no net)
- U1 pad 18: unconnected-(U1-GPIO35-Pad18) -> (no net)
- U1 pad 19: Net-(U1-GPIO36) -> (no net)
- U1 pad 2: +3V3 -> (no net)
- U1 pad 20: unconnected-(U1-GPIO39-Pad20) -> (no net)
- U1 pad 3: GND -> (no net)
- U1 pad 4: unconnected-(U1-ESP_EN-Pad4) -> (no net)
- U1 pad 5: unconnected-(U1-GPIO0-Pad5) -> (no net)
- U1 pad 6: unconnected-(U1-GPIO1-Pad6) -> (no net)
- U1 pad 7: Net-(U1-GPIO2) -> (no net)
- U1 pad 8: Net-(U1-GPIO3) -> (no net)
- U1 pad 9: Net-(U1-GPIO4) -> (no net)
- U2 pad 1: Net-(AE1-A) -> (no net)
- U2 pad 2: GND -> (no net)
- U2 pad 3: GND -> (no net)
- U2 pad 4: +3V3 -> (no net)
- U2 pad 5: +3V3 -> (no net)
- U2 pad 6: Net-(R2-Pad2) -> (no net)
- U2 pad 7: Net-(R2-Pad2) -> (no net)
- U2 pad 8: GND -> (no net)
- U3 pad 1: Net-(R9-Pad1) -> (no net)
- U3 pad 2: GND -> (no net)
- U3 pad 3: unconnected-(U3-NC-Pad3) -> (no net)
- U3 pad 4: Net-(Q1-G) -> (no net)
- U3 pad 5: unconnected-(U3-NC-Pad5) -> (no net)
- U3 pad 6: Net-(R13-Pad2) -> (no net)
- U4 pad 1: Net-(R10-Pad1) -> (no net)
- U4 pad 2: GND -> (no net)
- U4 pad 3: unconnected-(U4-NC-Pad3) -> (no net)
- U4 pad 4: Net-(Q2-G) -> (no net)
- U4 pad 5: unconnected-(U4-NC-Pad5) -> (no net)
- U4 pad 6: Net-(R14-Pad2) -> (no net)
- U5 pad 1: Net-(R11-Pad1) -> (no net)
- U5 pad 2: GND -> (no net)
- U5 pad 3: unconnected-(U5-NC-Pad3) -> (no net)
- U5 pad 4: Net-(Q3-G) -> (no net)
- U5 pad 5: unconnected-(U5-NC-Pad5) -> (no net)
- U5 pad 6: Net-(R15-Pad2) -> (no net)
- U6 pad 1: Net-(R12-Pad1) -> (no net)
- U6 pad 2: GND -> (no net)
- U6 pad 3: unconnected-(U6-NC-Pad3) -> (no net)
- U6 pad 4: Net-(Q4-G) -> (no net)
- U6 pad 5: unconnected-(U6-NC-Pad5) -> (no net)
- U6 pad 6: Net-(R16-Pad2) -> (no net)
Routing:
- net (no net): track 0.00 -> 1712.5 mm, vias 0 -> 25
- net GND: track 211.5 -> 0.00 mm, vias 3 -> 0
- net Net-(Q1-A2): track 194.8 -> 0.00 mm, vias 1 -> 0
- net LINE: track 145.6 -> 0.00 mm
- net Net-(Q4-G): track 99.0 -> 0.00 mm
- net Net-(Q2-G): track 98.1 -> 0.00 mm, vias 4 -> 0
- net Net-(Q3-G): track 90.2 -> 0.00 mm, vias 4 -> 0
- net +3V3: track 88.9 -> 0.00 mm, vias 2 -> 0
- net Net-(Q1-G): track 84.8 -> 0.00 mm, vias 4 -> 0
- net Net-(J2-Pin_3): track 75.7 -> 0.00 mm, vias 1 -> 0
- net Net-(J2-Pin_4): track 74.5 -> 0.00 mm
- net Net-(J2-Pin_5): track 68.1 -> 0.00 mm, vias 1 -> 0
- net Net-(J2-Pin_6): track 66.0 -> 0.00 mm
- net Net-(U1-GPIO2): track 53.1 -> 0.00 mm, vias 1 -> 0
- net Net-(U1-GPIO3): track 49.0 -> 0.00 mm, vias 1 -> 0
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Other:
- outline, holes or cut-outs redrawn

Commit message: wip pcb
Parts:
- removed AE1: Antenna, Connector_PinHeader_2.54mm:PinHeader_1x01_P2.54mm_Vertical
- U2: footprint mylife-footprints:AMRX12A433P -> mylife-footprints:QAM-RX10-433
- moved U2 0.89 mm to (194.9, 54.6)
Connections:
- D1 pad 1: (no net) -> GND
- D1 pad 2: (no net) -> Net-(D1-A)
- D2 pad 1: (no net) -> GND
- D2 pad 2: (no net) -> Net-(D2-A)
- D3 pad 1: (no net) -> GND
- D3 pad 2: (no net) -> Net-(D3-A)
- D4 pad 1: (no net) -> GND
- D4 pad 2: (no net) -> Net-(D4-A)
- F1 pad 1: (no net) -> LINE
- F1 pad 2: (no net) -> Net-(Q1-A2)
- J1 pad R1: (no net) -> Net-(U1-GPIO13)
- J1 pad R2: (no net) -> Net-(U1-GPIO13)
- J1 pad S: (no net) -> GND
- J1 pad T: (no net) -> +3V3
- J2 pad 1: (no net) -> LINE
- J2 pad 2: (no net) -> NEUT
- J2 pad 3: (no net) -> Net-(J2-Pin_3)
- J2 pad 4: (no net) -> Net-(J2-Pin_4)
- J2 pad 5: (no net) -> Net-(J2-Pin_5)
- J2 pad 6: (no net) -> Net-(J2-Pin_6)
- PS1 pad 1: (no net) -> LINE
- PS1 pad 14: (no net) -> GND
- PS1 pad 16: (no net) -> +5V
- PS1 pad 3: (no net) -> NEUT
- PS1 pad 5: (no net) -> unconnected-(PS1-NC-Pad5)
- Q1 pad 1: (no net) -> Net-(J2-Pin_3)
- Q1 pad 2: (no net) -> Net-(Q1-A2)
- Q1 pad 3: (no net) -> Net-(Q1-G)
- Q2 pad 1: (no net) -> Net-(J2-Pin_4)
- Q2 pad 2: (no net) -> Net-(Q1-A2)
- Q2 pad 3: (no net) -> Net-(Q2-G)
- Q3 pad 1: (no net) -> Net-(J2-Pin_5)
- Q3 pad 2: (no net) -> Net-(Q1-A2)
- Q3 pad 3: (no net) -> Net-(Q3-G)
- Q4 pad 1: (no net) -> Net-(J2-Pin_6)
- Q4 pad 2: (no net) -> Net-(Q1-A2)
- Q4 pad 3: (no net) -> Net-(Q4-G)
- R1 pad 1: (no net) -> +3V3
- R1 pad 2: (no net) -> Net-(U1-GPIO13)
- R10 pad 1: (no net) -> Net-(R10-Pad1)
- R10 pad 2: (no net) -> Net-(U1-GPIO3)
- R11 pad 1: (no net) -> Net-(R11-Pad1)
- R11 pad 2: (no net) -> Net-(U1-GPIO4)
- R12 pad 1: (no net) -> Net-(R12-Pad1)
- R12 pad 2: (no net) -> Net-(U1-GPIO5)
- R13 pad 1: (no net) -> Net-(Q1-A2)
- R13 pad 2: (no net) -> Net-(R13-Pad2)
- R14 pad 1: (no net) -> Net-(Q1-A2)
- R14 pad 2: (no net) -> Net-(R14-Pad2)
- R15 pad 1: (no net) -> Net-(Q1-A2)
- R15 pad 2: (no net) -> Net-(R15-Pad2)
- R16 pad 1: (no net) -> Net-(Q1-A2)
- R16 pad 2: (no net) -> Net-(R16-Pad2)
- R2 pad 1: (no net) -> Net-(U1-GPIO36)
- R2 pad 2: (no net) -> Net-(R2-Pad2)
- R3 pad 1: (no net) -> Net-(U1-GPIO36)
- R3 pad 2: (no net) -> Net-(R3-Pad2)
- R4 pad 1: (no net) -> Net-(R3-Pad2)
- R4 pad 2: (no net) -> GND
- R5 pad 1: (no net) -> Net-(U1-GPIO2)
- R5 pad 2: (no net) -> Net-(D1-A)
- R6 pad 1: (no net) -> Net-(U1-GPIO3)
- R6 pad 2: (no net) -> Net-(D2-A)
- R7 pad 1: (no net) -> Net-(U1-GPIO4)
- R7 pad 2: (no net) -> Net-(D3-A)
- R8 pad 1: (no net) -> Net-(U1-GPIO5)
- R8 pad 2: (no net) -> Net-(D4-A)
- R9 pad 1: (no net) -> Net-(R9-Pad1)
- R9 pad 2: (no net) -> Net-(U1-GPIO2)
- U1 pad 1: (no net) -> +5V
- U1 pad 10: (no net) -> Net-(U1-GPIO5)
- U1 pad 11: (no net) -> Net-(U1-GPIO13)
- U1 pad 12: (no net) -> unconnected-(U1-GPIO14-Pad12)
- U1 pad 13: (no net) -> unconnected-(U1-GPIO15-Pad13)
- U1 pad 14: (no net) -> unconnected-(U1-GPIO16-Pad14)
- U1 pad 15: (no net) -> unconnected-(U1-GPIO32-Pad15)
- U1 pad 16: (no net) -> unconnected-(U1-GPIO33-Pad16)
- U1 pad 17: (no net) -> unconnected-(U1-GPIO34-Pad17)
- U1 pad 18: (no net) -> unconnected-(U1-GPIO35-Pad18)
- U1 pad 19: (no net) -> Net-(U1-GPIO36)
- U1 pad 2: (no net) -> +3V3
- U1 pad 20: (no net) -> unconnected-(U1-GPIO39-Pad20)
- U1 pad 3: (no net) -> GND
- U1 pad 4: (no net) -> unconnected-(U1-ESP_EN-Pad4)
- U1 pad 5: (no net) -> unconnected-(U1-GPIO0-Pad5)
- U1 pad 6: (no net) -> unconnected-(U1-GPIO1-Pad6)
- U1 pad 7: (no net) -> Net-(U1-GPIO2)
- U1 pad 8: (no net) -> Net-(U1-GPIO3)
- U1 pad 9: (no net) -> Net-(U1-GPIO4)
- U2 pad 1: (no net) -> +3V3
- U2 pad 2: (no net) -> Net-(R2-Pad2)
- U2 pad 3: (no net) -> Net-(R2-Pad2)
- U2 pad 4: (no net) -> GND
- U3 pad 1: (no net) -> Net-(R9-Pad1)
- U3 pad 2: (no net) -> GND
- U3 pad 3: (no net) -> unconnected-(U3-NC-Pad3)
- U3 pad 4: (no net) -> Net-(Q1-G)
- U3 pad 5: (no net) -> unconnected-(U3-NC-Pad5)
- U3 pad 6: (no net) -> Net-(R13-Pad2)
- U4 pad 1: (no net) -> Net-(R10-Pad1)
- U4 pad 2: (no net) -> GND
- U4 pad 3: (no net) -> unconnected-(U4-NC-Pad3)
- U4 pad 4: (no net) -> Net-(Q2-G)
- U4 pad 5: (no net) -> unconnected-(U4-NC-Pad5)
- U4 pad 6: (no net) -> Net-(R14-Pad2)
- U5 pad 1: (no net) -> Net-(R11-Pad1)
- U5 pad 2: (no net) -> GND
- U5 pad 3: (no net) -> unconnected-(U5-NC-Pad3)
- U5 pad 4: (no net) -> Net-(Q3-G)
- U5 pad 5: (no net) -> unconnected-(U5-NC-Pad5)
- U5 pad 6: (no net) -> Net-(R15-Pad2)
- U6 pad 1: (no net) -> Net-(R12-Pad1)
- U6 pad 2: (no net) -> GND
- U6 pad 3: (no net) -> unconnected-(U6-NC-Pad3)
- U6 pad 4: (no net) -> Net-(Q4-G)
- U6 pad 5: (no net) -> unconnected-(U6-NC-Pad5)
- U6 pad 6: (no net) -> Net-(R16-Pad2)
Routing:
- net (no net): track 1712.5 -> 0.00 mm, vias 25 -> 0
- net Net-(Q1-A2): track 0.00 -> 194.8 mm, vias 0 -> 1
- net GND: track 0.00 -> 187.5 mm, vias 0 -> 3
- net LINE: track 0.00 -> 145.6 mm
- net Net-(Q4-G): track 0.00 -> 99.0 mm
- net Net-(Q2-G): track 0.00 -> 98.1 mm, vias 0 -> 4
- net Net-(Q3-G): track 0.00 -> 90.2 mm, vias 0 -> 4
- net Net-(Q1-G): track 0.00 -> 84.8 mm, vias 0 -> 4
- net Net-(J2-Pin_3): track 0.00 -> 75.7 mm, vias 0 -> 1
- net Net-(J2-Pin_4): track 0.00 -> 74.5 mm
- net Net-(J2-Pin_5): track 0.00 -> 68.1 mm, vias 0 -> 1
- net Net-(J2-Pin_6): track 0.00 -> 66.0 mm
- net +3V3: track 0.00 -> 64.8 mm, vias 0 -> 1
- net Net-(U1-GPIO2): track 0.00 -> 53.1 mm, vias 0 -> 1
- net Net-(U1-GPIO3): track 0.00 -> 49.0 mm, vias 0 -> 1
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
Commit message: pcb OK
Parts:
- moved HS1 5.86 mm to (86.3, 79.5)
- moved HS2 5.86 mm to (104.3, 79.5)
- moved Q1 5.86 mm to (82.8, 77.0)
- moved Q2 5.86 mm to (89.7, 82.0)
- moved Q3 5.86 mm to (100.8, 76.9)
- moved Q4 5.86 mm to (107.8, 82.0)
Routing:
- net Net-(Q1-A2): track 194.8 -> 187.1 mm
- net Net-(Q3-G): track 90.2 -> 92.9 mm
- net Net-(Q4-G): track 99.0 -> 101.4 mm
- net Net-(Q2-G): track 98.1 -> 100.5 mm
- net Net-(J2-Pin_4): track 74.5 -> 76.9 mm
- net Net-(J2-Pin_6): track 66.0 -> 68.4 mm
- net Net-(Q1-G): track 84.8 -> 86.8 mm

Commit message: update moc3021 to available part
Parts:
- U3, U4, U5, U6: value MOC3021M -> MOC3021S
Changed lines of the file:
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@@
     (descr "6-lead surface-mounted (SMD) DIP package, row spacing 9.53 mm (375 mils)")
     (tags "SMD DIP DIL PDIP SMDIP 2.54mm 9.53mm 375mil")
-    (property "LCSC" "C108500")
+    (property "LCSC" "C427436")
     (property "Sheetfile" "bed-smart-plug.kicad_sch")
     (property "Sheetname" "")
@@
         (effects (font (size 1 1) (thickness 0.15)))
     )
-    (fp_text value "MOC3021M" (at 0 4.87 90) (layer "F.Fab")
+    (fp_text value "MOC3021S" (at 0 4.87 90) (layer "F.Fab")
         (effects (font (size 1 1) (thickness 0.15)))
     )
@@
     (descr "6-lead surface-mounted (SMD) DIP package, row spacing 9.53 mm (375 mils)")
     (tags "SMD DIP DIL PDIP SMDIP 2.54mm 9.53mm 375mil")
-    (property "LCSC" "C108500")
+    (property "LCSC" "C427436")
     (property "Sheetfile" "bed-smart-plug.kicad_sch")
     (property "Sheetname" "")
@@
         (effects (font (size 1 1) (thickness 0.15)))
     )
-    (fp_text value "MOC3021M" (at 0 4.87 90) (layer "F.Fab")
+    (fp_text value "MOC3021S" (at 0 4.87 90) (layer "F.Fab")
         (effects (font (size 1 1) (thickness 0.15)))
     )
@@
     (descr "6-lead surface-mounted (SMD) DIP package, row spacing 9.53 mm (375 mils)")
     (tags "SMD DIP DIL PDIP SMDIP 2.54mm 9.53mm 375mil")
-    (property "LCSC" "C108500")
+    (property "LCSC" "C427436")
     (property "Sheetfile" "bed-smart-plug.kicad_sch")
     (property "Sheetname" "")
@@
         (effects (font (size 1 1) (thickness 0.15)))
     )
-    (fp_text value "MOC3021M" (at 0 4.87 90) (layer "F.Fab")
+    (fp_text value "MOC3021S" (at 0 4.87 90) (layer "F.Fab")
         (effects (font (size 1 1) (thickness 0.15)))
     )
@@
     (descr "6-lead surface-mounted (SMD) DIP package, row spacing 9.53 mm (375 mils)")
     (tags "SMD DIP DIL PDIP SMDIP 2.54mm 9.53mm 375mil")
-    (property "LCSC" "C108500")
+    (property "LCSC" "C427436")
     (property "Sheetfile" "bed-smart-plug.kicad_sch")
     (property "Sheetname" "")
@@
         (effects (font (size 1 1) (thickness 0.15)))
     )
-    (fp_text value "MOC3021M" (at 0 4.87 90) (layer "F.Fab")
-        (effects (font (size 1 1) (thickness 0.15)))
-    )
+    (fp_text value "MOC3021S" (at 0 4.87 90) (layer "F.Fab")
+        (effects (font (size 1 1) (thickness 0.15)))
+    )
