File: gate-driver/v1/gate-driver.kicad_sch (KiCad schematic)
At the start: 10 parts, among them J1 Conn_01x03_Male, J2 Screw_Terminal_01x02, J3 Conn_01x02_Pin, Q1 BSS138, U1 WeMos_D1_mini

Commit message: wip schematic
Parts:
- removed D1: LED, Diode_SMD:D_0805_2012Metric, symbol Device:LED
- removed J2: Screw_Terminal_01x02, TerminalBlock:TerminalBlock_bornier-2_P5.08mm, symbol Connector:Screw_Terminal_01x02
- removed J3: Conn_01x02_Pin, Connector_PinHeader_2.54mm:PinHeader_1x02_P2.54mm_Vertical, symbol Connector:Conn_01x02_Pin
- removed PS1: Alim RS PRO 5V 1A, Converter_ACDC:Converter_ACDC_MeanWell_IRM-03-xx_THT, symbol Converter_ACDC:IRM-03-5
- removed Q1: BSS138, Package_TO_SOT_SMD:SOT-23, symbol Transistor_FET:BS170
- removed R1: 4.7KΩ, Resistor_SMD:R_0402_1005Metric, symbol Device:R
- removed R2: 1KΩ, Resistor_SMD:R_0603_1608Metric, symbol Device:R
- removed R3: 18Ω/0.5W, Resistor_SMD:R_1210_3225Metric, symbol Device:R
Connections:
- net +5V: now also J1.2 (Pin_2)
- net at J1.3 (Pin_3): now also U1.13 (SDA/D2); no longer U1.15 (RX)
- net +3V3: no longer names the net of U1.8 (3V3)
- net +3V3: no longer J1.2 (Pin_2)
Other:
- note added: "FS1000A"
- note removed: "+"
- note removed: "-"
- note removed: "Alim"
- note removed: "DS18B20"
- note removed: "LED IR"
