File: gate-driver/v1/gate-driver.kicad_pcb (KiCad board)
At the start: 2 copper layers, 60 x 40 mm, 14 parts, among them J1 Conn_01x03_Male, J2 Screw_Terminal_01x02, J3 Conn_01x02_Pin, Q1 BSS138, U1 WeMos_D1_mini

Commit message: pcb
Parts:
- removed D1: LED, Diode_SMD:D_0805_2012Metric
- removed J2: Screw_Terminal_01x02, TerminalBlock:TerminalBlock_bornier-2_P5.08mm
- removed J3: Conn_01x02_Pin, Connector_PinHeader_2.54mm:PinHeader_1x02_P2.54mm_Vertical
- removed PS1: Alim RS PRO 5V 1A, Converter_ACDC:Converter_ACDC_MeanWell_IRM-03-xx_THT
- removed Q1: BSS138, Package_TO_SOT_SMD:SOT-23
- removed R1: 4.7KΩ, Resistor_SMD:R_0402_1005Metric
- removed R2: 1KΩ, Resistor_SMD:R_0603_1608Metric
- removed R3: 18Ω/0.5W, Resistor_SMD:R_1210_3225Metric
- moved J1 12.2 mm to (132.2, 62.9), turned to 0 degrees
- moved U1 5.32 mm to (114.6, 72.2)
Connections:
- J1 pad 2: +3V3 -> +5V
- U1 pad 13: unconnected-(U1-SDA/D2-Pad13) -> Net-(J1-Pin_3)
- U1 pad 14: Net-(Q1-G) -> unconnected-(U1-SCL/D1-Pad14)
- U1 pad 15: Net-(J1-Pin_3) -> unconnected-(U1-RX-Pad15)
- U1 pad 8: +3V3 -> unconnected-(U1-3V3-Pad8)
Routing:
- net GND: track 110.9 -> 48.4 mm, vias 1 -> 0
- net +3V3: track 34.4 -> 0.00 mm
- net Net-(J3-Pin_2): track 19.8 -> 0.00 mm
- net Net-(D1-K): track 16.4 -> 0.00 mm
- net Net-(J1-Pin_3): track 37.7 -> 53.6 mm
- net Net-(Q1-G): track 10.4 -> 0.00 mm, vias 1 -> 0
- net NEUT: track 8.15 -> 0.00 mm
- net LINE: track 8.15 -> 0.00 mm
- net Net-(Q1-D): track 7.92 -> 0.00 mm
- net +5V: track 65.1 -> 57.7 mm
Other:
- board text added: "5V"
- board text added: "DATA"
- board text removed: "+"
- board text removed: "-"
- board text removed: "3V3"
- board text removed: "DS18B20"
- board text removed: "IN"
- board text removed: "LED IR"
